File: Block Diagram.kicad_sch (KiCad schematic)
At the start: 0 parts

Commit message: [25/06/2025][Block Diagram] Update
Other:
- note added: "+3V3"
- note removed: "+??V"

Commit message: [25/06/2026][MCU-POWER] Update
Other:
- note added: "+??V"
- note removed: "+3V3"
