File: MCU - POWER.kicad_sch (KiCad schematic)
At the start: 22 parts, among them U1 STM32G474RET6, U2 STM32G474RET6

Commit message: [25/06/2025][MCU - IOs] Update
Connections:
- net GND: now also U1.15 (VSS), U1.27 (VSSA), U1.31 (VSS), U1.47 (VSS), U1.63 (VSS), U2.15 (VSS), U2.27 (VSSA), U2.31 (VSS), U2.47 (VSS), U2.63 (VSS)
- new net: C7., C9., FB1., U1.28 (VREF+), U1.29 (VDDA)
- new net: C14., C18., FB2., U2.28 (VREF+), U2.29 (VDDA)
Other:
- note removed: "STM32G474 Datasheet p.81"
- moved on the sheet: FB1, FB2

Commit message: [26/06/2026][MCU - IOs] Update
Parts:
- U1, U2: footprint Duc_Library:LQFP-64_L10.0-W10.0-P0.50-LS12.0-BL -> (none); private (none) -> Datasheet
Connections:
- new net: C7., C9., FB1., U1.28 (VREF+), U1.29 (VDDA)
- new net: C14., C18., FB2., U2.28 (VREF+), U2.29 (VDDA)
Changed lines of the file:
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@@
 	)
 	(symbol
-		(lib_name "CC0402KRX7R6BB105_4")
+		(lib_name "CC0402KRX7R6BB105_2")
 		(lib_id "Duc_Library:CC0402KRX7R6BB105")
 		(at 124.46 152.4 90)
@@
 	)
 	(symbol
-		(lib_name "CC0402KRX7R9BB104_2")
 		(lib_id "Duc_Library:CC0402KRX7R9BB104")
 		(at 116.84 68.58 90)
@@
 	)
 	(symbol
-		(lib_name "CC0402KRX7R9BB104_8")
+		(lib_name "CC0402KRX7R9BB104_1")
 		(lib_id "Duc_Library:CC0402KRX7R9BB104")
 		(at 139.7 134.62 90)
@@
 	)
 	(symbol
-		(lib_name "CC0402KRX7R6BB105_2")
 		(lib_id "Duc_Library:CC0402KRX7R6BB105")
 		(at 124.46 86.36 90)
@@
 	)
 	(symbol
+		(lib_name "CC0402KRX7R6BB105_1")
 		(lib_id "Duc_Library:CC0402KRX7R6BB105")
 		(at 182.88 48.26 90)
@@
 			)
 		)
-		(property "Footprint" "Duc_Library:LQFP-64_L10.0-W10.0-P0.50-LS12.0-BL"
+		(property private "Footprint" "Duc_Library:LQFP-64_L10.0-W10.0-P0.50-LS12.0-BL"
 			(at 225.552 98.044 0)
 			(effects
@@
 			)
 		)
-		(property "Datasheet" "https://lcsc.com/product-detail/No-specification-for-star-making-plan_STMicroelectronics-STM32G474RET6_C521608.html"
+		(property private "Datasheet" "https://lcsc.com/product-detail/No-specification-for-star-making-plan_STMicroelectronics-STM32G474RET6_C521608.html"
 			(at 233.68 100.33 0)
 			(do_not_autoplace yes)
@@
 			)
 		)
-		(property "Footprint" "Duc_Library:LQFP-64_L10.0-W10.0-P0.50-LS12.0-BL"
+		(property private "Footprint" "Duc_Library:LQFP-64_L10.0-W10.0-P0.50-LS12.0-BL"
 			(at 225.552 164.084 0)
 			(effects
@@
 			)
 		)
-		(property "Datasheet" "https://lcsc.com/product-detail/No-specification-for-star-making-plan_STMicroelectronics-STM32G474RET6_C521608.html"
+		(property private "Datasheet" "https://lcsc.com/product-detail/No-specification-for-star-making-plan_STMicroelectronics-STM32G474RET6_C521608.html"
 			(at 233.68 166.37 0)
 			(do_not_autoplace yes)
@@
 	)
 	(symbol
-		(lib_name "CC0402KRX7R6BB105_5")
+		(lib_name "CC0402KRX7R6BB105_3")
 		(lib_id "Duc_Library:CC0402KRX7R6BB105")
 		(at 182.88 114.3 90)
@@
 	)
 	(symbol
-		(lib_name "CC0402KRX7R9BB104_5")
+		(lib_name "CC0402KRX7R9BB104_3")
 		(lib_id "Duc_Library:CC0402KRX7R9BB104")
 		(at 182.88 152.4 90)
@@
 	)
 	(symbol
-		(lib_name "CC0402KRX7R9BB104_4")
+		(lib_name "CC0402KRX7R9BB104_9")
 		(lib_id "Duc_Library:CC0402KRX7R9BB104")
 		(at 182.88 86.36 90)
@@
 	)
 	(symbol
-		(lib_name "CC0402KRX7R9BB104_7")
+		(lib_name "CC0402KRX7R9BB104_2")
 		(lib_id "Duc_Library:CC0402KRX7R9BB104")
 		(at 182.88 134.62 90)
@@
 	)
 	(symbol
-		(lib_name "CC0402KRX7R9BB104_6")
+		(lib_name "CC0402KRX7R9BB104_8")
 		(lib_id "Duc_Library:CC0402KRX7R9BB104")
 		(at 162.56 134.62 90)
@@
 	)
 	(symbol
-		(lib_name "CC0402KRX7R9BB104_3")
+		(lib_name "CC0402KRX7R9BB104_4")
 		(lib_id "Duc_Library:CC0402KRX7R9BB104")
 		(at 162.56 68.58 90)
@@
 	)
 	(symbol
-		(lib_name "CC0402MRX5R7BB475_1")
 		(lib_id "Duc_Library:CC0402MRX5R7BB475")
 		(at 93.98 134.62 270)
@@
 	)
 	(symbol
-		(lib_name "CC0402KRX7R9BB104_1")
+		(lib_name "CC0402KRX7R9BB104_5")
 		(lib_id "Duc_Library:CC0402KRX7R9BB104")
 		(at 139.7 68.58 90)
@@
 	)
 	(symbol
-		(lib_name "CC0402KRX7R6BB105_1")
+		(lib_name "CC0402KRX7R6BB105_4")
 		(lib_id "Duc_Library:CC0402KRX7R6BB105")
 		(at 160.02 86.36 90)
@@
 	)
 	(symbol
-		(lib_name "CC0402KRX7R6BB105_3")
+		(lib_name "CC0402KRX7R6BB105_5")
 		(lib_id "Duc_Library:CC0402KRX7R6BB105")
 		(at 160.02 152.4 90)
@@
 	)
 	(symbol
+		(lib_name "CC0402KRX7R9BB104_6")
 		(lib_id "Duc_Library:CC0402KRX7R9BB104")
 		(at 182.88 68.58 90)
@@
 	)
 	(symbol
-		(lib_name "CC0402KRX7R9BB104_9")
+		(lib_name "CC0402KRX7R9BB104_7")
 		(lib_id "Duc_Library:CC0402KRX7R9BB104")
 		(at 116.84 134.62 90)
@@
 	)
 	(symbol
+		(lib_name "CC0402MRX5R7BB475_1")
 		(lib_id "Duc_Library:CC0402MRX5R7BB475")
 		(at 93.98 68.58 270)
