File: Sensing - Position.kicad_sch (KiCad schematic)
At the start: 0 parts

Commit message: [01/07/2026][MCU - IOs] Update
Other:
- company: (none) -> ${COMPANY}
Changed lines of the file:
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@@
 	(generator_version "9.0")
 	(paper "A4")
+	(title_block
+		(date "2026-06-27")
+		(company "${COMPANY}")
+	)
 )
