File: Project Architecture.kicad_sch (KiCad schematic)
At the start: 0 parts

Commit message: [01/07/2026][MCU - IOs] Update
Other:
- sheet Interface - FD-CAN1 renamed Interface - FD-CAN
- sheet Interface - RS-485 renamed Interface - RS - 485
- sheet Sensing - Temperature renamed Sensing - Temperature & Humidity
Changed lines of the file:
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@@
 	(title_block
 		(title "Project Architecture")
-		(date "2025-01-12")
+		(date "2026-06-27")
 		(rev "${REVISION}")
 		(company "${COMPANY}")
@@
 			(color 128 255 255 0.5000)
 		)
-		(property "Sheetname" "Sensing - Temperature"
+		(property "Sheetname" "Sensing - Temperature & Humidity"
 			(at 140.97 127.2409 0)
 			(effects
@@
 			(color 255 150 255 0.5000)
 		)
-		(property "Sheetname" "Interface - RS-485"
+		(property "Sheetname" "Interface - RS - 485"
 			(at 140.97 214.8709 0)
 			(effects
@@
 			(color 255 150 255 0.5000)
 		)
-		(property "Sheetname" "Interface - FD-CAN1"
+		(property "Sheetname" "Interface - FD-CAN"
 			(at 55.88 138.6709 0)
 			(effects

Commit message: Update Power Generation Schematic
Other:
- sheet MCU - POWER renamed MCU - Power
Changed lines of the file:
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@@
 			(color 128 255 128 0.5000)
 		)
-		(property "Sheetname" "MCU - POWER"
+		(property "Sheetname" "MCU - Power"
 			(at 190.5 75.1709 0)
 			(effects

Commit message: Update Power Connector & Motor Control Schematic
Other:
- sheet MCU - Power: file MCU - POWER.kicad_sch -> MCU - Power.kicad_sch
Changed lines of the file:
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@@
 			)
 		)
-		(property "Sheetfile" "MCU - POWER.kicad_sch"
+		(property "Sheetfile" "MCU - Power.kicad_sch"
 			(at 190.5 97.1046 0)
 			(effects
