File: Revision History.kicad_sch (KiCad schematic)
At the start: 0 parts

Commit message: Update Schematic
Other:
- title: Revision History -> (none)
Changed lines of the file:
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@@
 	(paper "A4")
 	(title_block
-		(title "Revision History")
 		(date "2026-06-27")
 		(rev "${REVISION}")
