File: Interface - RS-422.kicad_sch (KiCad schematic)
At the start: 0 parts

Commit message: [01/07/2026][MCU - IOs] Update
Other:
- company: (none) -> ${COMPANY}
Changed lines of the file:
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@@
 	(generator_version "9.0")
 	(paper "A4")
+	(title_block
+		(date "2026-06-27")
+		(company "${COMPANY}")
+	)
 )

Commit message: Update Schematic
Parts:
- added C73, C74: 4.7uF 35V 0603, Duc:C0603, symbol Duc-Capacitors:CAP CER 0603
- added D10, D15: USBLC6-2SC6, Duc:SOT-23-6_L2.9-W1.6-P0.95-LS2.8-BL, symbol Duc-Diodes:USBLC6-2SC6
- added D11, D14: SMAJ5.0A, Duc:SMA_L4.3-W2.6-LS5.2-RD, symbol Duc-Diodes:SMAJ5.0A
- added D12, D13: BLUE 0603, Duc:LED0603-RD_WHITE, symbol Duc-Diodes:LED 0603
- added J8, J9: TYPE-C 16PIN 2MD, Duc:USB-C-SMD_TYPE-C-16PIN-2MD-073, symbol Duc-Connectors:TYPE-C16PIN2MD
- added R29, R30, R43, R44: 5.1K 0.1% 0402, Duc_Library:R0402, symbol Duc-Resistors:RES SMD 0402
- added R39, R45: 430K 0.1% 0603, Duc:R0603, symbol Duc-Resistors:RES SMD 0603
- added R40, R46: 620K 0.1% 0603, Duc:R0603, symbol Duc-Resistors:RES SMD 0603
- added R41, R42: 1K 0.1% 0603, Duc:R0603, symbol Duc-Resistors:RES SMD 0603
Connections:
- new net: D12.2 (A), R41.2
- new net: J9.B5 (CC2), R44.1
- new net: J8.A5 (CC1), R29.1
- new net: J8.B5 (CC2), R30.1
- new net: J9.A5 (CC1), R43.1
- new net: D13.2 (A), R42.2
- new net GND: C73.1, C74.1, D10.2 (GND), D11.2 (A), D12.1 (C), D13.1 (C), D14.2 (A), D15.2 (GND), J8.13 (EH), J8.14 (EH), J8.A1B12 (GND), J8.B1A12 (GND), J9.13 (EH), J9.14 (EH), J9.A1B12 (GND), J9.B1A12 (GND), R29.2, R30.2, R40.2, R43.2, R44.2, R46.2
- new net USB-DM_1: D10.1 (IO1), D10.6 (IO1), D15.1 (IO1), D15.6 (IO1), J8.A7 (Dn1), J8.B7 (Dn2), J9.A7 (Dn1), J9.B7 (Dn2)
- new net USB-DP_1: D10.3 (IO2), D10.4 (IO2), D15.3 (IO2), D15.4 (IO2), J8.A6 (Dp1), J8.B6 (Dp2), J9.A6 (Dp1), J9.B6 (Dp2)
- new net VBUS_1: C73.2, C74.2, D11.1 (C), D14.1 (C), J8.A4B9 (VBUS), J8.B4A9 (VBUS), J9.A4B9 (VBUS), J9.B4A9 (VBUS), R39.1, R41.1, R42.1, R45.1
- new net VBUS_DET1: R39.2, R40.1, R45.2, R46.1
- no-connect marks 0 -> 6
