File: User - LED Indicators.kicad_sch (KiCad schematic)
At the start: 0 parts

Commit message: [01/07/2026][MCU - IOs] Update
Other:
- company: (none) -> ${COMPANY}
Changed lines of the file:
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@@
 	(generator_version "9.0")
 	(paper "A4")
+	(title_block
+		(date "2026-06-27")
+		(company "${COMPANY}")
+	)
 )

Commit message: Update Schematic
Parts:
- added D2, D8, D9: Red 0603, Duc:LED0603-RD_WHITE, symbol Duc-Diodes:LED 0603
- added D3: Orange 0603, Duc:LED0603-RD_WHITE, symbol Duc-Diodes:LED 0603
- added D4: Yellow 0603, Duc:LED0603-RD_WHITE, symbol Duc-Diodes:LED 0603
- added D5: Green 0603, Duc:LED0603-RD_WHITE, symbol Duc-Diodes:LED 0603
- added D6: Blue 0603, Duc:LED0603-RD_WHITE, symbol Duc-Diodes:LED 0603
- added D7: White 0603, Duc:LED0603-RD_WHITE, symbol Duc-Diodes:LED 0603
- added R27, R28, R31, R35, R36: 220R 0.1% 0402, Duc_Library:R0402, symbol Duc-Resistors:RES SMD 0402
- added R32, R33, R34: 100R 0.1% 0402, Duc_Library:R0402, symbol Duc-Resistors:RES SMD 0402
Connections:
- new net: D7.1 (C), R34.2
- new net: D4.1 (C), R31.2
- new net: D2.1 (C), R27.2
- new net: D9.1 (C), R36.2
- new net: D8.1 (C), R35.2
- new net: D6.1 (C), R33.2
- new net: D5.1 (C), R32.2
- new net: D3.1 (C), R28.2
- new net +3.3V: D2.2 (A), D3.2 (A), D4.2 (A), D5.2 (A), D6.2 (A), D7.2 (A), D8.2 (A), D9.2 (A)
- new net GPIO-LED_Debug_1: R35.1
- new net GPIO-LED_Debug_2: R36.1
- new net GPIO-LED_I: R27.1
- new net GPIO-LED_M: R34.1
- new net GPIO-LED_P: R32.1
- new net GPIO-LED_R: R33.1
- new net GPIO-LED_T1: R28.1
- new net GPIO-LED_T2: R31.1

Commit message: Update Schematic
Parts:
- added BZ1: MLT-8530, Duc:BUZ-SMD_4P-L8.5-W8.5-P8.50-BR, symbol Duc-Misc:MLT-8530
- added D16: SS34, Duc:SMA_L4.3-W2.5-LS5.0-RD, symbol Duc-Diodes:SS34
- added Q3: 2SC1815, Duc:SOT-23-3_L2.9-W1.3-P1.90-LS2.4-BR, symbol Duc-Transistors:2SC1815_C20069143
- added R55: 470R 0.1% 0603, Duc:R0603, symbol Duc-Resistors:RES SMD 0603
Connections:
- net +3.3V: now also BZ1.1 (+), D16.1 (C)
- new net: BZ1.2 (-), D16.2 (A), Q3.3 (C)
- new net: Q3.1 (B), R55.2
- new net GND: Q3.2 (E)
- new net PWM_BUZZER: R55.1
Other:
- moved on the sheet: D2, D3, D4, D5, D6, D7, D8, D9, R27, R28, R31, R32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
