File: Power - Connectors.kicad_sch (KiCad schematic)
At the start: 10 parts, among them J1 XT60PW-M, J2 DC-044A-20A, Q1 HV10N03, Q2 HV10N03, U4 LM74700QDBVRQ1, U5 LM74700QDBVRQ1

Commit message: Update Schematic
Parts:
- C1: renamed from C26; value CAP CER 0603 -> 100nF 50V 0603
- C2: renamed from C27; value CAP CER 0603 -> 100nF 50V 0603
- C3: renamed from C28; value CAP CER 0603 -> 100nF 50V 0603
- C4: renamed from C29; value CAP CER 0603 -> 100nF 50V 0603
- renumbered U4 to U1, U5 to U2

Commit message: Update Schematic & PCB
Parts:
- C1, C2, C3, C4: value 100nF 50V 0603 -> CAP CER 0603
- J1: value XT60PW-M -> XT30PW-F; footprint Duc:CONN-TH_XT60PW-M -> Duc:CONN-TH_XT30PW-F-1; symbol Duc-Connectors:XT60PW-M -> Duc-Connectors:XT30PW-F; LCSC Part C98732 -> C2913282; MPN XT60PW-M -> XT30PW-F20.G.Y
- J2: value DC-044A-20A -> KF350-3.5-2P; footprint Duc:DC-IN-TH_DC-044A-20A -> Duc:CONN-TH_P3.50_KF350-3.5-2P; symbol Duc-Connectors:DC-044A-20A -> Duc-Connectors:KF350-3.5-2P; LCSC Part C129006 -> C474892; MPN DC-044A-20A -> KF350-3.5-2P; Manufacturer 韩国韩荣 -> KEFA(科发)
Connections:
- net +V_ADAPTER: now also J2.2; no longer J2.1
- net +V_BAT2S: now also J1.1; no longer J1.2 (+)
- net GND: now also J1.2, J2.1; no longer J1.1 (-), J2.2, J2.3
- no-connect marks 4 -> 2
Other:
- moved on the sheet: C3, C4, Q2, U2
