File: Misc - Board Version DAC.kicad_sch (KiCad schematic)
At the start: 0 parts

Commit message: [01/07/2026][MCU - IOs] Update
Other:
- company: (none) -> ${COMPANY}
Changed lines of the file:
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@@
 	(generator_version "9.0")
 	(paper "A4")
+	(title_block
+		(date "2026-06-27")
+		(company "${COMPANY}")
+	)
 )

Commit message: Update Schematic
Parts:
- added R25, R26: 100K 0.1% 0603, Duc:R0603, symbol Duc-Resistors:RES SMD 0603
Connections:
- new net +3.3V: R25.2
- new net BOARD_VERSION: R25.1, R26.2
- new net GND: R26.1

Commit message: Update Schematic
Changed lines of the file:
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@@
 		)
 	)
-	(text_box "Amulet"
+	(text_box "MB\n"
 		(exclude_from_sim no)
 		(at 100.33 114.3 0)
@@
 		(stroke
 			(width -0.0001)
-			(type default)
+			(type solid)
 		)
 		(fill
@@
 		)
 	)
-	(text_box "moteus"
+	(text_box "MCB\n"
 		(exclude_from_sim no)
 		(at 100.33 102.87 0)
@@
 		(stroke
 			(width -0.0001)
-			(type default)
+			(type solid)
 		)
 		(fill

Commit message: Update Schematic
Parts:
- renumbered R25 to R56, R26 to R57
Connections:
- net +3.3V renamed +3V3
Changed lines of the file:
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@@
 		(effects
 			(font
-				(face "Arial")
+				(face "KiCad Font")
 				(size 1.27 1.27)
 			)
@@
 		)
 	)
-	(hierarchical_label "+3.3V"
+	(hierarchical_label "+3V3"
 		(shape input)
 		(at 144.78 41.91 180)
@@
 		(dnp no)
 		(fields_autoplaced yes)
-		(property "Reference" "#PWR078"
+		(property "Reference" "#PWR0105"
 			(at 147.32 78.74 0)
 			(do_not_autoplace yes)
@@
 			(project "Master_Hand_Kicad"
 				(path "/f9e05184-c88b-4a88-ae9c-ab2bdb32be7c/c5103ceb-5325-4a84-a025-9638a412984e/0bb1cb44-88fa-40dc-bea3-1adee4cb244a"
-					(reference "#PWR078")
+					(reference "#PWR0105")
 					(unit 1)
 				)
@@
 		(dnp no)
 		(fields_autoplaced yes)
-		(property "Reference" "R26"
+		(property "Reference" "R57"
 			(at 149.86 71.1199 90)
 			(effects
@@
 			(project "Master_Hand_Kicad"
 				(path "/f9e05184-c88b-4a88-ae9c-ab2bdb32be7c/c5103ceb-5325-4a84-a025-9638a412984e/0bb1cb44-88fa-40dc-bea3-1adee4cb244a"
-					(reference "R26")
+					(reference "R57")
 					(unit 1)
 				)
@@
 		(dnp no)
 		(fields_autoplaced yes)
-		(property "Reference" "R25"
+		(property "Reference" "R56"
 			(at 149.86 53.3399 90)
 			(effects
@@
 			(project "Master_Hand_Kicad"
 				(path "/f9e05184-c88b-4a88-ae9c-ab2bdb32be7c/c5103ceb-5325-4a84-a025-9638a412984e/0bb1cb44-88fa-40dc-bea3-1adee4cb244a"
-					(reference "R25")
+					(reference "R56")
 					(unit 1)
 				)
