File: MCU - Power.kicad_sch (KiCad schematic)
At the start: 22 parts, among them U1 STM32G474RET6, U2 STM32G474RET6

Commit message: Update Schematic
Connections:
- new net: C7., C9., FB1., U1.28 (VREF+), U1.29 (VDDA)
- new net: C14., C18., FB2., U2.28 (VREF+), U2.29 (VDDA)
Other:
- title: MCU - Power -> (none)
Changed lines of the file:
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@@
 	(paper "A3")
 	(title_block
-		(title "MCU - Power")
 		(date "2026-06-27")
 		(rev "${REVISION}")
@@
 	(text_box "Microcontroller Power Supply Scheme"
 		(exclude_from_sim no)
-		(at 88.9 129.54 0)
+		(at 88.9 130.81 0)
 		(size 144.78 7.62)
 		(margins 1.9049 1.9049 1.9049 1.9049)
@@
 		)
 	)
-	(text_box "[${#}] ${TITLE}"
-		(exclude_from_sim no)
-		(at 12.7 13.97 0)
-		(size 393.7 12.7)
-		(margins 4.4999 4.4999 4.4999 4.4999)
-		(stroke
-			(width -0.0001)
-			(type solid)
-		)
-		(fill
-			(type none)
-		)
-		(effects
-			(font
-				(face "Times New Roman")
-				(size 6 6)
-				(thickness 1.2)
-				(bold yes)
-				(color 162 22 34 1)
-			)
-		)
-	)

Commit message: Update Schematic
Connections:
- net +3V3: now also FB1.1, FB2.1; no longer FB1., FB2.
- new net: C7., C9., FB1.2, U1.28 (VREF+), U1.29 (VDDA)
- new net: C14., C18., FB2.2, U2.28 (VREF+), U2.29 (VDDA)
Changed lines of the file:
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@@
 	)
 	(symbol
-		(lib_name "PBBHAQ2012H-102T10_1")
 		(lib_id "Duc_Library:PBBHAQ2012H-102T10")
 		(at 198.12 104.14 0)
@@
 			)
 		)
-		(property "Description" "300mΩ 1 ±25% 1kΩ@100MHz 0805 Ferrite Beads and Chips RoHS"
+		(property "Description" "300m? 1 �25% 1k?@100MHz 0805 Ferrite Beads and Chips RoHS"
 			(at 198.12 104.14 0)
 			(effects
@@
 			)
 		)
-		(pin ""
-		)
-		(pin ""
+		(pin "2"
+		)
+		(pin "1"
 		)
 		(instances
@@
 	)
 	(symbol
-		(lib_name "PBBHAQ2012H-102T10_2")
 		(lib_id "Duc_Library:PBBHAQ2012H-102T10")
 		(at 198.12 187.96 0)
@@
 			)
 		)
-		(property "Description" "300mΩ 1 ±25% 1kΩ@100MHz 0805 Ferrite Beads and Chips RoHS"
+		(property "Description" "300m? 1 �25% 1k?@100MHz 0805 Ferrite Beads and Chips RoHS"
 			(at 198.12 187.96 0)
 			(effects
@@
 			)
 		)
-		(pin ""
-		)
-		(pin ""
+		(pin "2"
+		)
+		(pin "1"
 		)
 		(instances

Commit message: Update Schematic
Parts:
- renumbered C16 to C10, C10 to C11, C11 to C12, C15 to C14, C17 to C15, C12 to C16, C14 to C17, C6 to C2, C5 to C3, C3 to C5, C2 to C6, C8 to C7, C9 to C8, C7 to C9
Connections:
- net +3V3: no longer C11., C12., C13., C14., C15., C7., FB1.1, U2.16 (VDD), U2.32 (VDD), U2.48 (VDD), U2.64 (VDD)
- new net +A3V3: C11., C12., C13., C14., C15., C7., FB1.1, U2.16 (VDD), U2.32 (VDD), U2.48 (VDD), U2.64 (VDD)

Commit message: Update Schematic
Parts:
- renumbered C1 to C30, C2 to C31, C3 to C32, C4 to C33, C5 to C34, C6 to C35, C7 to C36, C8 to C37, C9 to C38, C10 to C39, C11 to C40, C12 to C41, C13 to C42, C14 to C43, C15 to C44, C16 to C45, C17 to C46, C18 to C47, FB1 to FB3, FB2 to FB4, U1 to U6, U2 to U7
