File: Motor Control - Index.kicad_sch (KiCad schematic)
At the start: 8 parts, among them U10 TB9051FTG,EL

Commit message: Update Schematic
Parts:
- added J2: BM09B-SRSS-TB, Duc:CONN-SMD_9P-P1.00_BM09B-SRSS-TB, symbol Duc-Connectors:BM09B-SRSS-TB
- C50: value CAP CER 0402 -> 100nF 16V 0402
- C51: value CAP CER 0402 -> 470nF 16V 0402
Connections:
- net +5V: now also J2.10, J2.11
- net ECA_I: now also J2.6
- net ECB_I: now also J2.7
- net GND: now also J2.1, J2.5
- net OCM_I: now also R8.1, R9.1; no longer C51.2, R8.2, U10.7 (OCM)
- net OUT1_I: now also J2.4
- net OUT2_I: now also J2.9
- new net +3.3V: J2.3, J2.8
- new net ECC_I: J2.2
- new net _OCM_I: C51.2, R8.2, U10.7 (OCM)
Other:
- moved on the sheet: C48, C49, C50, C51, R7, R8, R9, U10

Commit message: Update Schematic
Connections:
- net DGND is gone; now on net GND: C48.1, C49.1, C51.1, R9.2, U10.1 (OCC), U10.27 (TEST1), U10.28 (TEST2), U10.3 (ENB), U10.4 (AGND)

Commit message: Update Schematic
Changed lines of the file:
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@@
+	)
+	(rectangle
+		(start 177.8 25.4)
+		(end 254 76.2)
+		(stroke
+			(width 1)
+			(type default)
+			(color 200 0 0 1)
+		)
+		(fill
+			(type none)
+		)
 	)
 	(rectangle

Commit message: Update Schematic
Parts:
- removed R7: 1R 0.1% 0402, Duc_Library:R0402, symbol Duc-Resistors:RES SMD 0402
- added C86, C87: 100nF 16V 0402, Duc_Library:C0402, symbol Duc-Capacitors:CAP CER 0402
- added R58: 1R 0.1% 0402, Duc_Library:R0402, symbol Duc-Resistors:RES SMD 0402
- added R61: 1K 0.1% 0402, Duc_Library:R0402, symbol Duc-Resistors:RES SMD 0402
- added R62, R71: 220R 0.1% 0402, Duc_Library:R0402, symbol Duc-Resistors:RES SMD 0402
- R8: value 10K 0.1% 0402 -> 1K 0.1% 0402
- R9: value 510R 0.1% 0402 -> 220R 0.1% 0402
- renumbered J2 to J3, U10 to U8
Connections:
- net +5V: now also R58.1; no longer J3.10, J3.11
- net DIAG_I: now also R62.2; no longer U8.18 (DIAG)
- net ECC_I: now also C87.2, R71.2; no longer J3.2
- net GND: now also J3.10, J3.11, C86.1, C87.1
- net VCC_I: now also R58.2
- net +3.3V renamed +3V3
- net +3V3: now also R61.2; no longer J3.3
- new net +A3V3: C86.2, J3.3
- new net _DIAG_I: R61.1, R62.1, U8.18 (DIAG)
- new net _ECC_I: J3.2, R71.1
Other:
- moved on the sheet: C48, C49, C50, C51, J3, R8, R9

Commit message: Update Schematic
Parts:
- renumbered C48 to C52, C49 to C53, C50 to C54, C51 to C55, C86 to C56, C87 to C57, R9 to R10, R61 to R11, R71 to R12, R58 to R7, R62 to R9
Changed lines of the file:
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@@
 			"cfMAhEL3gWUtPFId99ULxB1+eYtLMsIzcfnajMwvPv9bJASuVL3ACzsxTrh3eurpPMjx7HZt97Tv"
 			"9ic6nqvOUZWbzSr76S7/6QH3tVsV2K58biW3lBmy0aLnUPFKcbfHoxt85Ncr+x41+rVt9uJ7bw8b"
-			"pJVYsjhjmAjOiYgA+P8VlfdVjgg0hgAAAABJRU5ErkJggg=="
+			"pJVYsjhjmAjOiYgA+P8VlfdVjgg0hgAAAABJRU5ErkJggk0AagAyAEEARQA5AE8AQQBGAHIAdQBq"
+			"AE0AeABuAFoAKwBGAHYATwBBAHQAcQB3AE4AYQArAGwATgA3AFcAYwBBAGQARwBJAEwAWQBqAEcA"
+			"RwBHAE8AYwBzAEYAdgByAFUARQBxAHIAWgBVAGgASwBPAGkASgBKAFQAQwBGAEkAagBDAFEAQgBo"
+			"AEoAMgBsAE0AVAB1AGgAegBYADcAegBZAFoAdgBrAEsATgBkAGEAbAAzAHkANgBHAHMANgBHAEoA"
+			"YgBxAE8AeQBUADEAUwBkAHcAWABIAHgAUgBjAGsATgBrADQATgBxAFIAaABwAHEAVgBCADYAZQA3"
+			"AHEAZwB6AFIAYQBJADkATgA3ADMAegBjAC8AbgA5AGEAYwBQADgAWABsAGIAVgBEAEUAeQB2AEwA"
+			"cwBOAFAAMwB4AEQAMwA3ADUAcAAzADkANwBaAGIAZgBLAGIAaQBHAHUAQQBSAEUAagBBAFoAawBE"
+			"AG0AUgAzADcAcQBEAHMAQwBBAFEAdwBqADkARgBWAGcAdgBQAGkAWgBGAEIAMABmAGIAWgA4AGYA"
+			"WQBoADAAUwBDAFQAWQBtAFcAZwAxADQAMgBvAGMALwBlAG8AWABhAHIAdABkAFoAUwBWAFIAVQBS"
+			"AGgAVQBsAEMARwBDAGIAZwBUAEIATwBkAE0ALwBOAGwAeABWAGEAaAAxAGQANQBhAFUAMgB1ADUA"
+			"dABOAGEAeABOAFYANwBXAEcAQQBLAEcAaABFAGcAQQBTAGcAWgBPAEEARQBJAHkATQBUAGMALwA2"
+			"AEUAdwBBAHYAYwBQAHoAOAAvADcANQAwADUAZgAzAHYALwB6ADYAOAA5AC8ALwA4AGMAcwAvADMA"
+			"agA4ADkAUAA1AFoANgAwAGQANwBOAEQAaQAyAC8ARQBRAFAAcwBrAEQAVQArAE4AZwBVAE8AUwBj"
+			"AFMAWABpAEQATgBQADYATgA2AGIASAA2AHcANQBoADkAbAB6AFUAKwAzAEgANwBMAEUATgBJAEEA"
+			"NABPAGwANABYAC8ASAA2ADgARAB3AFoAZwBnAHgAcABnAHkASQBFAFEAQQAxAFgANAArAFAAOQBW"
+			"AFMAOQB6ADAALwBQAHoAOAA5AFAARAB6ADgAMgA1AC8AKwAvAEkAYwAvAC8ASABoADMAZAA3AGUA"
+			"dQB5AFIAbgAzAHAAbAAxADcAMwA2AHMAcQBtADAAZQAxAEkASQBJAGkAeQBJAEgAQwBGAE4AWgBn"
+			"AGgAMQBkAEUAOAB5AFAAdwA0AEkARgA2AEgAYQB2AEQAdABYAG8AdAAyAGwAcgBaADkAegBHAEMA"
+			"VABqAEcARwBFAEkAWgA1ADYAMwBVAHUAZABhAHIAZAB6AA=="
 		)
 	)
@@
 		)
 	)
-	(hierarchical_label "{MD1}"
+	(hierarchical_label "{MD_I}"
 		(shape bidirectional)
 		(at 229.87 38.1 0)
@@
 		(dnp no)
 		(fields_autoplaced yes)
-		(property "Reference" "#PWR034"
+		(property "Reference" "#PWR038"
 			(at 101.6 115.57 0)
 			(do_not_autoplace yes)
@@
 			(project "Master_Hand_Kicad"
 				(path "/f9e05184-c88b-4a88-ae9c-ab2bdb32be7c/c5103ceb-5325-4a84-a025-9638a412984e/9fef4a7d-fe15-42af-a3b5-95e4268f1da7"
-					(reference "#PWR034")
+					(reference "#PWR038")
 					(unit 1)
 				)
@@
 		(dnp no)
 		(fields_autoplaced yes)
-		(property "Reference" "C50"
+		(property "Reference" "C54"
 			(at 105.41 109.2199 90)
 			(effects
@@
 			(project "Master_Hand_Kicad"
 				(path "/f9e05184-c88b-4a88-ae9c-ab2bdb32be7c/c5103ceb-5325-4a84-a025-9638a412984e/9fef4a7d-fe15-42af-a3b5-95e4268f1da7"
-					(reference "C50")
+					(reference "C54")
 					(unit 1)
 				)
@@
 		(dnp no)
 		(fields_autoplaced yes)
-		(property "Reference" "#PWR033"
+		(property "Reference" "#PWR037"
 			(at 50.8 115.57 0)
 			(do_not_autoplace yes)
@@
 			(project "Master_Hand_Kicad"
 				(path "/f9e05184-c88b-4a88-ae9c-ab2bdb32be7c/c5103ceb-5325-4a84-a025-9638a412984e/9fef4a7d-fe15-42af-a3b5-95e4268f1da7"
-					(reference "#PWR033")
+					(reference "#PWR037")
 					(unit 1)
 				)
@@
 		(dnp no)
 		(fields_autoplaced yes)
-		(property "Reference" "#PWR030"
+		(property "Reference" "#PWR033"
 			(at 139.7 86.36 0)
 			(do_not_autoplace yes)
@@
 			(project "Master_Hand_Kicad"
 				(path "/f9e05184-c88b-4a88-ae9c-ab2bdb32be7c/c5103ceb-5325-4a84-a025-9638a412984e/9fef4a7d-fe15-42af-a3b5-95e4268f1da7"
-					(reference "#PWR030")
+					(reference "#PWR033")
 					(unit 1)
 				)
@@
 		(dnp no)
 		(fields_autoplaced yes)
-		(property "Reference" "R9"
+		(property "Reference" "R10"
 			(at 152.4 109.2199 90)
 			(effects
@@
 			(project "Master_Hand_Kicad"
 				(path "/f9e05184-c88b-4a88-ae9c-ab2bdb32be7c/c5103ceb-5325-4a84-a025-9638a412984e/9fef4a7d-fe15-42af-a3b5-95e4268f1da7"
-					(reference "R9")
+					(reference "R10")
 					(unit 1)
 				)
@@
 		(on_board no)
 		(dnp no)
-		(property "Reference" "#PWR0107"
+		(property "Reference" "#PWR040"
 			(at 231.14 132.08 0)
 			(do_not_autoplace yes)
@@
 			(project "Master_Hand_Kicad"
 				(path "/f9e05184-c88b-4a88-ae9c-ab2bdb32be7c/c5103ceb-5325-4a84-a025-9638a412984e/9fef4a7d-fe15-42af-a3b5-95e4268f1da7"
-					(reference "#PWR0107")
+					(reference "#PWR040")
 					(unit 1)
 				)
@@
 		(on_board no)
 		(dnp no)
-		(property "Reference" "#PWR0119"
+		(property "Reference" "#PWR042"
 			(at 162.56 143.51 0)
 			(do_not_autoplace yes)
@@
 			(project "Master_Hand_Kicad"
 				(path "/f9e05184-c88b-4a88-ae9c-ab2bdb32be7c/c5103ceb-5325-4a84-a025-9638a412984e/9fef4a7d-fe15-42af-a3b5-95e4268f1da7"
-					(reference "#PWR0119")
+					(reference "#PWR042")
 					(unit 1)
 				)
@@
 		(dnp no)
 		(fields_autoplaced yes)
-		(property "Reference" "R61"
+		(property "Reference" "R11"
 			(at 180.34 110.4899 90)
 			(effects
@@
 			(project "Master_Hand_Kicad"
 				(path "/f9e05184-c88b-4a88-ae9c-ab2bdb32be7c/c5103ceb-5325-4a84-a025-9638a412984e/9fef4a7d-fe15-42af-a3b5-95e4268f1da7"
-					(reference "R61")
+					(reference "R11")
 					(unit 1)
 				)
@@
 		(dnp no)
 		(fields_autoplaced yes)
-		(property "Reference" "C87"
+		(property "Reference" "C57"
 			(at 166.37 137.1599 90)
 			(effects
@@
 			(project "Master_Hand_Kicad"
 				(path "/f9e05184-c88b-4a88-ae9c-ab2bdb32be7c/c5103ceb-5325-4a84-a025-9638a412984e/9fef4a7d-fe15-42af-a3b5-95e4268f1da7"
-					(reference "C87")
+					(reference "C57")
 					(unit 1)
 				)
@@
 		(dnp no)
 		(fields_autoplaced yes)
-		(property "Reference" "R58"
+		(property "Reference" "R7"
 			(at 62.23 97.79 0)
 			(effects
@@
 			(project "Master_Hand_Kicad"
 				(path "/f9e05184-c88b-4a88-ae9c-ab2bdb32be7c/c5103ceb-5325-4a84-a025-9638a412984e/9fef4a7d-fe15-42af-a3b5-95e4268f1da7"
-					(reference "R58")
+					(reference "R7")
 					(unit 1)
 				)
@@
 		(on_board yes)
 		(dnp no)
-		(property "Reference" "C86"
+		(property "Reference" "C56"
 			(at 116.84 137.16 90)
 			(effects
@@
 			(project "Master_Hand_Kicad"
 				(path "/f9e05184-c88b-4a88-ae9c-ab2bdb32be7c/c5103ceb-5325-4a84-a025-9638a412984e/9fef4a7d-fe15-42af-a3b5-95e4268f1da7"
-					(reference "C86")
+					(reference "C56")
 					(unit 1)
 				)
@@
 		(dnp no)
 		(fields_autoplaced yes)
-		(property "Reference" "#PWR035"
+		(property "Reference" "#PWR039"
 			(at 127 115.57 0)
 			(do_not_autoplace yes)
@@
 			(project "Master_Hand_Kicad"
 				(path "/f9e05184-c88b-4a88-ae9c-ab2bdb32be7c/c5103ceb-5325-4a84-a025-9638a412984e/9fef4a7d-fe15-42af-a3b5-95e4268f1da7"
-					(reference "#PWR035")
+					(reference "#PWR039")
 					(unit 1)
 				)
@@
 		(on_board no)
 		(dnp no)
-		(property "Reference" "#PWR032"
+		(property "Reference" "#PWR036"
 			(at 240.03 114.3 0)
 			(do_not_autoplace yes)
@@
 			(project "Master_Hand_Kicad"
 				(path "/f9e05184-c88b-4a88-ae9c-ab2bdb32be7c/c5103ceb-5325-4a84-a025-9638a412984e/9fef4a7d-fe15-42af-a3b5-95e4268f1da7"
-					(reference "#PWR032")
+					(reference "#PWR036")
 					(unit 1)
 				)
@@
 		(dnp no)
 		(fields_autoplaced yes)
-		(property "Reference" "C48"
+		(property "Reference" "C52"
 			(at 54.61 109.2199 90)
 			(effects
@@
 			(project "Master_Hand_Kicad"
 				(path "/f9e05184-c88b-4a88-ae9c-ab2bdb32be7c/c5103ceb-5325-4a84-a025-9638a412984e/9fef4a7d-fe15-42af-a3b5-95e4268f1da7"
-					(reference "C48")
+					(reference "C52")
 					(unit 1)
 				)
@@
 		(on_board yes)
 		(dnp no)
-		(property "Reference" "R71"
+		(property "Reference" "R12"
 			(at 153.67 127 0)
 			(effects
@@
 			(project "Master_Hand_Kicad"
 				(path "/f9e05184-c88b-4a88-ae9c-ab2bdb32be7c/c5103ceb-5325-4a84-a025-9638a412984e/9fef4a7d-fe15-42af-a3b5-95e4268f1da7"
-					(reference "R71")
+					(reference "R12")
 					(unit 1)
 				)
@@
 		(dnp no)
 		(fields_autoplaced yes)
-		(property "Reference" "C51"
+		(property "Reference" "C55"
 			(at 130.81 109.2199 90)
 			(effects
@@
 			(project "Master_Hand_Kicad"
 				(path "/f9e05184-c88b-4a88-ae9c-ab2bdb32be7c/c5103ceb-5325-4a84-a025-9638a412984e/9fef4a7d-fe15-42af-a3b5-95e4268f1da7"
-					(reference "C51")
+					(reference "C55")
 					(unit 1)
 				)
@@
 		(on_board no)
 		(dnp no)
-		(property "Reference" "#PWR0106"
+		(property "Reference" "#PWR034"
 			(at 231.14 96.52 0)
 			(do_not_autoplace yes)
@@
 			(project "Master_Hand_Kicad"
 				(path "/f9e05184-c88b-4a88-ae9c-ab2bdb32be7c/c5103ceb-5325-4a84-a025-9638a412984e/9fef4a7d-fe15-42af-a3b5-95e4268f1da7"
-					(reference "#PWR0106")
+					(reference "#PWR034")
 					(unit 1)
 				)
@@
 		(dnp no)
 		(fields_autoplaced yes)
-		(property "Reference" "C49"
+		(property "Reference" "C53"
 			(at 77.47 109.2199 90)
 			(effects
@@
 			(project "Master_Hand_Kicad"
 				(path "/f9e05184-c88b-4a88-ae9c-ab2bdb32be7c/c5103ceb-5325-4a84-a025-9638a412984e/9fef4a7d-fe15-42af-a3b5-95e4268f1da7"
-					(reference "C49")
+					(reference "C53")
 					(unit 1)
 				)
@@
 		(dnp no)
 		(fields_autoplaced yes)
-		(property "Reference" "#PWR0118"
+		(property "Reference" "#PWR041"
 			(at 114.3 143.51 0)
 			(do_not_autoplace yes)
@@
 			(project "Master_Hand_Kicad"
 				(path "/f9e05184-c88b-4a88-ae9c-ab2bdb32be7c/c5103ceb-5325-4a84-a025-9638a412984e/9fef4a7d-fe15-42af-a3b5-95e4268f1da7"
-					(reference "#PWR0118")
+					(reference "#PWR041")
 					(unit 1)
 				)
@@
 		(dnp no)
 		(fields_autoplaced yes)
-		(property "Reference" "R62"
+		(property "Reference" "R9"
 			(at 187.96 97.79 0)
 			(effects
@@
 			(project "Master_Hand_Kicad"
 				(path "/f9e05184-c88b-4a88-ae9c-ab2bdb32be7c/c5103ceb-5325-4a84-a025-9638a412984e/9fef4a7d-fe15-42af-a3b5-95e4268f1da7"
-					(reference "R62")
+					(reference "R9")
 					(unit 1)
 				)
@@
 		(on_board no)
 		(dnp no)
-		(property "Reference" "#PWR031"
+		(property "Reference" "#PWR035"
 			(at 240.03 104.14 0)
 			(do_not_autoplace yes)
@@
 			(project "Master_Hand_Kicad"
 				(path "/f9e05184-c88b-4a88-ae9c-ab2bdb32be7c/c5103ceb-5325-4a84-a025-9638a412984e/9fef4a7d-fe15-42af-a3b5-95e4268f1da7"
-					(reference "#PWR031")
+					(reference "#PWR035")
 					(unit 1)
 				)

Commit message: Update Schematic
Parts:
- C52: value 4.7uF 16V 0402 -> CAP CER 0402
- C53: value 100nF 16V 0603 -> CAP CER 0402
- C54, C56, C57: value 100nF 16V 0402 -> CAP CER 0402
- C55: value 470nF 16V 0402 -> CAP CER 0402
- R10, R12, R9: value 220R 0.1% 0402 -> RES 0402
- R11, R8: value 1K 0.1% 0402 -> RES 0402
- R7: value 1R 0.1% 0402 -> RES 0402

Commit message: Update Schematic
Parts:
- removed R12: RES 0402, Duc_Library:R0402, symbol Duc-Resistors:RES SMD 0402
- added R12: 220R 0.1% 0603, Duc:R0603, symbol Duc-Resistors:RES SMD 0603
- C52: value CAP CER 0402 -> 4.7uF 50V 0603; footprint Duc_Library:C0402 -> Duc:C0603; symbol Duc-Capacitors:CAP CER 0402 -> Duc-Capacitors:CAP CER 0603; LCSC Part C325464 -> C14663; MPN CC0402KRX5R7BB105 -> CAP CER 0603; Manufacturer (none) -> YAGEO(国巨)
- C53, C54, C56, C57: value CAP CER 0402 -> 100nF 50V 0603; footprint Duc_Library:C0402 -> Duc:C0603; symbol Duc-Capacitors:CAP CER 0402 -> Duc-Capacitors:CAP CER 0603; LCSC Part C325464 -> C14663; MPN CC0402KRX5R7BB105 -> CAP CER 0603; Manufacturer (none) -> YAGEO(国巨)
- C55: value CAP CER 0402 -> 470nF 50V 0603; footprint Duc_Library:C0402 -> Duc:C0603; symbol Duc-Capacitors:CAP CER 0402 -> Duc-Capacitors:CAP CER 0603; LCSC Part C325464 -> C14663; MPN CC0402KRX5R7BB105 -> CAP CER 0603; Manufacturer (none) -> YAGEO(国巨)
- R10, R9: value RES 0402 -> 220R 0.1% 0603; footprint Duc_Library:R0402 -> Duc:R0603; symbol Duc-Resistors:RES SMD 0402 -> Duc-Resistors:RES SMD 0603; LCSC Part C728576 -> C4107493; MPN RT0402FRE07100KL -> RT0603FRE13100KL; Manufacturer (none) -> YAGEO(国巨)
- R11, R8: value RES 0402 -> 1K 0.1% 0603; footprint Duc_Library:R0402 -> Duc:R0603; symbol Duc-Resistors:RES SMD 0402 -> Duc-Resistors:RES SMD 0603; LCSC Part C728576 -> C4107493; MPN RT0402FRE07100KL -> RT0603FRE13100KL; Manufacturer (none) -> YAGEO(国巨)
- R7: value RES 0402 -> 1R 0.1% 0603; footprint Duc_Library:R0402 -> Duc:R0603; symbol Duc-Resistors:RES SMD 0402 -> Duc-Resistors:RES SMD 0603; LCSC Part C728576 -> C4107493; MPN RT0402FRE07100KL -> RT0603FRE13100KL; Manufacturer (none) -> YAGEO(国巨)
Connections:
- net ECC_I: now also R12.2
- net _ECC_I: now also R12.1
