File: Motor Control - Thumb 2.kicad_sch (KiCad schematic)
At the start: 0 parts

Commit message: Update Schematic
Parts:
- added C68: 4.7uF 16V 0402, Duc_Library:C0402, symbol Duc-Capacitors:CAP CER 0402
- added C69: 100nF 16V 0603, Duc_Library:C0402, symbol Duc-Capacitors:CAP CER 0402
- added C70: 100nF 16V 0402, Duc_Library:C0402, symbol Duc-Capacitors:CAP CER 0402
- added C71: 470nF 16V 0402, Duc_Library:C0402, symbol Duc-Capacitors:CAP CER 0402
- added J7: BM09B-SRSS-TB, Duc:CONN-SMD_9P-P1.00_BM09B-SRSS-TB, symbol Duc-Connectors:BM09B-SRSS-TB
- added R22: 1R 0.1% 0402, Duc_Library:R0402, symbol Duc-Resistors:RES SMD 0402
- added R23: 10K 0.1% 0402, Duc_Library:R0402, symbol Duc-Resistors:RES SMD 0402
- added R24: 510R 0.1% 0402, Duc_Library:R0402, symbol Duc-Resistors:RES SMD 0402
- added U15: TB9051FTG,EL, Duc_Library:UQFN-28_L6.0-W6.0-P0.65-BL-EP4.0, symbol Duc-ICs:TB9051FTG,EL
Connections:
- new net: R23.1, R24.1
- new net +3.3V: J7.3, J7.8
- new net +5V: C68.2, J7.10, J7.11, R22.1
- new net +VBAT: C70.2, U15.11 (VBAT), U15.12 (VBAT), U15.24 (VBAT), U15.25 (VBAT)
- new net DGND: C68.1, C69.1, C71.1, R24.2, U15.1 (OCC), U15.27 (TEST1), U15.28 (TEST2), U15.3 (ENB), U15.4 (AGND)
- new net DIAG_M: U15.18 (DIAG)
- new net ECA_M: J7.6
- new net ECB_M: J7.7
- new net ECC_M: J7.2
- new net EN_M: U15.5 (EN)
- new net GND: C70.1, J7.1, J7.5, U15.15 (PGND), U15.16 (PGND), U15.17 (PGND), U15.19 (PGND), U15.20 (PGND), U15.21 (PGND), U15.29 (EP)
- new net OUT1_M: J7.4, U15.13 (OUT1), U15.14 (OUT1)
- new net OUT2_M: J7.9, U15.22 (OUT2), U15.23 (OUT2)
- new net PWMA_M: U15.8 (PWM1)
- new net PWMB_M: U15.9 (PWM2)
- new net VCC_M: C69.2, R22.2, U15.2 (VCC)
- new net _OCM_M: C71.2, R23.2, U15.7 (OCM)
- no-connect marks 0 -> 3

Commit message: Update Motor Schematic
Connections:
- net OCM_T2: now reaches R23.1, R24.1
- net DIAG_M renamed DIAG_T2
- net ECA_M renamed ECA_T2
- net ECB_M renamed ECB_T2
- net ECC_M renamed ECC_T2
- net EN_M renamed EN_T2
- net OUT1_M renamed OUT1_T2
- net OUT2_M renamed OUT2_T2
- net PWMA_M renamed PWMA_T2
- net PWMB_M renamed PWMB_T2
- net VCC_M renamed VCC_T2
- net _OCM_M renamed _OCM_T2

Commit message: Update Schematic
Connections:
- net DGND is gone; now on net GND: C68.1, C69.1, C71.1, R24.2, U15.1 (OCC), U15.27 (TEST1), U15.28 (TEST2), U15.3 (ENB), U15.4 (AGND)

Commit message: Update Schematic
Changed lines of the file:
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@@
+		)
+	)
+	(rectangle
+		(start 177.8 25.4)
+		(end 254 76.2)
+		(stroke
+			(width 1)
+			(type default)
+			(color 200 0 0 1)
+		)
+		(fill
+			(type none)
 		)
 	)

Commit message: Update Schematic
Parts:
- removed J7: BM09B-SRSS-TB, Duc:CONN-SMD_9P-P1.00_BM09B-SRSS-TB, symbol Duc-Connectors:BM09B-SRSS-TB
- added C96, C97: 100nF 16V 0402, Duc_Library:C0402, symbol Duc-Capacitors:CAP CER 0402
- added J8: BM09B-SRSS-TB, Duc:CONN-SMD_9P-P1.00_BM09B-SRSS-TB, symbol Duc-Connectors:BM09B-SRSS-TB
- added R69: 1K 0.1% 0402, Duc_Library:R0402, symbol Duc-Resistors:RES SMD 0402
- added R70, R76: 220R 0.1% 0402, Duc_Library:R0402, symbol Duc-Resistors:RES SMD 0402
- R23: value 10K 0.1% 0402 -> 1K 0.1% 0402
- R24: value 510R 0.1% 0402 -> 220R 0.1% 0402
- renumbered U15 to U13
Connections:
- net DIAG_T2: now also R70.2; no longer U13.18 (DIAG)
- net ECA_T2: now also J8.6
- net ECB_T2: now also J8.7
- net ECC_T2: now also C97.2, R76.2
- net GND: now also C96.1, C97.1, J8.1, J8.10, J8.11, J8.5
- net OUT1_T2: now also J8.4
- net OUT2_T2: now also J8.9
- new net +3V3: J8.8, R69.2
- new net +A3V3: C96.2, J8.3
- new net _DIAG_T2: R69.1, R70.1, U13.18 (DIAG)
- new net _ECC_T2: J8.2, R76.1
Other:
- moved on the sheet: C68, C69, C70, C71, R22, R23, R24

Commit message: Update Schematic
Parts:
- renumbered C68 to C82, C69 to C83, C70 to C84, C71 to C85, C96 to C86, C97 to C87, R22 to R37, R23 to R38, R70 to R39, R24 to R40, R69 to R41, R76 to R42

Commit message: Update Schematic
Parts:
- C82: value 4.7uF 16V 0402 -> CAP CER 0402
- C83: value 100nF 16V 0603 -> CAP CER 0402
- C84, C86, C87: value 100nF 16V 0402 -> CAP CER 0402
- C85: value 470nF 16V 0402 -> CAP CER 0402
- R37: value 1R 0.1% 0402 -> RES 0402
- R38, R41: value 1K 0.1% 0402 -> RES 0402
- R39, R40, R42: value 220R 0.1% 0402 -> RES 0402

Commit message: Update Schematic
Parts:
- removed C82, C83, C84, C85, C86, C87: CAP CER 0402, Duc_Library:C0402, symbol Duc-Capacitors:CAP CER 0402
- removed R37, R38, R39, R40, R41, R42: RES 0402, Duc_Library:R0402, symbol Duc-Resistors:RES SMD 0402
- added C82: 4.7uF 50V 0603, Duc:C0603, symbol Duc-Capacitors:CAP CER 0603
- added C83, C84, C86, C87: 100nF 50V 0603, Duc:C0603, symbol Duc-Capacitors:CAP CER 0603
- added C85: 470nF 50V 0603, Duc:C0603, symbol Duc-Capacitors:CAP CER 0603
- added R37: 1R 0.1% 0603, Duc:R0603, symbol Duc-Resistors:RES SMD 0603
- added R38, R41: 1K 0.1% 0603, Duc:R0603, symbol Duc-Resistors:RES SMD 0603
- added R39, R40, R42: 220R 0.1% 0603, Duc:R0603, symbol Duc-Resistors:RES SMD 0603
Connections:
- net +3V3: now also R41.2
- net +5V: now also C82.2, R37.1
- net +A3V3: now also C86.2
- net +VBAT: now also C84.2
- net DIAG_T2: now also R39.2
- net ECC_T2: now also C87.2, R42.2
- net GND: now also C82.1, C83.1, C84.1, C85.1, C86.1, C87.1, R40.2
- net OCM_T2: now also R38.1, R40.1
- net VCC_T2: now also C83.2, R37.2
- net _DIAG_T2: now also R39.1, R41.1
- net _ECC_T2: now also R42.1
- net _OCM_T2: now also C85.2, R38.2
