File: Master_Hand_Kicad.kicad_pcb (KiCad board)
At the start: 6 copper layers, 0 parts

Commit message: Update Schematic
Routing:
- net (no net): vias 0 -> 7
Other:
- board outline added: 42.2 x 28.9 mm

Commit message: Update Schematic
Other:
- board size 42.2 x 28.9 mm -> 79 x 65.8 mm

Commit message: Update Schematic
Parts:
- added BZ1: MLT-8530, Duc:BUZ-SMD_4P-L8.5-W8.5-P8.50-BR, F.Cu at (267.0, 50.8)
- added C1: 100nF 50V 0603, Duc:C0603, F.Cu at (281.0, 32.5)
- added C10: 10uF 50V 1206, Duc_Library:C1206, F.Cu at (231.5, 26.1)
- added C100: 100nF 50V 0603, Duc:C0603, F.Cu at (324.0, 103.2)
- added C101: 100nF 50V 0603, Duc:C0603, F.Cu at (264.5, 91.9)
- added C102: 100nF 50V 0603, Duc:C0603, F.Cu at (264.5, 94.5)
- added C11: 100nF 50V 1206, Duc_Library:C1206, F.Cu at (231.5, 29.4)
- added C12: 1uF 50V 0603, Duc:C0603, F.Cu at (236.6, 21.1)
- added C13: 22uF 50V 1206, Duc_Library:C1206, F.Cu at (231.5, 32.7)
- added C14: 2.2uF 100V 0603, Duc:C0603, F.Cu at (236.6, 23.7)
- added C15: 2.2uF 100V 0603, Duc:C0603, F.Cu at (236.6, 26.4)
- added C16: 10uF 50V 1206, Duc_Library:C1206, F.Cu at (231.5, 36.0)
- added C17: 1uF 50V 1206, Duc_Library:C1206, F.Cu at (231.5, 39.4)
- added C18: 1uF 50V 1206, Duc_Library:C1206, F.Cu at (231.5, 42.7)
- added C19: 25SVPF330M, Duc:CAP-SMD_BD10.0-L10.3-W10.3-LS11.0-FD, F.Cu at (167.3, 102.4)
- added C2: 100nF 50V 0603, Duc:C0603, F.Cu at (281.0, 35.1)
- added C20: 10uF 50V 0603, Duc:C0603, F.Cu at (236.6, 29.1)
- added C21: 10uF 50V 0603, Duc:C0603, F.Cu at (240.7, 15.7)
- added C22: 10uF 50V 0603, Duc:C0603, F.Cu at (240.7, 18.4)
- added C23: 10uF 50V 0603, Duc:C0603, F.Cu at (240.7, 21.1)
- added C24: 10uF 50V 0603, Duc:C0603, F.Cu at (240.7, 23.7)
- added C25: 10uF 50V 0603, Duc:C0603, F.Cu at (240.7, 26.4)
- added C26: 10uF 50V 0603, Duc:C0603, F.Cu at (240.7, 29.1)
- added C27: 10uF 50V 0603, Duc:C0603, F.Cu at (244.7, 15.7)
- added C28: 10uF 50V 0603, Duc:C0603, F.Cu at (244.7, 18.4)
- added C29: 10uF 50V 0603, Duc:C0603, F.Cu at (244.7, 21.1)
- added C3: 100nF 50V 0603, Duc:C0603, F.Cu at (281.0, 37.8)
- added C30: 1uF 10V 0603, Duc:C0603, F.Cu at (301.4, 15.7)
- added C31: 4.7uF 16V 0603, Duc:C0603, F.Cu at (301.4, 18.4)
- added C32: 100nF 50V 0603, Duc:C0603, F.Cu at (301.4, 21.1)
- added C33: 100nF 50V 0603, Duc:C0603, F.Cu at (301.4, 23.7)
- added C34: 100nF 50V 0603, Duc:C0603, F.Cu at (301.4, 26.4)
- added C35: 100nF 50V 0603, Duc:C0603, F.Cu at (301.4, 29.1)
- added C36: 1uF 10V 0603, Duc:C0603, F.Cu at (301.4, 31.8)
- added C37: 1uF 10V 0603, Duc:C0603, F.Cu at (305.5, 15.7)
- added C38: 100nF 50V 0603, Duc:C0603, F.Cu at (305.5, 18.4)
- added C39: 1uF 10V 0603, Duc:C0603, F.Cu at (305.5, 21.1)
- added C4: 100nF 50V 0603, Duc:C0603, F.Cu at (281.0, 40.5)
- added C40: 4.7uF 16V 0603, Duc:C0603, F.Cu at (305.5, 23.7)
- added C41: 100nF 50V 0603, Duc:C0603, F.Cu at (305.5, 26.4)
- added C42: 100nF 50V 0603, Duc:C0603, F.Cu at (305.5, 29.1)
- added C43: 100nF 50V 0603, Duc:C0603, F.Cu at (305.5, 31.8)
- added C44: 100nF 50V 0603, Duc:C0603, F.Cu at (309.5, 15.7)
- added C45: 1uF 10V 0603, Duc:C0603, F.Cu at (309.5, 18.4)
- added C46: 1uF 10V 0603, Duc:C0603, F.Cu at (309.5, 21.1)
- added C47: 100nF 50V 0603, Duc:C0603, F.Cu at (309.5, 23.7)
- added C48: 8pF 16V 0603, Duc:C0603, F.Cu at (287.3, 47.7)
- added C49: 8pF 16V 0603, Duc:C0603, F.Cu at (287.3, 50.4)
- added C5: 4.7uF 100V 1206, Duc_Library:C1206, F.Cu at (231.5, 16.1)
- added C50: 8pF 16V 0603, Duc:C0603, F.Cu at (287.3, 53.0)
- added C51: 8pF 16V 0603, Duc:C0603, F.Cu at (287.3, 55.7)
- added C52: 4.7uF 50V 0603, Duc:C0603, F.Cu at (296.2, 87.9)
- added C53: 100nF 50V 0603, Duc:C0603, F.Cu at (296.2, 90.5)
- added C54: 100nF 50V 0603, Duc:C0603, F.Cu at (296.2, 93.2)
- added C55: 470nF 50V 0603, Duc:C0603, F.Cu at (296.2, 95.9)
- added C56: 100nF 50V 0603, Duc:C0603, F.Cu at (296.2, 98.6)
- added C57: 100nF 50V 0603, Duc:C0603, F.Cu at (296.2, 101.2)
- added C58: 4.7uF 50V 0603, Duc:C0603, F.Cu at (230.4, 96.3)
- added C59: 100nF 50V 0603, Duc:C0603, F.Cu at (230.4, 99.0)
- added C6: 4.7uF 100V 1206, Duc_Library:C1206, F.Cu at (231.5, 19.4)
- added C60: 100nF 50V 0603, Duc:C0603, F.Cu at (230.4, 101.7)
- added C61: 470nF 50V 0603, Duc:C0603, F.Cu at (230.4, 104.3)
- added C62: 100nF 50V 0603, Duc:C0603, F.Cu at (230.4, 107.0)
- added C63: 100nF 50V 0603, Duc:C0603, F.Cu at (230.4, 109.7)
- added C64: 4.7uF 50V 0603, Duc:C0603, F.Cu at (274.9, 69.9)
- added C65: 100nF 50V 0603, Duc:C0603, F.Cu at (274.9, 72.5)
- added C66: 100nF 50V 0603, Duc:C0603, F.Cu at (274.9, 75.2)
- added C67: 470nF 50V 0603, Duc:C0603, F.Cu at (274.9, 77.9)
- added C68: 100nF 50V 0603, Duc:C0603, F.Cu at (274.9, 80.5)
- added C69: 100nF 50V 0603, Duc:C0603, F.Cu at (274.9, 83.2)
- added C7: 2.2uF 100V 0603, Duc:C0603, F.Cu at (236.6, 15.7)
- added C70: 4.7uF 50V 0603, Duc:C0603, F.Cu at (294.8, 47.7)
- added C71: 100nF 50V 0603, Duc:C0603, F.Cu at (294.8, 50.4)
- added C72: 100nF 50V 0603, Duc:C0603, F.Cu at (294.8, 53.0)
- added C73: 470nF 50V 0603, Duc:C0603, F.Cu at (294.8, 55.7)
- added C74: 100nF 50V 0603, Duc:C0603, F.Cu at (294.8, 58.4)
- added C75: 100nF 50V 0603, Duc:C0603, F.Cu at (294.8, 61.0)
- added C76: 4.7uF 50V 0603, Duc:C0603, F.Cu at (274.9, 87.9)
- added C77: 100nF 50V 0603, Duc:C0603, F.Cu at (274.9, 90.5)
- added C78: 100nF 50V 0603, Duc:C0603, F.Cu at (274.9, 93.2)
- added C79: 470nF 50V 0603, Duc:C0603, F.Cu at (274.9, 95.9)
- added C8: 2.2uF 100V 0603, Duc:C0603, F.Cu at (236.6, 18.4)
- added C80: 100nF 50V 0603, Duc:C0603, F.Cu at (274.9, 98.6)
- added C81: 100nF 50V 0603, Duc:C0603, F.Cu at (274.9, 101.2)
- added C82: 4.7uF 50V 0603, Duc:C0603, F.Cu at (296.2, 69.9)
- added C83: 100nF 50V 0603, Duc:C0603, F.Cu at (296.2, 72.5)
- added C84: 100nF 50V 0603, Duc:C0603, F.Cu at (296.2, 75.2)
- added C85: 470nF 50V 0603, Duc:C0603, F.Cu at (296.2, 77.9)
- added C86: 100nF 50V 0603, Duc:C0603, F.Cu at (296.2, 80.5)
- added C87: 100nF 50V 0603, Duc:C0603, F.Cu at (296.2, 83.2)
- added C88: 4.7uF 50V 0603, Duc:C0603, F.Cu at (245.1, 64.5)
- added C89: 4.7uF 50V 0603, Duc:C0603, F.Cu at (245.1, 67.1)
- added C9: 10uF 100V 1206, Duc_Library:C1206, F.Cu at (231.5, 22.7)
- added C90: CAP CER 0603, Duc:C0603, F.Cu at (255.2, 79.2)
- added C91: CAP CER 0603, Duc:C0603, F.Cu at (255.2, 81.9)
- added C92: CAP CER 0603, Duc:C0603, F.Cu at (255.2, 84.5)
- added C93: CAP CER 0603, Duc:C0603, F.Cu at (255.2, 87.2)
- added C94: 4.7uF 50V 0603, Duc:C0603, F.Cu at (239.2, 71.8)
- added C95: 100nF 50V 0603, Duc:C0603, F.Cu at (239.2, 74.5)
- added C96: 100nF 50V 0603, Duc:C0603, F.Cu at (239.2, 77.1)
- added C97: 100nF 50V 0603, Duc:C0603, F.Cu at (239.2, 79.8)
- added C98: 100nF 50V 0603, Duc:C0603, F.Cu at (320.6, 87.9)
- added C99: 100nF 50V 0603, Duc:C0603, F.Cu at (320.6, 90.5)
- added D1: SMAJ12A, Duc:SMA_L4.3-W2.6-LS5.2-RD, F.Cu at (250.4, 23.9)
- added D10: Orange 0603, Duc:LED0603-RD_WHITE, F.Cu at (255.3, 50.4)
- added D11: Yellow 0603, Duc:LED0603-RD_WHITE, F.Cu at (255.3, 53.0)
- added D12: Green 0603, Duc:LED0603-RD_WHITE, F.Cu at (255.3, 55.7)
- added D13: Blue 0603, Duc:LED0603-RD_WHITE, F.Cu at (255.3, 58.3)
- added D14: White 0603, Duc:LED0603-RD_WHITE, F.Cu at (255.3, 61.0)
- added D15: SS34, Duc:SMA_L4.3-W2.5-LS5.0-RD, F.Cu at (263.9, 58.9)
- added D16: Red 0603, Duc:LED0603-RD_WHITE, F.Cu at (255.3, 63.7)
- added D17: Red 0603, Duc:LED0603-RD_WHITE, F.Cu at (255.3, 66.3)
- added D2: Blue 0603, Duc:LED0603-RD_WHITE, F.Cu at (249.2, 64.5)
- added D3: SMAJ5.0A, Duc:SMA_L4.3-W2.6-LS5.2-RD, F.Cu at (246.8, 48.4)
- added D4: USBLC6-2SC6, Duc:SOT-23-6_L2.9-W1.6-P0.95-LS2.8-BL, F.Cu at (245.6, 56.6)
- added D5: Blue 0603, Duc:LED0603-RD_WHITE, F.Cu at (249.2, 67.1)
- added D6: SMAJ5.0A, Duc:SMA_L4.3-W2.6-LS5.2-RD, F.Cu at (246.8, 52.4)
- added D7: USBLC6-2SC6, Duc:SOT-23-6_L2.9-W1.6-P0.95-LS2.8-BL, F.Cu at (245.6, 60.9)
- added D8: PESD1CAN, Duc:SOT-23-3_L2.9-W1.3-P1.90-LS2.4-BR, F.Cu at (247.1, 72.6)
- added D9: RED 0603, Duc:LED0603-RD_WHITE, F.Cu at (255.3, 47.7)
- added FB1: 1k @ 100MHz, Duc_Library:L0805, F.Cu at (254.7, 32.1)
- added FB2: 1k @ 100MHz, Duc_Library:L0805, F.Cu at (254.7, 35.4)
- added FM1: ~, Duc:Fiducial_1mm_Mask2mm, F.Cu at (323.0, 16.0)
- added FM2: ~, Duc:Fiducial_1mm_Mask2mm, F.Cu at (323.0, 19.1)
- added FM3: ~, Duc:Fiducial_1mm_Mask2mm, F.Cu at (323.0, 22.3)
- added H1: M2.4, Duc:MountingHole_2.4mm_M2.4_Pad_Via, F.Cu at (197.4, 74.3)
- added H2: M2.4, Duc:MountingHole_2.4mm_M2.4_Pad_Via, F.Cu at (123.6, 81.4)
- added H3: M2.4, Duc:MountingHole_2.4mm_M2.4_Pad_Via, F.Cu at (131.6, 117.5)
- added J1: XT60PW-M, Duc:CONN-TH_XT60PW-M, F.Cu at (146.7, 118.4)
- added J10: TYPE-C 16PIN 2MD, Duc:USB-C-SMD_TYPE-C-16PIN-2MD-073, F.Cu at (130.4, 102.1)
- added J11: 1.25-3PLTDK, Duc:CONN-SMD_3P-P1.25_SHOU_1.25-3PLTDK, F.Cu at (241.3, 89.5)
- added J12: 5025982393, Duc:FPC-SMD_23P-P0.60_502598-2393, B.Cu at (183.8, 70.7)
- added J13: PH2.54-2X3P-H25, Duc:HDR-TH_6P-P2.54-V-M-R2-C3-S2.54-1, F.Cu at (232.8, 73.6)
- added J14: PH2.54-2X3P-H25, Duc:HDR-TH_6P-P2.54-V-M-R2-C3-S2.54-1, F.Cu at (232.8, 79.9)
- added J15: PH2.54-2X3P-H25, Duc:HDR-TH_6P-P2.54-V-M-R2-C3-S2.54-1, F.Cu at (232.8, 86.2)
- added J2: DC-044A-20A, Duc:DC-IN-TH_DC-044A-20A, F.Cu at (170.9, 116.3)
- added J3: BM09B-SRSS-TB, Duc:CONN-SMD_9P-P1.00_BM09B-SRSS-TB, B.Cu at (180.6, 84.1)
- added J4: BM09B-SRSS-TB, Duc:CONN-SMD_9P-P1.00_BM09B-SRSS-TB, B.Cu at (197.1, 84.1)
- added J5: BM09B-SRSS-TB, Duc:CONN-SMD_9P-P1.00_BM09B-SRSS-TB, B.Cu at (180.3, 90.6)
- added J6: BM09B-SRSS-TB, Duc:CONN-SMD_9P-P1.00_BM09B-SRSS-TB, B.Cu at (196.1, 91.1)
- added J7: BM09B-SRSS-TB, Duc:CONN-SMD_9P-P1.00_BM09B-SRSS-TB, B.Cu at (180.6, 97.1)
- added J8: BM09B-SRSS-TB, Duc:CONN-SMD_9P-P1.00_BM09B-SRSS-TB, B.Cu at (196.7, 98.0)
- added J9: TYPE-C 16PIN 2MD, Duc:USB-C-SMD_TYPE-C-16PIN-2MD-073, F.Cu at (128.6, 91.4)
- added L1: ANR3015T2R2M, Duc:IND-SMD_L3.0-W3.0_SMNR3015, F.Cu at (254.5, 39.4)
- added L2: PBBHAQ2012H-102T10, Duc_Library:L0805, F.Cu at (302.0, 34.7)
- added L3: PBBHAQ2012H-102T10, Duc_Library:L0805, F.Cu at (302.0, 38.0)
- added Q1: HV10N03, Duc:SOT-89-3_L4.5-W2.5-P1.50-LS4.0-BR, F.Cu at (276.3, 34.0)
- added Q2: HV10N03, Duc:SOT-89-3_L4.5-W2.5-P1.50-LS4.0-BR, F.Cu at (276.3, 39.9)
- added Q3: 2SC1815, Duc:SOT-23-3_L2.9-W1.3-P1.90-LS2.4-BR, F.Cu at (262.2, 63.0)
- added R1: 41.2K 0.1% 0603, Duc:R0603, F.Cu at (250.6, 31.5)
- added R10: 220R 0.1% 0603, Duc:R0603, F.Cu at (299.7, 94.1)
- added R11: 1K 0.1% 0603, Duc:R0603, F.Cu at (299.7, 96.2)
- added R12: 220R 0.1% 0603, Duc:R0603, F.Cu at (299.7, 98.4)
- added R13: 1R 0.1% 0603, Duc:R0603, F.Cu at (233.9, 96.1)
- added R14: 1K 0.1% 0603, Duc:R0603, F.Cu at (233.9, 98.2)
- added R15: 220R 0.1% 0603, Duc:R0603, F.Cu at (233.9, 100.4)
- added R16: 220R 0.1% 0603, Duc:R0603, F.Cu at (233.9, 102.5)
- added R17: 1K 0.1% 0603, Duc:R0603, F.Cu at (233.9, 104.7)
- added R18: 220R 0.1% 0603, Duc:R0603, F.Cu at (233.9, 106.8)
- added R19: 1R 0.1% 0603, Duc:R0603, F.Cu at (278.4, 69.6)
- added R2: 10K 0.1% 0603, Duc:R0603, F.Cu at (250.6, 33.6)
- added R20: 1K 0.1% 0603, Duc:R0603, F.Cu at (278.4, 71.8)
- added R21: 220R 0.1% 0603, Duc:R0603, F.Cu at (278.4, 73.9)
- added R22: 220R 0.1% 0603, Duc:R0603, F.Cu at (278.4, 76.0)
- added R23: 1K 0.1% 0603, Duc:R0603, F.Cu at (278.4, 78.2)
- added R24: 220R 0.1% 0603, Duc:R0603, F.Cu at (278.4, 80.3)
- added R25: 1R 0.1% 0603, Duc:R0603, F.Cu at (298.3, 47.4)
- added R26: 1K 0.1% 0603, Duc:R0603, F.Cu at (298.3, 49.6)
- added R27: 220R 0.1% 0603, Duc:R0603, F.Cu at (298.3, 51.7)
- added R28: 220R 0.1% 0603, Duc:R0603, F.Cu at (298.3, 53.9)
- added R29: 1K 0.1% 0603, Duc:R0603, F.Cu at (298.3, 56.0)
- added R3: 40.2K 0.1% 0603, Duc:R0603, F.Cu at (250.6, 35.8)
- added R30: 220R 0.1% 0603, Duc:R0603, F.Cu at (298.3, 58.2)
- added R31: 1R 0.1% 0603, Duc:R0603, F.Cu at (278.4, 87.6)
- added R32: 1K 0.1% 0603, Duc:R0603, F.Cu at (278.4, 89.8)
- added R33: 220R 0.1% 0603, Duc:R0603, F.Cu at (278.4, 91.9)
- added R34: 220R 0.1% 0603, Duc:R0603, F.Cu at (278.4, 94.1)
- added R35: 1K 0.1% 0603, Duc:R0603, F.Cu at (278.4, 96.2)
- added R36: 220R 0.1% 0603, Duc:R0603, F.Cu at (278.4, 98.4)
- added R37: 1R 0.1% 0603, Duc:R0603, F.Cu at (299.7, 69.6)
- added R38: 1K 0.1% 0603, Duc:R0603, F.Cu at (299.7, 71.8)
- added R39: 220R 0.1% 0603, Duc:R0603, F.Cu at (299.7, 73.9)
- added R4: 13K 0.1% 0603, Duc:R0603, F.Cu at (250.6, 37.9)
- added R40: 220R 0.1% 0603, Duc:R0603, F.Cu at (299.7, 76.0)
- added R41: 1K 0.1% 0603, Duc:R0603, F.Cu at (299.7, 78.2)
- added R42: 220R 0.1% 0603, Duc:R0603, F.Cu at (299.7, 80.3)
- added R43: 430K 0.1% 0603, Duc:R0603, F.Cu at (241.2, 47.6)
- added R44: 620K 0.1% 0603, Duc:R0603, F.Cu at (241.2, 50.1)
- added R45: 1K 0.1% 0603, Duc:R0603, F.Cu at (241.2, 52.5)
- added R46: 5.1K 0.1% 0603, Duc:R0603, F.Cu at (249.2, 55.5)
- added R47: 5.1K 0.1% 0603, Duc:R0603, F.Cu at (249.2, 57.6)
- added R48: 430K 0.1% 0603, Duc:R0603, F.Cu at (241.2, 55.0)
- added R49: 620K 0.1% 0603, Duc:R0603, F.Cu at (241.2, 57.5)
- added R5: 10K 0.1% 0603, Duc:R0603, F.Cu at (250.6, 40.1)
- added R50: 1K 0.1% 0603, Duc:R0603, F.Cu at (241.2, 60.0)
- added R51: 5.1K 0.1% 0603, Duc:R0603, F.Cu at (249.2, 59.8)
- added R52: 5.1K 0.1% 0603, Duc:R0603, F.Cu at (249.2, 61.9)
- added R53: 10K 0.1% 0603, Duc:R0603, F.Cu at (259.2, 79.1)
- added R54: 10K 0.1% 0603, Duc:R0603, F.Cu at (259.2, 81.6)
- added R55: 10K 0.1% 0603, Duc:R0603, F.Cu at (259.2, 84.0)
- added R56: 10K 0.1% 0603, Duc:R0603, F.Cu at (259.2, 86.5)
- added R57: 2.2K 0.1% 0603, Duc:R0603, F.Cu at (243.2, 71.7)
- added R58: 2.2K 0.1% 0603, Duc:R0603, F.Cu at (243.2, 74.2)
- added R59: 60R4 0.1% 0603, Duc:R0603, F.Cu at (243.2, 76.6)
- added R6: 100K 0.1% 0603, Duc:R0603, F.Cu at (254.8, 19.8)
- added R60: 60R4 0.1% 0603, Duc:R0603, F.Cu at (243.2, 79.1)
- added R61: 330R 0.1% 0603, Duc:R0603, F.Cu at (258.7, 47.4)
- added R62: 330R 0.1% 0603, Duc:R0603, F.Cu at (258.7, 49.6)
- added R63: 330R 0.1% 0603, Duc:R0603, F.Cu at (258.7, 51.7)
- added R64: 100R 0.1% 0603, Duc:R0603, F.Cu at (258.7, 53.9)
- added R65: 100R 0.1% 0603, Duc:R0603, F.Cu at (258.7, 56.0)
- added R66: 100R 0.1% 0603, Duc:R0603, F.Cu at (258.7, 58.2)
- added R67: 330R 0.1% 0603, Duc:R0603, F.Cu at (258.7, 60.3)
- added R68: 330R 0.1% 0603, Duc:R0603, F.Cu at (258.7, 62.5)
- added R69: 470R 0.1% 0603, Duc:R0603, F.Cu at (262.2, 66.4)
- added R7: 1R 0.1% 0603, Duc:R0603, F.Cu at (299.7, 87.6)
- added R70: 10K 0.1% 0603, Duc:R0603, F.Cu at (317.0, 87.6)
- added R71: 10K 0.1% 0603, Duc:R0603, F.Cu at (317.0, 89.8)
- added R72: 10K 0.1% 0603, Duc:R0603, F.Cu at (317.0, 91.9)
- added R73: 10K 0.1% 0603, Duc:R0603, F.Cu at (317.0, 94.1)
- added R74: 100K 0.1% 0603, Duc:R0603, F.Cu at (318.1, 105.5)
- added R75: 47K 0.1% 0603, Duc:R0603, F.Cu at (314.7, 106.4)
- added R76: 0R 0.1% 0603, Duc:R0603, F.Cu at (254.7, 91.6)
- added R77: 100K 0.1% 0603, Duc:R0603, F.Cu at (264.5, 97.1)
- added R78: 0R 0.1% 0603, Duc:R0603, F.Cu at (254.7, 93.8)
- added R79: 100K 0.1% 0603, Duc:R0603, F.Cu at (264.5, 99.6)
- added R8: 1K 0.1% 0603, Duc:R0603, F.Cu at (299.7, 89.8)
- added R80: 10K 0.1% 0603, Duc:R0603, F.Cu at (254.7, 95.9)
- added R81: 10K 0.1% 0603, Duc:R0603, F.Cu at (254.7, 98.1)
- added R82: 10K 0.1% 0603, Duc:R0603, F.Cu at (254.7, 100.2)
- added R83: 10K 0.1% 0603, Duc:R0603, F.Cu at (254.7, 102.4)
- added R9: 220R 0.1% 0603, Duc:R0603, F.Cu at (299.7, 91.9)
- added SW1: DSIC02LSGET, Duc:SW-SMD_DSIC02LSGET, F.Cu at (259.4, 96.5)
- added TP1: ~, Duc_Library:TestPoint_Pad_D0.5mm, F.Cu at (247.5, 26.7)
- added TP10: ~, Duc_Library:TestPoint_Pad_D0.5mm, F.Cu at (273.6, 48.7)
- added TP11: ~, Duc_Library:TestPoint_Pad_D0.5mm, F.Cu at (273.6, 50.3)
- added TP12: ~, Duc_Library:TestPoint_Pad_D0.5mm, F.Cu at (273.6, 51.8)
- added TP13: ~, Duc_Library:TestPoint_Pad_D0.5mm, F.Cu at (273.6, 53.4)
- added TP14: ~, Duc_Library:TestPoint_Pad_D0.5mm, F.Cu at (273.6, 54.9)
- added TP15: ~, Duc_Library:TestPoint_Pad_D0.5mm, F.Cu at (273.6, 56.5)
- added TP16: ~, Duc_Library:TestPoint_Pad_D0.5mm, F.Cu at (273.6, 58.1)
- added TP17: ~, Duc_Library:TestPoint_Pad_D0.5mm, F.Cu at (273.6, 59.6)
- added TP18: ~, Duc_Library:TestPoint_Pad_D0.5mm, F.Cu at (273.6, 61.2)
- added TP19: ~, Duc_Library:TestPoint_Pad_D0.5mm, F.Cu at (273.6, 62.7)
- added TP2: ~, Duc_Library:TestPoint_Pad_D0.5mm, F.Cu at (247.5, 28.2)
- added TP20: ~, Duc_Library:TestPoint_Pad_D0.5mm, F.Cu at (275.2, 47.1)
- added TP21: ~, Duc_Library:TestPoint_Pad_D0.5mm, F.Cu at (275.2, 48.7)
- added TP22: ~, Duc_Library:TestPoint_Pad_D0.5mm, F.Cu at (275.2, 50.3)
- added TP23: ~, Duc_Library:TestPoint_Pad_D0.5mm, F.Cu at (275.2, 51.8)
- added TP24: ~, Duc_Library:TestPoint_Pad_D0.5mm, F.Cu at (275.2, 53.4)
- added TP25: ~, Duc_Library:TestPoint_Pad_D0.5mm, F.Cu at (275.2, 54.9)
- added TP26: ~, Duc_Library:TestPoint_Pad_D0.5mm, F.Cu at (275.2, 56.5)
- added TP27: ~, Duc_Library:TestPoint_Pad_D0.5mm, F.Cu at (275.2, 58.1)
- added TP28: ~, Duc_Library:TestPoint_Pad_D0.5mm, F.Cu at (275.2, 59.6)
- added TP29: ~, Duc_Library:TestPoint_Pad_D0.5mm, F.Cu at (275.2, 61.2)
- added TP3: ~, Duc_Library:TestPoint_Pad_D0.5mm, F.Cu at (249.1, 26.7)
- added TP30: ~, Duc_Library:TestPoint_Pad_D0.5mm, F.Cu at (275.2, 62.7)
- added TP31: ~, Duc_Library:TestPoint_Pad_D0.5mm, F.Cu at (276.7, 47.1)
- added TP32: ~, Duc_Library:TestPoint_Pad_D0.5mm, F.Cu at (276.7, 48.7)
- added TP33: ~, Duc_Library:TestPoint_Pad_D0.5mm, F.Cu at (276.7, 50.3)
- added TP34: ~, Duc_Library:TestPoint_Pad_D0.5mm, F.Cu at (276.7, 51.8)
- added TP35: ~, Duc_Library:TestPoint_Pad_D0.5mm, F.Cu at (276.7, 53.4)
- added TP36: ~, Duc_Library:TestPoint_Pad_D0.5mm, F.Cu at (276.7, 54.9)
- added TP37: ~, Duc_Library:TestPoint_Pad_D0.5mm, F.Cu at (276.7, 56.5)
- added TP38: ~, Duc_Library:TestPoint_Pad_D0.5mm, F.Cu at (276.7, 58.1)
- added TP39: ~, Duc_Library:TestPoint_Pad_D0.5mm, F.Cu at (276.7, 59.6)
- added TP4: ~, Duc_Library:TestPoint_Pad_D0.5mm, F.Cu at (249.1, 28.2)
- added TP40: ~, Duc_Library:TestPoint_Pad_D0.5mm, F.Cu at (276.7, 61.2)
- added TP41: ~, Duc_Library:TestPoint_Pad_D0.5mm, F.Cu at (276.7, 62.7)
- added TP42: ~, Duc_Library:TestPoint_Pad_D0.5mm, F.Cu at (278.3, 47.1)
- added TP43: ~, Duc_Library:TestPoint_Pad_D0.5mm, F.Cu at (278.3, 48.7)
- added TP44: ~, Duc_Library:TestPoint_Pad_D0.5mm, F.Cu at (278.3, 50.3)
- added TP45: ~, Duc_Library:TestPoint_Pad_D0.5mm, F.Cu at (278.3, 51.8)
- added TP46: ~, Duc_Library:TestPoint_Pad_D0.5mm, F.Cu at (278.3, 53.4)
- added TP47: ~, Duc_Library:TestPoint_Pad_D0.5mm, F.Cu at (278.3, 54.9)
- added TP48: ~, Duc_Library:TestPoint_Pad_D0.5mm, F.Cu at (278.3, 56.5)
- added TP49: ~, Duc_Library:TestPoint_Pad_D0.5mm, F.Cu at (278.3, 58.1)
- added TP5: ~, Duc_Library:TestPoint_Pad_D0.5mm, F.Cu at (250.6, 26.7)
- added TP50: ~, Duc_Library:TestPoint_Pad_D0.5mm, F.Cu at (278.3, 59.6)
- added TP51: ~, Duc_Library:TestPoint_Pad_D0.5mm, F.Cu at (278.3, 61.2)
- added TP52: ~, Duc_Library:TestPoint_Pad_D0.5mm, F.Cu at (278.3, 62.7)
- added TP53: ~, Duc_Library:TestPoint_Pad_D0.5mm, F.Cu at (279.9, 47.1)
- added TP54: ~, Duc_Library:TestPoint_Pad_D0.5mm, F.Cu at (279.9, 48.7)
- added TP55: ~, Duc_Library:TestPoint_Pad_D0.5mm, F.Cu at (279.9, 50.3)
- added TP56: ~, Duc_Library:TestPoint_Pad_D0.5mm, F.Cu at (279.9, 51.8)
- added TP57: ~, Duc_Library:TestPoint_Pad_D0.5mm, F.Cu at (279.9, 53.4)
- added TP58: ~, Duc_Library:TestPoint_Pad_D0.5mm, F.Cu at (279.9, 54.9)
- added TP59: ~, Duc_Library:TestPoint_Pad_D0.5mm, F.Cu at (279.9, 56.5)
- added TP6: ~, Duc_Library:TestPoint_Pad_D0.5mm, F.Cu at (250.6, 28.2)
- added TP60: ~, Duc_Library:TestPoint_Pad_D0.5mm, F.Cu at (279.9, 58.1)
- added TP61: ~, Duc_Library:TestPoint_Pad_D0.5mm, F.Cu at (279.9, 59.6)
- added TP62: ~, Duc_Library:TestPoint_Pad_D0.5mm, F.Cu at (279.9, 61.2)
- added TP63: ~, Duc_Library:TestPoint_Pad_D0.5mm, F.Cu at (279.9, 62.7)
- added TP64: ~, Duc_Library:TestPoint_Pad_D0.5mm, F.Cu at (281.4, 47.1)
- added TP65: ~, Duc_Library:TestPoint_Pad_D0.5mm, F.Cu at (281.4, 48.7)
- added TP66: ~, Duc_Library:TestPoint_Pad_D0.5mm, F.Cu at (281.4, 50.3)
- added TP67: ~, Duc_Library:TestPoint_Pad_D0.5mm, F.Cu at (281.4, 51.8)
- added TP68: ~, Duc_Library:TestPoint_Pad_D0.5mm, F.Cu at (281.4, 53.4)
- added TP69: ~, Duc_Library:TestPoint_Pad_D0.5mm, F.Cu at (281.4, 54.9)
- added TP7: ~, Duc_Library:TestPoint_Pad_D0.5mm, F.Cu at (252.2, 26.7)
- added TP70: ~, Duc_Library:TestPoint_Pad_D0.5mm, F.Cu at (281.4, 56.5)
- added TP71: ~, Duc_Library:TestPoint_Pad_D0.5mm, F.Cu at (281.4, 58.1)
- added TP72: ~, Duc_Library:TestPoint_Pad_D0.5mm, F.Cu at (281.4, 59.6)
- added TP73: ~, Duc_Library:TestPoint_Pad_D0.5mm, F.Cu at (281.4, 61.2)
- added TP74: ~, Duc_Library:TestPoint_Pad_D0.5mm, F.Cu at (281.4, 62.7)
- added TP75: ~, Duc_Library:TestPoint_Pad_D0.5mm, F.Cu at (283.0, 47.1)
- added TP76: ~, Duc_Library:TestPoint_Pad_D0.5mm, F.Cu at (283.0, 48.7)
- added TP77: ~, Duc_Library:TestPoint_Pad_D0.5mm, F.Cu at (283.0, 50.3)
- added TP78: ~, Duc_Library:TestPoint_Pad_D0.5mm, F.Cu at (283.0, 51.8)
- added TP79: ~, Duc_Library:TestPoint_Pad_D0.5mm, F.Cu at (283.0, 53.4)
- added TP8: ~, Duc_Library:TestPoint_Pad_D0.5mm, F.Cu at (252.2, 28.2)
- added TP80: ~, Duc_Library:TestPoint_Pad_D0.5mm, F.Cu at (283.0, 54.9)
- added TP81: ~, Duc_Library:TestPoint_Pad_D0.5mm, F.Cu at (283.0, 56.5)
- added TP82: ~, Duc_Library:TestPoint_Pad_D0.5mm, F.Cu at (283.0, 58.1)
- added TP83: ~, Duc_Library:TestPoint_Pad_D0.5mm, F.Cu at (283.0, 59.6)
- added TP84: ~, Duc_Library:TestPoint_Pad_D0.5mm, F.Cu at (283.0, 61.2)
- added TP85: ~, Duc_Library:TestPoint_Pad_D0.5mm, F.Cu at (283.0, 62.7)
- added TP86: ~, Duc_Library:TestPoint_Pad_D0.5mm, F.Cu at (284.5, 47.1)
- added TP87: ~, Duc_Library:TestPoint_Pad_D0.5mm, F.Cu at (284.5, 48.7)
- added TP88: ~, Duc_Library:TestPoint_Pad_D0.5mm, F.Cu at (284.5, 50.3)
- added TP89: ~, Duc_Library:TestPoint_Pad_D0.5mm, F.Cu at (284.5, 51.8)
- added TP9: ~, Duc_Library:TestPoint_Pad_D0.5mm, F.Cu at (273.6, 47.1)
- added TP90: ~, Duc_Library:TestPoint_Pad_D0.5mm, F.Cu at (284.5, 53.4)
- added TP91: ~, Duc_Library:TestPoint_Pad_D0.5mm, F.Cu at (284.5, 54.9)
- added U1: LM74700QDBVRQ1, Duc:SOT-23-6_L2.9-W1.6-P0.95-LS2.8-BL, F.Cu at (281.4, 16.6)
- added U10: TB9051FTG,EL, Duc_Library:UQFN-28_L6.0-W6.0-P0.65-BL-EP4.0, F.Cu at (141.4, 95.9)
- added U11: TB9051FTG,EL, Duc_Library:UQFN-28_L6.0-W6.0-P0.65-BL-EP4.0, F.Cu at (141.4, 105.2)
- added U12: TB9051FTG,EL, Duc_Library:UQFN-28_L6.0-W6.0-P0.65-BL-EP4.0, F.Cu at (153.5, 105.1)
- added U13: TB9051FTG,EL, Duc_Library:UQFN-28_L6.0-W6.0-P0.65-BL-EP4.0, F.Cu at (153.5, 95.9)
- added U14: TJA1051T/3, Duc:SOP-8_L4.9-W3.9-P1.27-LS6.0-BL-1, F.Cu at (256.7, 73.8)
- added U15: TJA1051T/3, Duc:SOP-8_L4.9-W3.9-P1.27-LS6.0-BL-1, F.Cu at (263.3, 73.8)
- added U16: SHT40-N-NF, Duc:DFN-4_L1.5-W1.5-P0.80-TL-EP, F.Cu at (320.1, 93.3)
- added U17: SHT40-N-NF, Duc:DFN-4_L1.5-W1.5-P0.80-TL-EP, F.Cu at (320.1, 96.1)
- added U2: LM74700QDBVRQ1, Duc:SOT-23-6_L2.9-W1.6-P0.95-LS2.8-BL, F.Cu at (281.4, 21.0)
- added U3: TPSM63603RDHR, Duc_Library:QFN-30_L6.0-W4.0-P0.50_TLVM13630RDHR, F.Cu at (250.1, 18.1)
- added U4: TPS62162DSG, Duc:WSON-8_L2.0-W2.0-P0.50-TL-EP, F.Cu at (255.1, 27.7)
- added U5: TLV75533PDBVR, Duc:SOT-23-5_L3.0-W1.7-P0.95-LS2.8-BR, F.Cu at (255.2, 16.5)
- added U6: STM32G474RET6, Duc_Library:LQFP-64_L10.0-W10.0-P0.50-LS12.0-BL, F.Cu at (171.4, 68.8)
- added U7: STM32G474RET6, Duc_Library:LQFP-64_L10.0-W10.0-P0.50-LS12.0-BL, F.Cu at (147.1, 68.9)
- added U8: TB9051FTG,EL, Duc_Library:UQFN-28_L6.0-W6.0-P0.65-BL-EP4.0, F.Cu at (153.5, 86.7)
- added U9: TB9051FTG,EL, Duc_Library:UQFN-28_L6.0-W6.0-P0.65-BL-EP4.0, F.Cu at (141.4, 86.7)
- added X1: X322516MLB4SI, Duc:CRYSTAL-SMD_4P-L3.2-W2.5-BL, F.Cu at (288.2, 59.3)
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Routing:
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Other:
- rule pad_to_mask_clearance: 0.05 -> 0.025

Commit message: Update Schematic
Parts:
- added C103: 100nF 50V 0603, Duc:C0603, F.Cu at (115.1, 90.8)
- added C104: 100nF 50V 0603, Duc:C0603, F.Cu at (115.1, 93.5)
- BZ1, C10, C11, C12, C13, C14, C15, C16, C17, C18, C19, C5, C6, C7, C8, C9, D1, D15, FB1, FB2, L1, Q3, R1, R2, R3, R4, R5, R53, R54, R55, R56, R57, R58, R6, R69, U14, U15, U3, U4, U5: moved to B.Cu
- C89: value 4.7uF 50V 0603 -> 100nF 50V 0402; footprint Duc:C0603 -> Duc_Library:C0402
- C90: value CAP CER 0603 -> 4.7uF 50V 0603
- C91: value CAP CER 0603 -> 100nF 50V 0402; footprint Duc:C0603 -> Duc_Library:C0402
- C92, C93: value CAP CER 0603 -> 100nF 50V 0603; moved to B.Cu
- C94: value 4.7uF 50V 0603 -> 100nF 50V 0603
- C96: value 100nF 50V 0603 -> 4.7uF 50V 0603
- R43, R48: value 430K 0.1% 0603 -> 430K 0.1% 0402; footprint Duc:R0603 -> Duc_Library:R0402
- R44, R49: value 620K 0.1% 0603 -> 620K 0.1% 0402; footprint Duc:R0603 -> Duc_Library:R0402
- R45, R50: value 1K 0.1% 0603 -> 1K 0.1% 0402; footprint Duc:R0603 -> Duc_Library:R0402
- R46, R47, R51, R52: value 5.1K 0.1% 0603 -> 5.1K 0.1% 0402; footprint Duc:R0603 -> Duc_Library:R0402
- moved C64 213.0 mm to (64.6, 104.2)
- moved C65 213.0 mm to (64.6, 106.9)
- moved C66 213.0 mm to (64.6, 109.5)
- moved C67 213.0 mm to (64.6, 112.2)
- moved C68 213.0 mm to (64.6, 114.9)
- moved C69 213.0 mm to (64.6, 117.5)
- moved C76 213.0 mm to (64.6, 122.2)
- moved C77 213.0 mm to (64.6, 124.9)
- moved C78 213.0 mm to (64.6, 127.6)
- moved C79 213.0 mm to (64.6, 130.2)
- moved C80 213.0 mm to (64.6, 132.9)
- moved C81 213.0 mm to (64.6, 135.6)
- moved R10 213.0 mm to (89.5, 128.4)
- moved R11 213.0 mm to (89.5, 130.6)
- moved R12 213.0 mm to (89.5, 132.7)
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Connections:
- C100 pad 2: /Project Architecture/MCU - IOs/SENSE_VBAT -> +A3V3
- C101 pad 2: Net-(C101-Pad2) -> +A3V3
- C102 pad 2: Net-(C102-Pad2) -> /Project Architecture/MCU - IOs/SENSE_VBAT
- C89 pad 2: /Project Architecture/Interface - USB 2.0/VBUS_2 -> /Project Architecture/Interface - USB 2.0/VBUS_1
- C90 pad 2: +5V -> /Project Architecture/Interface - USB 2.0/VBUS_2
- C91 pad 2: +3V3 -> /Project Architecture/Interface - USB 2.0/VBUS_2
- C94 pad 2: Net-(C94-Pad2) -> +5V
- C96 pad 2: +3V3 -> Net-(C96-Pad2)
- C98 pad 2: +A3V3 -> +3V3
- C99 pad 2: +A3V3 -> +3V3
- D4 pad 1: /Project Architecture/Interface - USB 2.0/USB-DM_1 -> Net-(J9-Dn1)
- D4 pad 3: /Project Architecture/Interface - USB 2.0/USB-DP_1 -> Net-(J9-Dp1)
- D4 pad 5: unconnected-(D4-VBUS-Pad5) -> /Project Architecture/Interface - USB 2.0/VBUS_1
- D7 pad 1: /Project Architecture/Interface - USB 2.0/USB-DM_2 -> Net-(J10-Dn1)
- D7 pad 3: /Project Architecture/Interface - USB 2.0/USB-DP_2 -> Net-(J10-Dp1)
- D7 pad 5: unconnected-(D7-VBUS-Pad5) -> /Project Architecture/Interface - USB 2.0/VBUS_2
- J10 pad A6: /Project Architecture/Interface - USB 2.0/USB-DP_2 -> Net-(J10-Dp1)
- J10 pad A7: /Project Architecture/Interface - USB 2.0/USB-DM_2 -> Net-(J10-Dn1)
- J10 pad B6: /Project Architecture/Interface - USB 2.0/USB-DP_2 -> Net-(J10-Dp1)
- J10 pad B7: /Project Architecture/Interface - USB 2.0/USB-DM_2 -> Net-(J10-Dn1)
- J9 pad A6: /Project Architecture/Interface - USB 2.0/USB-DP_1 -> Net-(J9-Dp1)
- J9 pad A7: /Project Architecture/Interface - USB 2.0/USB-DM_1 -> Net-(J9-Dn1)
- J9 pad B6: /Project Architecture/Interface - USB 2.0/USB-DP_1 -> Net-(J9-Dp1)
- J9 pad B7: /Project Architecture/Interface - USB 2.0/USB-DM_1 -> Net-(J9-Dn1)
- R59 pad 1: Net-(C94-Pad2) -> Net-(C96-Pad2)
- R60 pad 2: Net-(C94-Pad2) -> Net-(C96-Pad2)
- R80 pad 2: Net-(C101-Pad2) -> Net-(C103-Pad2)
- R81 pad 1: Net-(C101-Pad2) -> Net-(C103-Pad2)
- R82 pad 2: Net-(C102-Pad2) -> Net-(C104-Pad2)
- R83 pad 1: Net-(C102-Pad2) -> Net-(C104-Pad2)
- SW1 pad 1: Net-(C101-Pad2) -> Net-(C103-Pad2)
- SW1 pad 2: Net-(C102-Pad2) -> Net-(C104-Pad2)
Routing:
- net /Project Architecture/Power - Connectors/+V_BAT2S: track 0.00 -> 40.6 mm, vias 0 -> 7
- net /Project Architecture/Power - Connectors/+V_ADAPTER: track 0.00 -> 34.9 mm, vias 0 -> 7
- net +VBAT: track 0.00 -> 29.1 mm, vias 0 -> 6
- net GND: track 0.00 -> 27.2 mm, vias 0 -> 24
- net +5V: track 0.00 -> 23.2 mm
- net /Project Architecture/Interface - USB 2.0/VBUS_1: track 0.00 -> 20.7 mm, vias 0 -> 3
- net /Project Architecture/Interface - USB 2.0/VBUS_2: track 0.00 -> 18.7 mm, vias 0 -> 3
- net /Project Architecture/Power - Generation/F_VIN_5V: track 0.00 -> 16.6 mm
- net /Project Architecture/Power - Generation/FB_5V: track 0.00 -> 9.87 mm
- net /Project Architecture/Power - Generation/EN_5V: track 0.00 -> 8.76 mm
- net Net-(U3-VCC): track 0.00 -> 5.17 mm
- net Net-(J9-Dn1): track 0.00 -> 4.87 mm
- net Net-(J10-Dn1): track 0.00 -> 4.68 mm
- net Net-(J10-Dp1): track 0.00 -> 4.15 mm
- net Net-(J9-Dp1): track 0.00 -> 4.15 mm
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
Commit message: Update Schematic
Parts:
- removed C14, C15: 2.2uF 100V 0603, Duc:C0603
- removed FB2: 1k @ 100MHz, Duc_Library:L0805
- C52, C58, C64, C70, C76, C82: value 4.7uF 50V 0603 -> 4.7uF 50V 0402; footprint Duc:C0603 -> Duc:C0402
- C53, C54, C56, C57, C59, C60, C62, C63, C65, C66, C68, C69, C71, C72, C74, C75, C77, C78, C80, C81, C83, C84, C86, C87: value 100nF 50V 0603 -> 100nF 50V 0402; footprint Duc:C0603 -> Duc:C0402
- C55, C61, C67, C73, C79, C85: value 470nF 50V 0603 -> 470nF 50V 0402; footprint Duc:C0603 -> Duc:C0402
- C89, C91: footprint Duc_Library:C0402 -> Duc:C0402
- R10, R12, R15, R16, R18, R21, R22, R24, R27, R28, R30, R33, R34, R36, R39, R40, R42, R9: value 220R 0.1% 0603 -> 220R 0.1% 0402; footprint Duc:R0603 -> Duc:R0402
- R11, R14, R17, R20, R23, R26, R29, R32, R35, R38, R41, R8: value 1K 0.1% 0603 -> 1K 0.1% 0402; footprint Duc:R0603 -> Duc:R0402
- R13, R19, R25, R31, R37, R7: value 1R 0.1% 0603 -> 1R 0.1% 0402; footprint Duc:R0603 -> Duc:R0402
- R43, R44, R45, R46, R47, R48, R49, R50, R51, R52: footprint Duc_Library:R0402 -> Duc:R0402
- moved R6 129.6 mm to (227.7, 53.8), turned to 0 degrees
- moved L1 129.6 mm to (223.9, 55.1), turned to 90 degrees
- moved U4 128.8 mm to (227.8, 55.9)
- moved C13 126.3 mm to (230.6, 55.7), turned to 90 degrees
- moved C78 126.2 mm to (186.8, 95.8)
- moved C16 122.2 mm to (228.3, 71.7), turned to 90 degrees
- moved C66 119.5 mm to (183.2, 95.1)
- moved C60 117.9 mm to (183.2, 85.2)
- moved C54 109.2 mm to (186.8, 85.7)
- moved C84 100.8 mm to (186.7, 105.5)
- moved C72 100.3 mm to (183.2, 105.1)
- moved C77 97.2 mm to (155.1, 89.3), turned to -90 degrees
- moved C76 95.2 mm to (153.9, 89.3), turned to -90 degrees
- moved C63 94.1 mm to (155.5, 68.8), turned to 90 degrees
- moved R31 91.9 mm to (154.6, 90.8)
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Connections:
- C16 pad 2: Net-(U4-VIN) -> +5V
- U4 pad 2: Net-(U4-VIN) -> +5V
Routing:
- net GND: track 27.2 -> 47.3 mm, vias 24 -> 9
- net +3V3: track 0.00 -> 19.7 mm
- net +5V: track 23.2 -> 41.9 mm
- net +VBAT: track 29.1 -> 35.1 mm
- net /Project Architecture/Power - Generation/SW_3V3: track 0.00 -> 5.04 mm
- net Net-(U4-FB): track 0.00 -> 4.50 mm
- net /Project Architecture/Power - Generation/EN_3V3: track 0.00 -> 4.15 mm, vias 0 -> 2
- net /Project Architecture/Motor Control - Pinky/VCC_P: track 0.00 -> 2.86 mm
- net /Project Architecture/Motor Control - Ring/VCC_R: track 0.00 -> 2.86 mm
- net /Project Architecture/Motor Control - Middle/VCC_M: track 0.00 -> 2.82 mm
- net /Project Architecture/Power - Generation/F_VIN_5V: track 16.6 -> 14.6 mm
- net /Project Architecture/Motor Control - Thumb 2/VCC_T2: track 0.00 -> 1.59 mm
- net Net-(U4-PG): track 0.00 -> 1.49 mm
- net Net-(U3-RT): track 1.73 -> 2.89 mm
- net /Project Architecture/Motor Control - Index/VCC_I: track 0.00 -> 1.14 mm
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
Commit message: Update Schematic
Parts:
- moved C20 63.0 mm to (168.8, 92.6)
- moved C21 63.0 mm to (168.8, 94.4)
- moved C22 62.9 mm to (168.8, 96.2)
- moved C23 62.9 mm to (168.8, 98.0)
- moved C24 62.8 mm to (168.8, 99.8)
- moved C25 56.9 mm to (168.8, 101.6), turned to 0 degrees
- moved C26 56.8 mm to (168.8, 103.4), turned to 0 degrees
- moved C27 56.8 mm to (168.8, 105.2), turned to 0 degrees
- moved C28 56.8 mm to (168.8, 107.0), turned to 0 degrees
- moved C29 56.7 mm to (168.8, 108.8), turned to 0 degrees
- moved C72 36.6 mm to (147.3, 111.9), turned to 90 degrees
- moved C66 36.2 mm to (147.3, 99.2), turned to 90 degrees
- moved C60 36.0 mm to (147.3, 86.3), turned to 90 degrees
- moved R16 35.1 mm to (123.0, 59.4)
- moved C61 35.1 mm to (123.0, 58.2)
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Routing:
- net /Project Architecture/Power - Connectors/+V_BAT2S: track 40.6 -> 6.21 mm, vias 7 -> 3
- net /Project Architecture/Power - Connectors/+V_ADAPTER: track 34.9 -> 7.39 mm, vias 7 -> 3
- net +VBAT: track 35.1 -> 11.0 mm, vias 6 -> 0
- net /Project Architecture/Interface - USB 2.0/VBUS_2: track 18.7 -> 31.8 mm, vias 3 -> 0
- net /Project Architecture/Interface - USB 2.0/VBUS_1: track 20.7 -> 27.6 mm, vias 3 -> 0
- net GND: track 47.3 -> 42.8 mm, vias 9 -> 5
- net /Project Architecture/Motor Control - Pinky/OUT2_P: track 0.00 -> 2.66 mm, vias 0 -> 1
- net /Project Architecture/Motor Control - Pinky/_DIAG_P: track 0.00 -> 1.01 mm, vias 0 -> 1
- net Net-(J10-Dp1): track 4.15 -> 4.95 mm
- net /Project Architecture/Interface - USB 2.0/VBUS_DET2: track 2.07 -> 1.34 mm, vias 1 -> 0
- net Net-(J9-Dp1): track 4.15 -> 4.87 mm
- net /Project Architecture/Interface - USB 2.0/VBUS_DET1: track 2.07 -> 1.37 mm, vias 1 -> 0

Commit message: Update Schematic & PCB
Parts:
- removed R54, R56: 10K 0.1% 0603, Duc:R0603
- C10, C11, C13, C16, C17, C18, C5, C6, C9: footprint Duc_Library:C1206 -> Duc:C1206
- C92, C93, R53, R55, U14, U15: moved to F.Cu
- FB1, L2, L3: footprint Duc_Library:L0805 -> Duc:L0805
- TP1, TP10, TP11, TP12, TP13, TP14, TP15, TP16, TP17, TP18, TP19, TP2, TP20, TP21, TP22, TP23, TP24, TP25, TP26, TP27, TP28, TP29, TP3, TP30, TP31, TP32, TP33, TP34, TP35, TP36, TP37, TP38, TP39, TP4, TP40, TP41, TP42, TP43, TP44, TP45, TP46, TP47, TP48, TP49, TP5, TP50, TP51, TP52, TP53, TP54, TP55, TP56, TP57, TP58, TP59, TP6, TP60, TP61, TP62, TP63, TP64, TP65, TP66, TP67, TP68, TP69, TP7, TP70, TP71, TP72, TP73, TP74, TP75, TP76, TP77, TP78, TP79, TP8, TP80, TP81, TP82, TP83, TP84, TP85, TP86, TP87, TP88, TP89, TP9, TP90, TP91: footprint Duc_Library:TestPoint_Pad_D0.5mm -> Duc:TestPoint_Pad_D0.5mm
- U10, U11, U12, U13, U8, U9: footprint Duc_Library:UQFN-28_L6.0-W6.0-P0.65-BL-EP4.0 -> Duc:UQFN-28_L6.0-W6.0-P0.65-BL-EP4.0
- U3: footprint Duc_Library:QFN-30_L6.0-W4.0-P0.50_TLVM13630RDHR -> Duc:QFN-30_L6.0-W4.0-P0.50_TLVM13630RDHR
- U6, U7: footprint Duc_Library:LQFP-64_L10.0-W10.0-P0.50-LS12.0-BL -> Duc:LQFP-64_L10.0-W10.0-P0.50-LS12.0-BL
- moved R34 133.9 mm to (189.4, 71.6), turned to -90 degrees
- moved R32 131.0 mm to (188.2, 71.6), turned to -90 degrees
- moved C57 121.7 mm to (188.2, 69.6), turned to 90 degrees
- moved R35 119.5 mm to (172.7, 72.7), turned to 90 degrees
- moved R33 118.5 mm to (173.9, 72.7), turned to 90 degrees
- moved R10 117.0 mm to (189.4, 67.6), turned to -90 degrees
- moved C69 114.2 mm to (168.3, 69.8), turned to 180 degrees
- moved R8 113.7 mm to (188.2, 67.6), turned to -90 degrees
- moved R36 105.4 mm to (165.2, 91.7), turned to -90 degrees
- moved R22 104.2 mm to (165.4, 73.1), turned to -90 degrees
- moved R20 103.9 mm to (166.6, 73.1), turned to -90 degrees
- moved R11 103.5 mm to (177.4, 76.0)
- moved R9 101.9 mm to (177.4, 74.8)
- moved R40 101.1 mm to (184.4, 75.5)
- moved R38 100.1 mm to (184.4, 74.3)
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Connections:
- net /Project Architecture/Interface - USB 2.0/USB-DM_1 renamed /Project Architecture/Interface - USB 2.0/USB1_N
- net /Project Architecture/Interface - USB 2.0/USB-DP_1 renamed /Project Architecture/Interface - USB 2.0/USB1_P
- D7 pad 1: Net-(J10-Dn1) -> Net-(J10-Dp1)
- D7 pad 3: Net-(J10-Dp1) -> Net-(J10-Dn1)
- D7 pad 4: /Project Architecture/Interface - USB 2.0/USB-DP_2 -> /Project Architecture/Interface - USB 2.0/USB2_N
- D7 pad 6: /Project Architecture/Interface - USB 2.0/USB-DM_2 -> /Project Architecture/Interface - USB 2.0/USB2_P
- D8 pad 1: /Project Architecture/Interface - FD-CAN/FDCAN_P -> /Project Architecture/Interface - FD-CAN/FDCAN_N
- D8 pad 2: /Project Architecture/Interface - FD-CAN/FDCAN_N -> /Project Architecture/Interface - FD-CAN/FDCAN_P
- J3 pad 4: /Project Architecture/Motor Control - Index/OUT1_I -> /Project Architecture/Motor Control - Index/OUT2_I
- J3 pad 9: /Project Architecture/Motor Control - Index/OUT2_I -> /Project Architecture/Motor Control - Index/OUT1_I
- J4 pad 4: /Project Architecture/Motor Control - Middle/OUT1_M -> /Project Architecture/Motor Control - Middle/OUT2_M
- J4 pad 9: /Project Architecture/Motor Control - Middle/OUT2_M -> /Project Architecture/Motor Control - Middle/OUT1_M
- J5 pad 4: /Project Architecture/Motor Control - Ring/OUT1_R -> /Project Architecture/Motor Control - Ring/OUT2_R
- J5 pad 9: /Project Architecture/Motor Control - Ring/OUT2_R -> /Project Architecture/Motor Control - Ring/OUT1_R
- J6 pad 4: /Project Architecture/Motor Control - Pinky/OUT1_P -> /Project Architecture/Motor Control - Pinky/OUT2_P
- J6 pad 9: /Project Architecture/Motor Control - Pinky/OUT2_P -> /Project Architecture/Motor Control - Pinky/OUT1_P
- J7 pad 4: /Project Architecture/Motor Control - Thumb 1/OUT1_T1 -> /Project Architecture/Motor Control - Thumb 1/OUT2_T1
- J7 pad 9: /Project Architecture/Motor Control - Thumb 1/OUT2_T1 -> /Project Architecture/Motor Control - Thumb 1/OUT1_T1
- J8 pad 4: /Project Architecture/Motor Control - Thumb 2/OUT1_T2 -> /Project Architecture/Motor Control - Thumb 2/OUT2_T2
- J8 pad 9: /Project Architecture/Motor Control - Thumb 2/OUT2_T2 -> /Project Architecture/Motor Control - Thumb 2/OUT1_T2
- R53 pad 1: /Project Architecture/Interface - FD-CAN/FDCAN1_TX -> /Project Architecture/Interface - FD-CAN/FDCAN2_TX
- R55 pad 1: /Project Architecture/Interface - FD-CAN/FDCAN2_TX -> /Project Architecture/Interface - FD-CAN/FDCAN1_TX
- TP69 pad 1: /Project Architecture/Interface - USB 2.0/USB-DP_2 -> /Project Architecture/Interface - USB 2.0/USB2_P
- TP71 pad 1: /Project Architecture/Interface - USB 2.0/USB-DM_2 -> /Project Architecture/Interface - USB 2.0/USB2_N
- U14 pad 1: /Project Architecture/Interface - FD-CAN/FDCAN1_TX -> /Project Architecture/Interface - FD-CAN/FDCAN2_TX
- U14 pad 4: /Project Architecture/Interface - FD-CAN/FDCAN1_RX -> /Project Architecture/Interface - FD-CAN/FDCAN2_RX
- U14 pad 8: Net-(U14-S) -> GND
- U15 pad 1: /Project Architecture/Interface - FD-CAN/FDCAN2_TX -> /Project Architecture/Interface - FD-CAN/FDCAN1_TX
- U15 pad 4: /Project Architecture/Interface - FD-CAN/FDCAN2_RX -> /Project Architecture/Interface - FD-CAN/FDCAN1_RX
- U15 pad 8: Net-(U15-S) -> GND
- U6 pad 36: /Project Architecture/MCU - IOs/PWMA_I -> /Project Architecture/MCU - IOs/PWMB_I
- U6 pad 37: /Project Architecture/MCU - IOs/PWMB_I -> /Project Architecture/MCU - IOs/PWMA_I
- U7 pad 10: /Project Architecture/MCU - IOs/PWMA_R -> /Project Architecture/MCU - IOs/PWMB_R
- U7 pad 11: /Project Architecture/MCU - IOs/PWMB_R -> /Project Architecture/MCU - IOs/PWMA_R
- U7 pad 12: /Project Architecture/MCU - IOs/ECA_M -> /Project Architecture/MCU - IOs/ECB_M
- U7 pad 13: /Project Architecture/MCU - IOs/ECB_M -> /Project Architecture/MCU - IOs/ECA_M
- U7 pad 20: /Project Architecture/MCU - IOs/ECA_R -> /Project Architecture/MCU - IOs/ECB_R
- U7 pad 21: /Project Architecture/MCU - IOs/ECB_R -> /Project Architecture/MCU - IOs/ECA_R
- U7 pad 38: /Project Architecture/MCU - IOs/ECA_P -> /Project Architecture/MCU - IOs/ECB_P
- U7 pad 39: /Project Architecture/MCU - IOs/ECB_P -> /Project Architecture/MCU - IOs/ECA_P
- U7 pad 45: /Project Architecture/Interface - USB 2.0/USB-DM_2 -> /Project Architecture/Interface - USB 2.0/USB2_N
- U7 pad 46: /Project Architecture/Interface - USB 2.0/USB-DP_2 -> /Project Architecture/Interface - USB 2.0/USB2_P
- U7 pad 8: /Project Architecture/MCU - IOs/PWMA_M -> /Project Architecture/MCU - IOs/PWMB_M
- U7 pad 9: /Project Architecture/MCU - IOs/PWMB_M -> /Project Architecture/MCU - IOs/PWMA_M
Routing:
- net /Project Architecture/Interface - USB 2.0/VBUS_DET2: track 1.34 -> 78.1 mm, vias 0 -> 2
- net /Project Architecture/Interface - USB 2.0/VBUS_DET1: track 1.37 -> 77.7 mm, vias 0 -> 2
- net /Project Architecture/MCU - IOs/PWMA_P: track 0.00 -> 75.5 mm, vias 0 -> 2
- net /Project Architecture/MCU - IOs/PWMB_P: track 0.00 -> 72.2 mm, vias 0 -> 2
- net /Project Architecture/MCU - IOs/ECA_P: track 0.00 -> 69.8 mm, vias 0 -> 2
- net /Project Architecture/Interface - USB 2.0/USB1_N: track 1.04 -> 70.4 mm, vias 1 -> 2
- net /Project Architecture/Interface - USB 2.0/USB1_P: track 1.04 -> 70.0 mm, vias 1 -> 2
- net /Project Architecture/Interface - USB 2.0/USB2_N: track 0.00 -> 68.3 mm, vias 0 -> 2
- net /Project Architecture/MCU - IOs/ECB_P: track 0.00 -> 66.8 mm, vias 0 -> 2
- net /Project Architecture/Interface - USB 2.0/USB2_P: track 0.00 -> 65.1 mm, vias 0 -> 2
- net /Project Architecture/MCU - IOs/ECC_P: track 0.00 -> 63.8 mm, vias 0 -> 3
- net /Project Architecture/MCU - IOs/EN_R: track 0.00 -> 54.4 mm, vias 0 -> 2
- net /Project Architecture/MCU - IOs/PWMA_T2: track 0.00 -> 50.7 mm, vias 0 -> 2
- net /Project Architecture/MCU - IOs/ECC_R: track 0.00 -> 50.6 mm, vias 0 -> 2
- net /Project Architecture/MCU - IOs/ECB_R: track 0.00 -> 50.2 mm, vias 0 -> 2
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Other:
- rule solder_mask_min_width: 0.1 -> 0.05
