File: Master_Hand_Kicad.kicad_pcb (KiCad board)
At the start: 6 copper layers, 79 x 65.8 mm, 340 parts, among them J1 XT60PW-M, J10 TYPE-C 16PIN 2MD, J11 1.25-3PLTDK, J12 5025982393, J13 PH2.54-2X3P-H25, J14 PH2.54-2X3P-H25, J15 PH2.54-2X3P-H25, J2 DC-044A-20A, J3 BM09B-SRSS-TB, J4 BM09B-SRSS-TB, J5 BM09B-SRSS-TB, J6 BM09B-SRSS-TB, J7 BM09B-SRSS-TB, J8 BM09B-SRSS-TB, J9 TYPE-C 16PIN 2MD, Q1 HV10N03, Q2 HV10N03, Q3 2SC1815, SW1 DSIC02LSGET, U1 LM74700QDBVRQ1, U10 TB9051FTG,EL, U11 TB9051FTG,EL, U12 TB9051FTG,EL, U13 TB9051FTG,EL, U14 TJA1051T/3, U15 TJA1051T/3, U16 SHT40-N-NF, U17 SHT40-N-NF, U2 LM74700QDBVRQ1, U3 TPSM63603RDHR, U4 TPS62162DSG, U5 TLV75533PDBVR, U6 STM32G474RET6, U7 STM32G474RET6, U8 TB9051FTG,EL, U9 TB9051FTG,EL, X1 X322516MLB4SI, X2 X322516MLB4SI

Commit message: Update SCH & PCB
Parts:
- moved C81 140.3 mm to (188.6, 69.8), turned to 180 degrees
- moved C87 112.2 mm to (188.2, 71.4), turned to 90 degrees
- moved C85 70.0 mm to (155.8, 108.3), turned to -90 degrees
- moved C10 28.5 mm to (236.4, 100.9)
- moved C11 28.5 mm to (236.4, 98.4)
- moved C12 28.5 mm to (240.7, 111.8)
- moved C13 28.5 mm to (234.4, 84.0)
- moved C16 28.5 mm to (232.1, 100.0)
- moved C17 28.5 mm to (235.5, 95.8)
- moved C18 28.5 mm to (235.0, 91.6)
- moved C5 28.5 mm to (232.2, 105.3)
- moved C6 28.5 mm to (240.3, 106.9)
- moved C7 28.5 mm to (228.3, 111.1)
- moved C8 28.5 mm to (227.6, 104.0)
- moved C9 28.5 mm to (229.7, 105.3)
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Connections:
- U6 pad 14: /Project Architecture/MCU - IOs/OCM_T2 -> /Project Architecture/MCU - IOs/OCM_T1
- U6 pad 17: /Project Architecture/MCU - IOs/OCM_T1 -> /Project Architecture/MCU - IOs/OCM_T2
- U6 pad 2: /Project Architecture/MCU - IOs/DIAG_T2 -> /Project Architecture/MCU - IOs/DIAG_T1
- U6 pad 20: /Project Architecture/MCU - IOs/ECA_T1 -> /Project Architecture/MCU - IOs/ECB_T1
- U6 pad 21: /Project Architecture/MCU - IOs/ECB_T1 -> /Project Architecture/MCU - IOs/ECA_T1
- U6 pad 3: /Project Architecture/MCU - IOs/DIAG_T1 -> /Project Architecture/MCU - IOs/DIAG_T2
- U6 pad 38: /Project Architecture/MCU - IOs/ECA_I -> /Project Architecture/MCU - IOs/ECB_I
- U6 pad 39: /Project Architecture/MCU - IOs/ECB_I -> /Project Architecture/MCU - IOs/ECA_I
Routing:
- net /Project Architecture/MCU - IOs/EN_T2: track 0.00 -> 62.0 mm, vias 0 -> 2
- net /Project Architecture/Motor Control - Thumb 2/_OCM_T2: track 2.05 -> 60.2 mm
- net /Project Architecture/Motor Control - Pinky/_OCM_P: track 3.58 -> 52.4 mm
- net /Project Architecture/Motor Control - Index/_OCM_I: track 2.94 -> 46.2 mm
- net /Project Architecture/Motor Control - Thumb 1/_OCM_T1: track 3.17 -> 46.2 mm
- net /Project Architecture/MCU - IOs/ECB_T1: track 3.02 -> 46.0 mm
- net /Project Architecture/MCU - IOs/PWMA_T1: track 2.44 -> 45.2 mm
- net /Project Architecture/Motor Control - Thumb 2/_DIAG_T2: track 0.00 -> 42.6 mm, vias 0 -> 2
- net /Project Architecture/MCU - IOs/PWMB_T1: track 3.69 -> 45.6 mm
- net /Project Architecture/MCU - IOs/ECA_T1: track 3.87 -> 45.4 mm
- net /Project Architecture/MCU - IOs/PWMA_I: track 1.27 -> 39.7 mm
- net /Project Architecture/MCU - IOs/EN_I: track 1.63 -> 39.8 mm, vias 1 -> 2
- net /Project Architecture/MCU - IOs/EN_T1: track 2.89 -> 40.7 mm
- net /Project Architecture/MCU - IOs/PWMB_I: track 2.06 -> 39.4 mm
- net GND: track 42.9 -> 6.55 mm
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