File: Master_Hand_Kicad.kicad_pcb (KiCad board)
At the start: 6 copper layers, 79 x 65.8 mm, 340 parts, among them J1 XT60PW-M, J10 TYPE-C 16PIN 2MD, J11 1.25-3PLTDK, J12 5025982393, J13 PH2.54-2X3P-H25, J14 PH2.54-2X3P-H25, J15 PH2.54-2X3P-H25, J2 DC-044A-20A, J3 BM09B-SRSS-TB, J4 BM09B-SRSS-TB, J5 BM09B-SRSS-TB, J6 BM09B-SRSS-TB, J7 BM09B-SRSS-TB, J8 BM09B-SRSS-TB, J9 TYPE-C 16PIN 2MD, Q1 HV10N03, Q2 HV10N03, Q3 2SC1815, SW1 DSIC02LSGET, U1 LM74700QDBVRQ1, U10 TB9051FTG,EL, U11 TB9051FTG,EL, U12 TB9051FTG,EL, U13 TB9051FTG,EL, U14 TJA1051T/3, U15 TJA1051T/3, U16 SHT40-N-NF, U17 SHT40-N-NF, U2 LM74700QDBVRQ1, U3 TPSM63603RDHR, U4 TPS62162DSG, U5 TLV75533PDBVR, U6 STM32G474RET6, U7 STM32G474RET6, U8 TB9051FTG,EL, U9 TB9051FTG,EL, X1 X322516MLB4SI, X2 X322516MLB4SI

Commit message: Update Schematic & PCB
Parts:
- removed L2, L3: PBBHAQ2012H-102T10, Duc:L0805
- added FB2: 1k @ 100MHz, Duc:L0805, F.Cu at (220.8, 92.5)
- added FB3: 1k @ 100MHz, Duc:L0805, F.Cu at (220.8, 95.8)
- C1, C100, C101, C102, C103, C104, C2, C3, C32, C33, C34, C35, C38, C4, C41, C42, C43, C44, C47, C92, C93, C94, C95, C97, C98, C99: value 100nF 50V 0603 -> CAP CER 0603
- C10, C16: value 10uF 50V 1206 -> CAP CER 1206
- C11: value 100nF 50V 1206 -> CAP CER 1206
- C12: value 1uF 50V 0603 -> CAP CER 0603
- C13: value 22uF 50V 1206 -> CAP CER 1206
- C17, C18: value 1uF 50V 1206 -> CAP CER 1206
- C20, C21, C22, C23, C24, C25, C26, C27, C28, C29: value 10uF 50V 0603 -> CAP CER 0603
- C30, C36, C37, C39, C45, C46: value 1uF 10V 0603 -> CAP CER 0603
- C31, C40: value 4.7uF 16V 0603 -> CAP CER 0603
- C48, C49, C50, C51: value 8pF 16V 0603 -> CAP CER 0603
- C5, C6: value 4.7uF 100V 1206 -> CAP CER 1206
- C52, C58, C64, C70, C76, C82: value 4.7uF 50V 0402 -> CAP CER 0402
- C53, C54, C56, C57, C59, C60, C62, C63, C65, C66, C68, C69, C71, C72, C74, C75, C77, C78, C80, C81, C83, C84, C86, C87, C89, C91: value 100nF 50V 0402 -> CAP CER 0402
- C55, C61, C67, C73, C79, C85: value 470nF 50V 0402 -> CAP CER 0402
- C7, C8: value 2.2uF 100V 0603 -> CAP CER 0603
- C88, C90, C96: value 4.7uF 50V 0603 -> CAP CER 0603
- C9: value 10uF 100V 1206 -> CAP CER 1206
- D10: value Orange 0603 -> LED 0603
- D11: value Yellow 0603 -> LED 0603
- D12: value Green 0603 -> LED 0603
- D13, D2, D5: value Blue 0603 -> LED 0603
- D14: value White 0603 -> LED 0603
- D16, D17: value Red 0603 -> LED 0603
- D9: value RED 0603 -> LED 0603
- J1: value XT60PW-M -> XT30PW-F; footprint Duc:CONN-TH_XT60PW-M -> Duc:CONN-TH_XT30PW-F-1; moved to B.Cu
- J2: value DC-044A-20A -> KF350-3.5-2P; footprint Duc:DC-IN-TH_DC-044A-20A -> Duc:CONN-TH_P3.50_KF350-3.5-2P; moved to B.Cu
- R1: value 41.2K 0.1% 0603 -> RES 0603
- R10, R12, R15, R16, R18, R21, R22, R24, R27, R28, R30, R33, R34, R36, R39, R40, R42, R9: value 220R 0.1% 0402 -> RES 0402
- R11, R14, R17, R20, R23, R26, R29, R32, R35, R38, R41, R45, R50, R8: value 1K 0.1% 0402 -> RES 0402
- R13, R19, R25, R31, R37, R7: value 1R 0.1% 0402 -> RES 0402
- R2, R5, R53, R55, R70, R71, R72, R73, R80, R81, R82, R83: value 10K 0.1% 0603 -> RES 0603
- R3: value 40.2K 0.1% 0603 -> RES 0603
- R4: value 13K 0.1% 0603 -> RES 0603
- R43, R48: value 430K 0.1% 0402 -> RES 0402
- R44, R49: value 620K 0.1% 0402 -> RES 0402
- R46, R47, R51, R52: value 5.1K 0.1% 0402 -> RES 0402
- R57, R58: value 2.2K 0.1% 0603 -> RES 0603
- R59, R60: value 60R4 0.1% 0603 -> RES 0603
- R6, R74, R77, R79: value 100K 0.1% 0603 -> RES 0603
- R61, R62, R63, R67, R68: value 330R 0.1% 0603 -> RES 0603
- R64, R65, R66: value 100R 0.1% 0603 -> RES 0603
- R69: value 470R 0.1% 0603 -> RES 0603
- R75: value 47K 0.1% 0603 -> RES 0603
- R76, R78: value 0R 0.1% 0603 -> RES 0603
- moved U3 63.5 mm to (173.4, 115.5)
- moved C72 9.61 mm to (147.7, 102.3), turned to 180 degrees
- moved C60 9.60 mm to (147.6, 76.7), turned to 180 degrees
- moved C66 9.60 mm to (147.6, 89.6), turned to 180 degrees
- moved J2 9.09 mm to (163.9, 119.5), turned to 180 degrees
- moved C2 7.50 mm to (147.1, 117.1)
- moved C1 7.45 mm to (147.1, 114.0)
- moved Q2 7.25 mm to (157.6, 116.6)
- moved U2 6.92 mm to (157.6, 121.1)
- moved C4 6.87 mm to (154.2, 121.5)
- moved C3 6.87 mm to (154.2, 118.4)
- moved Q1 6.24 mm to (150.8, 116.6)
- moved U1 6.22 mm to (150.8, 121.1)
- moved J8 5.10 mm to (161.5, 106.9)
- moved J3 5.10 mm to (161.6, 81.5)
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Connections:
- D7 pad 1: Net-(J10-Dp1) -> Net-(J10-Dn1)
- D7 pad 3: Net-(J10-Dn1) -> Net-(J10-Dp1)
- D7 pad 4: /Project Architecture/Interface - USB 2.0/USB2_N -> /Project Architecture/Interface - USB 2.0/USB2_P
- D7 pad 6: /Project Architecture/Interface - USB 2.0/USB2_P -> /Project Architecture/Interface - USB 2.0/USB2_N
- J1 pad 1: GND -> /Project Architecture/Power - Connectors/+V_BAT2S
- J1 pad 2: /Project Architecture/Power - Connectors/+V_BAT2S -> GND
- J2 pad 1: /Project Architecture/Power - Connectors/+V_ADAPTER -> GND
- J2 pad 2: GND -> /Project Architecture/Power - Connectors/+V_ADAPTER
Routing:
- net /Project Architecture/MCU - IOs/PWMA_P: track 76.5 -> 2.90 mm
- net /Project Architecture/MCU - IOs/ECA_P: track 74.8 -> 2.68 mm
- net /Project Architecture/MCU - IOs/ECB_P: track 71.9 -> 4.43 mm
- net /Project Architecture/MCU - IOs/PWMB_P: track 73.2 -> 6.67 mm
- net /Project Architecture/MCU - IOs/EN_T2: track 62.0 -> 4.08 mm
- net /Project Architecture/Motor Control - Thumb 2/_OCM_T2: track 60.2 -> 3.37 mm
- net /Project Architecture/MCU - IOs/ECC_P: track 63.3 -> 8.89 mm
- net /Project Architecture/MCU - IOs/EN_R: track 54.4 -> 2.47 mm
- net /Project Architecture/MCU - IOs/ECA_T2: track 53.4 -> 2.77 mm
- net /Project Architecture/MCU - IOs/PWMB_T2: track 53.5 -> 3.87 mm
- net /Project Architecture/MCU - IOs/PWMA_T2: track 53.3 -> 3.75 mm
- net /Project Architecture/Motor Control - Pinky/_OCM_P: track 52.4 -> 3.58 mm
- net /Project Architecture/MCU - IOs/ECB_T2: track 52.2 -> 4.26 mm
- net /Project Architecture/MCU - IOs/ECA_R: track 54.4 -> 7.21 mm
- net /Project Architecture/MCU - IOs/ECB_R: track 52.5 -> 6.87 mm
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
Commit message: Update SCH & PCB
Parts:
- moved R16 1.17 mm to (162.8, 74.4)
- moved R14 1.17 mm to (162.8, 75.6)
Connections:
- U7 pad 10: /Project Architecture/MCU - IOs/PWMB_R -> /Project Architecture/MCU - IOs/PWMB_M
- U7 pad 11: /Project Architecture/MCU - IOs/PWMA_R -> /Project Architecture/MCU - IOs/PWMA_M
- U7 pad 8: /Project Architecture/MCU - IOs/PWMB_M -> /Project Architecture/MCU - IOs/PWMA_R
- U7 pad 9: /Project Architecture/MCU - IOs/PWMA_M -> /Project Architecture/MCU - IOs/PWMB_R
Routing:
- net /Project Architecture/MCU - IOs/PWMA_P: track 2.90 -> 71.8 mm
- net /Project Architecture/MCU - IOs/EN_P: track 2.34 -> 70.6 mm
- net /Project Architecture/MCU - IOs/PWMB_P: track 6.67 -> 70.7 mm
- net /Project Architecture/MCU - IOs/ECA_P: track 2.68 -> 66.1 mm
- net /Project Architecture/MCU - IOs/ECB_P: track 4.43 -> 65.2 mm
- net /Project Architecture/MCU - IOs/PWMB_R: track 2.74 -> 55.3 mm
- net /Project Architecture/Motor Control - Pinky/_OCM_P: track 3.58 -> 52.7 mm
- net /Project Architecture/MCU - IOs/PWMA_R: track 3.64 -> 52.6 mm
- net /Project Architecture/MCU - IOs/ECA_R: track 7.21 -> 55.6 mm
- net /Project Architecture/MCU - IOs/EN_R: track 2.47 -> 50.5 mm
- net /Project Architecture/MCU - IOs/ECB_R: track 6.87 -> 53.6 mm
- net /Project Architecture/Motor Control - Pinky/_DIAG_P: track 3.08 -> 46.3 mm
- net /Project Architecture/Motor Control - Ring/_DIAG_R: track 3.06 -> 38.6 mm
- net /Project Architecture/Motor Control - Ring/_OCM_R: track 3.50 -> 31.7 mm
- net /Project Architecture/MCU - IOs/ECB_M: track 2.83 -> 26.8 mm
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
Commit message: Update Schematic & PCB
Parts:
- removed C9: CAP CER 1206, Duc:C1206
- C10, C11, C5, C6, D1, FB1, L1, U3, U4, U5: moved to F.Cu
- C12, C7, C8: value CAP CER 0603 -> CAP CER 0402; footprint Duc:C0603 -> Duc:C0402; moved to F.Cu
- C13, C18: value CAP CER 1206 -> CAP CER 0603; footprint Duc:C1206 -> Duc:C0603; moved to F.Cu
- C16, C17: value CAP CER 1206 -> CAP CER 0402; footprint Duc:C1206 -> Duc:C0402; moved to F.Cu
- C19: value 25SVPF330M -> SM337M025E0800; footprint Duc:CAP-SMD_BD10.0-L10.3-W10.3-LS11.0-FD -> Duc:CAP-SMD_BD6.3-L6.6-W6.6-FD-1
- C20, C21, C22, C23, C24, C25, C26, C27, C28, C29, C56, C62, C68, C74, C80, C86: moved to B.Cu
- R1, R2, R3, R4, R5, R6: value RES 0603 -> RES 0402; footprint Duc:R0603 -> Duc:R0402; moved to F.Cu
- moved D1 75.9 mm to (157.7, 119.5), turned to -90 degrees
- moved R3 69.6 mm to (173.6, 122.0), turned to -90 degrees
- moved C17 68.2 mm to (168.7, 109.7)
- moved C11 68.0 mm to (170.0, 113.1), turned to 90 degrees
- moved C18 67.5 mm to (168.7, 103.9), turned to 180 degrees
- moved C7 66.5 mm to (161.9, 113.7), turned to -90 degrees
- moved C12 65.0 mm to (176.5, 122.0)
- moved R5 64.9 mm to (174.9, 122.0), turned to 90 degrees
- moved U4 64.9 mm to (172.6, 111.2), turned to 90 degrees
- moved U5 64.9 mm to (168.7, 106.9)
- moved R6 63.6 mm to (174.5, 110.4), turned to 90 degrees
- moved C13 63.6 mm to (176.3, 109.9), turned to 110 degrees
- moved C5 63.6 mm to (170.0, 118.4)
- moved C6 63.1 mm to (178.6, 119.9)
- moved R1 61.2 mm to (168.2, 121.6)
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Connections:
- U6 pad 10: /Project Architecture/MCU - IOs/PWMA_T1 -> /Project Architecture/MCU - IOs/PWMA_T2
- U6 pad 11: /Project Architecture/MCU - IOs/PWMB_T1 -> /Project Architecture/MCU - IOs/PWMB_T2
- U6 pad 12: /Project Architecture/MCU - IOs/ECA_T2 -> /Project Architecture/MCU - IOs/ECA_T1
- U6 pad 13: /Project Architecture/MCU - IOs/ECB_T2 -> /Project Architecture/MCU - IOs/ECB_T1
- U6 pad 20: /Project Architecture/MCU - IOs/ECB_T1 -> /Project Architecture/MCU - IOs/ECB_T2
- U6 pad 21: /Project Architecture/MCU - IOs/ECA_T1 -> /Project Architecture/MCU - IOs/ECA_T2
- U6 pad 38: /Project Architecture/MCU - IOs/ECB_I -> /Project Architecture/MCU - IOs/ECA_I
- U6 pad 39: /Project Architecture/MCU - IOs/ECA_I -> /Project Architecture/MCU - IOs/ECB_I
- U6 pad 8: /Project Architecture/MCU - IOs/PWMA_T2 -> /Project Architecture/MCU - IOs/PWMA_T1
- U6 pad 9: /Project Architecture/MCU - IOs/PWMB_T2 -> /Project Architecture/MCU - IOs/PWMB_T1
Routing:
- net /Project Architecture/MCU - IOs/ECC_P: track 3.09 -> 68.0 mm
- net /Project Architecture/MCU - IOs/PWMB_T2: track 3.87 -> 57.6 mm
- net /Project Architecture/MCU - IOs/PWMA_T2: track 3.75 -> 57.4 mm
- net /Project Architecture/MCU - IOs/EN_T2: track 4.08 -> 57.0 mm
- net /Project Architecture/MCU - IOs/ECA_T2: track 2.77 -> 55.7 mm
- net /Project Architecture/MCU - IOs/ECB_T2: track 4.26 -> 56.0 mm
- net /Project Architecture/MCU - IOs/ECC_T2: track 4.37 -> 55.7 mm, vias 3 -> 2
- net /Project Architecture/MCU - IOs/ECC_R: track 3.31 -> 53.3 mm
- net /Project Architecture/MCU - IOs/EN_T1: track 2.89 -> 43.5 mm
- net /Project Architecture/MCU - IOs/ECC_T1: track 3.19 -> 42.1 mm
- net /Project Architecture/Motor Control - Thumb 2/_DIAG_T2: track 3.14 -> 42.0 mm
- net /Project Architecture/MCU - IOs/PWMB_T1: track 4.64 -> 43.2 mm
- net /Project Architecture/MCU - IOs/PWMA_T1: track 5.52 -> 43.3 mm
- net /Project Architecture/MCU - IOs/PWMB_I: track 3.87 -> 41.6 mm
- net /Project Architecture/MCU - IOs/ECB_T1: track 3.98 -> 41.3 mm
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- added copper zone on B.Cu, net +3V3
- added copper zone on B.Cu, net +5V
- added copper zone on B.Cu, net /Project Architecture/Power - Generation/F_VIN_5V

Commit message: Update SCH & PCB
Parts:
- removed the C7 at (161.9, 113.7)
- removed the C8 at (167.4, 113.7)
- removed the FB1 at (164.7, 113.7)
- removed the TP2 at (145.2, 28.3)
- C43: renamed from C48; moved to B.Cu
- C44: renamed from C49; moved to B.Cu
- C45: renamed from C50; moved to B.Cu
- C46: renamed from C51; moved to B.Cu
- C91: renamed from C96; moved to B.Cu
- C95: renamed from C100; value CAP CER 0603 -> CAP CER 0402; footprint Duc:C0603 -> Duc:C0402
- C96: renamed from C101; value CAP CER 0603 -> CAP CER 0402; footprint Duc:C0603 -> Duc:C0402
- C97: renamed from C102; moved to B.Cu
- C98: renamed from C103; value CAP CER 0603 -> CAP CER 0402; footprint Duc:C0603 -> Duc:C0402
- C99: renamed from C104; value CAP CER 0603 -> CAP CER 0402; footprint Duc:C0603 -> Duc:C0402
- R55: renamed from R57; value RES 0603 -> RES 0402; footprint Duc:R0603 -> Duc:R0402
- R56: renamed from R58; value RES 0603 -> RES 0402; footprint Duc:R0603 -> Duc:R0402
- R59: renamed from R61; value RES 0603 -> RES 0402; footprint Duc:R0603 -> Duc:R0402
- R60: renamed from R62; value RES 0603 -> RES 0402; footprint Duc:R0603 -> Duc:R0402
- R61: renamed from R63; value RES 0603 -> RES 0402; footprint Duc:R0603 -> Duc:R0402
- R62: renamed from R64; value RES 0603 -> RES 0402; footprint Duc:R0603 -> Duc:R0402
- R63: renamed from R65; value RES 0603 -> RES 0402; footprint Duc:R0603 -> Duc:R0402
- R64: renamed from R66; value RES 0603 -> RES 0402; footprint Duc:R0603 -> Duc:R0402
- R65: renamed from R67; value RES 0603 -> RES 0402; footprint Duc:R0603 -> Duc:R0402
- R66: renamed from R68; value RES 0603 -> RES 0402; footprint Duc:R0603 -> Duc:R0402
- R67: renamed from R69; value RES 0603 -> RES 0402; footprint Duc:R0603 -> Duc:R0402
- R68: renamed from R70; value RES 0603 -> RES 0402; footprint Duc:R0603 -> Duc:R0402
- R69: renamed from R71; value RES 0603 -> RES 0402; footprint Duc:R0603 -> Duc:R0402
- R70: renamed from R72; value RES 0603 -> RES 0402; footprint Duc:R0603 -> Duc:R0402
- R71: renamed from R73; value RES 0603 -> RES 0402; footprint Duc:R0603 -> Duc:R0402
- R72: renamed from R74; moved to B.Cu
- R73: renamed from R75; moved to B.Cu
- R74: renamed from R76; value RES 0603 -> RES 0402; footprint Duc:R0603 -> Duc:R0402
- R75: renamed from R77; value RES 0603 -> RES 0402; footprint Duc:R0603 -> Duc:R0402
- R76: renamed from R78; value RES 0603 -> RES 0402; footprint Duc:R0603 -> Duc:R0402
- R77: renamed from R79; value RES 0603 -> RES 0402; footprint Duc:R0603 -> Duc:R0402
- R78: renamed from R80; value RES 0603 -> RES 0402; footprint Duc:R0603 -> Duc:R0402
- R79: renamed from R81; value RES 0603 -> RES 0402; footprint Duc:R0603 -> Duc:R0402
- R80: renamed from R82; value RES 0603 -> RES 0402; footprint Duc:R0603 -> Duc:R0402
- R81: renamed from R83; value RES 0603 -> RES 0402; footprint Duc:R0603 -> Duc:R0402
- X1, X2: moved to B.Cu
- moved C51 107.0 mm to (165.1, 78.7), turned to -90 degrees
- moved R76 106.1 mm to (152.1, 66.7), turned to -90 degrees
- moved C81 102.3 mm to (165.1, 104.2), turned to -90 degrees
- moved C31 89.0 mm to (196.0, 64.0), turned to -90 degrees
- moved R74 86.9 mm to (172.5, 63.4), turned to 90 degrees
- moved D14 83.2 mm to (146.4, 60.5), turned to 180 degrees
- moved D17 83.0 mm to (169.1, 76.3), turned to -90 degrees
- moved C75 83.0 mm to (165.2, 91.6), turned to -90 degrees
- moved D16 81.8 mm to (170.9, 76.3), turned to -90 degrees
- moved R64 80.3 mm to (149.1, 60.5), turned to 180 degrees
- moved R66 80.2 mm to (169.1, 73.6), turned to -90 degrees
- moved C28 80.0 mm to (187.9, 62.5), turned to -90 degrees
- moved R65 79.4 mm to (170.9, 73.6), turned to -90 degrees
- moved C32 79.3 mm to (191.8, 64.0), turned to 90 degrees
- moved D13 78.9 mm to (146.4, 62.3), turned to 180 degrees
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- renumbered C13 to C10, C16 to C11, C17 to C12, C18 to C13, C19 to C14, C20 to C15, C21 to C16, C22 to C17, C23 to C18, C24 to C19, C25 to C20, C26 to C21, C27 to C22, C28 to C23, C29 to C24, C30 to C25, C31 to C26, C32 to C27, C33 to C28, C34 to C29, C35 to C30, C36 to C31, C37 to C32, C38 to C33, C39 to C34, C40 to C35, C41 to C36, C42 to C37, C43 to C38, C44 to C39, C45 to C40, C46 to C41, C47 to C42, C52 to C47, C53 to C48, C54 to C49, C55 to C50, C56 to C51, C57 to C52, C58 to C53, C59 to C54, C60 to C55, C61 to C56, C62 to C57, C63 to C58, C64 to C59, C65 to C60, C66 to C61, C67 to C62, C68 to C63, C69 to C64, C70 to C65, C71 to C66, C72 to C67, C73 to C68, C74 to C69, C10 to C7, C75 to C70, C76 to C71, C77 to C72, C78 to C73, C79 to C74, C80 to C75, C81 to C76, C82 to C77, C83 to C78, C84 to C79, C11 to C8, C85 to C80, C86 to C81, C87 to C82, C88 to C83, C89 to C84, C90 to C85, C91 to C86, C92 to C87, C93 to C88, C94 to C89, C12 to C9, C95 to C90, C97 to C92, C98 to C93, C99 to C94, FB2 to FB1, FB3 to FB2, R55 to R54, R59 to R57, R60 to R58, TP11 to TP10, TP12 to TP11, TP13 to TP12, TP14 to TP13, TP15 to TP14, TP16 to TP15, TP17 to TP16, TP18 to TP17, TP19 to TP18, TP20 to TP19, TP3 to TP2, TP21 to TP20, TP22 to TP21, TP23 to TP22, TP24 to TP23, TP25 to TP24, TP26 to TP25, TP27 to TP26, TP28 to TP27, TP29 to TP28, TP30 to TP29, TP4 to TP3, TP31 to TP30, TP32 to TP31, TP33 to TP32, TP34 to TP33, TP35 to TP34, TP36 to TP35, TP37 to TP36, TP38 to TP37, TP39 to TP38, TP40 to TP39, TP5 to TP4, TP41 to TP40, TP42 to TP41, TP43 to TP42, TP44 to TP43, TP45 to TP44, TP46 to TP45, TP47 to TP46, TP48 to TP47, TP49 to TP48, TP50 to TP49, TP6 to TP5, TP51 to TP50, TP52 to TP51, TP53 to TP52, TP54 to TP53, TP55 to TP54, TP56 to TP55, TP57 to TP56, TP58 to TP57, TP59 to TP58, TP60 to TP59, TP7 to TP6, TP61 to TP60, TP62 to TP61, TP63 to TP62, TP64 to TP63, TP65 to TP64, TP66 to TP65, TP67 to TP66, TP68 to TP67, TP69 to TP68, TP70 to TP69, TP8 to TP7, TP71 to TP70, TP72 to TP71, TP73 to TP72, TP74 to TP73, TP75 to TP74, TP76 to TP75, TP77 to TP76, TP78 to TP77, TP79 to TP78, TP80 to TP79, TP9 to TP8, TP81 to TP80, TP82 to TP81, TP83 to TP82, TP84 to TP83, TP85 to TP84, TP86 to TP85, TP87 to TP86, TP88 to TP87, TP89 to TP88, TP90 to TP89, TP10 to TP9, TP91 to TP90
Connections:
- C35 pad 1: +A3V3 -> +3V3
- C36 pad 2: +A3V3 -> +3V3
- C37 pad 2: +A3V3 -> +3V3
- C38 pad 2: +A3V3 -> +3V3
- C39 pad 2: +A3V3 -> +3V3
- C40 pad 2: +3V3 -> +A3V3
- C5 pad 2: /Project Architecture/Power - Generation/F_VIN_5V -> +VBAT
- C6 pad 2: /Project Architecture/Power - Generation/F_VIN_5V -> +VBAT
- FB2 pad 1: +3V3 -> +A3V3
- J12 pad 11: /Project Architecture/Interface - Interconnects/SWCLK1 -> /Project Architecture/Interface - Interconnects/SWDIO2
- J12 pad 13: /Project Architecture/Interface - Interconnects/NRST1 -> /Project Architecture/Interface - Interconnects/SWCLK2
- J12 pad 15: /Project Architecture/Interface - Interconnects/SWDIO2 -> /Project Architecture/Interface - Interconnects/SWCLK1
- J12 pad 17: /Project Architecture/Interface - Interconnects/SWCLK2 -> /Project Architecture/Interface - Interconnects/SWDIO1
- J12 pad 19: /Project Architecture/Interface - Interconnects/NRST2 -> /Project Architecture/Interface - Interconnects/NRST1
- J12 pad 9: /Project Architecture/Interface - Interconnects/SWDIO1 -> /Project Architecture/Interface - Interconnects/NRST2
- R1 pad 2: /Project Architecture/Power - Generation/F_VIN_5V -> +VBAT
- U3 pad 18: /Project Architecture/Power - Generation/F_VIN_5V -> +VBAT
- U3 pad 19: /Project Architecture/Power - Generation/F_VIN_5V -> +VBAT
- U3 pad 3: /Project Architecture/Power - Generation/F_VIN_5V -> +VBAT
- U3 pad 4: /Project Architecture/Power - Generation/F_VIN_5V -> +VBAT
- U7 pad 16: +A3V3 -> +3V3
- U7 pad 26: /Project Architecture/MCU - IOs/BOARD_VERSION -> unconnected-(U7B-PB2-Pad26)
- U7 pad 32: +A3V3 -> +3V3
- U7 pad 48: +A3V3 -> +3V3
- U7 pad 64: +A3V3 -> +3V3
Routing:
- net /Project Architecture/Motor Control - Thumb 2/_OCM_T2: track 3.23 -> 62.3 mm
- net /Project Architecture/Interface - Interconnects/I2C_SDA: track 0.00 -> 57.8 mm, vias 0 -> 2
- net /Project Architecture/Interface - Interconnects/I2C_SCL: track 0.00 -> 55.0 mm, vias 0 -> 1
- net /Project Architecture/MCU - IOs/BOOT_1: track 0.00 -> 51.3 mm, vias 0 -> 2
- net /Project Architecture/MCU - IOs/I2C-SCL_1: track 0.00 -> 46.0 mm, vias 0 -> 2
- net /Project Architecture/MCU - IOs/I2C-SDA_1: track 0.00 -> 45.0 mm, vias 0 -> 2
- net +3V3: track 6.25 -> 50.0 mm, vias 2 -> 1
- net /Project Architecture/Motor Control - Thumb 1/_OCM_T1: track 3.10 -> 46.5 mm
- net /Project Architecture/Motor Control - Index/_OCM_I: track 3.12 -> 44.5 mm
- net /Project Architecture/Interface - Interconnects/SWCLK2: track 0.00 -> 35.4 mm, vias 0 -> 1
- net /Project Architecture/Interface - Interconnects/SWDIO2: track 0.00 -> 34.2 mm, vias 0 -> 1
- net /Project Architecture/MCU - IOs/I2C-SCL_2: track 0.00 -> 31.4 mm, vias 0 -> 2
- net /Project Architecture/MCU - IOs/I2C-SDA_2: track 0.00 -> 29.2 mm, vias 0 -> 2
- net /Project Architecture/MCU - IOs/GPIO-LED_T2: track 0.00 -> 26.4 mm, vias 0 -> 2
- net /Project Architecture/MCU - IOs/GPIO-LED_Debug_1: track 0.00 -> 25.4 mm, vias 0 -> 2
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- added copper zone on F.Cu, net +5V
- added copper zone on F.Cu, net +VBAT
- removed copper zone on B.Cu, net +3V3
- removed copper zone on B.Cu, net +5V
- removed copper zone on B.Cu, net /Project Architecture/Power - Generation/F_VIN_5V

Commit message: Update SCH & PCB
Parts:
- removed BZ1: MLT-8530, Duc:BUZ-SMD_4P-L8.5-W8.5-P8.50-BR
- removed the D15 at (191.6, 72.4)
- removed Q3: 2SC1815, Duc:SOT-23-3_L2.9-W1.3-P1.90-LS2.4-BR
- removed the R67 at (183.3, 73.4)
- removed the TP80 at (163.3, 34.4)
- C10, C11, C12, C13, C5, C6, C7, C8, C9, D1, D8, J11, L1, R1, R2, R3, R4, R5, R57, R58, R6, U14, U15, U3, U4, U5: moved to B.Cu
- C87, C88, C89, C90: value CAP CER 0603 -> CAP CER 0402; footprint Duc:C0603 -> Duc:C0402; moved to B.Cu
- R53, R54: value RES 0603 -> RES 0402; footprint Duc:R0603 -> Duc:R0402; moved to B.Cu
- moved C69 126.9 mm to (269.7, 110.5)
- moved C15 126.9 mm to (280.9, 80.7)
- moved C16 126.9 mm to (280.9, 82.5)
- moved C17 126.9 mm to (280.9, 84.3)
- moved C18 126.9 mm to (280.9, 93.9)
- moved C19 126.9 mm to (280.9, 95.7)
- moved C20 126.9 mm to (280.9, 97.5)
- moved C21 126.9 mm to (280.9, 106.5)
- moved C22 126.9 mm to (280.9, 108.3)
- moved C23 126.9 mm to (280.9, 110.1)
- moved C24 126.9 mm to (280.9, 111.9)
- moved C57 126.9 mm to (269.6, 84.8)
- moved C75 126.9 mm to (292.1, 92.6)
- moved R71 126.9 mm to (280.9, 79.0)
- moved R72 126.9 mm to (280.9, 77.4)
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- renumbered C94 to C92, C92 to C94, D16 to D15, D17 to D16, J15 to J13, J13 to J15, R68 to R67, R69 to R68, R70 to R69, R71 to R70, R72 to R71, R73 to R72, R74 to R73, R75 to R74, R76 to R75, R77 to R76, R78 to R77, R79 to R78, R80 to R79, R81 to R80, TP81 to TP80, TP82 to TP81, TP83 to TP82, TP84 to TP83, TP85 to TP84, TP86 to TP85, TP87 to TP86, TP88 to TP87, TP89 to TP88, TP90 to TP89
Connections:
- net /Project Architecture/Motor Control - Index/_DIAG_I renamed /Project Architecture/Motor Control 1/_DIAG
- net /Project Architecture/Motor Control - Index/_ECC_I renamed /Project Architecture/Motor Control 1/_ECC
- net /Project Architecture/Motor Control - Index/_OCM_I renamed /Project Architecture/Motor Control 1/_OCM
- net /Project Architecture/Motor Control - Middle/_DIAG_M renamed /Project Architecture/Motor Control 2/_DIAG
- net /Project Architecture/Motor Control - Middle/_ECC_M renamed /Project Architecture/Motor Control 2/_ECC
- net /Project Architecture/Motor Control - Middle/_OCM_M renamed /Project Architecture/Motor Control 2/_OCM
- net /Project Architecture/Motor Control - Pinky/_DIAG_P renamed /Project Architecture/Motor Control 4/_DIAG
- net /Project Architecture/Motor Control - Pinky/_ECC_P renamed /Project Architecture/Motor Control 4/_ECC
- net /Project Architecture/Motor Control - Pinky/_OCM_P renamed /Project Architecture/Motor Control 4/_OCM
- net /Project Architecture/Motor Control - Ring/_DIAG_R renamed /Project Architecture/Motor Control 3/_DIAG
- net /Project Architecture/Motor Control - Ring/_ECC_R renamed /Project Architecture/Motor Control 3/_ECC
- net /Project Architecture/Motor Control - Ring/_OCM_R renamed /Project Architecture/Motor Control 3/_OCM
- net /Project Architecture/Motor Control - Thumb 1/_DIAG_T1 renamed /Project Architecture/Motor Control 5/_DIAG
- net /Project Architecture/Motor Control - Thumb 1/_ECC_T1 renamed /Project Architecture/Motor Control 5/_ECC
- net /Project Architecture/Motor Control - Thumb 1/_OCM_T1 renamed /Project Architecture/Motor Control 5/_OCM
- net /Project Architecture/Motor Control - Thumb 2/_DIAG_T2 renamed /Project Architecture/Motor Control 6/_DIAG
- net /Project Architecture/Motor Control - Thumb 2/_ECC_T2 renamed /Project Architecture/Motor Control 6/_ECC
- net /Project Architecture/Motor Control - Thumb 2/_OCM_T2 renamed /Project Architecture/Motor Control 6/_OCM
- C10 pad 1: Net-(U4-FB) -> GND
- C48 pad 2: /Project Architecture/Motor Control - Index/VCC_I -> /Project Architecture/Motor Control 1/VCC
- C51 pad 2: +A3V3 -> +3V3
- C54 pad 2: /Project Architecture/Motor Control - Middle/VCC_M -> /Project Architecture/Motor Control 2/VCC
- C57 pad 2: +A3V3 -> +3V3
- C60 pad 2: /Project Architecture/Motor Control - Ring/VCC_R -> /Project Architecture/Motor Control 3/VCC
- C63 pad 2: +A3V3 -> +3V3
- C66 pad 2: /Project Architecture/Motor Control - Pinky/VCC_P -> /Project Architecture/Motor Control 4/VCC
- C69 pad 2: +A3V3 -> +3V3
- C72 pad 2: /Project Architecture/Motor Control - Thumb 1/VCC_T1 -> /Project Architecture/Motor Control 5/VCC
- C75 pad 2: +A3V3 -> +3V3
- C78 pad 2: /Project Architecture/Motor Control - Thumb 2/VCC_T2 -> /Project Architecture/Motor Control 6/VCC
- C81 pad 2: +A3V3 -> +3V3
- D7 pad 1: Net-(J10-Dn1) -> Net-(J10-Dp1)
- D7 pad 3: Net-(J10-Dp1) -> Net-(J10-Dn1)
- D7 pad 4: /Project Architecture/Interface - USB 2.0/USB2_P -> /Project Architecture/Interface - USB 2.0/USB2_N
- D7 pad 6: /Project Architecture/Interface - USB 2.0/USB2_N -> /Project Architecture/Interface - USB 2.0/USB2_P
- J12 pad 10: +5V -> GND
- J12 pad 11: /Project Architecture/Interface - Interconnects/SWDIO2 -> /Project Architecture/Interface - Interconnects/USART1_TX1
- J12 pad 13: /Project Architecture/Interface - Interconnects/SWCLK2 -> GND
- J12 pad 15: /Project Architecture/Interface - Interconnects/SWCLK1 -> /Project Architecture/Interface - Interconnects/USART1_RX2
- J12 pad 16: +5V -> GND
- J12 pad 17: /Project Architecture/Interface - Interconnects/SWDIO1 -> /Project Architecture/Interface - Interconnects/USART1_TX2
- J12 pad 19: /Project Architecture/Interface - Interconnects/NRST1 -> GND
- J12 pad 9: /Project Architecture/Interface - Interconnects/NRST2 -> /Project Architecture/Interface - Interconnects/USART1_RX1
- J3 pad 3: +A3V3 -> +3V3
- J3 pad 4: /Project Architecture/Motor Control - Index/OUT2_I -> GND
- J3 pad 5: GND -> /Project Architecture/MCU - IOs/ECB_I
- J3 pad 7: /Project Architecture/MCU - IOs/ECB_I -> +3V3
- J3 pad 8: +3V3 -> /Project Architecture/Motor Control 1/OUT1
- J3 pad 9: /Project Architecture/Motor Control - Index/OUT1_I -> /Project Architecture/Motor Control 1/OUT2
- J4 pad 3: +A3V3 -> +3V3
- J4 pad 4: /Project Architecture/Motor Control - Middle/OUT2_M -> GND
- J4 pad 5: GND -> /Project Architecture/MCU - IOs/ECB_M
- J4 pad 7: /Project Architecture/MCU - IOs/ECB_M -> +3V3
- J4 pad 8: +3V3 -> /Project Architecture/Motor Control 2/OUT1
- J4 pad 9: /Project Architecture/Motor Control - Middle/OUT1_M -> /Project Architecture/Motor Control 2/OUT2
- J5 pad 3: +A3V3 -> +3V3
- J5 pad 4: /Project Architecture/Motor Control - Ring/OUT2_R -> GND
- J5 pad 5: GND -> /Project Architecture/MCU - IOs/ECB_R
- J5 pad 7: /Project Architecture/MCU - IOs/ECB_R -> +3V3
- J5 pad 8: +3V3 -> /Project Architecture/Motor Control 3/OUT1
- J5 pad 9: /Project Architecture/Motor Control - Ring/OUT1_R -> /Project Architecture/Motor Control 3/OUT2
- J6 pad 3: +A3V3 -> +3V3
- J6 pad 4: /Project Architecture/Motor Control - Pinky/OUT2_P -> GND
- J6 pad 5: GND -> /Project Architecture/MCU - IOs/ECB_P
- J6 pad 7: /Project Architecture/MCU - IOs/ECB_P -> +3V3
- J6 pad 8: +3V3 -> /Project Architecture/Motor Control 4/OUT1
- J6 pad 9: /Project Architecture/Motor Control - Pinky/OUT1_P -> /Project Architecture/Motor Control 4/OUT2
- J7 pad 3: +A3V3 -> +3V3
- J7 pad 4: /Project Architecture/Motor Control - Thumb 1/OUT2_T1 -> GND
- J7 pad 5: GND -> /Project Architecture/MCU - IOs/ECB_T1
- J7 pad 7: /Project Architecture/MCU - IOs/ECB_T1 -> +3V3
- J7 pad 8: +3V3 -> /Project Architecture/Motor Control 5/OUT1
- J7 pad 9: /Project Architecture/Motor Control - Thumb 1/OUT1_T1 -> /Project Architecture/Motor Control 5/OUT2
- J8 pad 3: +A3V3 -> +3V3
- J8 pad 4: /Project Architecture/Motor Control - Thumb 2/OUT2_T2 -> GND
- J8 pad 5: GND -> /Project Architecture/MCU - IOs/ECB_T2
- J8 pad 7: /Project Architecture/MCU - IOs/ECB_T2 -> +3V3
- J8 pad 8: +3V3 -> /Project Architecture/Motor Control 6/OUT1
- J8 pad 9: /Project Architecture/Motor Control - Thumb 2/OUT1_T2 -> /Project Architecture/Motor Control 6/OUT2
- R13 pad 1: +5V -> /Project Architecture/Motor Control 2/VCC
- R13 pad 2: /Project Architecture/Motor Control - Middle/VCC_M -> +5V
- R19 pad 1: +5V -> /Project Architecture/Motor Control 3/VCC
- R19 pad 2: /Project Architecture/Motor Control - Ring/VCC_R -> +5V
- R25 pad 1: +5V -> /Project Architecture/Motor Control 4/VCC
- R25 pad 2: /Project Architecture/Motor Control - Pinky/VCC_P -> +5V
- R31 pad 1: +5V -> /Project Architecture/Motor Control 5/VCC
- R31 pad 2: /Project Architecture/Motor Control - Thumb 1/VCC_T1 -> +5V
- R37 pad 1: +5V -> /Project Architecture/Motor Control 6/VCC
- R37 pad 2: /Project Architecture/Motor Control - Thumb 2/VCC_T2 -> +5V
- R7 pad 1: +5V -> /Project Architecture/Motor Control 1/VCC
- R7 pad 2: /Project Architecture/Motor Control - Index/VCC_I -> +5V
- U10 pad 13: /Project Architecture/Motor Control - Ring/OUT1_R -> /Project Architecture/Motor Control 3/OUT1
- U10 pad 14: /Project Architecture/Motor Control - Ring/OUT1_R -> /Project Architecture/Motor Control 3/OUT1
- U10 pad 2: /Project Architecture/Motor Control - Ring/VCC_R -> /Project Architecture/Motor Control 3/VCC
- U10 pad 22: /Project Architecture/Motor Control - Ring/OUT2_R -> /Project Architecture/Motor Control 3/OUT2
- U10 pad 23: /Project Architecture/Motor Control - Ring/OUT2_R -> /Project Architecture/Motor Control 3/OUT2
- U11 pad 13: /Project Architecture/Motor Control - Pinky/OUT1_P -> /Project Architecture/Motor Control 4/OUT1
- U11 pad 14: /Project Architecture/Motor Control - Pinky/OUT1_P -> /Project Architecture/Motor Control 4/OUT1
- U11 pad 2: /Project Architecture/Motor Control - Pinky/VCC_P -> /Project Architecture/Motor Control 4/VCC
- U11 pad 22: /Project Architecture/Motor Control - Pinky/OUT2_P -> /Project Architecture/Motor Control 4/OUT2
- U11 pad 23: /Project Architecture/Motor Control - Pinky/OUT2_P -> /Project Architecture/Motor Control 4/OUT2
- U12 pad 13: /Project Architecture/Motor Control - Thumb 1/OUT1_T1 -> /Project Architecture/Motor Control 5/OUT1
- U12 pad 14: /Project Architecture/Motor Control - Thumb 1/OUT1_T1 -> /Project Architecture/Motor Control 5/OUT1
- U12 pad 2: /Project Architecture/Motor Control - Thumb 1/VCC_T1 -> /Project Architecture/Motor Control 5/VCC
- U12 pad 22: /Project Architecture/Motor Control - Thumb 1/OUT2_T1 -> /Project Architecture/Motor Control 5/OUT2
- U12 pad 23: /Project Architecture/Motor Control - Thumb 1/OUT2_T1 -> /Project Architecture/Motor Control 5/OUT2
- U13 pad 13: /Project Architecture/Motor Control - Thumb 2/OUT1_T2 -> /Project Architecture/Motor Control 6/OUT1
- U13 pad 14: /Project Architecture/Motor Control - Thumb 2/OUT1_T2 -> /Project Architecture/Motor Control 6/OUT1
- U13 pad 2: /Project Architecture/Motor Control - Thumb 2/VCC_T2 -> /Project Architecture/Motor Control 6/VCC
- U13 pad 22: /Project Architecture/Motor Control - Thumb 2/OUT2_T2 -> /Project Architecture/Motor Control 6/OUT2
- U13 pad 23: /Project Architecture/Motor Control - Thumb 2/OUT2_T2 -> /Project Architecture/Motor Control 6/OUT2
- U4 pad 5: Net-(U4-FB) -> GND
- U6 pad 59: unconnected-(U6B-PB6-Pad59) -> /Project Architecture/Interface - Interconnects/USART1_TX1
- U6 pad 60: unconnected-(U6B-PB7-Pad60) -> /Project Architecture/Interface - Interconnects/USART1_RX1
- U6 pad 62: /Project Architecture/MCU - IOs/PWM_BUZZER -> unconnected-(U6B-PB9-Pad62)
- U7 pad 59: unconnected-(U7B-PB6-Pad59) -> /Project Architecture/Interface - Interconnects/USART1_TX2
- U7 pad 60: unconnected-(U7B-PB7-Pad60) -> /Project Architecture/Interface - Interconnects/USART1_RX2
- U8 pad 13: /Project Architecture/Motor Control - Index/OUT1_I -> /Project Architecture/Motor Control 1/OUT1
- U8 pad 14: /Project Architecture/Motor Control - Index/OUT1_I -> /Project Architecture/Motor Control 1/OUT1
- U8 pad 2: /Project Architecture/Motor Control - Index/VCC_I -> /Project Architecture/Motor Control 1/VCC
- U8 pad 22: /Project Architecture/Motor Control - Index/OUT2_I -> /Project Architecture/Motor Control 1/OUT2
- U8 pad 23: /Project Architecture/Motor Control - Index/OUT2_I -> /Project Architecture/Motor Control 1/OUT2
- U9 pad 13: /Project Architecture/Motor Control - Middle/OUT1_M -> /Project Architecture/Motor Control 2/OUT1
- U9 pad 14: /Project Architecture/Motor Control - Middle/OUT1_M -> /Project Architecture/Motor Control 2/OUT1
- U9 pad 2: /Project Architecture/Motor Control - Middle/VCC_M -> /Project Architecture/Motor Control 2/VCC
- U9 pad 22: /Project Architecture/Motor Control - Middle/OUT2_M -> /Project Architecture/Motor Control 2/OUT2
- U9 pad 23: /Project Architecture/Motor Control - Middle/OUT2_M -> /Project Architecture/Motor Control 2/OUT2
Routing:
- net /Project Architecture/MCU - IOs/EN_P: track 71.6 -> 3.12 mm
- net /Project Architecture/MCU - IOs/ECA_P: track 69.2 -> 4.58 mm
- net /Project Architecture/MCU - IOs/ECC_P: track 66.8 -> 2.39 mm, vias 2 -> 1
- net /Project Architecture/MCU - IOs/EN_T2: track 63.6 -> 3.04 mm
- net /Project Architecture/Motor Control 6/_OCM: track 62.3 -> 2.63 mm, vias 2 -> 1
- net /Project Architecture/MCU - IOs/PWMB_R: track 59.8 -> 4.03 mm
- net /Project Architecture/MCU - IOs/PWMA_R: track 59.1 -> 4.12 mm
- net /Project Architecture/MCU - IOs/ECA_R: track 58.8 -> 4.33 mm
- net /Project Architecture/MCU - IOs/ECB_R: track 57.3 -> 3.09 mm
- net /Project Architecture/MCU - IOs/PWMB_T2: track 57.7 -> 4.12 mm
- net /Project Architecture/MCU - IOs/PWMA_T2: track 57.6 -> 4.00 mm
- net /Project Architecture/MCU - IOs/ECB_T2: track 56.0 -> 3.04 mm
- net /Project Architecture/Motor Control 4/_OCM: track 55.2 -> 2.65 mm, vias 2 -> 1
- net /Project Architecture/MCU - IOs/ECA_T2: track 55.7 -> 4.25 mm
- net /Project Architecture/MCU - IOs/ECC_T2: track 55.1 -> 3.90 mm, vias 2 -> 1
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- removed copper zone on F.Cu, net +5V
- removed copper zone on F.Cu, net +VBAT
