File: Master_Hand_Kicad.kicad_pcb (KiCad board)
At the start: 6 copper layers, 79 x 65.8 mm, 330 parts, among them J1 XT30PW-F, J10 TYPE-C 16PIN 2MD, J11 1.25-3PLTDK, J12 5025982393, J13 PH2.54-2X3P-H25, J14 PH2.54-2X3P-H25, J15 PH2.54-2X3P-H25, J2 KF350-3.5-2P, J3 BM09B-SRSS-TB, J4 BM09B-SRSS-TB, J5 BM09B-SRSS-TB, J6 BM09B-SRSS-TB, J7 BM09B-SRSS-TB, J8 BM09B-SRSS-TB, J9 TYPE-C 16PIN 2MD, Q1 HV10N03, Q2 HV10N03, SW1 DSIC02LSGET, U1 LM74700QDBVRQ1, U10 TB9051FTG,EL, U11 TB9051FTG,EL, U12 TB9051FTG,EL, U13 TB9051FTG,EL, U14 TJA1051T/3, U15 TJA1051T/3, U16 SHT40-N-NF, U17 SHT40-N-NF, U2 LM74700QDBVRQ1, U3 TPSM63603RDHR, U4 TPS62162DSG, U5 TLV75533PDBVR, U6 STM32G474RET6, U7 STM32G474RET6, U8 TB9051FTG,EL, U9 TB9051FTG,EL, X1 X322516MLB4SI, X2 X322516MLB4SI

Commit message: Update SCH & PCB
Routing:
- net /Project Architecture/MCU - IOs/ECB_P: track 19.7 -> 70.3 mm
- net /Project Architecture/MCU - IOs/ECA_P: track 4.58 -> 52.5 mm
- net /Project Architecture/Motor Control 4/_DIAG: track 68.3 -> 70.0 mm
- net /Project Architecture/MCU - IOs/PWMA_P: track 65.1 -> 63.6 mm
- net /Project Architecture/MCU - IOs/PWMB_P: track 65.9 -> 64.5 mm
Changed lines of the file:
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@@
 	)
 	(segment
+		(start 152.145002 107.394954)
+		(end 146.964954 107.394954)
+		(width 0.2)
+		(layer "In1.Cu")
+		(net 81)
+	)
+	(segment
+		(start 141.39 101.82)
+		(end 141.39 67.724974)
+		(width 0.2)
+		(layer "In1.Cu")
+		(net 81)
+	)
+	(segment
+		(start 152.669997 106.869959)
+		(end 152.145002 107.394954)
+		(width 0.2)
+		(layer "In1.Cu")
+		(net 81)
+	)
+	(segment
+		(start 146.964954 107.394954)
+		(end 141.39 101.82)
+		(width 0.2)
+		(layer "In1.Cu")
+		(net 81)
+	)
+	(segment
 		(start 160.84 62.92319)
 		(end 160.84 61.3)
@@
 	)
 	(segment
+		(start 147.674974 61.44)
+		(end 159.73 61.44)
+		(width 0.2)
+		(layer "In1.Cu")
+		(net 82)
+	)
+	(segment
 		(start 151.799999 106.869954)
-		(end 143.919954 106.869954)
+		(end 147.089954 106.869954)
+		(width 0.2)
+		(layer "In1.Cu")
+		(net 82)
+	)
+	(segment
+		(start 147.089954 106.869954)
+		(end 141.74 101.52)
+		(width 0.2)
+		(layer "In1.Cu")
+		(net 82)
+	)
+	(segment
+		(start 141.74 67.374974)
+		(end 147.674974 61.44)
 		(width 0.2)
 		(layer "In1.Cu")
@@
 	)
 	(segment
-		(start 141.85 104.8)
-		(end 141.85 99.06)
+		(start 159.73 61.44)
+		(end 159.95 61.66)
 		(width 0.2)
 		(layer "In1.Cu")
@@
 	)
 	(segment
-		(start 143.919954 106.869954)
-		(end 141.85 104.8)
+		(start 141.74 101.52)
+		(end 141.74 67.374974)
 		(width 0.2)
 		(layer "In1.Cu")
@@
 	)
 	(segment
-		(start 162.09 61.68)
-		(end 163.27 62.86)
+		(start 162.21 61.08)
+		(end 163.61 62.48)
 		(width 0.2)
 		(layer "In1.Cu")
@@
 	)
 	(segment
-		(start 143.140001 106.889962)
-		(end 141.5 105.249961)
+		(start 163.61 62.48)
+		(end 164.24 62.48)
+		(width 0.2)
+		(layer "In1.Cu")
+		(net 133)
+	)
+	(segment
+		(start 147.54 61.08)
+		(end 162.21 61.08)
 		(width 0.2)
 		(layer "In1.Cu")
@@
 	)
 	(segment
-		(start 141.5 67.12)
-		(end 146.94 61.68)
+		(start 141.02 104.769961)
+		(end 141.02 67.6)
 		(width 0.2)
 		(layer "In1.Cu")
@@
 	)
 	(segment
-		(start 141.5 105.249961)
-		(end 141.5 67.12)
+		(start 143.140001 106.889962)
+		(end 141.02 104.769961)
 		(width 0.2)
 		(layer "In1.Cu")
@@
 	)
 	(segment
-		(start 146.94 61.68)
-		(end 162.09 61.68)
+		(start 141.02 67.6)
+		(end 147.54 61.08)
 		(width 0.2)
 		(layer "In1.Cu")
@@
 	)
 	(segment
-		(start 149.85 102.007497)
-		(end 149.372503 101.53)
+		(start 146.394974 101.53)
+		(end 142.56 97.695026)
 		(width 0.2)
 		(layer "In1.Cu")
@@
 	)
 	(segment
-		(start 146.394974 101.53)
-		(end 142.2 97.335026)
+		(start 149.85 102.069965)
+		(end 149.85 102.007497)
 		(width 0.2)
 		(layer "In1.Cu")
@@
 	)
 	(segment
-		(start 142.2 67.504974)
-		(end 147.324974 62.38)
+		(start 149.244974 62.38)
+		(end 161.46 62.38)
 		(width 0.2)
 		(layer "In1.Cu")
@@
 	)
 	(segment
-		(start 142.2 97.335026)
-		(end 142.2 67.504974)
+		(start 142.56 69.064974)
+		(end 149.244974 62.38)
 		(width 0.2)
 		(layer "In1.Cu")
@@
 	)
 	(segment
-		(start 149.85 102.069965)
-		(end 149.85 102.007497)
+		(start 149.372503 101.53)
+		(end 146.394974 101.53)
 		(width 0.2)
 		(layer "In1.Cu")
@@
 	)
 	(segment
-		(start 149.372503 101.53)
-		(end 146.394974 101.53)
+		(start 142.56 97.695026)
+		(end 142.56 69.064974)
 		(width 0.2)
 		(layer "In1.Cu")
@@
 	)
 	(segment
-		(start 147.324974 62.38)
-		(end 161.46 62.38)
+		(start 149.85 102.007497)
+		(end 149.372503 101.53)
 		(width 0.2)
 		(layer "In1.Cu")
@@
 	)
 	(segment
-		(start 161.84 62.03)
-		(end 162.14 62.33)
+		(start 142.21 97.84)
+		(end 142.21 68.92)
 		(width 0.2)
 		(layer "In1.Cu")
@@
 	)
 	(segment
-		(start 146.439957 102.069957)
-		(end 141.85 97.48)
+		(start 149.1 62.03)
+		(end 161.84 62.03)
 		(width 0.2)
 		(layer "In1.Cu")
@@
 	)
 	(segment
-		(start 141.85 67.36)
-		(end 147.18 62.03)
+		(start 149.169997 102.069957)
+		(end 146.439957 102.069957)
 		(width 0.2)
 		(layer "In1.Cu")
@@
 	)
 	(segment
-		(start 147.18 62.03)
-		(end 161.84 62.03)
+		(start 142.21 68.92)
+		(end 149.1 62.03)
 		(width 0.2)
 		(layer "In1.Cu")
@@
 	)
 	(segment
-		(start 141.85 97.48)
-		(end 141.85 67.36)
+		(start 161.84 62.03)
+		(end 162.14 62.33)
 		(width 0.2)
 		(layer "In1.Cu")
@@
 	)
 	(segment
-		(start 149.169997 102.069957)
-		(end 146.439957 102.069957)
+		(start 146.439957 102.069957)
+		(end 142.21 97.84)
 		(width 0.2)
 		(layer "In1.Cu")
