File: MCU - IOs.kicad_sch (KiCad schematic)
At the start: 8 parts, among them U6 STM32G474RET6, U7 STM32G474RET6, X1 X322516MLB4SI, X2 X322516MLB4SI

Commit message: Update Schematic
Parts:
- added TP10, TP11, TP12, TP13, TP14, TP15, TP16, TP17, TP18, TP19, TP20, TP21, TP22, TP23, TP24, TP25, TP26, TP27, TP28, TP29, TP30, TP31, TP32, TP33, TP34, TP35, TP36, TP37, TP38, TP39, TP40, TP41, TP42, TP43, TP44, TP45, TP46, TP47, TP48, TP49, TP50, TP51, TP52, TP53, TP54, TP55, TP56, TP57, TP58, TP59, TP60, TP61, TP62, TP63, TP64, TP65, TP66, TP67, TP68, TP69, TP70, TP71, TP72, TP73, TP74, TP75, TP76, TP77, TP78, TP79, TP80, TP81, TP82, TP83, TP84, TP85, TP86, TP87, TP88, TP89, TP9, TP90, TP91: ~, Duc_Library:TestPoint_Pad_D0.5mm, symbol Power_symbols:Test_Point
- C48, C49, C50, C51: value CAP CER 0402 -> 8pF 16V 0603; footprint Duc_Library:C0402 -> Duc:C0603; symbol Duc-Capacitors:CAP CER 0402 -> Duc-Capacitors:CAP CER 0603; LCSC Part C325464 -> C14663; MPN CC0402KRX5R7BB105 -> CAP CER 0603; Manufacturer (none) -> YAGEO(国巨)
Connections:
- net BOARD_VERSION: now also TP13.1
- net DIAG_I: now also TP14.1
- net DIAG_M: now also TP28.1
- net DIAG_P: now also TP59.1
- net DIAG_R: now also TP43.1
- net DIAG_T1: now also TP74.1
- net DIAG_T2: now also TP85.1
- net ECA_I: now also TP16.1
- net ECA_M: now also TP32.1
- net ECA_P: now also TP62.1
- net ECA_R: now also TP47.1
- net ECA_T1: now also TP76.1
- net ECA_T2: now also TP89.1
- net ECB_I: now also TP18.1
- net ECB_M: now also TP33.1
- net ECB_P: now also TP63.1
- net ECB_R: now also TP49.1
- net ECB_T1: now also TP78.1
- net ECB_T2: now also TP90.1
- net ECC_I: now also TP20.1
- net ECC_M: now also TP35.1
- net ECC_P: now also TP65.1
- net ECC_R: now also TP51.1
- net ECC_T1: now also TP80.1
- net ECC_T2: now also TP91.1
- net EN_I: now also TP12.1
- net EN_M: now also TP27.1
- net EN_P: now also TP57.1
- net EN_R: now also TP41.1
- net EN_T1: now also TP72.1
- net EN_T2: now also TP84.1
- net FDCAN1_RX: now also TP31.1
- net FDCAN1_TX: now also TP29.1
- net FDCAN2_RX: now also TP36.1
- net FDCAN2_TX: now also TP34.1
- net GPIO-LED_Debug_1: now also TP50.1
- net GPIO-LED_Debug_2: now also TP52.1
- net GPIO-LED_I: now also TP38.1
- net GPIO-LED_M: now also TP48.1
- net GPIO-LED_P: now also TP44.1
- net GPIO-LED_R: now also TP46.1
- net GPIO-LED_T1: now also TP40.1
- net GPIO-LED_T2: now also TP42.1
- net I2C-SCL_1: now also TP56.1
- net I2C-SCL_2: now also TP60.1
- net I2C-SDA_1: now also TP54.1
- net I2C-SDA_2: now also TP58.1
- net I2C_SCL: now also TP77.1
- net I2C_SDA: now also TP79.1
- net MCU_ID1: now also TP86.1
- net MCU_ID2: now also TP88.1
- net NRST1: now also TP22.1
- net NRST2: now also TP17.1
- net OCM_I: now also TP15.1
- net OCM_M: now also TP30.1
- net OCM_P: now also TP61.1
- net OCM_R: now also TP45.1
- net OCM_T1: now also TP75.1
- net OCM_T2: now also TP87.1
- net PWMA_I: now also TP10.1
- net PWMA_M: now also TP23.1
- net PWMA_P: now also TP53.1
- net PWMA_R: now also TP37.1
- net PWMA_T1: now also TP68.1
- net PWMA_T2: now also TP82.1
- net PWMB_I: now also TP11.1
- net PWMB_M: now also TP25.1
- net PWMB_P: now also TP55.1
- net PWMB_R: now also TP39.1
- net PWMB_T1: now also TP70.1
- net PWMB_T2: now also TP83.1
- net PWM_BUZZER: now also TP81.1
- net SENSE_VBAT: now also TP9.1
- net SWCLK1: now also TP24.1
- net SWCLK2: now also TP19.1
- net SWDIO1: now also TP26.1
- net SWDIO2: now also TP21.1
- net USB-DM_1: now also TP66.1
- net USB-DM_2: now also TP71.1
- net USB-DP_1: now also TP64.1
- net USB-DP_2: now also TP69.1
- net VBUS_DET1: now also TP67.1
- net VBUS_DET2: now also TP73.1
Other:
- note added: "5Mbps FD-CAN Bus"
- note added: "Battery Voltage Sense"
- note added: "Board Version Selection"
- note added: "Buzzer"
- note added: "LEDs"
- note added: "MCB to MB - I2C"
- note added: "MCU ID"
- note added: "MD Index"
- note added: "MD Middle"
- note added: "MD Pinky"
- note added: "MD Ring"
- note added: "MD Thumb 1"
- note added: "MD Thumb 2"
- note added: "SWD (Debug) Port"
- note added: "Temperature and Humidity"
- note added: "USB PORT"

Commit message: Update Schematic
Changed lines of the file:
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@@
 		)
 	)
-	(bus
-		(pts
-			(xy 153.67 213.36) (xy 153.67 214.63)
-		)
-		(stroke
-			(width 0)
-			(type default)
-		)
-	)
 	(wire
 		(pts
@@
 		)
 	)
-	(bus
-		(pts
-			(xy 232.41 219.71) (xy 232.41 220.98)
-		)
-		(stroke
-			(width 0)
-			(type default)
-		)
-	)
 	(wire
 		(pts
@@
 		)
 	)
-	(bus
-		(pts
-			(xy 157.48 127) (xy 157.48 128.27)
-		)
-		(stroke
-			(width 0)
-			(type default)
-		)
-	)
 	(wire
 		(pts
@@
 		)
 	)
-	(bus
-		(pts
-			(xy 157.48 114.3) (xy 157.48 115.57)
-		)
-		(stroke
-			(width 0)
-			(type default)
-		)
-	)
 	(wire
 		(pts
@@
 		)
 	)
-	(bus
-		(pts
-			(xy 160.02 69.85) (xy 160.02 71.12)
-		)
-		(stroke
-			(width 0)
-			(type default)
-		)
-	)
 	(wire
 		(pts
@@
 		)
 	)
-	(bus
-		(pts
-			(xy 160.02 82.55) (xy 160.02 83.82)
-		)
-		(stroke
-			(width 0)
-			(type default)
-		)
-	)
 	(wire
 		(pts
@@
 	(bus
 		(pts
-			(xy 153.67 226.06) (xy 153.67 227.33)
-		)
-		(stroke
-			(width 0)
-			(type default)
-		)
-	)
-	(bus
-		(pts
 			(xy 234.95 107.95) (xy 246.38 107.95)
 		)
@@
 		)
 		(instances
-			(project ""
+			(project "Master_Hand_Kicad"
 				(path "/f9e05184-c88b-4a88-ae9c-ab2bdb32be7c/c5103ceb-5325-4a84-a025-9638a412984e/e744f3ce-03a6-44a6-8792-1447ef232b9a"
 					(reference "TP9")

Commit message: Update Schematic & PCB
Parts:
- TP10, TP11, TP12, TP13, TP14, TP15, TP16, TP17, TP18, TP19, TP20, TP21, TP22, TP23, TP24, TP25, TP26, TP27, TP28, TP29, TP30, TP31, TP32, TP33, TP34, TP35, TP36, TP37, TP38, TP39, TP40, TP41, TP42, TP43, TP44, TP45, TP46, TP47, TP48, TP49, TP50, TP51, TP52, TP53, TP54, TP55, TP56, TP57, TP58, TP59, TP60, TP61, TP62, TP63, TP64, TP65, TP66, TP67, TP68, TP69, TP70, TP71, TP72, TP73, TP74, TP75, TP76, TP77, TP78, TP79, TP80, TP81, TP82, TP83, TP84, TP85, TP86, TP87, TP88, TP89, TP9, TP90, TP91: footprint Duc_Library:TestPoint_Pad_D0.5mm -> Duc:TestPoint_Pad_D0.5mm
- U6, U7: footprint Duc_Library:LQFP-64_L10.0-W10.0-P0.50-LS12.0-BL -> Duc:LQFP-64_L10.0-W10.0-P0.50-LS12.0-BL
Connections:
- net ECA_M: now also U7.13 (PA1); no longer U7.12 (PA0)
- net ECA_P: now also U7.39 (PC7); no longer U7.38 (PC6)
- net ECA_R: now also U7.21 (PA7); no longer U7.20 (PA6)
- net ECB_M: now also U7.12 (PA0); no longer U7.13 (PA1)
- net ECB_P: now also U7.38 (PC6); no longer U7.39 (PC7)
- net ECB_R: now also U7.20 (PA6); no longer U7.21 (PA7)
- net PWMA_I: now also U6.37 (PB15); no longer U6.36 (PB14)
- net PWMA_M: now also U7.9 (PC1); no longer U7.8 (PC0)
- net PWMA_R: now also U7.11 (PC3); no longer U7.10 (PC2)
- net PWMB_I: now also U6.36 (PB14); no longer U6.37 (PB15)
- net PWMB_M: now also U7.8 (PC0); no longer U7.9 (PC1)
- net PWMB_R: now also U7.10 (PC2); no longer U7.11 (PC3)
- net USB-DM_1 renamed USB1_N
- net USB-DM_2 renamed USB2_N
- net USB-DP_1 renamed USB1_P
- net USB-DP_2 renamed USB2_P

Commit message: Update SCH & PCB
Connections:
- net DIAG_T1: now also U6.2 (PC13); no longer U6.3 (PC14)
- net DIAG_T2: now also U6.3 (PC14); no longer U6.2 (PC13)
- net ECA_I: now also U6.39 (PC7); no longer U6.38 (PC6)
- net ECA_T1: now also U6.21 (PA7); no longer U6.20 (PA6)
- net ECB_I: now also U6.38 (PC6); no longer U6.39 (PC7)
- net ECB_T1: now also U6.20 (PA6); no longer U6.21 (PA7)
- net OCM_T1: now also U6.14 (PA2); no longer U6.17 (PA3)
- net OCM_T2: now also U6.17 (PA3); no longer U6.14 (PA2)
Changed lines of the file:
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@@
 	)
 	(label "ECB_I"
-		(at 21.59 107.95 0)
+		(at 21.59 105.41 0)
 		(effects
 			(font
@@
 	)
 	(label "ECB_T1"
-		(at 105.41 69.85 180)
+		(at 105.41 67.31 180)
 		(effects
 			(font
@@
 	)
 	(label "DIAG_T2"
-		(at 21.59 123.19 0)
+		(at 21.59 125.73 0)
 		(effects
 			(font
@@
 	)
 	(label "ECA_I"
-		(at 21.59 105.41 0)
+		(at 21.59 107.95 0)
 		(effects
 			(font
@@
 	)
 	(label "ECA_T1"
-		(at 105.41 67.31 180)
+		(at 105.41 69.85 180)
 		(effects
 			(font
@@
 	)
 	(label "OCM_T2"
-		(at 105.41 57.15 180)
+		(at 105.41 59.69 180)
 		(effects
 			(font
@@
 	)
 	(label "DIAG_T1"
-		(at 21.59 125.73 0)
+		(at 21.59 123.19 0)
 		(effects
 			(font
@@
 	)
 	(label "OCM_T1"
-		(at 105.41 59.69 180)
-		(effects
-			(font
+		(at 105.41 57.15 180)
+		(effects
+			(font

Commit message: Update Schematic & PCB
Parts:
- C48, C49, C50, C51: value 8pF 16V 0603 -> CAP CER 0603
Changed lines of the file:
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@@
 			)
 		)
-		(property "Value" "8pF 16V 0603"
+		(property "Value" "CAP CER 0603"
 			(at 251.46 151.13 90)
 			(effects
@@
 			)
 		)
-		(property "Value" "8pF 16V 0603"
+		(property "Value" "CAP CER 0603"
 			(at 196.85 176.53 90)
 			(effects
@@
 		(on_board no)
 		(dnp no)
-		(property "Reference" "#PWR034"
+		(property "Reference" "#PWR34"
 			(at 251.206 147.574 0)
 			(do_not_autoplace yes)
@@
 			(project "Master_Hand_Kicad"
 				(path "/f9e05184-c88b-4a88-ae9c-ab2bdb32be7c/c5103ceb-5325-4a84-a025-9638a412984e/e744f3ce-03a6-44a6-8792-1447ef232b9a"
-					(reference "#PWR034")
+					(reference "#PWR34")
 					(unit 1)
 				)
@@
 		(dnp no)
 		(fields_autoplaced yes)
-		(property "Reference" "#PWR035"
+		(property "Reference" "#PWR35"
 			(at 215.646 172.974 0)
 			(do_not_autoplace yes)
@@
 			(project "Master_Hand_Kicad"
 				(path "/f9e05184-c88b-4a88-ae9c-ab2bdb32be7c/c5103ceb-5325-4a84-a025-9638a412984e/e744f3ce-03a6-44a6-8792-1447ef232b9a"
-					(reference "#PWR035")
+					(reference "#PWR35")
 					(unit 1)
 				)
@@
 			)
 		)
-		(property "Value" "8pF 16V 0603"
+		(property "Value" "CAP CER 0603"
 			(at 196.85 151.13 90)
 			(effects
@@
 		(dnp no)
 		(fields_autoplaced yes)
-		(property "Reference" "#PWR036"
+		(property "Reference" "#PWR36"
 			(at 251.206 172.974 0)
 			(do_not_autoplace yes)
@@
 			(project "Master_Hand_Kicad"
 				(path "/f9e05184-c88b-4a88-ae9c-ab2bdb32be7c/c5103ceb-5325-4a84-a025-9638a412984e/e744f3ce-03a6-44a6-8792-1447ef232b9a"
-					(reference "#PWR036")
+					(reference "#PWR36")
 					(unit 1)
 				)
@@
 		(on_board no)
 		(dnp no)
-		(property "Reference" "#PWR033"
+		(property "Reference" "#PWR33"
 			(at 215.646 147.574 0)
 			(do_not_autoplace yes)
@@
 			(project "Master_Hand_Kicad"
 				(path "/f9e05184-c88b-4a88-ae9c-ab2bdb32be7c/c5103ceb-5325-4a84-a025-9638a412984e/e744f3ce-03a6-44a6-8792-1447ef232b9a"
-					(reference "#PWR033")
+					(reference "#PWR33")
 					(unit 1)
 				)
@@
 			)
 		)
-		(property "Value" "8pF 16V 0603"
+		(property "Value" "CAP CER 0603"
 			(at 251.46 176.53 90)
 			(effects

Commit message: Update SCH & PCB
Connections:
- net PWMA_M: now also U7.11 (PC3); no longer U7.9 (PC1)
- net PWMA_R: now also U7.8 (PC0); no longer U7.11 (PC3)
- net PWMB_M: now also U7.10 (PC2); no longer U7.8 (PC0)
- net PWMB_R: now also U7.9 (PC1); no longer U7.10 (PC2)
Changed lines of the file:
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@@
 	)
 	(label "PWMA_R"
-		(at 21.59 213.36 0)
+		(at 21.59 205.74 0)
 		(effects
 			(font
@@
 	)
 	(label "PWMB_M"
-		(at 21.59 205.74 0)
+		(at 21.59 210.82 0)
 		(effects
 			(font
@@
 	)
 	(label "PWMA_M"
-		(at 21.59 208.28 0)
+		(at 21.59 213.36 0)
 		(effects
 			(font
@@
 	)
 	(label "PWMB_R"
-		(at 21.59 210.82 0)
-		(effects
-			(font
+		(at 21.59 208.28 0)
+		(effects
+			(font

Commit message: Update Schematic & PCB
Connections:
- net ECA_I: now also U6.38 (PC6); no longer U6.39 (PC7)
- net ECA_T1: now also U6.12 (PA0); no longer U6.21 (PA7)
- net ECA_T2: now also U6.21 (PA7); no longer U6.12 (PA0)
- net ECB_I: now also U6.39 (PC7); no longer U6.38 (PC6)
- net ECB_T1: now also U6.13 (PA1); no longer U6.20 (PA6)
- net ECB_T2: now also U6.20 (PA6); no longer U6.13 (PA1)
- net PWMA_T1: now also U6.8 (PC0); no longer U6.10 (PC2)
- net PWMA_T2: now also U6.10 (PC2); no longer U6.8 (PC0)
- net PWMB_T1: now also U6.9 (PC1); no longer U6.11 (PC3)
- net PWMB_T2: now also U6.11 (PC3); no longer U6.9 (PC1)
Changed lines of the file:
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@@
 	)
 	(label "ECB_I"
-		(at 21.59 105.41 0)
+		(at 21.59 107.95 0)
 		(effects
 			(font
@@
 	)
 	(label "ECB_T2"
-		(at 105.41 54.61 180)
+		(at 105.41 67.31 180)
 		(effects
 			(font
@@
 	)
 	(label "ECB_T1"
-		(at 105.41 67.31 180)
+		(at 105.41 54.61 180)
 		(effects
 			(font
@@
 	)
 	(label "PWMA_T1"
-		(at 21.59 95.25 0)
+		(at 21.59 90.17 0)
 		(effects
 			(font
@@
 	)
 	(label "ECA_T2"
-		(at 105.41 52.07 180)
+		(at 105.41 69.85 180)
 		(effects
 			(font
@@
 	)
 	(label "ECA_I"
-		(at 21.59 107.95 0)
+		(at 21.59 105.41 0)
 		(effects
 			(font
@@
 	)
 	(label "ECA_T1"
-		(at 105.41 69.85 180)
+		(at 105.41 52.07 180)
 		(effects
 			(font
@@
 	)
 	(label "PWMB_T1"
-		(at 21.59 97.79 0)
+		(at 21.59 92.71 0)
 		(effects
 			(font
@@
 	)
 	(label "PWMA_T2"
-		(at 21.59 90.17 0)
+		(at 21.59 95.25 0)
 		(effects
 			(font
@@
 	)
 	(label "PWMB_T2"
-		(at 21.59 92.71 0)
-		(effects
-			(font
+		(at 21.59 97.79 0)
+		(effects
+			(font

Commit message: Update SCH & PCB
Parts:
- renumbered C48 to C43, C49 to C44, C50 to C45, C51 to C46, TP11 to TP10, TP12 to TP11, TP13 to TP12, TP14 to TP13, TP15 to TP14, TP16 to TP15, TP17 to TP16, TP18 to TP17, TP19 to TP18, TP20 to TP19, TP21 to TP20, TP22 to TP21, TP23 to TP22, TP24 to TP23, TP25 to TP24, TP26 to TP25, TP27 to TP26, TP28 to TP27, TP29 to TP28, TP30 to TP29, TP31 to TP30, TP32 to TP31, TP33 to TP32, TP34 to TP33, TP35 to TP34, TP36 to TP35, TP37 to TP36, TP38 to TP37, TP39 to TP38, TP40 to TP39, TP41 to TP40, TP42 to TP41, TP43 to TP42, TP44 to TP43, TP45 to TP44, TP46 to TP45, TP47 to TP46, TP48 to TP47, TP49 to TP48, TP50 to TP49, TP51 to TP50, TP52 to TP51, TP53 to TP52, TP54 to TP53, TP55 to TP54, TP56 to TP55, TP57 to TP56, TP58 to TP57, TP59 to TP58, TP60 to TP59, TP61 to TP60, TP62 to TP61, TP63 to TP62, TP64 to TP63, TP65 to TP64, TP66 to TP65, TP67 to TP66, TP68 to TP67, TP69 to TP68, TP70 to TP69, TP71 to TP70, TP72 to TP71, TP73 to TP72, TP74 to TP73, TP75 to TP74, TP76 to TP75, TP77 to TP76, TP78 to TP77, TP79 to TP78, TP80 to TP79, TP9 to TP8, TP81 to TP80, TP82 to TP81, TP83 to TP82, TP84 to TP83, TP85 to TP84, TP86 to TP85, TP87 to TP86, TP88 to TP87, TP89 to TP88, TP90 to TP89, TP10 to TP9, TP91 to TP90
Connections:
- net BOARD_VERSION: no longer U7.26 (PB2)
- no-connect marks 11 -> 12
