File: Interface - FD-CAN.kicad_sch (KiCad schematic)
At the start: 10 parts, among them U14 TJA1051T/3, U15 TJA1051T/3

Commit message: Update Schematic
Parts:
- R53, R54, R55, R56: value RES 0603 -> 10K 0.1% 0603
Changed lines of the file:
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@@
 	(wire
 		(pts
-			(xy 95.25 57.15) (xy 95.25 59.69)
+			(xy 95.25 57.15) (xy 95.25 60.96)
 		)
 		(stroke
@@
 	(wire
 		(pts
-			(xy 93.98 116.84) (xy 93.98 119.38)
+			(xy 93.98 115.57) (xy 93.98 119.38)
 		)
 		(stroke
@@
 	(wire
 		(pts
-			(xy 162.56 119.38) (xy 162.56 121.92)
+			(xy 162.56 118.11) (xy 162.56 121.92)
 		)
 		(stroke
@@
 	(wire
 		(pts
-			(xy 95.25 69.85) (xy 95.25 72.39)
+			(xy 95.25 68.58) (xy 95.25 72.39)
 		)
 		(stroke
@@
 	(wire
 		(pts
-			(xy 163.83 59.69) (xy 163.83 62.23)
+			(xy 163.83 59.69) (xy 163.83 63.5)
 		)
 		(stroke
@@
 	(wire
 		(pts
-			(xy 162.56 106.68) (xy 162.56 109.22)
+			(xy 162.56 106.68) (xy 162.56 110.49)
 		)
 		(stroke
@@
 	(wire
 		(pts
-			(xy 163.83 72.39) (xy 163.83 74.93)
+			(xy 163.83 71.12) (xy 163.83 74.93)
 		)
 		(stroke
@@
 	(wire
 		(pts
-			(xy 93.98 104.14) (xy 93.98 106.68)
+			(xy 93.98 104.14) (xy 93.98 107.95)
 		)
 		(stroke
@@
 			"AAAAAAAAAAAAAAAAAAAAAAAAAAAAAAAAAAAAAAAAAAAAAAAAAAAAAAAAAAAAAAAAAAAAAAAAAAAA"
 			"AAAAAAAAAAAAAAAAAAAAAAAAAAAAAAAAAAAAAAAAAAAAAAAAAAAAAAAAAAAAAAAAAAAAAAAAAAAA"
+			"AAAAAAAAAAAAAAAAAAAAAAAAAAAAADgAMQBtAHMAOQBsAHMANgBuAHMAQwBTAFMATgBEAEkAYgBo"
+			"AFMASwB2AEEAOQBwAFoAUwBMAHEAVgBoAGoAQwBLAHgAZwBFAGgAaQBpAEIAUQBKAHcAUwBiAFQA"
+			"NwBHAE4AZgBlAFEAKwAwAG4ALwAxAHAANQBnAEMAWABqAGUAagBiAHYAbwBSAGgAbgBUAEIARwBS"
+			"AHQAYwBBAFkAYwBxADYAaQBpAEgAbQArAHoAeABXADcAWQA4ADYAMAAxAGcAZwBvAHUAVgBEAEsA"
+			"bAAxAEsAYQBUAGwAdgBIAHUAOQBLADAARABKAGsAUQA0AG0AVQBnAEIAbQBPAHUAUgB0AGUAeQBv"
+			"AGYAVwBCADYANABEAHQAMQBNAGIAagB4ADQAKwBqAE8AUAA3AFcATgA3AC8ANQA3AFcAOQAvAE8A"
+			"NAA1AGoAcwBMAFoAcgAyADYAZABQAG4AegA1ADQAOABPAEQAWgBzADIAZABOADAAMABSAEIAYQBK"
+			"AHIATwBGAHkAcgB5AGcAeQB4AE4AeQAwADQAWABhAGYAYgAwADgAWgBQAEgARAB4AC8ATgBwADEA"
+			"TQBBAFkARQBJADQAcAA0AGQALwB6AHQATAA3AEkAeAArAEgATAArADgATAA0AFUAWABYAEoAZQBi"
+			"ADkATwBQAEMATgBxAGEAOAAyAEoAWABoAHAAOQA0AFoALwB2AFAARQBTAHYAKwBKAFcARwBxAGcA"
+			"WAAwAFYAYwBhAFUAcQBoAHUAbgBnAFAATABxAHAAWgBTAEMAUwBIAHoAbwByAGkANgBXAGwAVgBW"
+			"AE4AUgBxAFAAVAA4AC8ATwBrADkARQBZAEMATABJAHMAcgBhAHEARwBNAFYANABVADEAZgAzADMA"
+			"MwAvAC8ARgB6ADMALwArAGcAeAAvADgANwBZAGMAZgBmAGEAQgAxAEcAdwBSAGUARwBFAGQAVwB0"
+			"AHkANQBCAHkAMQBKAGYAOQBRAFgAQQBDAFUAQQB3ADcAbgBsAFMAMgB5ADcAUABVADIATQAxAFkA"
+			"NgBDAE4AVgBzAHEAUABvADcAZwBvAHEAMwBXADYAVwB5AHcAVwBUAGQAZAAxADIAawB4AG0ATQA5"
+			"AC8AMwBCAFcAZABhAEUAMQBsAHkATwBVAE4AMgBLAE8ARQArAFYAQgA3AFcAdwB0AEQASQBIAFEA"
+			"YwBoAFMAVQBhAGIAWABiAHIATAA4ADcAegBJAGkANwBxAHAAbABWAEwAagA4AFcAUQB5AEgAagB0"
+			"AHMAbwBlAHUAQQBNAFQAYQBkAGoAcQBJAG8ARgBKAHcAdABGAG8AdgBsAGEAcgBWAFkAWABMAGsA"
+			"cABtAHMANQBtAGgALwBOAEIAUgBNAAAAAAAAAAAAAAAAAAAAAAAAAAAAAAAAAAAAAAAAAAAAAAAA"
+			"AAAAAAAAAAAAAAAAAAAAAAAAAAAAAAAAAAAAAAAAAAAAAAAAAAAAAAAAAAAAAAAAAAAAAAAAAAAA"
+			"AAAAAAAAAAAAAAAAAAAAAAAAAAAAAAAAAAAAAAAAAAAAAAAAAAAAAAAAAAAAAAAAAAAAAAAAAAAA"
+			"AAAAAAAAAAAAAAAAAAAAAAAAAAAAAAAAAAAAAAAAAAAAAAAAAAAAAAAAAAAAAAAAAAAAAAAAAAAA"
+			"AAAAAAAAAAAAAAAAAAAAAAAAAAAAAAAAAAAAAAAAAAAAAAAAAAAAAAAAAAAAAAAAAAAAAAAAAAAA"
+			"AAAAAAAAAAAAAAAAAAAAAAAAAAAAAAAAAAAAAAAAAAAAAAAAAAAAAAAAAAAAAAAAAAAAAAAAAAAA"
+			"AAAAAAAAAAAAAAAAAAAAAAAAAAAAAAAAAAAAAAAAAAAAAAAAAAAAAAAAAAAAAAAAAAAAAAAAAAAA"
+			"AAAAAAAAAAAAAAAAAAAAAAAAAAAAAAAAAAAAAAAAAAAAAAAAAAAAAAAAAAAAAAAAAAAAAAAAAAAA"
+			"AAAAAAAAAAAAAAAAAAAAAAAAAAAAAAAAAAAAAAAAAAAAAAAAAAAAAAAAAAAAAAAAAAAAAAAAAAAA"
+			"AAAAAAAAAAAAAAAAAAAAAAAAAAAAAAAAAAAAAAAAAAAAAAAAAAAAAAAAAAAAAAAAAAAAAAAAAAAA"
+			"AAAAAAAAAAAAAAAAAAAAAAAAAAAAAAAAAAAAAAAAAAAAAAAAAAAAAAAAAAAAAAAAAAAAAAAAAAAA"
+			"AAAAAAAAAAAAAAAAAAAAAAAAAAAAAAAAAAAAAAAAAAAAAAAAAAAAAAAAAAAAAAAAAAAAAAAAAAAA"
+			"AAAAAAAAAAAAAAAAAAAAAAAAAAAAAAAAAAAAAAAAAAAAAAAAAAAAAAAAAAAAAAAAAAAAAAAAAAAA"
+			"AAAAAAAAAAAAAAAAAAAAAAAAAAAAAAAAAAAAAAAAAAAAAAAAAAAAAAAAAAAAAAAAAAAAAAAAAAAA"
+			"AAAAAAAAAAAAAAAAAAAAAAAAAAAAAAAAAAAAAAAAAAAAAAAAAAAAAAAAAAAAAAAAAAAAAAAAAAAA"
+			"AAAAAAAAAAAAAAAAAAAAAAAAAAAAAAAAAAAAAAAAAAAAAAAAAAAAAAAAAAAAAAAAAAAAAAAAAAAA"
+			"AAAAAAAAAAAAAAAAAAAAAAAAAAAAAAAAAAAAAAAAAAAAAAAAAAAAAAAAAAAAAAAAAAAAAAAAAAAA"
+			"AAAAAAAAAAAAAAAAAAAAAAAAAAAAAAAAAAAAAAAAAAAAAAAAAAAAAAAAAAAAAAAAAAAAAAAAAAAA"
 			"AAAAAAAAAAAAAAAAAAAAAAAAAAAAAA=="
 		)
@@
 			)
 		)
-		(property "Value" "RES 0603"
+		(property "Value" "10K 0.1% 0603"
 			(at 107.95 95.25 90)
 			(effects
@@
 			)
 		)
-		(property "Value" "RES 0603"
+		(property "Value" "10K 0.1% 0603"
 			(at 153.67 49.53 0)
 			(effects
@@
 			)
 		)
-		(property "Value" "RES 0603"
+		(property "Value" "10K 0.1% 0603"
 			(at 152.4 96.52 0)
 			(effects
@@
 			)
 		)
-		(property "Value" "RES 0603"
+		(property "Value" "10K 0.1% 0603"
 			(at 109.22 48.26 90)
 			(effects

Commit message: Update Schematic
Parts:
- C92: renamed from C90; value CAP CER 0603 -> 100nF 50V 0603
- C93: renamed from C91; value CAP CER 0603 -> 100nF 50V 0603
- C94: renamed from C92; value CAP CER 0603 -> 100nF 50V 0603
- C95: renamed from C93; value CAP CER 0603 -> 100nF 50V 0603
Other:
- moved on the sheet: C92, C93, R53, R54, U14

Commit message: Update Schematic & PCB
Parts:
- removed R54, R56: 10K 0.1% 0603, Duc:R0603, symbol Duc-Resistors:RES SMD 0603
Connections:
- net FDCAN1_RX: now also U15.4 (RXD); no longer U14.4 (RXD)
- net FDCAN1_TX: now also R55.1, U15.1 (TXD); no longer R53.1, U14.1 (TXD)
- net FDCAN2_RX: now also U14.4 (RXD); no longer U15.4 (RXD)
- net FDCAN2_TX: now also R53.1, U14.1 (TXD); no longer R55.1, U15.1 (TXD)
- net GND: now also U14.8 (S), U15.8 (S)

Commit message: Update Schematic & PCB
Parts:
- C92, C93, C94, C95: value 100nF 50V 0603 -> CAP CER 0603
- R53, R55: value 10K 0.1% 0603 -> RES 0603
Changed lines of the file:
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@@
 			"cgAAAAAAAAAAAAAAAAAAAAAADwAAAAAAAAAAaXJtYWxhIFVJAAAAAAAAAAAAAAAAAAAPAAAAAAAA"
 			"AAAAAAAAAAAAAAAAAAAAAAAAAAAAAAAAAACPfSgeAgAAAAAAAAAAAAAAAAAAAAAAAA8AAAAAAAAA"
-			"AG9sZAAAAAAAAAAAAAAAAAAAAAAAAA=="
+			"AG9sZAAAAAAAAAAAAAAAAAAAAAAAAAAA1mtqFQCoBoBGw6lsa8O2dsOpcgBjAAAAAAAAAAAAAADU"
+			"a2gVAKkGgGt1cnrDrXZhAAAAAAAAAAAAAAAAAAAAANJrZhVQqgaAVGltZXMgTmV3IFJvbWFuAA8A"
+			"AAAAAAAA0GtkFQCrBoDOoM67zqzOs865zrEAAAAADwAAAAAAAADOa2IVdawGgEt1cnNpdm9pdHUA"
+			"AAAAAAAPAAAAAAAAAMxrYBUArQaASXRhbGlxdWUAAAAAAAAAAAAPnJxQAgAAymt+FQCuBoBJdMOh"
+			"bGljbwAAAAAAAAAAAGVndWxhcgDIa3wVAK8GgNCa0YPRgNGB0LjQsgAAAAAAYWxndW4gR8ZrehVj"
+			"sAaAUG/FoWV2bm8AAAAAAAAAAAAAAAAAAAAAxGt4FQCxBoAAAAAAAAAAAKbA/4ZQAgAA4AfKx1AC"
+			"AADCa3YVALIGgAYAAAAQAAAAcNQSAQAAAAAAAAAAAAAAAMBrdBUAswaAUG9ncnViaW9uYSBrdXJz"
+			"eXdhAGljAAAAPmtyFQC0BoBIYWx2ZmV0IEt1cnNpdgAAAAAAAAAAAAA8a3AVALUGgAAAAAAAAAAA"
+			"AB5yMwAAAAAABsrHUAIAADprjhUAtgaAUG/FoWV2bm8AAAAAAAAAAAAAAAAAAAAAOGuMFQC3BoBU"
+			"aW1lcyBOZXcgUm9tYW4AAAAAAAAAAAA2a4oVALgGgEthbMSxbiDEsHRhbGlrAAAAAAAAAAAAADRr"
+			"iBVQuQaAzprOsc69zr/Ovc65zrrOrAAAAAAAAAAAMmuGFQC6BoBOZWdyaXRvIEl0w6FsaWNvAAAA"
+			"AAAAAAAwa4QVdbsGgE5vcm1hYWxpAAAAAAAAAAAPAAAAAAAAAC5rghUAvAaAAAAAAAAAAADRMYEN"
+			"AAAAAOADysdQAgAALGuAFQC9BoBLcmVwa28gcG/FoWV2bm8AAAAAAAAAAAAqa54VAL4GgFN0YW5k"
+			"YXJkAAAAAAAAAAAAAAAAAAAAAChrnBUAvwaAUG9ncnViaW9uYQAAAAAAAHAAAAAAAAAAJmuaFQDA"
+			"BoBOb3JtYWFsaQAAAAAAAAAAAAAAAAAAAAAka5gVAMEGgFl1IEdvdGhpYwBpYwAAAAAAAAAAAAAA"
+			"ACJrlhUAwgaABgAAABAAAADA+RIBAAAAAAAAAAAAAAAAIGuUFQDDBoBTdGFuZGFhcmQAAAAAAAAA"
+			"AAAAAAAAAAAea5IVUMQGgNCe0LHRi9GH0L3Ri9C5AAAPAAAAAAAAABxrkBVrxQaAV2luQ0NfZmxl"
+			"eGlibGVfaGlnaAAAAAAAGmuuFW7GBoBOb3JtYWFsaQAAAAAAAAAADwAAAAAAAAAYa6wVAMcGgENv"
+			"bmRlbnNlZCBSZWd1bGFyAADGUAIAAAAAAAAAAAAAAAAAAAAAAAAAAAAAAAAAAAAAAAAAAAAAAAAA"
+			"AAAAAAAAAAAAAAAAAAAAAAAAAAAAAAAAAAAAAAAAAAAAAAAAAAAAAAAAAAAAAAAAAAAAAAAAAAAA"
+			"AAAAAAAAAAAAAAAAAAAAAAAAAAAAAAAAAAAAAAAAAAAAAAAAAAAAAAAAAAAAAAAAAAAAAAAAAAAA"
+			"AAAAAAAAAAAAAAAAAAAAAAAAAAAAAAAAAAAAAAAAAAAAAAAAAAAAAAAAAAAAAAAAAAAAAAAAAAAA"
+			"AAAAAAAAAAAAAAAAAAAAAAAAAAAAAAAAAAAAAAAAAAAAAAAAAAAAAAAAAAAAAAAAAAAAAAAAAAAA"
+			"AAAAAAAAAAAAAAAAAAAAAAAAAAAAAAAAAAAAAAAAAAAAAAAAAAAAAAAAAAAAAAAAAAAAAAAAAAAA"
+			"AAAAAAAAAAAAAAAAAAAAAAAAAAAAAAAAAAAAAAAAAAAAAAAAAAAAAAAAAAAAAAAAAAAAAAAAAAAA"
+			"AAAAAAAAAAAAAAAAAAAAAAAAAAAAAAAAAAAAAAAAAAAAAAAAAAAAAAAAAAAAAAAAAAAAAAAAAAAA"
+			"AAAAAAAAAAAAAAAAAAAAAAAAAAAAAAAAAAAAAAAAAAAAAAAAAAAAAAAAAAAAAAAAAAAAAAAAAAAA"
+			"AAAAAAAAAAAAAAAAAAAAAAAAAAAAAAAAAAAAAAAAAAAAAAAAAAAAAAAAAAAAAAAAAAAAAAAAAAAA"
+			"AAAAAAAAAAAAAAAAAAAAAAAAAAAAAAAAAAAAAAAAAAAAAAAAAAAAAAAAAAAAAAAAAAAAAAAAAAAA"
+			"AAAAAAAAAAAAAAAAAAAAAAAAAAAAAAAAAAAAAAAAAAAAAAAAAAAAAAAAAAAAAAAAAAAAAAAAAAAA"
+			"AAAAAAAAAAAAAAAAAAAAAAAAAAAAAAAAAAAAAAAAAAAAAAAAAAAAAAAAAAAAAAAAAAAAAAAAAAAA"
+			"AAAAAAAAAAAAAAAAAAAAAAAAAAAAAAAAAAAAAAAAAAAAAAAAAAAAAAAAAAAAAAAAAAAAAAAAAAAA"
+			"AAAAAAAAAAAAAAAAAAAAAAAAAAAAAAAAAAAAAAAAAAAAAAAAAAAAAAAAAAAAAAAAAAAAAAAAAAAA"
+			"AAAAAAAAAAAAAAAAAAAAAAAAAAAAAAAAAAAAAAAAAAAAAAAAAAAAAAAAAAAAAAAAAAAAAAAAAAAA"
+			"AAAAAAAAAAAAAAAAAAAAAAAAAAAAAAAAAAAAAAAAAAAAAAAAAAAAAAAAAAAAAAAAAAAAAAAAAAAA"
+			"AAAAAAAAAAAAAAAAAAAAAAAAAAAAAAAAAAAAAAAAAAAAAAAAAAAAAAAAAAAAAAAAAAAAAAAAAAAA"
+			"AAAAAAAAAAAAAAAAAAAAAAAAAAAAAA=="
 		)
 	)
@@
 			)
 		)
-		(property "Value" "10K 0.1% 0603"
+		(property "Value" "RES 0603"
 			(at 107.95 95.25 90)
 			(effects
@@
 		(dnp no)
 		(fields_autoplaced yes)
-		(property "Reference" "#PWR0115"
+		(property "Reference" "#PWR115"
 			(at 97.536 62.484 0)
 			(do_not_autoplace yes)
@@
 			(project "Master_Hand_Kicad"
 				(path "/f9e05184-c88b-4a88-ae9c-ab2bdb32be7c/c5103ceb-5325-4a84-a025-9638a412984e/f2e2e46b-bf48-4385-80eb-484ec861c9a9"
-					(reference "#PWR0115")
+					(reference "#PWR115")
 					(unit 1)
 				)
@@
 		(dnp no)
 		(fields_autoplaced yes)
-		(property "Reference" "#PWR0113"
+		(property "Reference" "#PWR113"
 			(at 155.194 48.514 0)
 			(do_not_autoplace yes)
@@
 			(project "Master_Hand_Kicad"
 				(path "/f9e05184-c88b-4a88-ae9c-ab2bdb32be7c/c5103ceb-5325-4a84-a025-9638a412984e/f2e2e46b-bf48-4385-80eb-484ec861c9a9"
-					(reference "#PWR0113")
+					(reference "#PWR113")
 					(unit 1)
 				)
@@
 		(dnp no)
 		(fields_autoplaced yes)
-		(property "Reference" "#PWR0119"
+		(property "Reference" "#PWR119"
 			(at 96.266 110.744 0)
 			(do_not_autoplace yes)
@@
 			(project "Master_Hand_Kicad"
 				(path "/f9e05184-c88b-4a88-ae9c-ab2bdb32be7c/c5103ceb-5325-4a84-a025-9638a412984e/f2e2e46b-bf48-4385-80eb-484ec861c9a9"
-					(reference "#PWR0119")
+					(reference "#PWR119")
 					(unit 1)
 				)
@@
 			)
 		)
-		(property "Value" "100nF 50V 0603"
+		(property "Value" "CAP CER 0603"
 			(at 74.93 113.03 90)
 			(effects
@@
 			)
 		)
-		(property "Value" "100nF 50V 0603"
+		(property "Value" "CAP CER 0603"
 			(at 166.37 67.31 90)
 			(effects
@@
 			)
 		)
-		(property "Value" "100nF 50V 0603"
+		(property "Value" "CAP CER 0603"
 			(at 76.2 64.77 90)
 			(effects
@@
 		(dnp no)
 		(fields_autoplaced yes)
-		(property "Reference" "#PWR0114"
+		(property "Reference" "#PWR114"
 			(at 117.856 55.626 0)
 			(do_not_autoplace yes)
@@
 			(project "Master_Hand_Kicad"
 				(path "/f9e05184-c88b-4a88-ae9c-ab2bdb32be7c/c5103ceb-5325-4a84-a025-9638a412984e/f2e2e46b-bf48-4385-80eb-484ec861c9a9"
-					(reference "#PWR0114")
+					(reference "#PWR114")
 					(unit 1)
 				)
@@
 			)
 		)
-		(property "Value" "100nF 50V 0603"
+		(property "Value" "CAP CER 0603"
 			(at 165.1 115.57 90)
 			(effects
@@
 		(dnp no)
 		(fields_autoplaced yes)
-		(property "Reference" "#PWR0120"
+		(property "Reference" "#PWR120"
 			(at 164.846 113.284 0)
 			(do_not_autoplace yes)
@@
 			(project "Master_Hand_Kicad"
 				(path "/f9e05184-c88b-4a88-ae9c-ab2bdb32be7c/c5103ceb-5325-4a84-a025-9638a412984e/f2e2e46b-bf48-4385-80eb-484ec861c9a9"
-					(reference "#PWR0120")
+					(reference "#PWR120")
 					(unit 1)
 				)
@@
 		(dnp no)
 		(fields_autoplaced yes)
-		(property "Reference" "#PWR0116"
+		(property "Reference" "#PWR116"
 			(at 166.116 65.024 0)
 			(do_not_autoplace yes)
@@
 			(project "Master_Hand_Kicad"
 				(path "/f9e05184-c88b-4a88-ae9c-ab2bdb32be7c/c5103ceb-5325-4a84-a025-9638a412984e/f2e2e46b-bf48-4385-80eb-484ec861c9a9"
-					(reference "#PWR0116")
+					(reference "#PWR116")
 					(unit 1)
 				)
@@
 			)
 		)
-		(property "Value" "10K 0.1% 0603"
+		(property "Value" "RES 0603"
 			(at 109.22 46.99 90)
 			(effects
@@
 		(dnp no)
 		(fields_autoplaced yes)
-		(property "Reference" "#PWR0117"
+		(property "Reference" "#PWR117"
 			(at 153.924 96.774 0)
 			(do_not_autoplace yes)
@@
 			(project "Master_Hand_Kicad"
 				(path "/f9e05184-c88b-4a88-ae9c-ab2bdb32be7c/c5103ceb-5325-4a84-a025-9638a412984e/f2e2e46b-bf48-4385-80eb-484ec861c9a9"
-					(reference "#PWR0117")
+					(reference "#PWR117")
 					(unit 1)
 				)
@@
 		(dnp no)
 		(fields_autoplaced yes)
-		(property "Reference" "#PWR0118"
+		(property "Reference" "#PWR118"
 			(at 116.586 103.886 0)
 			(do_not_autoplace yes)
@@
 			(project "Master_Hand_Kicad"
 				(path "/f9e05184-c88b-4a88-ae9c-ab2bdb32be7c/c5103ceb-5325-4a84-a025-9638a412984e/f2e2e46b-bf48-4385-80eb-484ec861c9a9"
-					(reference "#PWR0118")
+					(reference "#PWR118")
 					(unit 1)
 				)

Commit message: Update SCH & PCB
Parts:
- renumbered C92 to C87, C93 to C88, C94 to C89, C95 to C90, R55 to R54
Changed lines of the file:
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@@
 		(on_board yes)
 		(dnp no)
-		(property "Reference" "R55"
+		(property "Reference" "R54"
 			(at 113.03 92.71 90)
 			(effects
@@
 			(project "Master_Hand_Kicad"
 				(path "/f9e05184-c88b-4a88-ae9c-ab2bdb32be7c/c5103ceb-5325-4a84-a025-9638a412984e/f2e2e46b-bf48-4385-80eb-484ec861c9a9"
-					(reference "R55")
+					(reference "R54")
 					(unit 1)
 				)
@@
 		(dnp no)
 		(fields_autoplaced yes)
-		(property "Reference" "#PWR115"
+		(property "Reference" "#PWR0115"
 			(at 97.536 62.484 0)
 			(do_not_autoplace yes)
@@
 			(project "Master_Hand_Kicad"
 				(path "/f9e05184-c88b-4a88-ae9c-ab2bdb32be7c/c5103ceb-5325-4a84-a025-9638a412984e/f2e2e46b-bf48-4385-80eb-484ec861c9a9"
-					(reference "#PWR115")
+					(reference "#PWR0115")
 					(unit 1)
 				)
@@
 		(dnp no)
 		(fields_autoplaced yes)
-		(property "Reference" "#PWR113"
+		(property "Reference" "#PWR0113"
 			(at 155.194 48.514 0)
 			(do_not_autoplace yes)
@@
 			(project "Master_Hand_Kicad"
 				(path "/f9e05184-c88b-4a88-ae9c-ab2bdb32be7c/c5103ceb-5325-4a84-a025-9638a412984e/f2e2e46b-bf48-4385-80eb-484ec861c9a9"
-					(reference "#PWR113")
+					(reference "#PWR0113")
 					(unit 1)
 				)
@@
 		(dnp no)
 		(fields_autoplaced yes)
-		(property "Reference" "#PWR119"
+		(property "Reference" "#PWR0119"
 			(at 96.266 110.744 0)
 			(do_not_autoplace yes)
@@
 			(project "Master_Hand_Kicad"
 				(path "/f9e05184-c88b-4a88-ae9c-ab2bdb32be7c/c5103ceb-5325-4a84-a025-9638a412984e/f2e2e46b-bf48-4385-80eb-484ec861c9a9"
-					(reference "#PWR119")
+					(reference "#PWR0119")
 					(unit 1)
 				)
@@
 		(on_board yes)
 		(dnp no)
-		(property "Reference" "C94"
+		(property "Reference" "C89"
 			(at 87.63 110.49 90)
 			(effects
@@
 			(project "Master_Hand_Kicad"
 				(path "/f9e05184-c88b-4a88-ae9c-ab2bdb32be7c/c5103ceb-5325-4a84-a025-9638a412984e/f2e2e46b-bf48-4385-80eb-484ec861c9a9"
-					(reference "C94")
+					(reference "C89")
 					(unit 1)
 				)
@@
 		(on_board yes)
 		(dnp no)
-		(property "Reference" "C93"
+		(property "Reference" "C88"
 			(at 166.37 64.77 90)
 			(effects
@@
 			(project "Master_Hand_Kicad"
 				(path "/f9e05184-c88b-4a88-ae9c-ab2bdb32be7c/c5103ceb-5325-4a84-a025-9638a412984e/f2e2e46b-bf48-4385-80eb-484ec861c9a9"
-					(reference "C93")
+					(reference "C88")
 					(unit 1)
 				)
@@
 		(on_board yes)
 		(dnp no)
-		(property "Reference" "C92"
+		(property "Reference" "C87"
 			(at 88.9 62.23 90)
 			(effects
@@
 			(project "Master_Hand_Kicad"
 				(path "/f9e05184-c88b-4a88-ae9c-ab2bdb32be7c/c5103ceb-5325-4a84-a025-9638a412984e/f2e2e46b-bf48-4385-80eb-484ec861c9a9"
-					(reference "C92")
+					(reference "C87")
 					(unit 1)
 				)
@@
 		(dnp no)
 		(fields_autoplaced yes)
-		(property "Reference" "#PWR114"
+		(property "Reference" "#PWR0114"
 			(at 117.856 55.626 0)
 			(do_not_autoplace yes)
@@
 			(project "Master_Hand_Kicad"
 				(path "/f9e05184-c88b-4a88-ae9c-ab2bdb32be7c/c5103ceb-5325-4a84-a025-9638a412984e/f2e2e46b-bf48-4385-80eb-484ec861c9a9"
-					(reference "#PWR114")
+					(reference "#PWR0114")
 					(unit 1)
 				)
@@
 		(on_board yes)
 		(dnp no)
-		(property "Reference" "C95"
+		(property "Reference" "C90"
 			(at 165.1 113.03 90)
 			(effects
@@
 			(project "Master_Hand_Kicad"
 				(path "/f9e05184-c88b-4a88-ae9c-ab2bdb32be7c/c5103ceb-5325-4a84-a025-9638a412984e/f2e2e46b-bf48-4385-80eb-484ec861c9a9"
-					(reference "C95")
+					(reference "C90")
 					(unit 1)
 				)
@@
 		(dnp no)
 		(fields_autoplaced yes)
-		(property "Reference" "#PWR120"
+		(property "Reference" "#PWR0120"
 			(at 164.846 113.284 0)
 			(do_not_autoplace yes)
@@
 			(project "Master_Hand_Kicad"
 				(path "/f9e05184-c88b-4a88-ae9c-ab2bdb32be7c/c5103ceb-5325-4a84-a025-9638a412984e/f2e2e46b-bf48-4385-80eb-484ec861c9a9"
-					(reference "#PWR120")
+					(reference "#PWR0120")
 					(unit 1)
 				)
@@
 		(dnp no)
 		(fields_autoplaced yes)
-		(property "Reference" "#PWR116"
+		(property "Reference" "#PWR0116"
 			(at 166.116 65.024 0)
 			(do_not_autoplace yes)
@@
 			(project "Master_Hand_Kicad"
 				(path "/f9e05184-c88b-4a88-ae9c-ab2bdb32be7c/c5103ceb-5325-4a84-a025-9638a412984e/f2e2e46b-bf48-4385-80eb-484ec861c9a9"
-					(reference "#PWR116")
+					(reference "#PWR0116")
 					(unit 1)
 				)
@@
 		(dnp no)
 		(fields_autoplaced yes)
-		(property "Reference" "#PWR117"
+		(property "Reference" "#PWR0117"
 			(at 153.924 96.774 0)
 			(do_not_autoplace yes)
@@
 			(project "Master_Hand_Kicad"
 				(path "/f9e05184-c88b-4a88-ae9c-ab2bdb32be7c/c5103ceb-5325-4a84-a025-9638a412984e/f2e2e46b-bf48-4385-80eb-484ec861c9a9"
-					(reference "#PWR117")
+					(reference "#PWR0117")
 					(unit 1)
 				)
@@
 		(dnp no)
 		(fields_autoplaced yes)
-		(property "Reference" "#PWR118"
+		(property "Reference" "#PWR0118"
 			(at 116.586 103.886 0)
 			(do_not_autoplace yes)
@@
 			(project "Master_Hand_Kicad"
 				(path "/f9e05184-c88b-4a88-ae9c-ab2bdb32be7c/c5103ceb-5325-4a84-a025-9638a412984e/f2e2e46b-bf48-4385-80eb-484ec861c9a9"
-					(reference "#PWR118")
-					(unit 1)
-				)
+					(reference "#PWR0118")
+					(unit 1)
+				)

Commit message: Update SCH & PCB
Parts:
- C87, C88, C89, C90: value CAP CER 0603 -> CAP CER 0402; footprint Duc:C0603 -> Duc:C0402; symbol Duc-Capacitors:CAP CER 0603 -> Duc-Capacitors:CAP CER 0402; LCSC Part C14663 -> C325464; MPN CAP CER 0603 -> CC0402KRX5R7BB105
- R53, R54: value RES 0603 -> RES 0402; footprint Duc:R0603 -> Duc:R0402; symbol Duc-Resistors:RES SMD 0603 -> Duc-Resistors:RES SMD 0402; LCSC Part C4107493 -> C728576; MPN RT0603FRE13100KL -> RT0402FRE07100KL
