File: Interface - Interconnects.kicad_sch (KiCad schematic)
At the start: 14 parts, among them J11 1.25-3PLTDK, J12 5025982393, J13 PH2.54-2X3P-H25, J14 PH2.54-2X3P-H25, J15 PH2.54-2X3P-H25

Commit message: Update Schematic
Parts:
- C94: value CAP CER 0603 -> 4.7uF 50V 0603
- C95, C96, C97: value CAP CER 0603 -> 100nF 50V 0603
- R57, R58: value RES 0603 -> 2.2K 0.1% 0603
- R59, R60: value RES 0603 -> 60R4 0.1% 0603

Commit message: Update Schematic
Parts:
- renumbered C94 to C96, C95 to C97, C96 to C98, C97 to C99
Changed lines of the file:
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@@
 		(on_board yes)
 		(dnp no)
-		(property "Reference" "C96"
+		(property "Reference" "C98"
 			(at 153.67 121.92 90)
 			(effects
@@
 			(project "Master_Hand_Kicad"
 				(path "/f9e05184-c88b-4a88-ae9c-ab2bdb32be7c/c5103ceb-5325-4a84-a025-9638a412984e/17a3bf50-6382-4412-b8e5-9c1afeb8fb2e"
-					(reference "C96")
+					(reference "C98")
 					(unit 1)
 				)
@@
 		(on_board yes)
 		(dnp no)
-		(property "Reference" "C95"
+		(property "Reference" "C97"
 			(at 90.17 121.92 90)
 			(effects
@@
 			(project "Master_Hand_Kicad"
 				(path "/f9e05184-c88b-4a88-ae9c-ab2bdb32be7c/c5103ceb-5325-4a84-a025-9638a412984e/17a3bf50-6382-4412-b8e5-9c1afeb8fb2e"
-					(reference "C95")
+					(reference "C97")
 					(unit 1)
 				)
@@
 		(on_board yes)
 		(dnp no)
-		(property "Reference" "C97"
+		(property "Reference" "C99"
 			(at 217.17 121.92 90)
 			(effects
@@
 			(project "Master_Hand_Kicad"
 				(path "/f9e05184-c88b-4a88-ae9c-ab2bdb32be7c/c5103ceb-5325-4a84-a025-9638a412984e/17a3bf50-6382-4412-b8e5-9c1afeb8fb2e"
-					(reference "C97")
+					(reference "C99")
 					(unit 1)
 				)
@@
 		(on_board yes)
 		(dnp no)
-		(property "Reference" "C94"
+		(property "Reference" "C96"
 			(at 195.58 71.12 90)
 			(effects
@@
 			(project "Master_Hand_Kicad"
 				(path "/f9e05184-c88b-4a88-ae9c-ab2bdb32be7c/c5103ceb-5325-4a84-a025-9638a412984e/17a3bf50-6382-4412-b8e5-9c1afeb8fb2e"
-					(reference "C94")
-					(unit 1)
-				)
+					(reference "C96")
+					(unit 1)
+				)

Commit message: Update Schematic & PCB
Connections:
- net FDCAN_N: now also D8.1; no longer D8.2
- net FDCAN_P: now also D8.2; no longer D8.1

Commit message: Update Schematic & PCB
Parts:
- C96: value 4.7uF 50V 0603 -> CAP CER 0603
- C97, C98, C99: value 100nF 50V 0603 -> CAP CER 0603
- R57, R58: value 2.2K 0.1% 0603 -> RES 0603
- R59, R60: value 60R4 0.1% 0603 -> RES 0603

Commit message: Update SCH & PCB
Parts:
- renumbered C96 to C91, C97 to C92, C98 to C93, C99 to C94, R57 to R55, R58 to R56, R59 to R57, R60 to R58
Connections:
- net NRST1: now also J12.19; no longer J12.13
- net NRST2: now also J12.9; no longer J12.19
- net SWCLK1: now also J12.15; no longer J12.11
- net SWCLK2: now also J12.13; no longer J12.17
- net SWDIO1: now also J12.17; no longer J12.9
- net SWDIO2: now also J12.11; no longer J12.15
Changed lines of the file:
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@@
 	)
 	(label "SWCLK1"
-		(at 80.01 74.93 0)
+		(at 80.01 80.01 0)
 		(effects
 			(font
@@
 	)
 	(label "SWCLK2"
-		(at 80.01 82.55 0)
+		(at 80.01 77.47 0)
 		(effects
 			(font
@@
 	)
 	(label "SWDIO1"
-		(at 80.01 72.39 0)
+		(at 80.01 82.55 0)
 		(effects
 			(font
@@
 	)
 	(label "SWDIO2"
-		(at 80.01 80.01 0)
+		(at 80.01 74.93 0)
 		(effects
 			(font
@@
 	)
 	(label "NRST1"
-		(at 80.01 77.47 0)
+		(at 80.01 85.09 0)
 		(effects
 			(font
@@
 	)
 	(label "NRST2"
-		(at 80.01 85.09 0)
+		(at 80.01 72.39 0)
 		(effects
 			(font
@@
 		(on_board no)
 		(dnp no)
-		(property "Reference" "#PWR129"
+		(property "Reference" "#PWR0129"
 			(at 225.806 123.444 0)
 			(do_not_autoplace yes)
@@
 			(project "Master_Hand_Kicad"
 				(path "/f9e05184-c88b-4a88-ae9c-ab2bdb32be7c/c5103ceb-5325-4a84-a025-9638a412984e/17a3bf50-6382-4412-b8e5-9c1afeb8fb2e"
-					(reference "#PWR129")
+					(reference "#PWR0129")
 					(unit 1)
 				)
@@
 		(on_board yes)
 		(dnp no)
-		(property "Reference" "C98"
+		(property "Reference" "C93"
 			(at 153.67 121.92 90)
 			(effects
@@
 			(project "Master_Hand_Kicad"
 				(path "/f9e05184-c88b-4a88-ae9c-ab2bdb32be7c/c5103ceb-5325-4a84-a025-9638a412984e/17a3bf50-6382-4412-b8e5-9c1afeb8fb2e"
-					(reference "C98")
+					(reference "C93")
 					(unit 1)
 				)
@@
 		(on_board no)
 		(dnp no)
-		(property "Reference" "#PWR130"
+		(property "Reference" "#PWR0130"
 			(at 230.886 123.444 0)
 			(do_not_autoplace yes)
@@
 			(project "Master_Hand_Kicad"
 				(path "/f9e05184-c88b-4a88-ae9c-ab2bdb32be7c/c5103ceb-5325-4a84-a025-9638a412984e/17a3bf50-6382-4412-b8e5-9c1afeb8fb2e"
-					(reference "#PWR130")
+					(reference "#PWR0130")
 					(unit 1)
 				)
@@
 		(dnp no)
 		(fields_autoplaced yes)
-		(property "Reference" "#PWR121"
+		(property "Reference" "#PWR0121"
 			(at 78.994 59.944 0)
 			(do_not_autoplace yes)
@@
 			(project "Master_Hand_Kicad"
 				(path "/f9e05184-c88b-4a88-ae9c-ab2bdb32be7c/c5103ceb-5325-4a84-a025-9638a412984e/17a3bf50-6382-4412-b8e5-9c1afeb8fb2e"
-					(reference "#PWR121")
+					(reference "#PWR0121")
 					(unit 1)
 				)
@@
 		(dnp no)
 		(fields_autoplaced yes)
-		(property "Reference" "R59"
+		(property "Reference" "R57"
 			(at 171.45 57.1499 90)
 			(effects
@@
 			(project "Master_Hand_Kicad"
 				(path "/f9e05184-c88b-4a88-ae9c-ab2bdb32be7c/c5103ceb-5325-4a84-a025-9638a412984e/17a3bf50-6382-4412-b8e5-9c1afeb8fb2e"
-					(reference "R59")
+					(reference "R57")
 					(unit 1)
 				)
@@
 		(on_board no)
 		(dnp no)
-		(property "Reference" "#PWR127"
+		(property "Reference" "#PWR0127"
 			(at 162.306 123.444 0)
 			(do_not_autoplace yes)
@@
 			(project "Master_Hand_Kicad"
 				(path "/f9e05184-c88b-4a88-ae9c-ab2bdb32be7c/c5103ceb-5325-4a84-a025-9638a412984e/17a3bf50-6382-4412-b8e5-9c1afeb8fb2e"
-					(reference "#PWR127")
+					(reference "#PWR0127")
 					(unit 1)
 				)
@@
 		(on_board yes)
 		(dnp no)
-		(property "Reference" "C97"
+		(property "Reference" "C92"
 			(at 90.17 121.92 90)
 			(effects
@@
 			(project "Master_Hand_Kicad"
 				(path "/f9e05184-c88b-4a88-ae9c-ab2bdb32be7c/c5103ceb-5325-4a84-a025-9638a412984e/17a3bf50-6382-4412-b8e5-9c1afeb8fb2e"
-					(reference "C97")
+					(reference "C92")
 					(unit 1)
 				)
@@
 		(dnp no)
 		(fields_autoplaced yes)
-		(property "Reference" "#PWR123"
+		(property "Reference" "#PWR0123"
 			(at 195.326 68.834 0)
 			(do_not_autoplace yes)
@@
 			(project "Master_Hand_Kicad"
 				(path "/f9e05184-c88b-4a88-ae9c-ab2bdb32be7c/c5103ceb-5325-4a84-a025-9638a412984e/17a3bf50-6382-4412-b8e5-9c1afeb8fb2e"
-					(reference "#PWR123")
+					(reference "#PWR0123")
 					(unit 1)
 				)
@@
 		(on_board yes)
 		(dnp no)
-		(property "Reference" "R57"
+		(property "Reference" "R55"
 			(at 76.2 34.29 0)
 			(effects
@@
 			(project "Master_Hand_Kicad"
 				(path "/f9e05184-c88b-4a88-ae9c-ab2bdb32be7c/c5103ceb-5325-4a84-a025-9638a412984e/17a3bf50-6382-4412-b8e5-9c1afeb8fb2e"
-					(reference "R57")
+					(reference "R55")
 					(unit 1)
 				)
@@
 		(dnp no)
 		(fields_autoplaced yes)
-		(property "Reference" "R60"
+		(property "Reference" "R58"
 			(at 171.45 69.8499 90)
 			(effects
@@
 			(project "Master_Hand_Kicad"
 				(path "/f9e05184-c88b-4a88-ae9c-ab2bdb32be7c/c5103ceb-5325-4a84-a025-9638a412984e/17a3bf50-6382-4412-b8e5-9c1afeb8fb2e"
-					(reference "R60")
+					(reference "R58")
 					(unit 1)
 				)
@@
 		(on_board yes)
 		(dnp no)
-		(property "Reference" "R58"
+		(property "Reference" "R56"
 			(at 76.2 43.18 0)
 			(effects
@@
 			(project "Master_Hand_Kicad"
 				(path "/f9e05184-c88b-4a88-ae9c-ab2bdb32be7c/c5103ceb-5325-4a84-a025-9638a412984e/17a3bf50-6382-4412-b8e5-9c1afeb8fb2e"
-					(reference "R58")
+					(reference "R56")
 					(unit 1)
 				)
@@
 		(on_board no)
 		(dnp no)
-		(property "Reference" "#PWR125"
+		(property "Reference" "#PWR0125"
 			(at 98.806 123.444 0)
 			(do_not_autoplace yes)
@@
 			(project "Master_Hand_Kicad"
 				(path "/f9e05184-c88b-4a88-ae9c-ab2bdb32be7c/c5103ceb-5325-4a84-a025-9638a412984e/17a3bf50-6382-4412-b8e5-9c1afeb8fb2e"
-					(reference "#PWR125")
+					(reference "#PWR0125")
 					(unit 1)
 				)
@@
 		(on_board yes)
 		(dnp no)
-		(property "Reference" "C99"
+		(property "Reference" "C94"
 			(at 217.17 121.92 90)
 			(effects
@@
 			(project "Master_Hand_Kicad"
 				(path "/f9e05184-c88b-4a88-ae9c-ab2bdb32be7c/c5103ceb-5325-4a84-a025-9638a412984e/17a3bf50-6382-4412-b8e5-9c1afeb8fb2e"
-					(reference "C99")
+					(reference "C94")
 					(unit 1)
 				)
@@
 		(on_board no)
 		(dnp no)
-		(property "Reference" "#PWR126"
+		(property "Reference" "#PWR0126"
 			(at 103.886 123.444 0)
 			(do_not_autoplace yes)
@@
 			(project "Master_Hand_Kicad"
 				(path "/f9e05184-c88b-4a88-ae9c-ab2bdb32be7c/c5103ceb-5325-4a84-a025-9638a412984e/17a3bf50-6382-4412-b8e5-9c1afeb8fb2e"
-					(reference "#PWR126")
+					(reference "#PWR0126")
 					(unit 1)
 				)
@@
 		(dnp no)
 		(fields_autoplaced yes)
-		(property "Reference" "#PWR124"
+		(property "Reference" "#PWR0124"
 			(at 149.606 72.644 0)
 			(do_not_autoplace yes)
@@
 			(project "Master_Hand_Kicad"
 				(path "/f9e05184-c88b-4a88-ae9c-ab2bdb32be7c/c5103ceb-5325-4a84-a025-9638a412984e/17a3bf50-6382-4412-b8e5-9c1afeb8fb2e"
-					(reference "#PWR124")
+					(reference "#PWR0124")
 					(unit 1)
 				)
@@
 		(on_board yes)
 		(dnp no)
-		(property "Reference" "C96"
+		(property "Reference" "C91"
 			(at 195.58 71.12 90)
 			(effects
@@
 			(project "Master_Hand_Kicad"
 				(path "/f9e05184-c88b-4a88-ae9c-ab2bdb32be7c/c5103ceb-5325-4a84-a025-9638a412984e/17a3bf50-6382-4412-b8e5-9c1afeb8fb2e"
-					(reference "C96")
+					(reference "C91")
 					(unit 1)
 				)
@@
 		(dnp no)
 		(fields_autoplaced yes)
-		(property "Reference" "#PWR122"
+		(property "Reference" "#PWR0122"
 			(at 134.366 58.674 0)
 			(do_not_autoplace yes)
@@
 			(project "Master_Hand_Kicad"
 				(path "/f9e05184-c88b-4a88-ae9c-ab2bdb32be7c/c5103ceb-5325-4a84-a025-9638a412984e/17a3bf50-6382-4412-b8e5-9c1afeb8fb2e"
-					(reference "#PWR122")
+					(reference "#PWR0122")
 					(unit 1)
 				)
@@
 		(on_board no)
 		(dnp no)
-		(property "Reference" "#PWR128"
+		(property "Reference" "#PWR0128"
 			(at 167.386 123.444 0)
 			(do_not_autoplace yes)
@@
 			(project "Master_Hand_Kicad"
 				(path "/f9e05184-c88b-4a88-ae9c-ab2bdb32be7c/c5103ceb-5325-4a84-a025-9638a412984e/17a3bf50-6382-4412-b8e5-9c1afeb8fb2e"
-					(reference "#PWR128")
+					(reference "#PWR0128")
 					(unit 1)
 				)

Commit message: Update SCH & PCB
Parts:
- R55, R56: value RES 0603 -> RES 0402; footprint Duc:R0603 -> Duc:R0402; symbol Duc-Resistors:RES SMD 0603 -> Duc-Resistors:RES SMD 0402; LCSC Part C4107493 -> C728576; MPN RT0603FRE13100KL -> RT0402FRE07100KL
- renumbered C94 to C92, C92 to C94, J15 to J13, J13 to J15
Connections:
- net +5V: no longer J12.10, J12.16
- net GND: now also J12.10, J12.13, J12.16, J12.19
- net NRST1: no longer J12.19
- net NRST2: no longer J12.9
- net SWCLK1: no longer J12.15
- net SWCLK2: no longer J12.13
- net SWDIO1: no longer J12.17
- net SWDIO2: no longer J12.11
- new net USART1_RX1: J12.9
- new net USART1_RX2: J12.15
- new net USART1_TX1: J12.11
- new net USART1_TX2: J12.17
Other:
- moved on the sheet: C92, C93, C94, J13, J14, J15
