File: Interface - USB 2.0.kicad_sch (KiCad schematic)
At the start: 20 parts, among them J10 TYPE-C 16PIN 2MD, J9 TYPE-C 16PIN 2MD

Commit message: Update Schematic
Parts:
- removed R51, R52: RES 0402, Duc_Library:R0402, symbol Duc-Resistors:RES SMD 0402
- added R51, R52: 5.1K 0.1% 0603, Duc:R0603, symbol Duc-Resistors:RES SMD 0603
- C88, C89: value CAP CER 0603 -> 4.7uF 50V 0603
- D2, D5: value LED 0603 -> Blue 0603
- R43, R48: value RES 0603 -> 430K 0.1% 0603
- R44, R49: value RES 0603 -> 620K 0.1% 0603
- R45, R50: value RES 0603 -> 1K 0.1% 0603
- R46, R47: value RES 0402 -> 5.1K 0.1% 0603; footprint Duc_Library:R0402 -> Duc:R0603; symbol Duc-Resistors:RES SMD 0402 -> Duc-Resistors:RES SMD 0603; LCSC Part C728576 -> C4107493; MPN RT0402FRE07100KL -> RT0603FRE13100KL; Manufacturer (none) -> YAGEO(国巨)
Connections:
- net GND: now also R51.2, R52.2
- net at J10.B5 (CC2): now also R52.1
- net at J10.A5 (CC1): now also R51.1
Other:
- moved on the sheet: D3

Commit message: Update Schematic
Parts:
- added C89, C91: 100nF 50V 0402, Duc_Library:C0402, symbol Duc-Capacitors:CAP CER 0402
- R43, R48: value 430K 0.1% 0603 -> 430K 0.1% 0402; footprint Duc:R0603 -> Duc_Library:R0402; symbol Duc-Resistors:RES SMD 0603 -> Duc-Resistors:RES SMD 0402; LCSC Part C4107493 -> C728576; MPN RT0603FRE13100KL -> RT0402FRE07100KL
- R44, R49: value 620K 0.1% 0603 -> 620K 0.1% 0402; footprint Duc:R0603 -> Duc_Library:R0402; symbol Duc-Resistors:RES SMD 0603 -> Duc-Resistors:RES SMD 0402; LCSC Part C4107493 -> C728576; MPN RT0603FRE13100KL -> RT0402FRE07100KL
- R45, R50: value 1K 0.1% 0603 -> 1K 0.1% 0402; footprint Duc:R0603 -> Duc_Library:R0402; symbol Duc-Resistors:RES SMD 0603 -> Duc-Resistors:RES SMD 0402; LCSC Part C4107493 -> C728576; MPN RT0603FRE13100KL -> RT0402FRE07100KL
- R46, R47, R51, R52: value 5.1K 0.1% 0603 -> 5.1K 0.1% 0402; footprint Duc:R0603 -> Duc_Library:R0402; symbol Duc-Resistors:RES SMD 0603 -> Duc-Resistors:RES SMD 0402; LCSC Part C4107493 -> C728576; MPN RT0603FRE13100KL -> RT0402FRE07100KL
- renumbered C89 to C90
Connections:
- net GND: now also C89.1, C91.1
- net USB-DM_1: no longer D4.1 (IO1), J9.A7 (Dn1), J9.B7 (Dn2)
- net USB-DM_2: no longer D7.1 (IO1), J10.A7 (Dn1), J10.B7 (Dn2)
- net USB-DP_1: no longer D4.3 (IO2), J9.A6 (Dp1), J9.B6 (Dp2)
- net USB-DP_2: no longer D7.3 (IO2), J10.A6 (Dp1), J10.B6 (Dp2)
- net VBUS_1: now also D4.5 (VBUS), C89.2
- net VBUS_2: now also D7.5 (VBUS), C91.2
- new net: D7.1 (IO1), J10.A7 (Dn1), J10.B7 (Dn2)
- new net: D7.3 (IO2), J10.A6 (Dp1), J10.B6 (Dp2)
- new net: D4.3 (IO2), J9.A6 (Dp1), J9.B6 (Dp2)
- new net: D4.1 (IO1), J9.A7 (Dn1), J9.B7 (Dn2)
- no-connect marks 6 -> 4
Other:
- moved on the sheet: D4

Commit message: Update Schematic
Parts:
- C89, C91: footprint Duc_Library:C0402 -> Duc:C0402
- R43, R44, R45, R46, R47, R48, R49, R50, R51, R52: footprint Duc_Library:R0402 -> Duc:R0402
Changed lines of the file:
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@@
 			"AHcAKwAwAGcAQgBUAFMAcABLAFYATQBuAG0AZQBKADcAbABzAEsAVwBVAEkAYwBSAGkARwByAHUA"
 			"LwB0AE8ASwBhAGkANQA5AFMASwA1ADQAbABRAEYAVQAvAFYAeAB2AEYANABQAEQAYQBOAEgAVQBj"
-			"AGkAeQBvAHgAWgBWAEkAdQBpAEsASQB1AGkAMABDAFoATg=="
+			"AGkAeQBvAHgAWgBWAEkAdQBpAEsASQB1AGkAMABDAFoATgBpAGoAaQBvAGkAVABGAFIAbwBJAFAA"
+			"egBlAG4AOABQAEIAdAB0AHAATwBjAGwAQgBRAHkASABUADQAOAA1AEEAWQBIAFkAVQBnAFkAQwA2"
+			"AGIAdQBxAHEASABvADEARwBYAGQAZABpAFkARgBUAGUAcAA1AEMAKwBqAEYAOAA2AGoARQB6AHoA"
+			"NwBNAGkAcAA4AFEAYwBFAHYASQAvAGkAZABqAFUAagBxAEMAQwBvAFUAYQAvAFoAYgBOAHoAdAA4"
+			"AGUANgB1AFAAYgAvAGIAZgAxAGoAMQBkAHoAdQBaADcANgBRAFYANgBvADEAMwBpAFkAawBqAFUA"
+			"VgBBAGkAdABZAEUAUQA3AG8AQQBoAE0AUQBHAE8AcQB3AEIAUQBWAFcAWgBTAFoAVgBYAFYATABx"
+			"AHQAcgBjAEkANQBNAHYASABRADAAdQAvAEoAWgB4AGMATgBqAGUAeABDAFUAQQByAHMATgB5AFUA"
+			"MAAwAGkARABTAGwAbgBQAGEANAA3AC8AaABuAG0AYQA4AFoAWQBsAEEAQgBRAE4ARgAzAC8ARABE"
+			"AFEAcQAyAGoASQBOAEIAdwBHAGsAQgBzADEAZQA5AE4AWgB6ADUAZgBEAEUAeQBHAEIAVABTADEA"
+			"SgBNAHMAZgB2AGkASQBPAFgAZABnADgAWABjADIARAA2AHEASgBnAE0ASABCAHMAbQByACsAawB6"
+			"AE4AUQB4AEIAawA2AG0AYQBpAEEANwBDAGkANABTAEIAMQA2AHQAaQB2AFMAbABNAFkAdwB3AGgA"
+			"UgBPAE0AQwBaAG8AdABXAHUAOQBRAGIAYgBaAE0AbQBzADAAYQBQAHcAMABsAE4AeABvAFUARgBQ"
+			"ADAAOAB3AE0AUABEAGoATABCAE0ASgBoAG4AVABOAFkARQBMACsAMQBuAG4AcQBkAEIAQgArAEIA"
+			"QQA1ACsASABJAEgAbwBRAFMAdQBUAFkAYgBPAHgAKwA1ADMAMwBKADgAWQBqADcAbABqADIAcwBC"
+			"ADkANwBQAFgAcwAzACsATgBHAHQAUgAwAFMANwB2AHQAdAB1AHQAdQB2AE4AZQByAFAAWgBpAGsA"
+			"aABnAG4AcwAyAG0AeAA4AGYASABkAGQAMwBFADYATgBwAGwAUgBrAHgAcwBUAHMAUQBkAFIARwA2"
+			"AEcAQwAzADEANABYAEwAKwBhAGcAeABYAEoARgB6ADMAUQA1AHcASgBBAEIAQQBYADYASgBPADEA"
+			"bQB0ADkAbABzAHQAcAB0AFYAdQA5ADEAQwBwAEIAZwAxAE4AWQA4AG4AMAAvAEgANAA1AEsAUQBx"
+			"AFIAagBnACsAZQAzAFoANgBWAEIAeABOACsAbwB2AEwAOQ=="
 		)
 	)
@@
 			"UUJwQUhFQVRBQnJBRzhBYWdCMkFFc0Fkd0JKQUdrQU1nQjZBRVFBT0FCdEFIa0FUQUJJQUcwQWJ3"
 			"QXhBSFFBYVFCNEFISUFiZ0JoQUZjQVJ3QldBRFlBUlFCM0FIb0FTd0J3QUhNQWNRQTVBQzhBZGdB"
-			"ckFFNEFPUUJpQUd3QVdBQmlBRmdBU1FCU0FFZ0FVUUJwQQ=="
+			"ckFFNEFPUUJpQUd3QVdBQmlBRmdBU1FCU0FFZ0FVUUJwQQAvAGYAdgBQAEgAYgA1ADYAZABuAFIA"
+			"RQBJAHYAYQA0AHIAWgA3AFUAVQAvAEUAMABoAEgAagA1ADQAVQBPADAAcgBSAFAAaQBsAGoALwA5"
+			"AFMARwBJAFYAagBYAGgARgBoAHEAbwAyAC8AdwA1AGcAeQBnAGQATQBEAC8AcwAvAGoANQB6AFcA"
+			"dQA3AHMAWABQAHgAagB3AGoAdwBvAEUATgBHAFUAZgB4AHQAagBHAHAASwBhAFgAdwBQAGgAQgBD"
+			"AFUAZwBkAHUAWABWAFcASQBEAE0ARQBCAEUASQBtADkAQgAwAEEAUwBSAEsASwBDAG0AZABGAG0A"
+			"YwBOAFoANQBPADIAagBxAEwAMAA2AEcAUQBXAHYAZABsAGUAVgBtADYATABXADEATgBvAG4AVABN"
+			"AEUAeQBNADAAZABWACsAVAB4AGUAUwBGAEEAbQA4ADQAbwA1AEsAMABZAFkAMQBYAGQAOQBXADEA"
+			"YgA2AHUASwA2AHIAWQBGAFUAVgArAGMAbgBwAE0AZQBTAEcAawBXAEUAWQBTACsAZwB2AFcAUQBw"
+			"AHkAZgBuAFcAMwBMAGIAZABzADAAeAB0AGoAagA0ADYATQBrAGoAcQBVAEEARwBJAGsAOQBiADQA"
+			"MQB2AEQAaABHAHEAYwAwAEMARgA1AEsANwByAFMAYQBQAFEATwA1AGUAbQBhAFoANwBsAHkAVgBT"
+			"AEUATgBzAFkARwBnAFcASwBTAEcAVwBzADUANAA4AHUAagBaAFIAUgBGAFoAKwBkAG4AcQA5AFgA"
+			"cQAvAE8ATABjAGUAWAAvAC8ALwByADMARgBmAE8AWgBlACsAYgBIAGcASABMAFEAYgAyAGQAMgBy"
+			"AHEAbQA2AGEAWgB1AGoANwBJAEEAcQBMAG8AcABqAE4AWgBrAHEAcQBBADYAbAB6AG0AawBTAEEA"
+			"WQBMAFMAYgBZAEUAWABlAGMAeQBFAFcAOAA3AGwAUwBpAHYAagBQAEMAVQBxADAAMgArADEATwBU"
+			"AGsANwBTAEoATwBtADYAYgBsAHQAdQBtADcAWgB4AHoAawBkAGgAbQBCAGMANQA1AFcAMgBrAFYA"
+			"SgB3AHoAYQA2AHcAMQBkAHUAUwBkAGYAegA0AFYANgBnAEgAQQBqAFIAUQBLAEgAbwBDAGEAcQBL"
+			"ACsAZABNAFgAZgBXAFMAUwBXAFAAbABrAGYAVQBGAHYAagAwAHkAZABNAEgAYgB6ADkAWQByADkA"
+			"WgA1AG4AaABlAHoAQQBqAHgAUQBQAFoAdwB4AGwAdQBkADUAVQBSAFIAQgBvAEoAUgBVAHoAagBs"
+			"AGoAegBWAFIARwBRADAAcQBIAGoAUgBIAHMAUwAvAE4AbA=="
 		)
 	)
@@
 			)
 		)
-		(property "Footprint" "Duc_Library:C0402"
+		(property "Footprint" "Duc:C0402"
 			(at 187.96 78.74 0)
 			(effects
@@
 			)
 		)
-		(property "Footprint" "Duc_Library:C0402"
+		(property "Footprint" "Duc:C0402"
 			(at 187.96 129.54 0)
 			(effects
@@
 			)
 		)
-		(property "Footprint" "Duc_Library:R0402"
+		(property "Footprint" "Duc:R0402"
 			(at 144.78 104.14 0)
 			(effects
@@
 			)
 		)
-		(property "Footprint" "Duc_Library:R0402"
+		(property "Footprint" "Duc:R0402"
 			(at 144.78 66.04 0)
 			(effects
@@
 			)
 		)
-		(property "Footprint" "Duc_Library:R0402"
+		(property "Footprint" "Duc:R0402"
 			(at 210.82 38.1 0)
 			(effects
@@
 			)
 		)
-		(property "Footprint" "Duc_Library:R0402"
+		(property "Footprint" "Duc:R0402"
 			(at 210.82 88.9 0)
 			(effects
@@
 			)
 		)
-		(property "Footprint" "Duc_Library:R0402"
+		(property "Footprint" "Duc:R0402"
 			(at 144.78 116.84 0)
 			(effects
@@
 			)
 		)
-		(property "Footprint" "Duc_Library:R0402"
+		(property "Footprint" "Duc:R0402"
 			(at 144.78 53.34 0)
 			(effects
@@
 			)
 		)
-		(property "Footprint" "Duc_Library:R0402"
+		(property "Footprint" "Duc:R0402"
 			(at 233.68 88.9 0)
 			(effects
@@
 			)
 		)
-		(property "Footprint" "Duc_Library:R0402"
+		(property "Footprint" "Duc:R0402"
 			(at 144.78 44.45 0)
 			(effects
@@
 			)
 		)
-		(property "Footprint" "Duc_Library:R0402"
+		(property "Footprint" "Duc:R0402"
 			(at 144.78 95.25 0)
 			(effects
@@
 			)
 		)
-		(property "Footprint" "Duc_Library:R0402"
+		(property "Footprint" "Duc:R0402"
 			(at 233.68 38.1 0)
 			(effects

Commit message: Update Schematic & PCB
Connections:
- net at J10.A7 (Dn1), J10.B7 (Dn2): now also D7.3 (IO2); no longer D7.1 (IO1)
- net at J10.A6 (Dp1), J10.B6 (Dp2): now also D7.1 (IO1); no longer D7.3 (IO2)
- net USB-DM_1 renamed USB1_N
- net USB-DM_2 renamed USB2_P
- net USB-DP_1 renamed USB1_P
- net USB-DP_2 renamed USB2_N

Commit message: Update Schematic & PCB
Parts:
- C88, C90: value 4.7uF 50V 0603 -> CAP CER 0603
- C89, C91: value 100nF 50V 0402 -> CAP CER 0402
- D2, D5: value Blue 0603 -> LED 0603
- R43, R48: value 430K 0.1% 0402 -> RES 0402; Manufacturer YAGEO(国巨) -> (none)
- R44, R49: value 620K 0.1% 0402 -> RES 0402; Manufacturer YAGEO(国巨) -> (none)
- R45, R50: value 1K 0.1% 0402 -> RES 0402; Manufacturer YAGEO(国巨) -> (none)
- R46, R47, R51, R52: value 5.1K 0.1% 0402 -> RES 0402; Manufacturer YAGEO(国巨) -> (none)
Connections:
- net USB2_N: now also D7.6 (IO1); no longer D7.4 (IO2)
- net USB2_P: now also D7.4 (IO2); no longer D7.6 (IO1)
- net at J10.A6 (Dp1), J10.B6 (Dp2): now also D7.3 (IO2); no longer D7.1 (IO1)
- net at J10.A7 (Dn1), J10.B7 (Dn2): now also D7.1 (IO1); no longer D7.3 (IO2)

Commit message: Update SCH & PCB
Parts:
- renumbered C88 to C83, C89 to C84, C90 to C85, C91 to C86
Changed lines of the file:
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@@
 		(on_board yes)
 		(dnp no)
-		(property "Reference" "C89"
+		(property "Reference" "C84"
 			(at 187.706 62.484 0)
 			(effects
@@
 			(project "Master_Hand_Kicad"
 				(path "/f9e05184-c88b-4a88-ae9c-ab2bdb32be7c/c5103ceb-5325-4a84-a025-9638a412984e/7164844d-ef2d-4ed9-93c6-2b7c97a3348e"
-					(reference "C89")
+					(reference "C84")
 					(unit 1)
 				)
@@
 		(on_board yes)
 		(dnp no)
-		(property "Reference" "C91"
+		(property "Reference" "C86"
 			(at 187.706 113.284 0)
 			(effects
@@
 			(project "Master_Hand_Kicad"
 				(path "/f9e05184-c88b-4a88-ae9c-ab2bdb32be7c/c5103ceb-5325-4a84-a025-9638a412984e/7164844d-ef2d-4ed9-93c6-2b7c97a3348e"
-					(reference "C91")
+					(reference "C86")
 					(unit 1)
 				)
@@
 		(dnp no)
 		(fields_autoplaced yes)
-		(property "Reference" "#PWR104"
+		(property "Reference" "#PWR0104"
 			(at 116.586 70.866 0)
 			(do_not_autoplace yes)
@@
 			(project "Master_Hand_Kicad"
 				(path "/f9e05184-c88b-4a88-ae9c-ab2bdb32be7c/c5103ceb-5325-4a84-a025-9638a412984e/7164844d-ef2d-4ed9-93c6-2b7c97a3348e"
-					(reference "#PWR104")
+					(reference "#PWR0104")
 					(unit 1)
 				)
@@
 		(dnp no)
 		(fields_autoplaced yes)
-		(property "Reference" "#PWR107"
+		(property "Reference" "#PWR0107"
 			(at 151.384 94.234 0)
 			(do_not_autoplace yes)
@@
 			(project "Master_Hand_Kicad"
 				(path "/f9e05184-c88b-4a88-ae9c-ab2bdb32be7c/c5103ceb-5325-4a84-a025-9638a412984e/7164844d-ef2d-4ed9-93c6-2b7c97a3348e"
-					(reference "#PWR107")
+					(reference "#PWR0107")
 					(unit 1)
 				)
@@
 		(dnp no)
 		(fields_autoplaced yes)
-		(property "Reference" "#PWR112"
+		(property "Reference" "#PWR0112"
 			(at 116.586 121.666 0)
 			(do_not_autoplace yes)
@@
 			(project "Master_Hand_Kicad"
 				(path "/f9e05184-c88b-4a88-ae9c-ab2bdb32be7c/c5103ceb-5325-4a84-a025-9638a412984e/7164844d-ef2d-4ed9-93c6-2b7c97a3348e"
-					(reference "#PWR112")
+					(reference "#PWR0112")
 					(unit 1)
 				)
@@
 		(dnp no)
 		(fields_autoplaced yes)
-		(property "Reference" "#PWR102"
+		(property "Reference" "#PWR0102"
 			(at 128.524 66.294 0)
 			(do_not_autoplace yes)
@@
 			(project "Master_Hand_Kicad"
 				(path "/f9e05184-c88b-4a88-ae9c-ab2bdb32be7c/c5103ceb-5325-4a84-a025-9638a412984e/7164844d-ef2d-4ed9-93c6-2b7c97a3348e"
-					(reference "#PWR102")
+					(reference "#PWR0102")
 					(unit 1)
 				)
@@
 		(dnp no)
 		(fields_autoplaced yes)
-		(property "Reference" "#PWR108"
+		(property "Reference" "#PWR0108"
 			(at 177.546 85.344 0)
 			(do_not_autoplace yes)
@@
 			(project "Master_Hand_Kicad"
 				(path "/f9e05184-c88b-4a88-ae9c-ab2bdb32be7c/c5103ceb-5325-4a84-a025-9638a412984e/7164844d-ef2d-4ed9-93c6-2b7c97a3348e"
-					(reference "#PWR108")
+					(reference "#PWR0108")
 					(unit 1)
 				)
@@
 		(dnp no)
 		(fields_autoplaced yes)
-		(property "Reference" "#PWR106"
+		(property "Reference" "#PWR0106"
 			(at 116.586 93.726 0)
 			(do_not_autoplace yes)
@@
 			(project "Master_Hand_Kicad"
 				(path "/f9e05184-c88b-4a88-ae9c-ab2bdb32be7c/c5103ceb-5325-4a84-a025-9638a412984e/7164844d-ef2d-4ed9-93c6-2b7c97a3348e"
-					(reference "#PWR106")
+					(reference "#PWR0106")
 					(unit 1)
 				)
@@
 		(dnp no)
 		(fields_autoplaced yes)
-		(property "Reference" "#PWR111"
+		(property "Reference" "#PWR0111"
 			(at 171.704 110.744 0)
 			(do_not_autoplace yes)
@@
 			(project "Master_Hand_Kicad"
 				(path "/f9e05184-c88b-4a88-ae9c-ab2bdb32be7c/c5103ceb-5325-4a84-a025-9638a412984e/7164844d-ef2d-4ed9-93c6-2b7c97a3348e"
-					(reference "#PWR111")
+					(reference "#PWR0111")
 					(unit 1)
 				)
@@
 		(dnp no)
 		(fields_autoplaced yes)
-		(property "Reference" "#PWR110"
+		(property "Reference" "#PWR0110"
 			(at 128.524 117.094 0)
 			(do_not_autoplace yes)
@@
 			(project "Master_Hand_Kicad"
 				(path "/f9e05184-c88b-4a88-ae9c-ab2bdb32be7c/c5103ceb-5325-4a84-a025-9638a412984e/7164844d-ef2d-4ed9-93c6-2b7c97a3348e"
-					(reference "#PWR110")
+					(reference "#PWR0110")
 					(unit 1)
 				)
@@
 		(dnp no)
 		(fields_autoplaced yes)
-		(property "Reference" "#PWR109"
+		(property "Reference" "#PWR0109"
 			(at 151.384 106.934 0)
 			(do_not_autoplace yes)
@@
 			(project "Master_Hand_Kicad"
 				(path "/f9e05184-c88b-4a88-ae9c-ab2bdb32be7c/c5103ceb-5325-4a84-a025-9638a412984e/7164844d-ef2d-4ed9-93c6-2b7c97a3348e"
-					(reference "#PWR109")
+					(reference "#PWR0109")
 					(unit 1)
 				)
@@
 		(dnp no)
 		(fields_autoplaced yes)
-		(property "Reference" "#PWR97"
+		(property "Reference" "#PWR097"
 			(at 236.474 28.194 0)
 			(do_not_autoplace yes)
@@
 			(project "Master_Hand_Kicad"
 				(path "/f9e05184-c88b-4a88-ae9c-ab2bdb32be7c/c5103ceb-5325-4a84-a025-9638a412984e/7164844d-ef2d-4ed9-93c6-2b7c97a3348e"
-					(reference "#PWR97")
+					(reference "#PWR097")
 					(unit 1)
 				)
@@
 		(dnp no)
 		(fields_autoplaced yes)
-		(property "Reference" "#PWR99"
+		(property "Reference" "#PWR099"
 			(at 151.384 43.434 0)
 			(do_not_autoplace yes)
@@
 			(project "Master_Hand_Kicad"
 				(path "/f9e05184-c88b-4a88-ae9c-ab2bdb32be7c/c5103ceb-5325-4a84-a025-9638a412984e/7164844d-ef2d-4ed9-93c6-2b7c97a3348e"
-					(reference "#PWR99")
+					(reference "#PWR099")
 					(unit 1)
 				)
@@
 		(dnp no)
 		(fields_autoplaced yes)
-		(property "Reference" "#PWR103"
+		(property "Reference" "#PWR0103"
 			(at 171.704 59.944 0)
 			(do_not_autoplace yes)
@@
 			(project "Master_Hand_Kicad"
 				(path "/f9e05184-c88b-4a88-ae9c-ab2bdb32be7c/c5103ceb-5325-4a84-a025-9638a412984e/7164844d-ef2d-4ed9-93c6-2b7c97a3348e"
-					(reference "#PWR103")
+					(reference "#PWR0103")
 					(unit 1)
 				)
@@
 		(on_board no)
 		(dnp no)
-		(property "Reference" "#PWR100"
+		(property "Reference" "#PWR0100"
 			(at 178.816 34.544 0)
 			(do_not_autoplace yes)
@@
 			(project "Master_Hand_Kicad"
 				(path "/f9e05184-c88b-4a88-ae9c-ab2bdb32be7c/c5103ceb-5325-4a84-a025-9638a412984e/7164844d-ef2d-4ed9-93c6-2b7c97a3348e"
-					(reference "#PWR100")
+					(reference "#PWR0100")
 					(unit 1)
 				)
@@
 		(dnp no)
 		(fields_autoplaced yes)
-		(property "Reference" "C88"
+		(property "Reference" "C83"
 			(at 198.12 35.5599 90)
 			(effects
@@
 			(project "Master_Hand_Kicad"
 				(path "/f9e05184-c88b-4a88-ae9c-ab2bdb32be7c/c5103ceb-5325-4a84-a025-9638a412984e/7164844d-ef2d-4ed9-93c6-2b7c97a3348e"
-					(reference "C88")
+					(reference "C83")
 					(unit 1)
 				)
@@
 		(dnp no)
 		(fields_autoplaced yes)
-		(property "Reference" "#PWR101"
+		(property "Reference" "#PWR0101"
 			(at 151.384 56.134 0)
 			(do_not_autoplace yes)
@@
 			(project "Master_Hand_Kicad"
 				(path "/f9e05184-c88b-4a88-ae9c-ab2bdb32be7c/c5103ceb-5325-4a84-a025-9638a412984e/7164844d-ef2d-4ed9-93c6-2b7c97a3348e"
-					(reference "#PWR101")
+					(reference "#PWR0101")
 					(unit 1)
 				)
@@
 		(dnp no)
 		(fields_autoplaced yes)
-		(property "Reference" "#PWR105"
+		(property "Reference" "#PWR0105"
 			(at 236.474 78.994 0)
 			(do_not_autoplace yes)
@@
 			(project "Master_Hand_Kicad"
 				(path "/f9e05184-c88b-4a88-ae9c-ab2bdb32be7c/c5103ceb-5325-4a84-a025-9638a412984e/7164844d-ef2d-4ed9-93c6-2b7c97a3348e"
-					(reference "#PWR105")
+					(reference "#PWR0105")
 					(unit 1)
 				)
@@
 		(dnp no)
 		(fields_autoplaced yes)
-		(property "Reference" "C90"
+		(property "Reference" "C85"
 			(at 198.12 86.3599 90)
 			(effects
@@
 			(project "Master_Hand_Kicad"
 				(path "/f9e05184-c88b-4a88-ae9c-ab2bdb32be7c/c5103ceb-5325-4a84-a025-9638a412984e/7164844d-ef2d-4ed9-93c6-2b7c97a3348e"
-					(reference "C90")
+					(reference "C85")
 					(unit 1)
 				)
@@
 		(dnp no)
 		(fields_autoplaced yes)
-		(property "Reference" "#PWR98"
+		(property "Reference" "#PWR098"
 			(at 116.586 42.926 0)
 			(do_not_autoplace yes)
@@
 			(project "Master_Hand_Kicad"
 				(path "/f9e05184-c88b-4a88-ae9c-ab2bdb32be7c/c5103ceb-5325-4a84-a025-9638a412984e/7164844d-ef2d-4ed9-93c6-2b7c97a3348e"
-					(reference "#PWR98")
+					(reference "#PWR098")
 					(unit 1)
 				)
