File: Misc - Board Version, Switch.kicad_sch (KiCad schematic)
At the start: 11 parts, among them SW1 DSIC02LSGET

Commit message: Update Schematic
Parts:
- C101, C102: value CAP CER 0402 -> 100nF 50V 0603; footprint Duc_Library:C0402 -> Duc:C0603; symbol Duc-Capacitors:CAP CER 0402 -> Duc-Capacitors:CAP CER 0603; LCSC Part C325464 -> C14663; MPN CC0402KRX5R7BB105 -> CAP CER 0603; Manufacturer (none) -> YAGEO(国巨)
- R76, R78: value RES 0402 -> 0R 0.1% 0603; footprint Duc_Library:R0402 -> Duc:R0603; symbol Duc-Resistors:RES SMD 0402 -> Duc-Resistors:RES SMD 0603; LCSC Part C728576 -> C4107493; MPN RT0402FRE07100KL -> RT0603FRE13100KL; Manufacturer (none) -> YAGEO(国巨)
- R77, R79: value RES 0603 -> 100K 0.1% 0603
- R80, R81, R82, R83: value RES 0402 -> 10K 0.1% 0603; footprint Duc_Library:R0402 -> Duc:R0603; symbol Duc-Resistors:RES SMD 0402 -> Duc-Resistors:RES SMD 0603; LCSC Part C728576 -> C4107493; MPN RT0402FRE07100KL -> RT0603FRE13100KL; Manufacturer (none) -> YAGEO(国巨)

Commit message: Update Schematic
Parts:
- renumbered C101 to C103, C102 to C104
Changed lines of the file:
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@@
 		(dnp no)
 		(fields_autoplaced yes)
-		(property "Reference" "C101"
+		(property "Reference" "C103"
 			(at 163.83 110.4899 90)
 			(effects
@@
 			(project "Master_Hand_Kicad"
 				(path "/f9e05184-c88b-4a88-ae9c-ab2bdb32be7c/c5103ceb-5325-4a84-a025-9638a412984e/0bb1cb44-88fa-40dc-bea3-1adee4cb244a"
-					(reference "C101")
+					(reference "C103")
 					(unit 1)
 				)
@@
 		(dnp no)
 		(fields_autoplaced yes)
-		(property "Reference" "#PWR0137"
+		(property "Reference" "#PWR0136"
 			(at 92.456 75.184 0)
 			(do_not_autoplace yes)
@@
 			(project "Master_Hand_Kicad"
 				(path "/f9e05184-c88b-4a88-ae9c-ab2bdb32be7c/c5103ceb-5325-4a84-a025-9638a412984e/0bb1cb44-88fa-40dc-bea3-1adee4cb244a"
-					(reference "#PWR0137")
+					(reference "#PWR0136")
 					(unit 1)
 				)
@@
 		(dnp no)
 		(fields_autoplaced yes)
-		(property "Reference" "#PWR0136"
+		(property "Reference" "#PWR0135"
 			(at 161.544 67.564 0)
 			(do_not_autoplace yes)
@@
 			(project "Master_Hand_Kicad"
 				(path "/f9e05184-c88b-4a88-ae9c-ab2bdb32be7c/c5103ceb-5325-4a84-a025-9638a412984e/0bb1cb44-88fa-40dc-bea3-1adee4cb244a"
-					(reference "#PWR0136")
+					(reference "#PWR0135")
 					(unit 1)
 				)
@@
 		(dnp no)
 		(fields_autoplaced yes)
-		(property "Reference" "#PWR0139"
+		(property "Reference" "#PWR0138"
 			(at 185.166 129.794 0)
 			(do_not_autoplace yes)
@@
 			(project "Master_Hand_Kicad"
 				(path "/f9e05184-c88b-4a88-ae9c-ab2bdb32be7c/c5103ceb-5325-4a84-a025-9638a412984e/0bb1cb44-88fa-40dc-bea3-1adee4cb244a"
-					(reference "#PWR0139")
+					(reference "#PWR0138")
 					(unit 1)
 				)
@@
 		(dnp no)
 		(fields_autoplaced yes)
-		(property "Reference" "C102"
+		(property "Reference" "C104"
 			(at 163.83 130.8099 90)
 			(effects
@@
 			(project "Master_Hand_Kicad"
 				(path "/f9e05184-c88b-4a88-ae9c-ab2bdb32be7c/c5103ceb-5325-4a84-a025-9638a412984e/0bb1cb44-88fa-40dc-bea3-1adee4cb244a"
-					(reference "C102")
+					(reference "C104")
 					(unit 1)
 				)
@@
 		(dnp no)
 		(fields_autoplaced yes)
-		(property "Reference" "#PWR0138"
+		(property "Reference" "#PWR0137"
 			(at 185.166 109.474 0)
 			(do_not_autoplace yes)
@@
 			(project "Master_Hand_Kicad"
 				(path "/f9e05184-c88b-4a88-ae9c-ab2bdb32be7c/c5103ceb-5325-4a84-a025-9638a412984e/0bb1cb44-88fa-40dc-bea3-1adee4cb244a"
-					(reference "#PWR0138")
-					(unit 1)
-				)
+					(reference "#PWR0137")
+					(unit 1)
+				)

Commit message: Update Schematic & PCB
Parts:
- C103, C104: value 100nF 50V 0603 -> CAP CER 0603
- R76, R78: value 0R 0.1% 0603 -> RES 0603
- R77, R79: value 100K 0.1% 0603 -> RES 0603; Manufacturer Part Number RT0402FRE07100KL -> (none); Supplier 1 Digikey -> (none); Supplier Part Number 1 YAG2307CT-ND -> (none)
- R80, R81, R82, R83: value 10K 0.1% 0603 -> RES 0603
Changed lines of the file:
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@@
 			"aQBnAG8AcQBFAG8AZQB1AEcALwBKADUALwBmAEgAeQBPADQANwBUAGQANwBzADYAbgBpAC8AZgBz"
 			"AHYAYgAvAGYAYwBoAEEAOABuADgAOAB2AEwAOQBmAE4ATgBoAEUAQgA3AHoARwBJADUALwAvAE4A"
-			"cQB4AHcASQBuADEAQwA3AHcAVQ=="
+			"cQB4AHcASQBuADEAQwA3AHcAVQAvAGYAUABmADUAUwBwAGcASQBBAFkAQgAyAFAAdwB6AGcATQB3"
+			"AC8AdgA3AGUANQBIAG4AegBQAHoAbAB5ADUAYwAwAFQAYQBkAHAAYQB0AHYAdQAxADEALwAvADEA"
+			"dgBjAGQAaQB6AC8AaABJAFMAagBQAFIAZQBSAGIAUQA2AGIALwB0AGsAcwBDAGUAdgBKADIANQBt"
+			"AEUAWQBiAHYAZAA3AGYAcwArAGQAOQBkAHYATgBiAHIAVQBLAEkAbABuAFYAZABWADEAVgBsAFcA"
+			"VgBWAEEAWQBDAEoATgBOAEUAcABpAG0ATgBFACsARABrAEQAOABFAGYAZABzAEEAZwBSAHcATQB2"
+			"AFQASgBBAFMAMgBFAFoAeQBEAHIAdQAyAHIAcQByAHIAbgA5ADYAcQBxAEIATwBSADgAUABsADgA"
+			"dQBsADEAVwAyAFMAcABMAEUAVwBWAGMAVQB4AGYAMQArAEgANABhAHUAcgB1AHIAUAA1AE4ATgBh"
+			"AEYAOABjAHgAUwBBAGgAYgBnADYANQBEAGYAagB6AG8AUAB6AEUAeQBqAHYAMQBDAEEAaQB6AEkA"
+			"egBGAHEAcABxAGkAcQAvADUAMwBsAGUAegBOAE4AawBqAE4AbQBzAE4ANQB2AHQANwBuAHcAKwBB"
+			"ADQAQwB3AHIATgBmAHIASwBEAEoARgBXAFEAUgBoAHgAdgB2ADcAUgAxAEEAaQBiAHoAWQBiAHAA"
+			"WgBSAGUANQBQAEsAZwBBAGMAQgBvAFQAVQBTAEkAWgByADMAWgBtAEMAaABTADIAbwBCAEEAVQBl"
+			"AFQALwA4AHIAZAAvAHEAYQBvAHkAVABkAE4AcABuAHEAZABwAGkAdQBQADQAKwB2AEsAeQAyADIA"
+			"NAAzAG0ANgAzAFcAUgBrAFMARQBGADkAcwBZADUAdQBoAGYAZABYAGQATAByAEkAZwBJAGcATAB6"
+			"AFUAMABnAFYARQBnAEUAUgBLAEsANQBXAHQAMQA0AGcAawBEAE0ANgA3AHIAeAA5AGYALwA4AHQA"
+			"ZgAvAG0ASwBkAFcANgBXAHIAbAA5AGUAWAB5ACsAVgB5AHYAbAB5AHkAMQBRAG8AUgBRADkAeQBu"
+			"AGQAVwBCAHoASABwAG0ARQBIADYARQBsAHEAUwBVAFkALwA4ADQAWgBNADUAQQBIAEEAaABGADAA"
+			"UQBrAEcAcwBEAGkASwBvAEkANwBVADkAYgBLAEoAWQBKADgAYQBMAG0AKwAwAG8AMwBwAEsAMQA0"
+			"AEQAMABnAG8AbQBoAGkAcwAwAGIAWgBhAFkAcgBaAGcAcAB1AEIAVgBLAFIASQBhAFkAVQBLAHIA"
+			"QQBmADkANAAyAE0AdgAwAFAASQBMAEEAZwBuADYAbQBNAEMAZgBPAEwAOQBuAE0AawBBAGsAbABI"
+			"AHkATABTAE8AZwBXAEkAVQBBAEsARQBiAFYAVwBTAFoASgBrAFcAWgBhAHUAVQBtAGIATwBpADIA"
+			"SQBhAHAALwBQAGwAagBJAGgASgBrAG0AYQByAGwAWQBsAFUATQBKAFMAaABIAHQAWQB6AEMARABN"
+			"ADkAOAA3AC8AZgBLAEsAMQB2AE8ARwA2AFoAWABrAEkAQQA5AE8ASQBFAFMARgBCADUAQQBBADgA"
+			"UwBHAHUAeABvAGIAVwBKAEYAUwBSAEoAcABqAGUAUABZAGwAWABVADUAZAB5ADAAdwBHAHkASgBB"
+			"AFkARwBIAGwASABkAGwAUgBoAG4AYQB1AEMAZwAyAGkARQBDAE8AVABlAEYARABPAGcAMwBWAGcA"
+			"TgBDAEQAdwBrAHUAZABmAHMAZwBxAC8AbQA0AEEASABoAFMAbwBDAC8ARwBpAFkAOQBGAHgAdwA1"
+			"ADcAMQBZADkAcwB6AGoATgBFADMAVAA3AEoAMQBMADQAZwBSAFIARwBXAFAAbQAyAGYAYgA5AHMA"
+			"RgA3AFAAVQBXAFIAZwA2AFEAZwBRADQAZwBMADUAdABqAE4AKwBOAHUASAA0AEIANgBmAHEAQgA3"
+			"ADgAYwBxAHMAdgB0AHoATQB4AE4AMAArAFQAMwB2AEsAbwBxAHIAZgBVAHYAdgAvAHkAUwBKAHUA"
+			"dAA1AG4AcABqADkANQArAGUASAA5ACsANwAxADkAVwBXADMAMwAwAFcAUgBmAHIANgBXAEgAcgBM"
+			"AFQAWgA1AGIANQB1AGYAUwB5ADEARgBaACsARwAvAHUAQgBNAFUAZwBrADEAUABBAEIARQBnAGwA"
+			"NwA1ADEAeABaAFYAZgBrADkAdgA5AC8AdgAxAHQAcgAxAGUAbgAwADgAbgB2AGIANwB3AHoAQQBP"
+			"AFQAZAB2AFcAZABWAFYAVgBsAGYAZgBlAHUAbQBtADMAMwBSADQATwBCADYASwBnAEcAVgB6AHMA"
+			"TgBRAEEAbwBRAGcARQBHAEEAVgBJAEsAQgBVAEsARgBKAFMASQBDAEEAdwBFAFIATQBDAEcAZwBn"
+			"AEEASgBNAEUARgBEAEEAVwB6AHQAMgB6AFYAVABrAGMAMwBVAGIAeQB2AHYAVQAxAGMAQQAyAGkA"
+			"cwAxAHEAcwA5AG4AcwBqADEARwA2AEUAVABJAGQAawBIAEkAeQBXAGwAZgBPADEAbgA3AGUAZQBs"
+			"AEwANwA2AHkAWABPAEUAbABTAEEASwBzAEIAWQBlAFMASwB0AGIAOAA4AFoAVABzAEkAUwBvAEMA"
+			"KwBGAGwAbwB0AEYAeABXAGQARw=="
 		)
 	)
@@
 			)
 		)
-		(property "Value" "100nF 50V 0603"
+		(property "Value" "CAP CER 0603"
 			(at 163.83 113.0299 90)
 			(effects
@@
 			)
 		)
-		(property "Value" "10K 0.1% 0603"
+		(property "Value" "RES 0603"
 			(at 185.42 133.3499 90)
 			(effects
@@
 			)
 		)
-		(property "Value" "0R 0.1% 0603"
+		(property "Value" "RES 0603"
 			(at 160.02 72.39 0)
 			(effects
@@
 			)
 		)
-		(property "Value" "10K 0.1% 0603"
+		(property "Value" "RES 0603"
 			(at 149.86 101.6 0)
 			(effects
@@
 		(dnp no)
 		(fields_autoplaced yes)
-		(property "Reference" "#PWR0136"
+		(property "Reference" "#PWR136"
 			(at 92.456 75.184 0)
 			(do_not_autoplace yes)
@@
 			(project "Master_Hand_Kicad"
 				(path "/f9e05184-c88b-4a88-ae9c-ab2bdb32be7c/c5103ceb-5325-4a84-a025-9638a412984e/0bb1cb44-88fa-40dc-bea3-1adee4cb244a"
-					(reference "#PWR0136")
+					(reference "#PWR136")
 					(unit 1)
 				)
@@
 		(dnp no)
 		(fields_autoplaced yes)
-		(property "Reference" "#PWR0135"
+		(property "Reference" "#PWR135"
 			(at 161.544 67.564 0)
 			(do_not_autoplace yes)
@@
 			(project "Master_Hand_Kicad"
 				(path "/f9e05184-c88b-4a88-ae9c-ab2bdb32be7c/c5103ceb-5325-4a84-a025-9638a412984e/0bb1cb44-88fa-40dc-bea3-1adee4cb244a"
-					(reference "#PWR0135")
+					(reference "#PWR135")
 					(unit 1)
 				)
@@
 			)
 		)
-		(property "Value" "0R 0.1% 0603"
+		(property "Value" "RES 0603"
 			(at 160.02 58.42 0)
 			(effects
@@
 			)
 		)
-		(property "Value" "10K 0.1% 0603"
+		(property "Value" "RES 0603"
 			(at 149.86 123.19 0)
 			(effects
@@
 		(dnp no)
 		(fields_autoplaced yes)
-		(property "Reference" "#PWR0138"
+		(property "Reference" "#PWR138"
 			(at 185.166 129.794 0)
 			(do_not_autoplace yes)
@@
 			(project "Master_Hand_Kicad"
 				(path "/f9e05184-c88b-4a88-ae9c-ab2bdb32be7c/c5103ceb-5325-4a84-a025-9638a412984e/0bb1cb44-88fa-40dc-bea3-1adee4cb244a"
-					(reference "#PWR0138")
+					(reference "#PWR138")
 					(unit 1)
 				)
@@
 			)
 		)
-		(property "Value" "100K 0.1% 0603"
+		(property "Value" "RES 0603"
 			(at 92.71 77.4699 90)
 			(effects
@@
 		(property "Manufacturer" "YAGEO(国巨)"
 			(at 102.87 76.2 0)
-			(effects
-				(font
-					(size 1.27 1.27)
-				)
-				(hide yes)
-			)
-		)
-		(property "Manufacturer Part Number" "RT0402FRE07100KL"
-			(at 90.17 76.2 0)
-			(effects
-				(font
-					(size 1.27 1.27)
-				)
-				(hide yes)
-			)
-		)
-		(property "Supplier 1" "Digikey"
-			(at 90.17 76.2 0)
-			(effects
-				(font
-					(size 1.27 1.27)
-				)
-				(hide yes)
-			)
-		)
-		(property "Supplier Part Number 1" "YAG2307CT-ND"
-			(at 90.17 76.2 0)
 			(effects
 				(font
@@
 			)
 		)
-		(property "Value" "100K 0.1% 0603"
+		(property "Value" "RES 0603"
 			(at 92.71 59.6899 90)
 			(effects
@@
 		(property "Manufacturer" "YAGEO(国巨)"
 			(at 102.87 58.42 0)
-			(effects
-				(font
-					(size 1.27 1.27)
-				)
-				(hide yes)
-			)
-		)
-		(property "Manufacturer Part Number" "RT0402FRE07100KL"
-			(at 90.17 58.42 0)
-			(effects
-				(font
-					(size 1.27 1.27)
-				)
-				(hide yes)
-			)
-		)
-		(property "Supplier 1" "Digikey"
-			(at 90.17 58.42 0)
-			(effects
-				(font
-					(size 1.27 1.27)
-				)
-				(hide yes)
-			)
-		)
-		(property "Supplier Part Number 1" "YAG2307CT-ND"
-			(at 90.17 58.42 0)
 			(effects
 				(font
@@
 			)
 		)
-		(property "Value" "10K 0.1% 0603"
+		(property "Value" "RES 0603"
 			(at 185.42 113.0299 90)
 			(effects
@@
 			)
 		)
-		(property "Value" "100nF 50V 0603"
+		(property "Value" "CAP CER 0603"
 			(at 163.83 133.3499 90)
 			(effects
@@
 		(dnp no)
 		(fields_autoplaced yes)
-		(property "Reference" "#PWR0137"
+		(property "Reference" "#PWR137"
 			(at 185.166 109.474 0)
 			(do_not_autoplace yes)
@@
 			(project "Master_Hand_Kicad"
 				(path "/f9e05184-c88b-4a88-ae9c-ab2bdb32be7c/c5103ceb-5325-4a84-a025-9638a412984e/0bb1cb44-88fa-40dc-bea3-1adee4cb244a"
-					(reference "#PWR0137")
+					(reference "#PWR137")
 					(unit 1)
 				)

Commit message: Update SCH & PCB
Parts:
- C98: renamed from C103; value CAP CER 0603 -> CAP CER 0402; footprint Duc:C0603 -> Duc:C0402; symbol Duc-Capacitors:CAP CER 0603 -> Duc-Capacitors:CAP CER 0402; LCSC Part C14663 -> C325464; MPN CAP CER 0603 -> CC0402KRX5R7BB105
- C99: renamed from C104; value CAP CER 0603 -> CAP CER 0402; footprint Duc:C0603 -> Duc:C0402; symbol Duc-Capacitors:CAP CER 0603 -> Duc-Capacitors:CAP CER 0402; LCSC Part C14663 -> C325464; MPN CAP CER 0603 -> CC0402KRX5R7BB105
- R78: renamed from R80; value RES 0603 -> RES 0402; footprint Duc:R0603 -> Duc:R0402; symbol Duc-Resistors:RES SMD 0603 -> Duc-Resistors:RES SMD 0402; LCSC Part C4107493 -> C728576; MPN RT0603FRE13100KL -> RT0402FRE07100KL
- R79: renamed from R81; value RES 0603 -> RES 0402; footprint Duc:R0603 -> Duc:R0402; symbol Duc-Resistors:RES SMD 0603 -> Duc-Resistors:RES SMD 0402; LCSC Part C4107493 -> C728576; MPN RT0603FRE13100KL -> RT0402FRE07100KL
- R80: renamed from R82; value RES 0603 -> RES 0402; footprint Duc:R0603 -> Duc:R0402; symbol Duc-Resistors:RES SMD 0603 -> Duc-Resistors:RES SMD 0402; LCSC Part C4107493 -> C728576; MPN RT0603FRE13100KL -> RT0402FRE07100KL
- R81: renamed from R83; value RES 0603 -> RES 0402; footprint Duc:R0603 -> Duc:R0402; symbol Duc-Resistors:RES SMD 0603 -> Duc-Resistors:RES SMD 0402; LCSC Part C4107493 -> C728576; MPN RT0603FRE13100KL -> RT0402FRE07100KL
- renumbered R76 to R74, R77 to R75, R78 to R76, R79 to R77

Commit message: Update SCH & PCB
Parts:
- R73: renamed from R74; value RES 0603 -> RES 0402; footprint Duc:R0603 -> Duc:R0402; symbol Duc-Resistors:RES SMD 0603 -> Duc-Resistors:RES SMD 0402; LCSC Part C4107493 -> C728576; MPN RT0603FRE13100KL -> RT0402FRE07100KL
- R74: renamed from R75; value RES 0603 -> RES 0402; footprint Duc:R0603 -> Duc:R0402; symbol Duc-Resistors:RES SMD 0603 -> Duc-Resistors:RES SMD 0402; LCSC Part C4107493 -> C728576; MPN RT0603FRE13100KL -> RT0402FRE07100KL
- R75: renamed from R76; value RES 0603 -> RES 0402; footprint Duc:R0603 -> Duc:R0402; symbol Duc-Resistors:RES SMD 0603 -> Duc-Resistors:RES SMD 0402; LCSC Part C4107493 -> C728576; MPN RT0603FRE13100KL -> RT0402FRE07100KL
- R76: renamed from R77; value RES 0603 -> RES 0402; footprint Duc:R0603 -> Duc:R0402; symbol Duc-Resistors:RES SMD 0603 -> Duc-Resistors:RES SMD 0402; LCSC Part C4107493 -> C728576; MPN RT0603FRE13100KL -> RT0402FRE07100KL
- renumbered R78 to R77, R79 to R78, R80 to R79, R81 to R80
Changed lines of the file:
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@@
 		(dnp no)
 		(fields_autoplaced yes)
-		(property "Reference" "R81"
+		(property "Reference" "R80"
 			(at 185.42 130.8099 90)
 			(effects
@@
 			(project "Master_Hand_Kicad"
 				(path "/f9e05184-c88b-4a88-ae9c-ab2bdb32be7c/c5103ceb-5325-4a84-a025-9638a412984e/0bb1cb44-88fa-40dc-bea3-1adee4cb244a"
-					(reference "R81")
+					(reference "R80")
 					(unit 1)
 				)
@@
 	)
 	(symbol
-		(lib_id "Duc-Resistors:RES SMD 0603")
+		(lib_id "Duc-Resistors:RES SMD 0402")
 		(at 160.02 69.85 0)
 		(unit 1)
@@
 		(on_board yes)
 		(dnp no)
-		(property "Reference" "R76"
-			(at 160.02 67.31 0)
-			(effects
-				(font
-					(size 1.27 1.27)
-				)
-			)
-		)
-		(property "Value" "RES 0603"
-			(at 160.02 72.39 0)
-			(effects
-				(font
-					(size 1.27 1.27)
-				)
-			)
-		)
-		(property "Footprint" "Duc:R0603"
+		(property "Reference" "R75"
+			(at 160.02 64.77 0)
+			(effects
+				(font
+					(size 1.27 1.27)
+				)
+			)
+		)
+		(property "Value" "RES 0402"
+			(at 160.02 72.898 0)
+			(effects
+				(font
+					(size 1.27 1.27)
+				)
+			)
+		)
+		(property "Footprint" "Duc:R0402"
 			(at 160.02 77.47 0)
 			(effects
@@
 			)
 		)
-		(property "Description" "RES SMD 0603"
-			(at 160.02 69.85 0)
+		(property "Description" "RES SMD 0402"
+			(at 159.512 72.898 0)
 			(effects
 				(font
@@
 			)
 		)
-		(property "MPN" "RT0603FRE13100KL"
+		(property "MPN" "RT0402FRE07100KL"
 			(at 160.02 85.09 0)
 			(effects
@@
 			)
 		)
-		(property "LCSC Part" "C4107493"
+		(property "LCSC Part" "C728576"
 			(at 160.02 87.63 0)
 			(effects
@@
 			(project "Master_Hand_Kicad"
 				(path "/f9e05184-c88b-4a88-ae9c-ab2bdb32be7c/c5103ceb-5325-4a84-a025-9638a412984e/0bb1cb44-88fa-40dc-bea3-1adee4cb244a"
-					(reference "R76")
+					(reference "R75")
 					(unit 1)
 				)
@@
 		(dnp no)
 		(fields_autoplaced yes)
-		(property "Reference" "R78"
+		(property "Reference" "R77"
 			(at 149.86 99.06 0)
 			(effects
@@
 			(project "Master_Hand_Kicad"
 				(path "/f9e05184-c88b-4a88-ae9c-ab2bdb32be7c/c5103ceb-5325-4a84-a025-9638a412984e/0bb1cb44-88fa-40dc-bea3-1adee4cb244a"
-					(reference "R78")
+					(reference "R77")
 					(unit 1)
 				)
@@
 		(dnp no)
 		(fields_autoplaced yes)
-		(property "Reference" "#PWR0136"
+		(property "Reference" "#PWR0140"
 			(at 92.456 75.184 0)
 			(do_not_autoplace yes)
@@
 			(project "Master_Hand_Kicad"
 				(path "/f9e05184-c88b-4a88-ae9c-ab2bdb32be7c/c5103ceb-5325-4a84-a025-9638a412984e/0bb1cb44-88fa-40dc-bea3-1adee4cb244a"
-					(reference "#PWR0136")
+					(reference "#PWR0140")
 					(unit 1)
 				)
@@
 		(dnp no)
 		(fields_autoplaced yes)
-		(property "Reference" "#PWR0135"
+		(property "Reference" "#PWR0139"
 			(at 161.544 67.564 0)
 			(do_not_autoplace yes)
@@
 			(project "Master_Hand_Kicad"
 				(path "/f9e05184-c88b-4a88-ae9c-ab2bdb32be7c/c5103ceb-5325-4a84-a025-9638a412984e/0bb1cb44-88fa-40dc-bea3-1adee4cb244a"
-					(reference "#PWR0135")
-					(unit 1)
-				)
-			)
-		)
-	)
-	(symbol
-		(lib_id "Duc-Resistors:RES SMD 0603")
+					(reference "#PWR0139")
+					(unit 1)
+				)
+			)
+		)
+	)
+	(symbol
+		(lib_id "Duc-Resistors:RES SMD 0402")
 		(at 160.02 55.88 0)
 		(unit 1)
@@
 		(on_board yes)
 		(dnp no)
-		(property "Reference" "R74"
-			(at 160.02 53.34 0)
-			(effects
-				(font
-					(size 1.27 1.27)
-				)
-			)
-		)
-		(property "Value" "RES 0603"
-			(at 160.02 58.42 0)
-			(effects
-				(font
-					(size 1.27 1.27)
-				)
-			)
-		)
-		(property "Footprint" "Duc:R0603"
+		(property "Reference" "R73"
+			(at 160.02 50.8 0)
+			(effects
+				(font
+					(size 1.27 1.27)
+				)
+			)
+		)
+		(property "Value" "RES 0402"
+			(at 160.02 58.928 0)
+			(effects
+				(font
+					(size 1.27 1.27)
+				)
+			)
+		)
+		(property "Footprint" "Duc:R0402"
 			(at 160.02 63.5 0)
 			(effects
@@
 			)
 		)
-		(property "Description" "RES SMD 0603"
-			(at 160.02 55.88 0)
+		(property "Description" "RES SMD 0402"
+			(at 159.512 58.928 0)
 			(effects
 				(font
@@
 			)
 		)
-		(property "MPN" "RT0603FRE13100KL"
+		(property "MPN" "RT0402FRE07100KL"
 			(at 160.02 71.12 0)
 			(effects
@@
 			)
 		)
-		(property "LCSC Part" "C4107493"
+		(property "LCSC Part" "C728576"
 			(at 160.02 73.66 0)
 			(effects
@@
 			(project "Master_Hand_Kicad"
 				(path "/f9e05184-c88b-4a88-ae9c-ab2bdb32be7c/c5103ceb-5325-4a84-a025-9638a412984e/0bb1cb44-88fa-40dc-bea3-1adee4cb244a"
-					(reference "R74")
+					(reference "R73")
 					(unit 1)
 				)
@@
 		(on_board yes)
 		(dnp no)
-		(property "Reference" "R80"
+		(property "Reference" "R79"
 			(at 149.86 120.65 0)
 			(effects
@@
 			(project "Master_Hand_Kicad"
 				(path "/f9e05184-c88b-4a88-ae9c-ab2bdb32be7c/c5103ceb-5325-4a84-a025-9638a412984e/0bb1cb44-88fa-40dc-bea3-1adee4cb244a"
-					(reference "R80")
+					(reference "R79")
 					(unit 1)
 				)
@@
 		(dnp no)
 		(fields_autoplaced yes)
-		(property "Reference" "#PWR0138"
+		(property "Reference" "#PWR0142"
 			(at 185.166 129.794 0)
 			(do_not_autoplace yes)
@@
 			(project "Master_Hand_Kicad"
 				(path "/f9e05184-c88b-4a88-ae9c-ab2bdb32be7c/c5103ceb-5325-4a84-a025-9638a412984e/0bb1cb44-88fa-40dc-bea3-1adee4cb244a"
-					(reference "#PWR0138")
-					(unit 1)
-				)
-			)
-		)
-	)
-	(symbol
-		(lib_id "Duc-Resistors:RES SMD 0603")
+					(reference "#PWR0142")
+					(unit 1)
+				)
+			)
+		)
+	)
+	(symbol
+		(lib_id "Duc-Resistors:RES SMD 0402")
 		(at 90.17 76.2 90)
 		(unit 1)
@@
 		(dnp no)
 		(fields_autoplaced yes)
-		(property "Reference" "R77"
+		(property "Reference" "R76"
 			(at 92.71 74.9299 90)
 			(effects
@@
 			)
 		)
-		(property "Value" "RES 0603"
+		(property "Value" "RES 0402"
 			(at 92.71 77.4699 90)
 			(effects
@@
 			)
 		)
-		(property "Footprint" "Duc:R0603"
+		(property "Footprint" "Duc:R0402"
 			(at 97.79 76.2 0)
 			(effects
@@
 			)
 		)
-		(property "Description" "RES SMD 0603"
-			(at 90.17 76.2 0)
+		(property "Description" "RES SMD 0402"
+			(at 93.218 76.708 0)
 			(effects
 				(font
@@
 			)
 		)
-		(property "MPN" "RT0603FRE13100KL"
+		(property "MPN" "RT0402FRE07100KL"
 			(at 105.41 76.2 0)
 			(effects
@@
 			)
 		)
-		(property "LCSC Part" "C4107493"
+		(property "LCSC Part" "C728576"
 			(at 107.95 76.2 0)
 			(effects
@@
 			(project "Master_Hand_Kicad"
 				(path "/f9e05184-c88b-4a88-ae9c-ab2bdb32be7c/c5103ceb-5325-4a84-a025-9638a412984e/0bb1cb44-88fa-40dc-bea3-1adee4cb244a"
-					(reference "R77")
-					(unit 1)
-				)
-			)
-		)
-	)
-	(symbol
-		(lib_id "Duc-Resistors:RES SMD 0603")
+					(reference "R76")
+					(unit 1)
+				)
+			)
+		)
+	)
+	(symbol
+		(lib_id "Duc-Resistors:RES SMD 0402")
 		(at 90.17 58.42 90)
 		(unit 1)
@@
 		(dnp no)
 		(fields_autoplaced yes)
-		(property "Reference" "R75"
+		(property "Reference" "R74"
 			(at 92.71 57.1499 90)
 			(effects
@@
 			)
 		)
-		(property "Value" "RES 0603"
+		(property "Value" "RES 0402"
 			(at 92.71 59.6899 90)
 			(effects
@@
 			)
 		)
-		(property "Footprint" "Duc:R0603"
+		(property "Footprint" "Duc:R0402"
 			(at 97.79 58.42 0)
 			(effects
@@
 			)
 		)
-		(property "Description" "RES SMD 0603"
-			(at 90.17 58.42 0)
+		(property "Description" "RES SMD 0402"
+			(at 93.218 58.928 0)
 			(effects
 				(font
@@
 			)
 		)
-		(property "MPN" "RT0603FRE13100KL"
+		(property "MPN" "RT0402FRE07100KL"
 			(at 105.41 58.42 0)
 			(effects
@@
 			)
 		)
-		(property "LCSC Part" "C4107493"
+		(property "LCSC Part" "C728576"
 			(at 107.95 58.42 0)
 			(effects
@@
 			(project "Master_Hand_Kicad"
 				(path "/f9e05184-c88b-4a88-ae9c-ab2bdb32be7c/c5103ceb-5325-4a84-a025-9638a412984e/0bb1cb44-88fa-40dc-bea3-1adee4cb244a"
-					(reference "R75")
+					(reference "R74")
 					(unit 1)
 				)
@@
 		(dnp no)
 		(fields_autoplaced yes)
-		(property "Reference" "R79"
+		(property "Reference" "R78"
 			(at 185.42 110.4899 90)
 			(effects
@@
 			(project "Master_Hand_Kicad"
 				(path "/f9e05184-c88b-4a88-ae9c-ab2bdb32be7c/c5103ceb-5325-4a84-a025-9638a412984e/0bb1cb44-88fa-40dc-bea3-1adee4cb244a"
-					(reference "R79")
+					(reference "R78")
 					(unit 1)
 				)
@@
 		(dnp no)
 		(fields_autoplaced yes)
-		(property "Reference" "#PWR0137"
+		(property "Reference" "#PWR0141"
 			(at 185.166 109.474 0)
 			(do_not_autoplace yes)
@@
 			(project "Master_Hand_Kicad"
 				(path "/f9e05184-c88b-4a88-ae9c-ab2bdb32be7c/c5103ceb-5325-4a84-a025-9638a412984e/0bb1cb44-88fa-40dc-bea3-1adee4cb244a"
-					(reference "#PWR0137")
-					(unit 1)
-				)
+					(reference "#PWR0141")
+					(unit 1)
+				)
