File: Power - Generation.kicad_sch (KiCad schematic)
At the start: 38 parts, among them U1 TPSM63603RDHR, U2 TPS62162DSG, U3 TLV75533PDBVR

Commit message: Update Schematic
Parts:
- added TP1, TP2, TP3, TP4, TP5, TP6, TP7, TP8: ~, Duc_Library:TestPoint_Pad_D0.5mm, symbol Power_symbols:Test_Point
- C10: renamed from C6; value CAP CER 1206 -> 10uF 50V 1206
- C11: renamed from C7; value CAP CER 1206 -> 100nF 50V 1206
- C12: renamed from C8; value CAP CER 0402 -> 1uF 50V 0603; footprint Duc_Library:C0402 -> Duc:C0603; symbol Duc-Capacitors:CAP CER 0402 -> Duc-Capacitors:CAP CER 0603; LCSC Part C325464 -> C14663; MPN CC0402KRX5R7BB105 -> CAP CER 0603; Manufacturer (none) -> YAGEO(国巨)
- C13: renamed from C9; value CAP CER 1206 -> 22uF 50V 1206
- C14: renamed from C10; value CAP CER 0402 -> 2.2uF 100V 0603; footprint Duc_Library:C0402 -> Duc:C0603; symbol Duc-Capacitors:CAP CER 0402 -> Duc-Capacitors:CAP CER 0603; LCSC Part C325464 -> C14663; MPN CC0402KRX5R7BB105 -> CAP CER 0603; Manufacturer (none) -> YAGEO(国巨)
- C15: renamed from C11; value CAP CER 0402 -> 2.2uF 100V 0603; footprint Duc_Library:C0402 -> Duc:C0603; symbol Duc-Capacitors:CAP CER 0402 -> Duc-Capacitors:CAP CER 0603; LCSC Part C325464 -> C14663; MPN CC0402KRX5R7BB105 -> CAP CER 0603; Manufacturer (none) -> YAGEO(国巨)
- C16: renamed from C12; value CAP CER 1206 -> 10uF 50V 1206
- C17: renamed from C13; value CAP CER 1206 -> 1uF 50V 1206
- C18: renamed from C14; value CAP CER 1206 -> 1uF 50V 1206
- C20: renamed from C16; value CAP CER 0603 -> 10uF 50V 0603
- C21: renamed from C17; value CAP CER 0603 -> 10uF 50V 0603
- C22: renamed from C18; value CAP CER 0603 -> 10uF 50V 0603
- C23: renamed from C19; value CAP CER 0603 -> 10uF 50V 0603
- C24: renamed from C20; value CAP CER 0603 -> 10uF 50V 0603
- C25: renamed from C21; value CAP CER 0603 -> 10uF 50V 0603
- C26: renamed from C22; value CAP CER 0603 -> 10uF 50V 0603
- C27: renamed from C23; value CAP CER 0603 -> 10uF 50V 0603
- C28: renamed from C24; value CAP CER 0603 -> 10uF 50V 0603
- C29: renamed from C25; value CAP CER 0603 -> 10uF 50V 0603
- C5: renamed from C2; value CAP CER 1206 -> 4.7uF 100V 1206
- C6: renamed from C1; value CAP CER 1206 -> 4.7uF 100V 1206
- C7: renamed from C3; value CAP CER 0402 -> 2.2uF 100V 0603; footprint Duc_Library:C0402 -> Duc:C0603; symbol Duc-Capacitors:CAP CER 0402 -> Duc-Capacitors:CAP CER 0603; LCSC Part C325464 -> C14663; MPN CC0402KRX5R7BB105 -> CAP CER 0603; Manufacturer (none) -> YAGEO(国巨)
- C8: renamed from C4; value CAP CER 0402 -> 2.2uF 100V 0603; footprint Duc_Library:C0402 -> Duc:C0603; symbol Duc-Capacitors:CAP CER 0402 -> Duc-Capacitors:CAP CER 0603; LCSC Part C325464 -> C14663; MPN CC0402KRX5R7BB105 -> CAP CER 0603; Manufacturer (none) -> YAGEO(国巨)
- C9: renamed from C5; value CAP CER 1206 -> 10uF 100V 1206
- R1: value RES 0402 -> 41.2K 0.1% 0603; footprint Duc_Library:R0402 -> Duc:R0603; symbol Duc-Resistors:RES SMD 0402 -> Duc-Resistors:RES SMD 0603; LCSC Part C728576 -> C4107493; MPN RT0402FRE07100KL -> RT0603FRE13100KL; Manufacturer (none) -> YAGEO(国巨)
- R2, R5: value RES 0402 -> 10K 0.1% 0603; footprint Duc_Library:R0402 -> Duc:R0603; symbol Duc-Resistors:RES SMD 0402 -> Duc-Resistors:RES SMD 0603; LCSC Part C728576 -> C4107493; MPN RT0402FRE07100KL -> RT0603FRE13100KL; Manufacturer (none) -> YAGEO(国巨)
- R3: value RES 0402 -> 40.2K 0.1% 0603; footprint Duc_Library:R0402 -> Duc:R0603; symbol Duc-Resistors:RES SMD 0402 -> Duc-Resistors:RES SMD 0603; LCSC Part C728576 -> C4107493; MPN RT0402FRE07100KL -> RT0603FRE13100KL; Manufacturer (none) -> YAGEO(国巨)
- R4: value RES 0402 -> 13K 0.1% 0603; footprint Duc_Library:R0402 -> Duc:R0603; symbol Duc-Resistors:RES SMD 0402 -> Duc-Resistors:RES SMD 0603; LCSC Part C728576 -> C4107493; MPN RT0402FRE07100KL -> RT0603FRE13100KL; Manufacturer (none) -> YAGEO(国巨)
- R6: value RES 0603 -> 100K 0.1% 0603
- renumbered C15 to C19, U1 to U3, U2 to U4, U3 to U5
Connections:
- net +3V3: now also TP5.1
- net +5V: now also TP3.1
- net +A3V3: now also TP7.1
- net +VBAT: now also TP1.1
- net EN_3V3: now also TP6.1
- net FB_5V: now also TP4.1
- net SW_3V3: now reaches L1.1, U4.7 (SW)
- net SW_3V3: now also TP8.1
- net F_VIN_5V: now reaches C5.2, C6.2, C8.2, C9.2, FB1.2, R1.2, U3.18 (VIN), U3.19 (VIN), U3.3 (VIN), U3.4 (VIN)
- net F_VIN_5V: now also TP2.1
Other:
- moved on the sheet: C12, C19, C20, C21, C22, C23, C24, C25, C26, C27, C28, C29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

Commit message: Update Schematic
Parts:
- removed C14, C15: 2.2uF 100V 0603, Duc:C0603, symbol Duc-Capacitors:CAP CER 0603
- removed FB2: 1k @ 100MHz, Duc_Library:L0805, symbol Duc-Inductors:PBBHAQ2012H-102T10
Connections:
- net +5V: now also C16.2, U4.2 (VIN)
Other:
- moved on the sheet: C16, C17

Commit message: Update Schematic & PCB
Parts:
- C10, C11, C13, C16, C17, C18, C5, C6, C9: footprint Duc_Library:C1206 -> Duc:C1206
- FB1: footprint Duc_Library:L0805 -> Duc:L0805
- TP1, TP2, TP3, TP4, TP5, TP6, TP7, TP8: footprint Duc_Library:TestPoint_Pad_D0.5mm -> Duc:TestPoint_Pad_D0.5mm
- U3: footprint Duc_Library:QFN-30_L6.0-W4.0-P0.50_TLVM13630RDHR -> Duc:QFN-30_L6.0-W4.0-P0.50_TLVM13630RDHR

Commit message: Update Schematic & PCB
Parts:
- C10, C16: value 10uF 50V 1206 -> CAP CER 1206
- C11: value 100nF 50V 1206 -> CAP CER 1206
- C12: value 1uF 50V 0603 -> CAP CER 0603
- C13: value 22uF 50V 1206 -> CAP CER 1206
- C17, C18: value 1uF 50V 1206 -> CAP CER 1206
- C20, C21, C22, C23, C24, C25, C26, C27, C28, C29: value 10uF 50V 0603 -> CAP CER 0603
- C5, C6: value 4.7uF 100V 1206 -> CAP CER 1206
- C7, C8: value 2.2uF 100V 0603 -> CAP CER 0603
- C9: value 10uF 100V 1206 -> CAP CER 1206
- R1: value 41.2K 0.1% 0603 -> RES 0603
- R2, R5: value 10K 0.1% 0603 -> RES 0603
- R3: value 40.2K 0.1% 0603 -> RES 0603
- R4: value 13K 0.1% 0603 -> RES 0603
- R6: value 100K 0.1% 0603 -> RES 0603

Commit message: Update Schematic & PCB
Parts:
- removed C9: CAP CER 1206, Duc:C1206, symbol Duc-Capacitors:CAP CER 1206
- C12, C7, C8: value CAP CER 0603 -> CAP CER 0402; footprint Duc:C0603 -> Duc:C0402; symbol Duc-Capacitors:CAP CER 0603 -> Duc-Capacitors:CAP CER 0402; LCSC Part C14663 -> C325464; MPN CAP CER 0603 -> CC0402KRX5R7BB105
- C13, C18: value CAP CER 1206 -> CAP CER 0603; footprint Duc:C1206 -> Duc:C0603; symbol Duc-Capacitors:CAP CER 1206 -> Duc-Capacitors:CAP CER 0603; LCSC Part C132170 -> C14663; MPN CC1206KKX7R9BB475 -> CAP CER 0603; Manufacturer (none) -> YAGEO(国巨)
- C16, C17: value CAP CER 1206 -> CAP CER 0402; footprint Duc:C1206 -> Duc:C0402; symbol Duc-Capacitors:CAP CER 1206 -> Duc-Capacitors:CAP CER 0402; LCSC Part C132170 -> C325464; MPN CC1206KKX7R9BB475 -> CC0402KRX5R7BB105; Manufacturer (none) -> YAGEO(国巨)
- C19: value 25SVPF330M -> SM337M025E0800; footprint Duc:CAP-SMD_BD10.0-L10.3-W10.3-LS11.0-FD -> Duc:CAP-SMD_BD6.3-L6.6-W6.6-FD-1; symbol Duc-Capacitors:25SVPF330M -> Duc-Capacitors:SM337M025E0800; LCSC Part C178367 -> C44606382; MPN 25SVPF330M -> SM337M025E0800; Manufacturer PANASONIC(松下) -> SHENGYANG(升阳)
- R1, R2, R3, R4, R5, R6: value RES 0603 -> RES 0402; footprint Duc:R0603 -> Duc:R0402; symbol Duc-Resistors:RES SMD 0603 -> Duc-Resistors:RES SMD 0402; LCSC Part C4107493 -> C728576; MPN RT0603FRE13100KL -> RT0402FRE07100KL
Other:
- moved on the sheet: C7, C8, D1, FB1

Commit message: Update SCH & PCB
Parts:
- removed C7, C8: CAP CER 0402, Duc:C0402, symbol Duc-Capacitors:CAP CER 0402
- removed FB1: 1k @ 100MHz, Duc:L0805, symbol Duc-Inductors:PBBHAQ2012H-102T10
- removed TP2: ~, Duc:TestPoint_Pad_D0.5mm, symbol Power_symbols:Test_Point
- renumbered C13 to C10, C16 to C11, C17 to C12, C18 to C13, C19 to C14, C20 to C15, C21 to C16, C22 to C17, C23 to C18, C24 to C19, C25 to C20, C26 to C21, C27 to C22, C28 to C23, C29 to C24, C10 to C7, C11 to C8, C12 to C9, TP3 to TP2, TP4 to TP3, TP5 to TP4, TP6 to TP5, TP7 to TP6, TP8 to TP7
Connections:
- net F_VIN_5V is gone; now on net +VBAT: C5.2, C6.2, R1.2, U3.18 (VIN), U3.19 (VIN), U3.3 (VIN), U3.4 (VIN)
Other:
- moved on the sheet: D1

Commit message: Update SCH & PCB
Connections:
- net GND: now also C10.1, U4.5 (FB)
Other:
- moved on the sheet: C10
Changed lines of the file:
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@@
 	)
 	(junction
-		(at 289.56 71.12)
+		(at 309.88 144.78)
 		(diameter 0)
 		(color 0 0 0 0)
 	)
 	(junction
-		(at 256.54 73.66)
+		(at 289.56 71.12)
 		(diameter 0)
 		(color 0 0 0 0)
 	)
 	(junction
-		(at 311.15 127)
+		(at 256.54 73.66)
 		(diameter 0)
 		(color 0 0 0 0)
@@
 	)
 	(junction
+		(at 309.88 127)
+		(diameter 0)
+		(color 0 0 0 0)
+	)
+	(junction
 		(at 237.49 107.95)
 		(diameter 0)
@@
 	(wire
 		(pts
-			(xy 311.15 127) (xy 318.77 127)
-		)
-		(stroke
-			(width 0)
-			(type default)
-		)
-	)
-	(wire
-		(pts
 			(xy 332.74 83.82) (xy 332.74 81.28)
 		)
@@
 	(wire
 		(pts
-			(xy 251.46 144.78) (xy 311.15 144.78)
+			(xy 251.46 144.78) (xy 309.88 144.78)
 		)
 		(stroke
@@
 	(wire
 		(pts
-			(xy 302.26 127) (xy 311.15 127)
+			(xy 302.26 127) (xy 309.88 127)
 		)
 		(stroke
@@
 	(wire
 		(pts
-			(xy 311.15 137.16) (xy 311.15 144.78)
+			(xy 309.88 137.16) (xy 309.88 144.78)
 		)
 		(stroke
@@
 	(wire
 		(pts
-			(xy 311.15 127) (xy 311.15 129.54)
+			(xy 309.88 127) (xy 309.88 129.54)
 		)
 		(stroke
@@
 	(wire
 		(pts
+			(xy 309.88 127) (xy 318.77 127)
+		)
+		(stroke
+			(width 0)
+			(type default)
+		)
+	)
+	(wire
+		(pts
 			(xy 293.37 223.52) (xy 316.23 223.52)
 		)
@@
 	)
 	(symbol
+		(lib_id "Power_symbols:GND")
+		(at 312.42 144.78 0)
+		(unit 1)
+		(exclude_from_sim no)
+		(in_bom no)
+		(on_board no)
+		(dnp no)
+		(property "Reference" "#PWR021"
+			(at 312.166 136.144 0)
+			(do_not_autoplace yes)
+			(effects
+				(font
+					(size 1.27 1.27)
+				)
+				(hide yes)
+			)
+		)
+		(property "Value" "GND"
+			(at 309.88 148.844 0)
+			(effects
+				(font
+					(size 1.27 1.27)
+				)
+			)
+		)
+		(property "Footprint" ""
+			(at 312.42 144.78 0)
+			(effects
+				(font
+					(size 1.27 1.27)
+				)
+				(hide yes)
+			)
+		)
+		(property "Datasheet" ""
+			(at 312.42 144.78 0)
+			(effects
+				(font
+					(size 1.27 1.27)
+				)
+				(hide yes)
+			)
+		)
+		(property "Description" "Power Symbol - Global Ground"
+			(at 312.42 151.638 0)
+			(effects
+				(font
+					(size 1.27 1.27)
+				)
+				(hide yes)
+			)
+		)
+		(pin "1"
+		)
+		(instances
+			(project "Master_Hand_Kicad"
+				(path "/f9e05184-c88b-4a88-ae9c-ab2bdb32be7c/c5103ceb-5325-4a84-a025-9638a412984e/042ebd96-5d8b-461b-acb5-c7c1300dab56"
+					(reference "#PWR021")
+					(unit 1)
+				)
+			)
+		)
+	)
+	(symbol
 		(lib_id "Duc-Resistors:RES SMD 0402")
 		(at 204.47 101.6 90)
@@
 			)
 		)
-		(property "Description" "330uF ±20% 25V SMD"
+		(property "Description" "CAP ALUM POLY 330uF ±20% 25V SMD"
 			(at 116.84 218.44 90)
 			(effects
@@
 		(on_board no)
 		(dnp no)
-		(property "Reference" "#PWR021"
+		(property "Reference" "#PWR022"
 			(at 225.806 138.684 0)
 			(do_not_autoplace yes)
@@
 			(project "Master_Hand_Kicad"
 				(path "/f9e05184-c88b-4a88-ae9c-ab2bdb32be7c/c5103ceb-5325-4a84-a025-9638a412984e/042ebd96-5d8b-461b-acb5-c7c1300dab56"
-					(reference "#PWR021")
+					(reference "#PWR022")
 					(unit 1)
 				)
@@
 		(on_board no)
 		(dnp no)
-		(property "Reference" "#PWR022"
+		(property "Reference" "#PWR023"
 			(at 258.826 141.224 0)
 			(do_not_autoplace yes)
@@
 			(project "Master_Hand_Kicad"
 				(path "/f9e05184-c88b-4a88-ae9c-ab2bdb32be7c/c5103ceb-5325-4a84-a025-9638a412984e/042ebd96-5d8b-461b-acb5-c7c1300dab56"
-					(reference "#PWR022")
+					(reference "#PWR023")
 					(unit 1)
 				)
@@
 	(symbol
 		(lib_id "Duc-Capacitors:CAP CER 0603")
-		(at 311.15 133.35 90)
+		(at 309.88 133.35 90)
 		(unit 1)
 		(exclude_from_sim no)
@@
 		(fields_autoplaced yes)
 		(property "Reference" "C10"
-			(at 314.96 132.0799 90)
+			(at 313.69 132.0799 90)
 			(effects
 				(font
@@
 		)
 		(property "Value" "CAP CER 0603"
-			(at 314.96 134.6199 90)
+			(at 313.69 134.6199 90)
 			(effects
 				(font
@@
 		)
 		(property "Footprint" "Duc:C0603"
-			(at 318.77 133.35 0)
+			(at 317.5 133.35 0)
 			(effects
 				(font
@@
 		)
 		(property "Datasheet" "https://lcsc.com/product-detail/Multilayer-Ceramic-Capacitors-MLCC-SMD-SMT_100nF-104-10-50V_C14663.html"
-			(at 321.31 133.35 0)
+			(at 320.04 133.35 0)
 			(effects
 				(font
@@
 		)
 		(property "Description" "CAP CER 0603"
-			(at 311.15 133.35 0)
+			(at 309.88 133.35 0)
 			(effects
 				(font
@@
 		)
 		(property "Manufacturer" "YAGEO(国巨)"
-			(at 323.85 133.35 0)
+			(at 322.58 133.35 0)
 			(effects
 				(font
@@
 		)
 		(property "MPN" "CAP CER 0603"
-			(at 326.39 133.35 0)
+			(at 325.12 133.35 0)
 			(effects
 				(font
@@
 		)
 		(property "LCSC Part" "C14663"
-			(at 328.93 133.35 0)
+			(at 327.66 133.35 0)
 			(effects
 				(font
@@
 		(on_board no)
 		(dnp no)
-		(property "Reference" "#PWR024"
+		(property "Reference" "#PWR025"
 			(at 106.426 217.424 0)
 			(do_not_autoplace yes)
@@
 			(project "Master_Hand_Kicad"
 				(path "/f9e05184-c88b-4a88-ae9c-ab2bdb32be7c/c5103ceb-5325-4a84-a025-9638a412984e/042ebd96-5d8b-461b-acb5-c7c1300dab56"
-					(reference "#PWR024")
+					(reference "#PWR025")
 					(unit 1)
 				)
@@
 		(on_board no)
 		(dnp no)
-		(property "Reference" "#PWR023"
+		(property "Reference" "#PWR024"
 			(at 192.786 171.704 0)
 			(do_not_autoplace yes)
@@
 			(project "Master_Hand_Kicad"
 				(path "/f9e05184-c88b-4a88-ae9c-ab2bdb32be7c/c5103ceb-5325-4a84-a025-9638a412984e/042ebd96-5d8b-461b-acb5-c7c1300dab56"
-					(reference "#PWR023")
+					(reference "#PWR024")
 					(unit 1)
 				)
