File: Sensing - Temperature.kicad_sch (KiCad schematic)
At the start: 8 parts, among them U16 SHT40-N-NF, U17 SHT40-N-NF

Commit message: Update Schematic
Parts:
- C98, C99: value CAP CER 0402 -> 100nF 50V 0603; footprint Duc_Library:C0402 -> Duc:C0603; symbol Duc-Capacitors:CAP CER 0402 -> Duc-Capacitors:CAP CER 0603; LCSC Part C325464 -> C14663; MPN CC0402KRX5R7BB105 -> CAP CER 0603; Manufacturer (none) -> YAGEO(国巨)
- R70, R71, R72, R73: value RES 0402 -> 10K 0.1% 0603; footprint Duc_Library:R0402 -> Duc:R0603; symbol Duc-Resistors:RES SMD 0402 -> Duc-Resistors:RES SMD 0603; LCSC Part C728576 -> C4107493; MPN RT0402FRE07100KL -> RT0603FRE13100KL; Manufacturer (none) -> YAGEO(国巨)
Connections:
- net +3V3 renamed +A3V3

Commit message: Update Schematic
Parts:
- renumbered C98 to C100, C99 to C101
Changed lines of the file:
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@@
 		(dnp no)
 		(fields_autoplaced yes)
-		(property "Reference" "C98"
+		(property "Reference" "C100"
 			(at 168.91 68.5799 90)
 			(effects
@@
 			(project "Master_Hand_Kicad"
 				(path "/f9e05184-c88b-4a88-ae9c-ab2bdb32be7c/c5103ceb-5325-4a84-a025-9638a412984e/2e63ad8d-085e-4704-a18e-2216b579ffe6"
-					(reference "C98")
+					(reference "C100")
 					(unit 1)
 				)
@@
 		(dnp no)
 		(fields_autoplaced yes)
-		(property "Reference" "#PWR0133"
+		(property "Reference" "#PWR0132"
 			(at 167.386 71.374 0)
 			(do_not_autoplace yes)
@@
 			(project "Master_Hand_Kicad"
 				(path "/f9e05184-c88b-4a88-ae9c-ab2bdb32be7c/c5103ceb-5325-4a84-a025-9638a412984e/2e63ad8d-085e-4704-a18e-2216b579ffe6"
-					(reference "#PWR0133")
+					(reference "#PWR0132")
 					(unit 1)
 				)
@@
 		(dnp no)
 		(fields_autoplaced yes)
-		(property "Reference" "C99"
+		(property "Reference" "C101"
 			(at 168.91 111.7599 90)
 			(effects
@@
 			(project "Master_Hand_Kicad"
 				(path "/f9e05184-c88b-4a88-ae9c-ab2bdb32be7c/c5103ceb-5325-4a84-a025-9638a412984e/2e63ad8d-085e-4704-a18e-2216b579ffe6"
-					(reference "C99")
+					(reference "C101")
 					(unit 1)
 				)
@@
 		(dnp no)
 		(fields_autoplaced yes)
-		(property "Reference" "#PWR0134"
+		(property "Reference" "#PWR0133"
 			(at 167.386 114.554 0)
 			(do_not_autoplace yes)
@@
 			(project "Master_Hand_Kicad"
 				(path "/f9e05184-c88b-4a88-ae9c-ab2bdb32be7c/c5103ceb-5325-4a84-a025-9638a412984e/2e63ad8d-085e-4704-a18e-2216b579ffe6"
-					(reference "#PWR0134")
-					(unit 1)
-				)
+					(reference "#PWR0133")
+					(unit 1)
+				)

Commit message: Update Schematic & PCB
Parts:
- C100, C101: value 100nF 50V 0603 -> CAP CER 0603
- R70, R71, R72, R73: value 10K 0.1% 0603 -> RES 0603
Changed lines of the file:
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@@
 			"AAAAAABT3rg5ZvMEgFRlcm1pbmFsAAB5AHgAMQBsAG8AawBRAFHevjlu9ASAAAAAAAAAAACLlrPZ"
 			"VABpAGANeygeAgAAr9+8OUr1BIAGAAAAEAAAAKCh7f//////AAAAAAAAAACt30I6c/YEgAAAAAAA"
-			"AAAAEzay2WEAWgDADnsoHgIAAKvfQDpy9wSAVGVybWluYWwAAGgAeQBuAA=="
+			"AAAAEzay2WEAWgDADnsoHgIAAKvfQDpy9wSAVGVybWluYWwAAGgAeQBuAAAAAAAAAAAAAAAAAAAA"
+			"AAAAAAAAAAAAAAAAAAAAAAAAAAAAAAAAAAAAAAAAAAAAAAAAAAAAAAAAAAAAAAAAAAAAAAAAAAAA"
+			"AAAAAAAAAAAAAAAAAAAAAAAAAAAAAAAAAAAAAAAAAAAAAAAAAAAAAAAAAAAAAAAAAAAAAAAAAAAA"
+			"AAAAAAAAAAAAAAAAAAAAAAAAAAAAAAAAAAAAAAAAAAAAAAAAAAAAAAAAAAAAAAAAAAAAAAAAAAAA"
+			"AAAAAAAAAAAAAAAAAAAAAAAAAAAAAAAAAAAAAAAAAAAAAAAAAAAAAAAAAAAAAAAAAAAAAAAAAAAA"
+			"AAAAAAAAAAAAAAAAAAAAAAAAAAAAAAAAAAAAAAAAAAAAAAAAAAAAAAAAAAAAAAAAAAAAAAAAAAAA"
+			"AAAAAAAAAAAAAAAAAAAAAAAAAAAAAAAAAAAAAAAAAAAAAAAAAAAAAAAAAAAAAAAAAAAAAAAAAAAA"
+			"AAAAAAAAAAAAAAAAAAAAAAAAAAAAAAAAAAAAAAAAAAAAAAAAAAAAAAAAAAAAAAAAAAAAAAAAAAAA"
+			"AAAAAAAAAAAAAAAAAAAAAAAAAAAAAAAAAAAAAAAAAAAAAAAAAAAAAAAAAAAAAAAAAAAAAAAAAAAA"
+			"AAAAAAAAAAAAAAAAAAAAAAAAAAAAAAAAAAAAAAAAAAAAAAAAAAAAAAAAAAAAAAAAAAAAAAAAAAAA"
+			"AAAAAAAAAAAAAAAAAAAAAAAAAAAAAAAAAAAAAAAAAAAAAAAAAAAAAAAAAAAAAAAAAAAAAAAAAAAA"
+			"AAAAAAAAAAAAAAAAAAAAAAAAAAAAAAAAAAAAAAAAAAAAAAAAAAAAAAAAAAAAAAAAAAAAAAAAAAAA"
+			"AAAAAAAAAAAAAAAAAAAAAAAAAAAAAAAAAAAAAAAAAAAAAAAAAAAAAAAAAAAAAAAAAAAAAAAAAAAA"
+			"AAAAAAAAAAAAAAAAAAAAAAAAAAAAAAAAAAAAAAAAAAAAAAAAAAAAAAAAAAAAAAAAAAAAAAAAAAAA"
+			"AAAAAAAAAAAAAAAAAAAAAAAAAAAAAAAAAAAAAAAAAAAAAAAAAAAAAAAAAAAAAAAAAAAAAAAAAAAA"
+			"AAAAAAAAAAAAAAAAAAAAAAAAAAAAAAAAAAAAAAAAAAAAAAAAAAAAAAAAAAAAAAAAAAAAAAAAAAAA"
+			"AAAAAAAAAAAAAAAAAAAAAAAAAAAAAAAAAAAAAAAAAAAAAAAAAAAAAAAAAAAAAAAAAAAAAAAAAAAA"
+			"AAAAAAAAAAAAAAAAAAAAAAAAAAAAAAAAAAAAAAAAAAAAAAAAAAAAAAAAAAAAAAAAAAAAAAAAAAAA"
+			"AAAAAAAAAAAAAAAAAAAAAAAAAAAAAAAAAAAAAAAAAAAAAAAAAAAAAAAAAAAAAAAAAAAAAAAAAAAA"
+			"AAAAAAAAAAAAAAAAAAAAAAAAAAAAAAAAAAAAAAAAAAAAAAAAAAAAAAAAAAAAAAAAAAAAAAAAAAAA"
+			"AAAAAAAAAAAAAAAAAAAAAAAAAAAAAAAAAAAAAAAAAAAAAAAAAAAAAAAAAAAAAAAAAAAAAAAAAAAA"
+			"AAAAAAAAAAAAAAAAAAAAAAAAAAAAAAAAAAAAAAAAAAAAAAAAAAAAAAAAAAAAAAAAAAAAAAAAAAAA"
+			"AAAAAAAAAAAAAAAAAAAAAAAAAAAAAAAAAAAAAAAAAAAAAAAAAAAAAAAAAAAAAAAAAAAAAAAAAAAA"
+			"AAAAAAAAAAAAAAAAAAAAAAAAAAAAAAAAAAAAAAAAAAAAAAAAAAAAAAAAAAAAAAAAAAAAAAAAAAAA"
+			"AAAAAAAAAAAAAAAAAAAAAAAAAAAAAAAAAAAAAAAAAAAAAAAAAAAAAAAAAAAAAAAAAAAAAAAAAAAA"
+			"AAAAAAAAAAAAAAAAAAAAAAAAAAAAAAAAAAAAAAAAAAAAAAAAAAAAAAAAAAAAAAAAAAAAAAAAAAAA"
+			"AAAAAAAAAAAAAAAAAAAAAAAAAAAAAAAAAAAAAAAAAAAAAAAAAAAAAAAAAAAAAAAAAAAAAAAAAAAA"
+			"AAAAAAAAAAAAAAAAAAAAAAAAAAAAAAAAAAAAAAAAAAAAAAAAAAAAAAAAAAAAAAAAAAAAAAAAAAAA"
+			"AAAAAAAAAAAAAAAAAAAAAAAAAAAAAAAAAAAAAAAAAAAAAAAAAAAAAAAAAAAAAAAAAAAAAAAAAAAA"
+			"AAAAAAAAAAAAAAAAAAAAAAAAAAAAAAAAAAAAAAAAAAAAAAAAAAAAAAAAAAAAAAAAAAAAAAAAAAAA"
+			"AAAAAAAAAAAAAAAAAAAAAAAAAAAAAAAAAAAAAAAAAAAAAAAAAAAAAAAAAAAAAAAAAAAAAAAAAAAA"
+			"AAAAAAAAAAAAAAAAAAAAAAAAAAAAAAAAAAAAAAAAAAAAAAAAAAAAAAAAAAAAAAAAAAAAAAAAAAAA"
+			"AAAAAAAAAAAAAAAAAAAAAAAAAAAAAAAAAAAAAAAAAAAAAAAAAAAAAAAAAAAAAAAAAAAAAAAAAAAA"
+			"AAAAAAAAAAAAAAAAAAAAAAAAAAAAAAAAAAAAAAAAAAAAAAAAAAAAAAAAAAAAAAAAAAAAAAAAAAAA"
+			"AAAAAAAAAAAAAAAAAAAAAAAAAAAAAAAAAAAAAAAAAAAAAAAAAAAAAAAAAAAAAAAAAAAAAAAAAAAA"
+			"AAAAAAAAAAAAAAAAAAAAAAAAAAAAAAAAAAAAAAAAAAAAAAAAAAAAAAAAAAAAAAAAAAAAAAAAAAAA"
+			"AAAAAAAAAAAAAAAAAAAAAAAAAAAAAAAAAAAAAAAAAAAAAAAAAAAAAAAAAA=="
 		)
 	)
@@
 			"AEUAbQBJAHoASwAxADkAMgBOAG8ANgBUADUARQBhAGEATQBmAGUAbgBZAHcAUgBwADkAWgBPAEsA"
 			"VwBjADcAdgBkAC8AdQBIAGgALwB1ADcAdQByAHUAdgA3AHkAOAB1AHIAaQA0AHUATABzAGkAeQA2"
-			"AHIAcQB1AGIANQB1AFgAbAA1AFgAQQA0ADMATwBJAHQAQwA2ADkAWAA2AA=="
+			"AHIAcQB1AGIANQB1AFgAbAA1AFgAQQA0ADMATwBJAHQAQwA2ADkAWAA2AGFnYzNrTlp2Q08ySHZw"
+			"cnNMRDRaMVU5NytuOFBtZGorOHM0TjhZbld2WnFya0R4TGpOMC8yWUZ5SnkrRW9DSFdMcEhvWUkz"
+			"bXFwdFpxMXJaUlNpb2prbkpnSkJGVVZrWlFVUkNrbEVBQUhjUmlJNEk1MXhib1dzK2dBbGQ3Vzc3"
+			"cUxRQ09PUEhDdlNFVUV3dnJSYzVmU0pBWm83MUVCamJYbVhHY3hEaG9zamFOOUl1TUd2N0pGQ0xG"
+			"Q1FCSmhVYjFHZnlBY1lRaG9JRFhudGZyU3JKSkdUalFOR0RJbWpkUGdIMDcyYnBMN0FlL3VjQklJ"
+			"ZGdtdHNBNXFFeElDek5GS3NWckorMlhhOS9aK0lWbERsRVdpbzZGWlhqQ3hYZEdDRlJyQ0pTM2Jw"
+			"WnFUS0xzVFM0QnFzMlZkVTZZeEl5VWRSeVNGaC9zM09BajB1Q2VLUURWVTYyWVZRckh2L0YyOWg1"
+			"bFVSZDdzd3YvbHgvY2Q4TlRMU0xWR2JRMWdKamFQM1IzNnlOMUZhTWo5R05scGN1NE4xc2lkcjlm"
+			"clZqZHI1dUVSa1ZOT0tZc29FWGZOTE5YRUlpS0F4VTE3SlFBekxHdXJyWUdrRnc1QTRMMzM3aXll"
+			"QngwSDZiWU9DRHQ4WTJpWHF3eWdtMk01ekZFOFZxQW1kVkhKd2NNZzFKZ3FxREEzUlNnRldvVTFk"
+			"dXRLem5zVzdPeEFoNHkzQ0JmbWxPVjBrbW5pYWJCSjQ1VDlmbXAzSTZaVUJrbXBwemtNZ01IdWxS"
+			"ZzcvOXloektkcGRJOEE3LzI0dlpVUm1rZ1ZLVFBJSEdBNHdUdEJNWUxNd2VoaUJCNEIwVFJPd3VL"
+			"QWdNVGNsM1ZwUmttekNGUWhETWZCc25uRnNRRVFjU0NHSGRVaUlEc1hKL1pqVVJDWU9LWDAvOVJt"
+			"Nm84N3Z2T3JRZ1F6MUZhdEdVR0kyTTFaUUllY0d3akNPS1F1SThMTnJMV3dDak1xcGRUYUFJaW9p"
+			"QXpEcUpvN0k1c2d6RWhKZW8wcStqcENML1duclZUM0lHYno4RGdPRXdFUHk0SnhUTU1BQXF4Vlp0"
+			"L3A2UjBzaHQ1Yk9rQ3hnZUt4QmFwSWFIS0JNQ2M3SlRJUko0MWNObWtiYWtVMGhKRTdSWkFIbk9B"
+			"YW9CQjFaaWRFVnBtbWRIZVMwOHluc1k1U0ovVlRibVBhS0JKQmdBUklRQUV3Y1JCMWFkd0FBOU9n"
+			"WTFaTlI0Wk44R09McnhiTXpoMDEwenNOYmt4Q1BWVUJkV1dRVWd1UjVEd1FXV3VsbjdmTnpNTVA4"
+			"SnQ3aUFNRXAzNmkyRG11eDNwOC9ER0grNUhvSDlFT2RDWWxxK0lQYWRiOGoASwA2ADAATQBDAGIA"
+			"cwBIADMANAAyAFoAZwBQAFgAWgBFAE4AQgBlADkARABkAFUASgBvAGQAYQA2ADIAKwAyAG0AYQBU"
+			"AEsAawBCAG4ANQBrAEsAVAAvAEsAcgBPAEQAOABOAGkAMgBnAEsAcgBrAFkAdABjAFMARQA2ADEA"
+			"YgBMADUAWABKAGwAZABFACsAeABrAGMATQBIAEcAKwBXADMAaAArADcAaAAvAFIAbgB3AEQAVwBy"
+			"AFQARgA0AEUAWgBpAGYAdwB4AEwAawBEAEUATQBVAGMARQBpAEQARwBPAHcAMABCAEEAeQArAFYA"
+			"aQAwAFMAOQBDADIANQBCAHoAeQBDAEMAQQBWAFIAUgBBAEIAZABEAFoAVwBmAFgAUQBMAFYAQQBC"
+			"AFMAZwBVAEYAcQBCAFgAMgBZADcANQBaADUAOQAyAFEAOQAyAFAAYwA3AGQAdgByAGoAUgA5AEcA"
+			"egBnAFYATABwAGEAcQBxAGsARQBRAEwAQQB2AG8AQQBpAHgANABYAEgAYQA0AFcALwB2AEkAQwBM"
+			"AHMANwBoAHYASABjADkAUQBpAGkAQwBRADQASQBwAGEAMABrAFIAVgBaAFoAdAA2AFIAdABjAHQA"
+			"RwBkADMATAA3AFQAdABSAHUAYwB0AEgAQQBVAEEASgBIAFoAcwA5AEUAQQA1AFIARQBNAEMAQQBB"
+			"AGUASQA2AHgAOAA2ADMAcQBpADYAMgBVAE8AagA0AEoAZgBuAFoANgBGAHQATgArAHYAMQBPAEUA"
+			"WAB2AHEAZQB0ADcAUQBxAHkANQA3AGoAZQA3AG0AawBvAFQARwBoAFYASgB1AFUAegBqAFYARQBy"
+			"AE4ASgBRAG4AbwBvAHUAdQBiAHIAbwBsAHgAYQB0AG8AVwBFAGUAawBRAE0AcwBCAGIAcwAvAGYA"
+			"MABuAGIAMQA5AEgAQQBHAGUAdwAwAHMAOQBKAGgAQgBxAHgAZwB0AE0AcQBJADQAUgAwAFQAdQBI"
+			"AEIATABXAEMAYwArADcATwB4AFUAWABUAGgAUABYADYAWgByAGYAYgBiAHoAZgBiAGMAUgB4AFYA"
+			"QgBIAEYAdQByAGgAUwBaAHUAOAByAHQAUgBnACsANgA1AGMAYgBvAHcAcQBZAEoAWgBsAGUAeQAy"
+			"ACsAMwBHAGMAYwB5AGwAaABCAEMAOABkADgAeQBVAFUAMQBKAFEAUgBHAFYAeQBSAFcAUwAzADIA"
+			"OQBjAGkAcQA5AFcAeQA2ADcAcABhAGQAUgByAFQAcwB1ADkAVwB5ADIAVwBOAFcAYQBzAE0AKwAr"
+			"AEgATAB2ADMANgA1ADMAKwAvAC8ALwBkAC8ALwAvAFQAZQAvACsAOAAxAA=="
 		)
 	)
@@
 			)
 		)
-		(property "Value" "100nF 50V 0603"
+		(property "Value" "CAP CER 0603"
 			(at 168.91 71.1199 90)
 			(effects
@@
 			)
 		)
-		(property "Value" "10K 0.1% 0603"
+		(property "Value" "RES 0603"
 			(at 124.46 76.2 90)
 			(effects
@@
 		(dnp no)
 		(fields_autoplaced yes)
-		(property "Reference" "#PWR0132"
+		(property "Reference" "#PWR132"
 			(at 167.386 71.374 0)
 			(do_not_autoplace yes)
@@
 			(project "Master_Hand_Kicad"
 				(path "/f9e05184-c88b-4a88-ae9c-ab2bdb32be7c/c5103ceb-5325-4a84-a025-9638a412984e/2e63ad8d-085e-4704-a18e-2216b579ffe6"
-					(reference "#PWR0132")
+					(reference "#PWR132")
 					(unit 1)
 				)
@@
 			)
 		)
-		(property "Value" "10K 0.1% 0603"
+		(property "Value" "RES 0603"
 			(at 102.87 119.3799 90)
 			(effects
@@
 			)
 		)
-		(property "Value" "10K 0.1% 0603"
+		(property "Value" "RES 0603"
 			(at 102.87 76.1999 90)
 			(effects
@@
 			)
 		)
-		(property "Value" "10K 0.1% 0603"
+		(property "Value" "RES 0603"
 			(at 124.46 119.38 90)
 			(effects
@@
 			)
 		)
-		(property "Value" "100nF 50V 0603"
+		(property "Value" "CAP CER 0603"
 			(at 168.91 114.2999 90)
 			(effects
@@
 		(dnp no)
 		(fields_autoplaced yes)
-		(property "Reference" "#PWR0133"
+		(property "Reference" "#PWR133"
 			(at 167.386 114.554 0)
 			(do_not_autoplace yes)
@@
 			(project "Master_Hand_Kicad"
 				(path "/f9e05184-c88b-4a88-ae9c-ab2bdb32be7c/c5103ceb-5325-4a84-a025-9638a412984e/2e63ad8d-085e-4704-a18e-2216b579ffe6"
-					(reference "#PWR0133")
+					(reference "#PWR133")
 					(unit 1)
 				)

Commit message: Update SCH & PCB
Parts:
- C95: renamed from C100; value CAP CER 0603 -> CAP CER 0402; footprint Duc:C0603 -> Duc:C0402; symbol Duc-Capacitors:CAP CER 0603 -> Duc-Capacitors:CAP CER 0402; LCSC Part C14663 -> C325464; MPN CAP CER 0603 -> CC0402KRX5R7BB105
- C96: renamed from C101; value CAP CER 0603 -> CAP CER 0402; footprint Duc:C0603 -> Duc:C0402; symbol Duc-Capacitors:CAP CER 0603 -> Duc-Capacitors:CAP CER 0402; LCSC Part C14663 -> C325464; MPN CAP CER 0603 -> CC0402KRX5R7BB105
- R68: renamed from R70; value RES 0603 -> RES 0402; footprint Duc:R0603 -> Duc:R0402; symbol Duc-Resistors:RES SMD 0603 -> Duc-Resistors:RES SMD 0402; LCSC Part C4107493 -> C728576; MPN RT0603FRE13100KL -> RT0402FRE07100KL
- R69: renamed from R71; value RES 0603 -> RES 0402; footprint Duc:R0603 -> Duc:R0402; symbol Duc-Resistors:RES SMD 0603 -> Duc-Resistors:RES SMD 0402; LCSC Part C4107493 -> C728576; MPN RT0603FRE13100KL -> RT0402FRE07100KL
- R70: renamed from R72; value RES 0603 -> RES 0402; footprint Duc:R0603 -> Duc:R0402; symbol Duc-Resistors:RES SMD 0603 -> Duc-Resistors:RES SMD 0402; LCSC Part C4107493 -> C728576; MPN RT0603FRE13100KL -> RT0402FRE07100KL
- R71: renamed from R73; value RES 0603 -> RES 0402; footprint Duc:R0603 -> Duc:R0402; symbol Duc-Resistors:RES SMD 0603 -> Duc-Resistors:RES SMD 0402; LCSC Part C4107493 -> C728576; MPN RT0603FRE13100KL -> RT0402FRE07100KL

Commit message: Update SCH & PCB
Parts:
- renumbered R68 to R67, R69 to R68, R70 to R69, R71 to R70
Changed lines of the file:
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@@
 		(on_board yes)
 		(dnp no)
-		(property "Reference" "R69"
+		(property "Reference" "R68"
 			(at 124.46 73.406 90)
 			(effects
@@
 			(project "Master_Hand_Kicad"
 				(path "/f9e05184-c88b-4a88-ae9c-ab2bdb32be7c/c5103ceb-5325-4a84-a025-9638a412984e/2e63ad8d-085e-4704-a18e-2216b579ffe6"
-					(reference "R69")
+					(reference "R68")
 					(unit 1)
 				)
@@
 		(dnp no)
 		(fields_autoplaced yes)
-		(property "Reference" "#PWR0132"
+		(property "Reference" "#PWR0136"
 			(at 167.386 71.374 0)
 			(do_not_autoplace yes)
@@
 			(project "Master_Hand_Kicad"
 				(path "/f9e05184-c88b-4a88-ae9c-ab2bdb32be7c/c5103ceb-5325-4a84-a025-9638a412984e/2e63ad8d-085e-4704-a18e-2216b579ffe6"
-					(reference "#PWR0132")
+					(reference "#PWR0136")
 					(unit 1)
 				)
@@
 		(dnp no)
 		(fields_autoplaced yes)
-		(property "Reference" "R70"
+		(property "Reference" "R69"
 			(at 102.87 116.8399 90)
 			(effects
@@
 			(project "Master_Hand_Kicad"
 				(path "/f9e05184-c88b-4a88-ae9c-ab2bdb32be7c/c5103ceb-5325-4a84-a025-9638a412984e/2e63ad8d-085e-4704-a18e-2216b579ffe6"
-					(reference "R70")
+					(reference "R69")
 					(unit 1)
 				)
@@
 		(dnp no)
 		(fields_autoplaced yes)
-		(property "Reference" "R68"
+		(property "Reference" "R67"
 			(at 102.87 73.6599 90)
 			(effects
@@
 			(project "Master_Hand_Kicad"
 				(path "/f9e05184-c88b-4a88-ae9c-ab2bdb32be7c/c5103ceb-5325-4a84-a025-9638a412984e/2e63ad8d-085e-4704-a18e-2216b579ffe6"
-					(reference "R68")
+					(reference "R67")
 					(unit 1)
 				)
@@
 		(on_board yes)
 		(dnp no)
-		(property "Reference" "R71"
+		(property "Reference" "R70"
 			(at 124.968 116.84 90)
 			(effects
@@
 			(project "Master_Hand_Kicad"
 				(path "/f9e05184-c88b-4a88-ae9c-ab2bdb32be7c/c5103ceb-5325-4a84-a025-9638a412984e/2e63ad8d-085e-4704-a18e-2216b579ffe6"
-					(reference "R71")
+					(reference "R70")
 					(unit 1)
 				)
@@
 		(dnp no)
 		(fields_autoplaced yes)
-		(property "Reference" "#PWR0133"
+		(property "Reference" "#PWR0137"
 			(at 167.386 114.554 0)
 			(do_not_autoplace yes)
@@
 			(project "Master_Hand_Kicad"
 				(path "/f9e05184-c88b-4a88-ae9c-ab2bdb32be7c/c5103ceb-5325-4a84-a025-9638a412984e/2e63ad8d-085e-4704-a18e-2216b579ffe6"
-					(reference "#PWR0133")
-					(unit 1)
-				)
+					(reference "#PWR0137")
+					(unit 1)
+				)
