File: User - LED Indicators & Buzzer.kicad_sch (KiCad schematic)
At the start: 20 parts, among them Q3 2SC1815

Commit message: Update Schematic
Parts:
- D10: value LED 0603 -> Orange 0603
- D11: value LED 0603 -> Yellow 0603
- D12: value LED 0603 -> Green 0603
- D13: value LED 0603 -> Blue 0603
- D14: value LED 0603 -> White 0603
- D16, D17: value LED 0603 -> Red 0603
- D9: value LED 0603 -> RED 0603
- R61, R62, R63, R67, R68: value RES 0402 -> 330R 0.1% 0603; footprint Duc_Library:R0402 -> Duc:R0603; symbol Duc-Resistors:RES SMD 0402 -> Duc-Resistors:RES SMD 0603; LCSC Part C728576 -> C4107493; MPN RT0402FRE07100KL -> RT0603FRE13100KL; Manufacturer (none) -> YAGEO(国巨)
- R64, R65, R66: value RES 0402 -> 100R 0.1% 0603; footprint Duc_Library:R0402 -> Duc:R0603; symbol Duc-Resistors:RES SMD 0402 -> Duc-Resistors:RES SMD 0603; LCSC Part C728576 -> C4107493; MPN RT0402FRE07100KL -> RT0603FRE13100KL; Manufacturer (none) -> YAGEO(国巨)
- R69: value RES 0603 -> 470R 0.1% 0603
Connections:
- net +3V3: now also D10.2 (A), D11.2 (A), D12.2 (A), D13.2 (A), D14.2 (A), D16.2 (A), D17.2 (A), D9.2 (A)
- net GND: no longer D10.1 (C), D11.1 (C), D12.1 (C), D13.1 (C), D14.1 (C), D16.1 (C), D17.1 (C), D9.1 (C)
- net at R66.2: now also D14.1 (C); no longer D14.2 (A)
- net at R63.2: now also D11.1 (C); no longer D11.2 (A)
- net at R61.2: now also D9.1 (C); no longer D9.2 (A)
- net at R68.2: now also D17.1 (C); no longer D17.2 (A)
- net at R67.2: now also D16.1 (C); no longer D16.2 (A)
- net at R65.2: now also D13.1 (C); no longer D13.2 (A)
- net at R64.2: now also D12.1 (C); no longer D12.2 (A)
- net at R62.2: now also D10.1 (C); no longer D10.2 (A)
- no-connect marks 0 -> 2
Other:
- moved on the sheet: D15, Q3, R69

Commit message: Update Schematic & PCB
Parts:
- D10: value Orange 0603 -> LED 0603
- D11: value Yellow 0603 -> LED 0603
- D12: value Green 0603 -> LED 0603
- D13: value Blue 0603 -> LED 0603
- D14: value White 0603 -> LED 0603
- D16, D17: value Red 0603 -> LED 0603
- D9: value RED 0603 -> LED 0603
- R61, R62, R63, R67, R68: value 330R 0.1% 0603 -> RES 0603
- R64, R65, R66: value 100R 0.1% 0603 -> RES 0603
- R69: value 470R 0.1% 0603 -> RES 0603
Changed lines of the file:
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@@
 			"AHkaJVR5ODFt0Ld0KB4CAADOJX4+ZxQHgFNlZ29lIE1ETDIgQXNzZXRzAFduVXVmSMwlfD5tFQeA"
 			"AAAAAAAAAAAqmfghRTVPNfC5dCgeAgAAyiUCPloWB4DOiM69z4TOv869zrEAMlpnUFhaRU5CZTnI"
-			"JQA+bxcHgFNlZ29lIFByaW50AEtUL0tyT0Q4TmkyZ8YlBg=="
+			"JQA+bxcHgFNlZ29lIFByaW50AEtUL0tyT0Q4TmkyZ8YlBgAAAAAAAAAAAAAAAAAAAAAAAAAAAAAA"
+			"AAAAAAAAAAAAAAAAAAAAAAAAAAAAAAAAAAAAAAAAAAAAAAAAAAAAAAAAAAAAAAAAAAAAAAAAAAAA"
+			"AAAAAAAAAAAAAAAAAAAAAAAAAAAAAAAAAAAAAAAAAAAAAAAAAAAAAAAAAAAAAAAAAAAAAAAAAAAA"
+			"AAAAAAAAAAAAAAAAAAAAAAAAAAAAAAAAAAAAAAAAAAAAAAAAAAAAAAAAAAAAAAAAAAAAAAAAAAAA"
+			"AAAAAAAAAAAAAAAAAAAAAAAAAAAAAAAAAAAAAAAAAAAAAAAAAAAAAAAAAAAAAAAAAAAAAAAAAAAA"
+			"AAAAAAAAAAAAAAAAAAAAAAAAAAAAAAAAAAAAAAAAAAAAAAAAAAAAAAAAAAAAAAAAAAAAAAAAAAAA"
+			"AAAAAAAAAAAAAAAAAAAAAAAAAAAAAAAAAAAAAAAAAAAAAAAAAAAAAAAAAAAAAAAAAAAAAAAAAAAA"
+			"AAAAAAAAAAAAAAAAAAAAAAAAAAAAAAAAAAAAAAAAAAAAAAAAAAAAAAAAAAAAAAAAAAAAAAAAAAAA"
+			"AAAAAAAAAAAAAAAAAAAAAAAAAAAAAAAAAAAAAAAAAAAAAAAAAAAAAAAAAAAAAAAAAAAAAAAAAAAA"
+			"AAAAAAAAAAAAAAAAAAAAAAAAAAAAAAAAAAAAAAAAAAAAAAAAAAAAAAAAAAAAAAAAAAAAAAAAAAAA"
+			"AAAAAAAAAAAAAAAAAAAAAAAAAAAAAAAAAAAAAAAAAAAAAAAAAAAAAAAAAAAAAAAAAAAAAAAAAAAA"
+			"AAAAAAAAAAAAAAAAAAAAAAAAAAAAAAAAAAAAAAAAAAAAAAAAAAAAAAAAAAAAAAAAAAAAAAAAAAAA"
+			"AAAAAAAAAAAAAAAAAAAAAAAAAAAAAAAAAAAAAAAAAAAAAAAAAAAAAAAAAAAAAAAAAAAAAAAAAAAA"
+			"AAAAAAAAAAAAAAAAAAAAAAAAAAAAAAAAAAAAAAAAAAAAAAAAAAAAAAAAAAAAAAAAAAAAAAAAAAAA"
+			"AAAAAAAAAAAAAAAAAAAAAAAAAAAAAAAAAAAAAAAAAAAAAAAAAAAAAAAAAAAAAAAAAAAAAAAAAAAA"
+			"AAAAAAAAAAAAAAAAAAAAAAAAAAAAAAAAAAAAAAAAAAAAAAAAAAAAAAAAAAAAAAAAAAAAAAAAAAAA"
+			"AAAAAAAAAAAAAAAAAAAAAAAAAAAAAAAAAAAAAAAAAAAAAAAAAAAAAAAAAAAAAAAAAAAAAAAAAAAA"
+			"AAAAAAAAAAAAAAAAAAAAAAAAAAAAAAAAAAAAAAAAAAAAAAAAAAAAAAAAAAAAAAAAAAAAAAAAAAAA"
+			"AAAAAAAAAAAAAAAAAAAAAAAAAAAAAAAAAAAAAAAAAAAAANIEgAAAAAAAAAAAAwAAAAAAAABALjtb"
+			"/QEAAAEAAAAAAAAAAAAAAAAAAADWLlTNANMEgAAAAAAAAAAABAAAAAAAAAAAAAAAAAAAAAEAAAAA"
+			"AAAAAAAAAAAAAADRLlfNANQEgAAAAAAAAAAAAwAAAAAAAACwTTlb/QEAAAEAAAAAAAAAAAAAAAAA"
+			"AADMLlLNANUEgAAAAAAAAAAAAwAAAAAAAAAwLztb/QEAAAEAAAAAAAAAAAAAAAAAAADPLk3NANYE"
+			"gAAAAAAAAAAAAwAAAAAAAABALTtb/QEAAAEAAAAAAAAAAAAAAAAAAADKLkjNANcEgAAAAAAAAAAA"
+			"AwAAAAAAAABAMDtb/QEAAAEAAAAAAAAAAAAAAAAAAADFLkvNANgEgAAAAAAAAAAACAAAAAAAAACg"
+			"yTFb/QEAAAEAAAAAAAAAAAAAAAAAAADALkbNANkEgAAAAAAAAAAAAwAAAAAAAAAgLjxb/QEAAAEA"
+			"AAAAAAAAAAAAAAAAAADDLkHNANoEgAAAAAAAAAAABAAAAAAAAAAAAAAAAAAAAAEAAAAAAAAAAAAA"
+			"AAAAAAD+LnzNANsEgAAAAAAAAAAAAwAAAAAAAABQSzlb/QEAAAEAAAAAAAAAAAAAAAAAAAD5Ln/N"
+			"ANwEgAAAAAAAAAAAAwAAAAAAAABQMDtb/QEAAAEAAAAAAAAAAAAAAAAAAAD0LnrNAN0EgAAAAAAA"
+			"AAAAAwAAAAAAAACwLjtb/QEAAAEAAAAAAAAAAAAAAAAAAAD3LnXNAN4EgAAAAAAAAAAABAAAAAAA"
+			"AAAAAAAAAAAAAAEAAAAAAAAAAAAAAAAAAADyLnDNAN8EgAAAAAAAAAAACAAAAAAAAADgxzFb/QEA"
+			"AAEAAAAAAAAAAAAAAAAAAADtLnPNAOAEgAAAAAAAAAAAAwAAAAAAAACQSDlb/QEAAAEAAAAAAAAA"
+			"AAAAAAAAAADoLm7NAOEEgEM6L1dpbmRvd3MvZm9udHNcc2VyaWZldC5mb24AAAAAAAAAAAAAAADr"
+			"LmnNAOIEgAAAAAAAAAAAAwAAAAAAAABAJjxb/QEAAAEAAAAAAAAAAAAAAAAAAADmLmTNAOMEgAAA"
+			"AAAAAAAAAwAAAAAAAAAgMDtb/QEAAAEAAAAAAAAAAAAAAAAAAADhLmfNAOQEgAAAAAAAAAAACAAA"
+			"AAAAAACgzzFb/QEAAAEAAAAAAAAAAAAAAAAAAACcLmLNAOUEgAAAAAAAAAAAAwAAAAAAAACgLTtb"
+			"/QEAAAEAAAAAAAAAAAAAAAAAAACfLh3NAOYEgAAAAAAAAAAAAwAAAAAAAADALTtb/QEAAAEAAAAA"
+			"AAAAAAAAAAAAAACaLhjNAOcEgAAAAAAAAAAAAwAAAAAAAA=="
 		)
 	)
@@
 			"aABlAHIAMAAvAFAAeAA2AGUAbgBvADUAbQBNAFUAbABvAHAAbgBTAEwAUQBxAG0AOQBHAEgAaABB"
 			"AFEAdwBBAGQAbgBqAEMARgA3AGcAUABuAEcAVABQAE0AQwBCAHAAYQBHADQARgBiAEMAUwBDAEUA"
-			"ZgBRAHEAVAB6AEgAcABZAHQASAArAGQARQ=="
+			"ZgBRAHEAVAB6AEgAcABZAHQASAArAGQARQBsADAASwB1AFYAbABXAE0AcgAzAE8AdAB1ADcARwAv"
+			"AHQATgBjAFEAZwBqAEgAVwBHAGkAKwBGAGUAdgBQADYAOQBYAHEAOQAwAGwAcQBhAHMAWQA4AHgA"
+			"MAB4AGsAQwAyAE0AdgBsAG0ATwBmAEYAYgAvADcAcwAxADEAcABuADMAdAB1AGgANgB5AGgATQBK"
+			"AEMAVQBJAFAAaQBBAFQAUwB1AHAATQBpAGEAcgBJAE0AaQBVAFEASQBpAFEASwBDAG4ARwBrAGsA"
+			"NABjAEUASQBVAFIAagBhAEwATQA2ADcAegBDAHAAUAByAHIAUgBrAEIAUABlAE8ARQB4ADkAMwAw"
+			"AC8ARwBJAEsAQgB6AGYAcgBXAHEAaQBpAEoAVABTAGwAVgBWAEYAVgBOAHkAMQBpAFkAWQBzAHIA"
+			"egBZAEgAUQA3AGoAYQBDAFoAcgB2AC8AcgA2AG0ANABmAEgANQA3AHEAcQBsAGQAWgBTAEMAcwA3"
+			"AFIAZQAwAGMAQgBXAGkARgBFADUANwAyAHoAbgB2AEYANQBtAFUAeQBwAEoAcABGAG8AbAA4AEYA"
+			"SgBLAFkAbQBEAFIAUQBXAGEAKwB0AGwAYgBVAHMARgB0ADEAaQBGAEsAcABvACsATwBlAE4AeABV"
+			"AGUAYwBsADcAZgAyAEcAZwBzAGcAWABIAG0ATwA5AFcAeABoAGcAaQBEAHgANgBJAHAAVQBmAHcA"
+			"UwBCAFEAaABSAGIARgBFAEMAbgBqAG4ALwBIAEsASgB4AFoAZABGADcARQBYAFkAUABWAHQAdQBU"
+			"AEMANgBFADkAbwBHAFoAYQBmAGoAZAA3ADMANwBuAHIAUABVACsAdgBIADcAOQBoAGkAaAA2AFMA"
+			"aQBuAE8AeABhAHQAWAByAHgARABaADgAOQBQAHoANAA4AE8AagBNAFIAWQBRADkALwBzAHQAWgBS"
+			"AHcAaQBRAGcAZwBFADMAMwA4AGEAUgBPAFUAYwBuAEEAdAA5ADMAeAB0AGoAMgA3AFoAcABtAHoA"
+			"YgBHAFMARQAxAGUAVgBWAFYANQBVAFEAZwBoAFoANABZAG4AUQBBAEsASQBFAGEAcQA2AC8AUAB6"
+			"AHoAegA3AFYAVwBIAHgANABlACsAcQA3AC8ANABZAGMAZgB6AEcAUgBlAHYAMwBtADEAMgBhAHcA"
+			"WgBBACsAYwArACsAaQBQACsAdwBZAE4AZQBNAEQAVQBiAEsAUwBVAGYAZwBqAFgAZQBtAEQAQQBN"
+			"AFEAOQB1ADIAZgBkAGUARwA2AE0AdQB5AHIASwBwAHkAdgBhADYAcgBxAG8AQgBFAEoAeAA5AGYA"
+			"cgBjAHAAWQBGAGMAWgBhADYAMQB4AHoAdgBRAFcAdABzAFkAKwBHAC8ATABRACsASQBhAEMAZAB6"
+			"AHgAZgBJAGsAawBzAFoAWQAxAHoAQwBLAHMAMQB0ADIANgB5AFYAUgBFAFEARQBGAHUATQBNADkA"
+			"ZABLAEIAegBSAEEAQgBFADIATwBvAHQATgBaAGEAQwBjAEcAUAB6ADgALwB2ADMALwA4AHcARABF"
+			"AE4AWgBWAHEAdgBWAHUAaQBoAHkAUQBHAFMAYwBTADYAVwBxAHEAbABKAGEAVwAyAHYANwB2AGgA"
+			"KwBHAGcAVwB3AGwAcwBrAHgAeQBEAGsAUwBzACsAcQBYAEYARAB3AEIAMAAzAFgAQQA4AEgAbwBu"
+			"ADIANgBwAHoATABzAG0AeQA3ADIAeAA0AE8AaAArADEAMgBxADcAWABrAEgAQgBtAEgARQBNAEIA"
+			"NQBzAGsANABEADcANQBNAFEAdgBDAGgAeQB4AHAAaAB6AHQAaAAvADYAbwBSADgANABZADAAVgBa"
+			"AFMAaQBsAG8ATABmADkAVABhAFAAYQAyAFgAcwBJADAANQA3ADgAZwBKAEgAVABXAFQAWgBOAHAA"
+			"bQBzADUATQAwAHoAQQBPADMAcgB1AHEATAB1AC8AdgA3ADMAYgA3AGIAWgA1AG4AZQBTAEYARABD"
+			"AEQANAA0AFkAbwBFAGgATQBxADAAegBVAHIAaABNAFoAcQBTAE0AYwBDAEcAMQAxAHUAcQBuAE4A"
+			"UQBVAFgANwBPAFEAUAB5ADAAMgBLAEgANQBkADgALwBIAC8ALwBEAC8AOAB4AHAAWQBoAEkARQBE"
+			"AHUAeABjAHgARAA1AGIAWABuADYAawAxADgAVQBPAFUANABUAE8AcwB3AGMAQgBrAFIAZwBpAEIA"
+			"dwBwAHcAQgBOAGgASABQADMAbABjAGgAMwBIAHcAVgByAGoAbgBQAEgAZQBUAGQATwBJAEMATwB2"
+			"ADEAKwB1ADUAdwBWADUAYQBWADEAcABnAGkANgBmAGQANQBpAHIARABZAGEAYgBIAFoAYgBlAHEA"
+			"WABQAGgAMQBDAHUAZQBmAC8AdABlAFIAQgAwAEkAbQB5AG8AQQBaAEYAawBRAHMAcABmAHYAegB4"
+			"AHgAdwA4AGYAUABuAHoANwA3AGQAZQBjAHMAMwBmAHYAUABpAHUASwBmAEwATgBaADcAMwBaAGIA"
+			"SwBUAGsAaQBKADAAZwBoAEoAZQBSAE0ASgBGAGoAUwBFAFAANwBnAEkAMgBJAFkAWQB3AEEARwBu"
+			"AEQAUAB2AEgAUwBCAHcAdwBaAHEAMgAvACsATAAzAFgANQAzAFAAWgAwAFIAcQBoAFgARwBjAEIA"
+			"dQA5ADgAVwBHAEwASwB2AFAAZgBUAFoATQ=="
 		)
 	)
@@
 			)
 		)
-		(property "Value" "100R 0.1% 0603"
+		(property "Value" "RES 0603"
 			(at 71.12 104.14 0)
 			(effects
@@
 			)
 		)
-		(property "Value" "Yellow 0603"
+		(property "Value" "LED 0603"
 			(at 86.36 67.31 0)
 			(effects
@@
 			)
 		)
-		(property "Value" "330R 0.1% 0603"
+		(property "Value" "RES 0603"
 			(at 71.12 66.04 0)
 			(effects
@@
 			)
 		)
-		(property "Value" "330R 0.1% 0603"
+		(property "Value" "RES 0603"
 			(at 71.12 40.64 0)
 			(effects
@@
 			)
 		)
-		(property "Value" "Red 0603"
+		(property "Value" "LED 0603"
 			(at 86.36 130.81 0)
 			(effects
@@
 			)
 		)
-		(property "Value" "Red 0603"
+		(property "Value" "LED 0603"
 			(at 86.36 118.11 0)
 			(effects
@@
 			)
 		)
-		(property "Value" "470R 0.1% 0603"
+		(property "Value" "RES 0603"
 			(at 208.28 129.54 0)
 			(effects
@@
 			)
 		)
-		(property "Value" "330R 0.1% 0603"
+		(property "Value" "RES 0603"
 			(at 71.12 116.84 0)
 			(effects
@@
 			)
 		)
-		(property "Value" "Blue 0603"
+		(property "Value" "LED 0603"
 			(at 86.36 92.71 0)
 			(effects
@@
 			)
 		)
-		(property "Value" "100R 0.1% 0603"
+		(property "Value" "RES 0603"
 			(at 71.12 78.74 0)
 			(effects
@@
 			)
 		)
-		(property "Value" "RED 0603"
+		(property "Value" "LED 0603"
 			(at 86.36 40.64 0)
 			(effects
@@
 			)
 		)
-		(property "Value" "White 0603"
+		(property "Value" "LED 0603"
 			(at 86.36 105.41 0)
 			(effects
@@
 			)
 		)
-		(property "Value" "100R 0.1% 0603"
+		(property "Value" "RES 0603"
 			(at 71.12 91.44 0)
 			(effects
@@
 			)
 		)
-		(property "Value" "330R 0.1% 0603"
+		(property "Value" "RES 0603"
 			(at 71.12 129.54 0)
 			(effects
@@
 			)
 		)
-		(property "Value" "330R 0.1% 0603"
+		(property "Value" "RES 0603"
 			(at 71.12 53.34 0)
 			(effects
@@
 			)
 		)
-		(property "Value" "Green 0603"
+		(property "Value" "LED 0603"
 			(at 86.36 80.01 0)
 			(effects
@@
 		(dnp no)
 		(fields_autoplaced yes)
-		(property "Reference" "#PWR0131"
+		(property "Reference" "#PWR131"
 			(at 225.806 128.524 0)
 			(do_not_autoplace yes)
@@
 			(project "Master_Hand_Kicad"
 				(path "/f9e05184-c88b-4a88-ae9c-ab2bdb32be7c/c5103ceb-5325-4a84-a025-9638a412984e/28daf353-f3ef-4ecd-aedd-b1b76d334dfe"
-					(reference "#PWR0131")
+					(reference "#PWR131")
 					(unit 1)
 				)
@@
 			)
 		)
-		(property "Value" "Orange 0603"
+		(property "Value" "LED 0603"
 			(at 86.36 54.61 0)
 			(effects

Commit message: Update SCH & PCB
Parts:
- renumbered R61 to R59, R62 to R60, R63 to R61, R64 to R62, R65 to R63, R66 to R64, R67 to R65, R68 to R66, R69 to R67
Changed lines of the file:
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@@
 		(on_board yes)
 		(dnp no)
-		(property "Reference" "R66"
+		(property "Reference" "R64"
 			(at 71.12 99.06 0)
 			(effects
@@
 			(project "Master_Hand_Kicad"
 				(path "/f9e05184-c88b-4a88-ae9c-ab2bdb32be7c/c5103ceb-5325-4a84-a025-9638a412984e/28daf353-f3ef-4ecd-aedd-b1b76d334dfe"
-					(reference "R66")
+					(reference "R64")
 					(unit 1)
 				)
@@
 		(on_board yes)
 		(dnp no)
-		(property "Reference" "R63"
+		(property "Reference" "R61"
 			(at 71.12 60.96 0)
 			(effects
@@
 			(project "Master_Hand_Kicad"
 				(path "/f9e05184-c88b-4a88-ae9c-ab2bdb32be7c/c5103ceb-5325-4a84-a025-9638a412984e/28daf353-f3ef-4ecd-aedd-b1b76d334dfe"
-					(reference "R63")
+					(reference "R61")
 					(unit 1)
 				)
@@
 		(on_board yes)
 		(dnp no)
-		(property "Reference" "R61"
+		(property "Reference" "R59"
 			(at 71.12 35.56 0)
 			(effects
@@
 			(project "Master_Hand_Kicad"
 				(path "/f9e05184-c88b-4a88-ae9c-ab2bdb32be7c/c5103ceb-5325-4a84-a025-9638a412984e/28daf353-f3ef-4ecd-aedd-b1b76d334dfe"
-					(reference "R61")
+					(reference "R59")
 					(unit 1)
 				)
@@
 		(on_board yes)
 		(dnp no)
-		(property "Reference" "R69"
+		(property "Reference" "R67"
 			(at 208.28 124.46 0)
 			(effects
@@
 			(project "Master_Hand_Kicad"
 				(path "/f9e05184-c88b-4a88-ae9c-ab2bdb32be7c/c5103ceb-5325-4a84-a025-9638a412984e/28daf353-f3ef-4ecd-aedd-b1b76d334dfe"
-					(reference "R69")
+					(reference "R67")
 					(unit 1)
 				)
@@
 		(on_board yes)
 		(dnp no)
-		(property "Reference" "R67"
+		(property "Reference" "R65"
 			(at 71.12 111.76 0)
 			(effects
@@
 			(project "Master_Hand_Kicad"
 				(path "/f9e05184-c88b-4a88-ae9c-ab2bdb32be7c/c5103ceb-5325-4a84-a025-9638a412984e/28daf353-f3ef-4ecd-aedd-b1b76d334dfe"
-					(reference "R67")
+					(reference "R65")
 					(unit 1)
 				)
@@
 		(on_board yes)
 		(dnp no)
-		(property "Reference" "R64"
+		(property "Reference" "R62"
 			(at 71.12 73.66 0)
 			(effects
@@
 			(project "Master_Hand_Kicad"
 				(path "/f9e05184-c88b-4a88-ae9c-ab2bdb32be7c/c5103ceb-5325-4a84-a025-9638a412984e/28daf353-f3ef-4ecd-aedd-b1b76d334dfe"
-					(reference "R64")
+					(reference "R62")
 					(unit 1)
 				)
@@
 		(on_board yes)
 		(dnp no)
-		(property "Reference" "R65"
+		(property "Reference" "R63"
 			(at 71.12 86.36 0)
 			(effects
@@
 			(project "Master_Hand_Kicad"
 				(path "/f9e05184-c88b-4a88-ae9c-ab2bdb32be7c/c5103ceb-5325-4a84-a025-9638a412984e/28daf353-f3ef-4ecd-aedd-b1b76d334dfe"
-					(reference "R65")
+					(reference "R63")
 					(unit 1)
 				)
@@
 		(on_board yes)
 		(dnp no)
-		(property "Reference" "R68"
+		(property "Reference" "R66"
 			(at 71.12 124.46 0)
 			(effects
@@
 			(project "Master_Hand_Kicad"
 				(path "/f9e05184-c88b-4a88-ae9c-ab2bdb32be7c/c5103ceb-5325-4a84-a025-9638a412984e/28daf353-f3ef-4ecd-aedd-b1b76d334dfe"
-					(reference "R68")
+					(reference "R66")
 					(unit 1)
 				)
@@
 		(on_board yes)
 		(dnp no)
-		(property "Reference" "R62"
+		(property "Reference" "R60"
 			(at 71.12 48.26 0)
 			(effects
@@
 			(project "Master_Hand_Kicad"
 				(path "/f9e05184-c88b-4a88-ae9c-ab2bdb32be7c/c5103ceb-5325-4a84-a025-9638a412984e/28daf353-f3ef-4ecd-aedd-b1b76d334dfe"
-					(reference "R62")
+					(reference "R60")
 					(unit 1)
 				)
@@
 		(dnp no)
 		(fields_autoplaced yes)
-		(property "Reference" "#PWR131"
+		(property "Reference" "#PWR0131"
 			(at 225.806 128.524 0)
 			(do_not_autoplace yes)
@@
 			(project "Master_Hand_Kicad"
 				(path "/f9e05184-c88b-4a88-ae9c-ab2bdb32be7c/c5103ceb-5325-4a84-a025-9638a412984e/28daf353-f3ef-4ecd-aedd-b1b76d334dfe"
-					(reference "#PWR131")
-					(unit 1)
-				)
+					(reference "#PWR0131")
+					(unit 1)
+				)

Commit message: Update SCH & PCB
Parts:
- removed BZ1: MLT-8530, Duc:BUZ-SMD_4P-L8.5-W8.5-P8.50-BR, symbol Duc-Misc:MLT-8530
- removed D15: SS34, Duc:SMA_L4.3-W2.5-LS5.0-RD, symbol Duc-Diodes:SS34
- removed Q3: 2SC1815, Duc:SOT-23-3_L2.9-W1.3-P1.90-LS2.4-BR, symbol Duc-Transistors:2SC1815_C20069143
- removed R67: RES 0603, Duc:R0603, symbol Duc-Resistors:RES SMD 0603
- R59, R60, R61, R62, R63, R64, R65, R66: value RES 0603 -> RES 0402; footprint Duc:R0603 -> Duc:R0402; symbol Duc-Resistors:RES SMD 0603 -> Duc-Resistors:RES SMD 0402; LCSC Part C4107493 -> C728576; MPN RT0603FRE13100KL -> RT0402FRE07100KL
- renumbered D16 to D15, D17 to D16
Connections:
- no-connect marks 2 -> 0
