File: Sensing - Battery.kicad_sch (KiCad schematic)
At the start: 3 parts

Commit message: Update Schematic
Parts:
- C100: value CAP CER 0603 -> 100nF 50V 0603
- R74: value RES 0603 -> 100K 0.1% 0603
- R75: value RES 0603 -> 47K 0.1% 0603
Changed lines of the file:
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@@
 	(wire
 		(pts
-			(xy 190.5 83.82) (xy 190.5 81.28)
+			(xy 190.5 81.28) (xy 190.5 85.09)
 		)
 		(stroke
@@
 	(wire
 		(pts
-			(xy 190.5 93.98) (xy 190.5 97.79)
+			(xy 190.5 92.71) (xy 190.5 97.79)
 		)
 		(stroke
@@
 			)
 		)
-		(property "Value" "RES 0603"
+		(property "Value" "100K 0.1% 0603"
 			(at 168.91 74.9299 90)
 			(effects
@@
 			)
 		)
-		(property "Value" "CAP CER 0603"
+		(property "Value" "100nF 50V 0603"
 			(at 194.31 90.1699 90)
 			(effects
@@
 			)
 		)
-		(property "Value" "RES 0603"
+		(property "Value" "47K 0.1% 0603"
 			(at 168.91 90.1699 90)
 			(effects

Commit message: Update Schematic
Parts:
- renumbered C100 to C102
Changed lines of the file:
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@@
 		(dnp no)
 		(fields_autoplaced yes)
-		(property "Reference" "#PWR0135"
+		(property "Reference" "#PWR0134"
 			(at 168.656 94.234 0)
 			(do_not_autoplace yes)
@@
 			(project "Master_Hand_Kicad"
 				(path "/f9e05184-c88b-4a88-ae9c-ab2bdb32be7c/c5103ceb-5325-4a84-a025-9638a412984e/d30056b5-4391-456e-bc80-2bde1ca0d521"
-					(reference "#PWR0135")
+					(reference "#PWR0134")
 					(unit 1)
 				)
@@
 		(dnp no)
 		(fields_autoplaced yes)
-		(property "Reference" "C100"
+		(property "Reference" "C102"
 			(at 194.31 87.6299 90)
 			(effects
@@
 			(project "Master_Hand_Kicad"
 				(path "/f9e05184-c88b-4a88-ae9c-ab2bdb32be7c/c5103ceb-5325-4a84-a025-9638a412984e/d30056b5-4391-456e-bc80-2bde1ca0d521"
-					(reference "C100")
+					(reference "C102")
 					(unit 1)
 				)

Commit message: Update Schematic & PCB
Parts:
- C102: value 100nF 50V 0603 -> CAP CER 0603
- R74: value 100K 0.1% 0603 -> RES 0603
- R75: value 47K 0.1% 0603 -> RES 0603
Changed lines of the file:
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@@
 		(dnp no)
 		(fields_autoplaced yes)
-		(property "Reference" "#PWR0134"
+		(property "Reference" "#PWR134"
 			(at 168.656 94.234 0)
 			(do_not_autoplace yes)
@@
 			(project "Master_Hand_Kicad"
 				(path "/f9e05184-c88b-4a88-ae9c-ab2bdb32be7c/c5103ceb-5325-4a84-a025-9638a412984e/d30056b5-4391-456e-bc80-2bde1ca0d521"
-					(reference "#PWR0134")
+					(reference "#PWR134")
 					(unit 1)
 				)
@@
 			)
 		)
-		(property "Value" "100K 0.1% 0603"
+		(property "Value" "RES 0603"
 			(at 168.91 74.9299 90)
 			(effects
@@
 			)
 		)
-		(property "Value" "100nF 50V 0603"
+		(property "Value" "CAP CER 0603"
 			(at 194.31 90.1699 90)
 			(effects
@@
 			)
 		)
-		(property "Value" "47K 0.1% 0603"
+		(property "Value" "RES 0603"
 			(at 168.91 90.1699 90)
 			(effects

Commit message: Update SCH & PCB
Parts:
- renumbered C102 to C97, R74 to R72, R75 to R73
Changed lines of the file:
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@@
 		(dnp no)
 		(fields_autoplaced yes)
-		(property "Reference" "#PWR134"
+		(property "Reference" "#PWR0134"
 			(at 168.656 94.234 0)
 			(do_not_autoplace yes)
@@
 			(project "Master_Hand_Kicad"
 				(path "/f9e05184-c88b-4a88-ae9c-ab2bdb32be7c/c5103ceb-5325-4a84-a025-9638a412984e/d30056b5-4391-456e-bc80-2bde1ca0d521"
-					(reference "#PWR134")
+					(reference "#PWR0134")
 					(unit 1)
 				)
@@
 		(dnp no)
 		(fields_autoplaced yes)
-		(property "Reference" "R74"
+		(property "Reference" "R72"
 			(at 168.91 72.3899 90)
 			(effects
@@
 			(project "Master_Hand_Kicad"
 				(path "/f9e05184-c88b-4a88-ae9c-ab2bdb32be7c/c5103ceb-5325-4a84-a025-9638a412984e/d30056b5-4391-456e-bc80-2bde1ca0d521"
-					(reference "R74")
+					(reference "R72")
 					(unit 1)
 				)
@@
 		(dnp no)
 		(fields_autoplaced yes)
-		(property "Reference" "C102"
+		(property "Reference" "C97"
 			(at 194.31 87.6299 90)
 			(effects
@@
 			(project "Master_Hand_Kicad"
 				(path "/f9e05184-c88b-4a88-ae9c-ab2bdb32be7c/c5103ceb-5325-4a84-a025-9638a412984e/d30056b5-4391-456e-bc80-2bde1ca0d521"
-					(reference "C102")
+					(reference "C97")
 					(unit 1)
 				)
@@
 		(dnp no)
 		(fields_autoplaced yes)
-		(property "Reference" "R75"
+		(property "Reference" "R73"
 			(at 168.91 87.6299 90)
 			(effects
@@
 			(project "Master_Hand_Kicad"
 				(path "/f9e05184-c88b-4a88-ae9c-ab2bdb32be7c/c5103ceb-5325-4a84-a025-9638a412984e/d30056b5-4391-456e-bc80-2bde1ca0d521"
-					(reference "R75")
+					(reference "R73")
 					(unit 1)
 				)

Commit message: Update SCH & PCB
Parts:
- renumbered R72 to R71, R73 to R72
Changed lines of the file:
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@@
 		(dnp no)
 		(fields_autoplaced yes)
-		(property "Reference" "#PWR0134"
+		(property "Reference" "#PWR0138"
 			(at 168.656 94.234 0)
 			(do_not_autoplace yes)
@@
 			(project "Master_Hand_Kicad"
 				(path "/f9e05184-c88b-4a88-ae9c-ab2bdb32be7c/c5103ceb-5325-4a84-a025-9638a412984e/d30056b5-4391-456e-bc80-2bde1ca0d521"
-					(reference "#PWR0134")
+					(reference "#PWR0138")
 					(unit 1)
 				)
@@
 		(dnp no)
 		(fields_autoplaced yes)
-		(property "Reference" "R72"
+		(property "Reference" "R71"
 			(at 168.91 72.3899 90)
 			(effects
@@
 			(project "Master_Hand_Kicad"
 				(path "/f9e05184-c88b-4a88-ae9c-ab2bdb32be7c/c5103ceb-5325-4a84-a025-9638a412984e/d30056b5-4391-456e-bc80-2bde1ca0d521"
-					(reference "R72")
+					(reference "R71")
 					(unit 1)
 				)
@@
 		(dnp no)
 		(fields_autoplaced yes)
-		(property "Reference" "R73"
+		(property "Reference" "R72"
 			(at 168.91 87.6299 90)
 			(effects
@@
 			(project "Master_Hand_Kicad"
 				(path "/f9e05184-c88b-4a88-ae9c-ab2bdb32be7c/c5103ceb-5325-4a84-a025-9638a412984e/d30056b5-4391-456e-bc80-2bde1ca0d521"
-					(reference "R73")
+					(reference "R72")
 					(unit 1)
 				)

Commit message: Update Schematic & PCB & STM32 IOC
Parts:
- C97: value CAP CER 0603 -> CAP CER 0402; footprint Duc:C0603 -> Duc:C0402; symbol Duc-Capacitors:CAP CER 0603 -> Duc-Capacitors:CAP CER 0402; LCSC Part C14663 -> C325464; MPN CAP CER 0603 -> CC0402KRX5R7BB105
- R71, R72: value RES 0603 -> RES 0402; footprint Duc:R0603 -> Duc:R0402; symbol Duc-Resistors:RES SMD 0603 -> Duc-Resistors:RES SMD 0402; LCSC Part C4107493 -> C728576; MPN RT0603FRE13100KL -> RT0402FRE07100KL
Changed lines of the file:
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@@
 	)
 	(symbol
-		(lib_id "Duc-Resistors:RES SMD 0603")
+		(lib_id "Duc-Resistors:RES SMD 0402")
 		(at 166.37 73.66 90)
 		(unit 1)
@@
 			)
 		)
-		(property "Value" "RES 0603"
+		(property "Value" "RES 0402"
 			(at 168.91 74.9299 90)
 			(effects
@@
 			)
 		)
-		(property "Footprint" "Duc:R0603"
+		(property "Footprint" "Duc:R0402"
 			(at 173.99 73.66 0)
 			(effects
@@
 			)
 		)
-		(property "Description" "RES SMD 0603"
-			(at 166.37 73.66 0)
+		(property "Description" "RES SMD 0402"
+			(at 169.418 74.168 0)
 			(effects
 				(font
@@
 			)
 		)
-		(property "MPN" "RT0603FRE13100KL"
+		(property "MPN" "RT0402FRE07100KL"
 			(at 181.61 73.66 0)
 			(effects
@@
 			)
 		)
-		(property "LCSC Part" "C4107493"
+		(property "LCSC Part" "C728576"
 			(at 184.15 73.66 0)
 			(effects
@@
 	)
 	(symbol
-		(lib_id "Duc-Capacitors:CAP CER 0603")
+		(lib_id "Duc-Capacitors:CAP CER 0402")
 		(at 190.5 88.9 90)
 		(unit 1)
@@
 			)
 		)
-		(property "Value" "CAP CER 0603"
+		(property "Value" "CAP CER 0402"
 			(at 194.31 90.1699 90)
 			(effects
@@
 			)
 		)
-		(property "Footprint" "Duc:C0603"
-			(at 198.12 88.9 0)
+		(property "Footprint" "Duc:C0402"
+			(at 203.2 88.9 0)
 			(effects
 				(font
@@
 		)
 		(property "Datasheet" "https://lcsc.com/product-detail/Multilayer-Ceramic-Capacitors-MLCC-SMD-SMT_100nF-104-10-50V_C14663.html"
-			(at 200.66 88.9 0)
-			(effects
-				(font
-					(size 1.27 1.27)
-				)
-				(hide yes)
-			)
-		)
-		(property "Description" "CAP CER 0603"
-			(at 190.5 88.9 0)
+			(at 205.74 88.9 0)
+			(effects
+				(font
+					(size 1.27 1.27)
+				)
+				(hide yes)
+			)
+		)
+		(property "Description" "CAP CER 0402"
+			(at 197.866 88.9 0)
 			(effects
 				(font
@@
 		)
 		(property "Manufacturer" "YAGEO(国巨)"
-			(at 203.2 88.9 0)
-			(effects
-				(font
-					(size 1.27 1.27)
-				)
-				(hide yes)
-			)
-		)
-		(property "MPN" "CAP CER 0603"
-			(at 205.74 88.9 0)
-			(effects
-				(font
-					(size 1.27 1.27)
-				)
-				(hide yes)
-			)
-		)
-		(property "LCSC Part" "C14663"
 			(at 208.28 88.9 0)
+			(effects
+				(font
+					(size 1.27 1.27)
+				)
+				(hide yes)
+			)
+		)
+		(property "MPN" "CC0402KRX5R7BB105"
+			(at 210.82 88.9 0)
+			(effects
+				(font
+					(size 1.27 1.27)
+				)
+				(hide yes)
+			)
+		)
+		(property "LCSC Part" "C325464"
+			(at 213.36 88.9 0)
 			(effects
 				(font
@@
 	)
 	(symbol
-		(lib_id "Duc-Resistors:RES SMD 0603")
+		(lib_id "Duc-Resistors:RES SMD 0402")
 		(at 166.37 88.9 90)
 		(unit 1)
@@
 			)
 		)
-		(property "Value" "RES 0603"
+		(property "Value" "RES 0402"
 			(at 168.91 90.1699 90)
 			(effects
@@
 			)
 		)
-		(property "Footprint" "Duc:R0603"
+		(property "Footprint" "Duc:R0402"
 			(at 173.99 88.9 0)
 			(effects
@@
 			)
 		)
-		(property "Description" "RES SMD 0603"
-			(at 166.37 88.9 0)
+		(property "Description" "RES SMD 0402"
+			(at 169.418 89.408 0)
 			(effects
 				(font
@@
 			)
 		)
-		(property "MPN" "RT0603FRE13100KL"
+		(property "MPN" "RT0402FRE07100KL"
 			(at 181.61 88.9 0)
 			(effects
@@
 			)
 		)
-		(property "LCSC Part" "C4107493"
+		(property "LCSC Part" "C728576"
 			(at 184.15 88.9 0)
 			(effects

Commit message: Update project
Parts:
- C97: value CAP CER 0402 -> 100nF 50V
- R71: value RES 0402 -> 100K 0.1%
- R72: value RES 0402 -> 47K 0.1%
Changed lines of the file:
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@@
 		(dnp no)
 		(fields_autoplaced yes)
-		(property "Reference" "#PWR0138"
+		(property "Reference" "#PWR138"
 			(at 168.656 94.234 0)
 			(do_not_autoplace yes)
@@
 			(project "Master_Hand_Kicad"
 				(path "/f9e05184-c88b-4a88-ae9c-ab2bdb32be7c/c5103ceb-5325-4a84-a025-9638a412984e/d30056b5-4391-456e-bc80-2bde1ca0d521"
-					(reference "#PWR0138")
+					(reference "#PWR138")
 					(unit 1)
 				)
@@
 		(on_board yes)
 		(dnp no)
-		(fields_autoplaced yes)
 		(property "Reference" "R71"
-			(at 168.91 72.3899 90)
-			(effects
-				(font
-					(size 1.27 1.27)
-				)
-				(justify right)
-			)
-		)
-		(property "Value" "RES 0402"
-			(at 168.91 74.9299 90)
+			(at 168.91 70.485 90)
+			(effects
+				(font
+					(size 1.27 1.27)
+				)
+				(justify right)
+			)
+		)
+		(property "Value" "100K 0.1%"
+			(at 168.91 73.025 90)
 			(effects
 				(font
@@
 		)
 		(property "Footprint" "Duc:R0402"
-			(at 173.99 73.66 0)
-			(effects
-				(font
-					(size 1.27 1.27)
-				)
-				(hide yes)
+			(at 168.91 75.565 90)
+			(effects
+				(font
+					(size 1.27 1.27)
+				)
+				(justify right)
 			)
 		)
@@
 		(on_board yes)
 		(dnp no)
-		(fields_autoplaced yes)
 		(property "Reference" "C97"
-			(at 194.31 87.6299 90)
-			(effects
-				(font
-					(size 1.27 1.27)
-				)
-				(justify right)
-			)
-		)
-		(property "Value" "CAP CER 0402"
-			(at 194.31 90.1699 90)
+			(at 193.04 86.995 90)
+			(effects
+				(font
+					(size 1.27 1.27)
+				)
+				(justify right)
+			)
+		)
+		(property "Value" "100nF 50V"
+			(at 193.04 89.535 90)
 			(effects
 				(font
@@
 		)
 		(property "Footprint" "Duc:C0402"
-			(at 203.2 88.9 0)
-			(effects
-				(font
-					(size 1.27 1.27)
-				)
-				(hide yes)
+			(at 193.04 92.075 90)
+			(effects
+				(font
+					(size 1.27 1.27)
+				)
+				(justify right)
 			)
 		)
@@
 		(on_board yes)
 		(dnp no)
-		(fields_autoplaced yes)
 		(property "Reference" "R72"
-			(at 168.91 87.6299 90)
-			(effects
-				(font
-					(size 1.27 1.27)
-				)
-				(justify right)
-			)
-		)
-		(property "Value" "RES 0402"
-			(at 168.91 90.1699 90)
+			(at 168.91 85.725 90)
+			(effects
+				(font
+					(size 1.27 1.27)
+				)
+				(justify right)
+			)
+		)
+		(property "Value" "47K 0.1%"
+			(at 168.91 88.265 90)
 			(effects
 				(font
@@
 		)
 		(property "Footprint" "Duc:R0402"
-			(at 173.99 88.9 0)
-			(effects
-				(font
-					(size 1.27 1.27)
-				)
-				(hide yes)
-			)
-		)
+			(at 168.91 90.805 90)
+			(effects
+				(font
+					(size 1.27 1.27)
+				)
+				(justify right)
+			)
+		)
