File: sch_backup_20260820_225926/Interface - FD-CAN.kicad_sch (KiCad schematic)
At the start: 10 parts, among them U14 TJA1051T/3, U15 TJA1051T/3

Commit message: Update Schematic
Connections:
- net FDCAN_N renamed FDCAN1_N
- net FDCAN1_N: no longer U15.6 (CANL)
- net FDCAN_P renamed FDCAN1_P
- net FDCAN1_P: no longer U15.7 (CANH)
- new net FDCAN2_N: U15.6 (CANL)
- new net FDCAN2_P: U15.7 (CANH)
