File: sch_backup_20260820_225926/Interface - Interconnects.kicad_sch (KiCad schematic)
At the start: 14 parts, among them J11 1.25-3PLTDK, J12 5025982393, J13 PH2.54-2X3P-H25, J14 PH2.54-2X3P-H25, J15 PH2.54-2X3P-H25

Commit message: Update Schematic
Connections:
- net CAN_TERM_MID: now reaches C94.2, R59.1, R60.2
- net FDCAN_N renamed CAN_TERM_B
- net FDCAN_P renamed CAN_TERM_T
- no-connect marks 4 -> 2
