File: sch_backup_20260820_225926/MCU - IOs.kicad_sch (KiCad schematic)
At the start: 8 parts, among them U6 STM32G474RET6, U7 STM32G474RET6, X1 X322516MLB4SI, X2 X322516MLB4SI

Commit message: Update Schematic
Changed lines of the file:
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@@
 		(company "${COMPANY}")
 	)
+	(bus_alias "SW_BOOT"
+		(members "BOOT_1" "BOOT_2")
+	)
 	(rectangle
 		(start 118.11 241.3)
@@
 		)
 	)
+	(wire
+		(pts
+			(xy 213.36 180.34) (xy 213.36 181.61)
+		)
+		(stroke
+			(width 0)
+			(type default)
+		)
+	)
 	(bus
 		(pts
@@
 	(wire
 		(pts
-			(xy 213.36 181.61) (xy 213.36 180.34)
-		)
-		(stroke
-			(width 0)
-			(type default)
-		)
-	)
-	(wire
-		(pts
 			(xy 82.55 110.49) (xy 105.41 110.49)
 		)
@@
 		)
 	)
-	(label "BOARD_VERSION"
+	(label "BOARD_VER"
 		(at 214.63 35.56 0)
 		(effects
@@
 		)
 	)
-	(label "BOARD_VERSION"
+	(label "BOARD_VER"
 		(at 105.41 210.82 180)
 		(effects
@@
 		)
 	)
-	(label "BOARD_VERSION"
+	(label "BOARD_VER"
 		(at 105.41 95.25 180)
 		(effects
@@
 		)
 	)
-	(hierarchical_label "{LED_Finger2}"
+	(hierarchical_label "{LED_Finger 2}"
 		(shape output)
 		(at 167.64 165.1 0)
@@
 		)
 	)
-	(hierarchical_label "{LED_Finger1}"
+	(hierarchical_label "{LED_Finger 1}"
 		(shape output)
 		(at 167.64 152.4 0)
@@
 	(symbol
 		(lib_id "Power_symbols:GND")
-		(at 251.46 156.21 0)
+		(at 248.92 154.94 180)
 		(unit 1)
 		(exclude_from_sim no)
@@
 		(on_board no)
 		(dnp no)
-		(property "Reference" "#PWR034"
-			(at 251.206 147.574 0)
+		(property "Reference" "#PWR30"
+			(at 248.92 154.94 0)
 			(do_not_autoplace yes)
 			(effects
@@
 		)
 		(property "Value" "GND"
-			(at 248.92 160.274 0)
+			(at 248.92 161.29 0)
 			(effects
 				(font
@@
 		)
 		(property "Footprint" ""
-			(at 251.46 156.21 0)
+			(at 248.92 154.94 0)
 			(effects
 				(font
@@
 		)
 		(property "Datasheet" ""
-			(at 251.46 156.21 0)
+			(at 248.92 154.94 0)
 			(effects
 				(font
@@
 		)
 		(property "Description" "Power Symbol - Global Ground"
-			(at 251.46 163.068 0)
+			(at 248.92 154.94 0)
 			(effects
 				(font
@@
 			(project "Master_Hand_Kicad"
 				(path "/f9e05184-c88b-4a88-ae9c-ab2bdb32be7c/c5103ceb-5325-4a84-a025-9638a412984e/e744f3ce-03a6-44a6-8792-1447ef232b9a"
-					(reference "#PWR034")
+					(reference "#PWR30")
 					(unit 1)
 				)
@@
 	(symbol
 		(lib_id "Power_symbols:GND")
-		(at 215.9 181.61 0)
+		(at 213.36 180.34 180)
 		(unit 1)
 		(exclude_from_sim no)
@@
 		(dnp no)
 		(fields_autoplaced yes)
-		(property "Reference" "#PWR035"
-			(at 215.646 172.974 0)
+		(property "Reference" "#PWR31"
+			(at 213.36 180.34 0)
 			(do_not_autoplace yes)
 			(effects
@@
 		)
 		(property "Footprint" ""
-			(at 215.9 181.61 0)
+			(at 213.36 180.34 0)
 			(effects
 				(font
@@
 		)
 		(property "Datasheet" ""
-			(at 215.9 181.61 0)
+			(at 213.36 180.34 0)
 			(effects
 				(font
@@
 		)
 		(property "Description" "Power Symbol - Global Ground"
-			(at 215.9 188.468 0)
+			(at 213.36 180.34 0)
 			(effects
 				(font
@@
 			(project "Master_Hand_Kicad"
 				(path "/f9e05184-c88b-4a88-ae9c-ab2bdb32be7c/c5103ceb-5325-4a84-a025-9638a412984e/e744f3ce-03a6-44a6-8792-1447ef232b9a"
-					(reference "#PWR035")
+					(reference "#PWR31")
 					(unit 1)
 				)
@@
 	(symbol
 		(lib_id "Power_symbols:GND")
-		(at 251.46 181.61 0)
+		(at 248.92 180.34 180)
 		(unit 1)
 		(exclude_from_sim no)
@@
 		(dnp no)
 		(fields_autoplaced yes)
-		(property "Reference" "#PWR036"
-			(at 251.206 172.974 0)
+		(property "Reference" "#PWR32"
+			(at 248.92 180.34 0)
 			(do_not_autoplace yes)
 			(effects
@@
 		)
 		(property "Footprint" ""
-			(at 251.46 181.61 0)
+			(at 248.92 180.34 0)
 			(effects
 				(font
@@
 		)
 		(property "Datasheet" ""
-			(at 251.46 181.61 0)
+			(at 248.92 180.34 0)
 			(effects
 				(font
@@
 		)
 		(property "Description" "Power Symbol - Global Ground"
-			(at 251.46 188.468 0)
+			(at 248.92 180.34 0)
 			(effects
 				(font
@@
 			(project "Master_Hand_Kicad"
 				(path "/f9e05184-c88b-4a88-ae9c-ab2bdb32be7c/c5103ceb-5325-4a84-a025-9638a412984e/e744f3ce-03a6-44a6-8792-1447ef232b9a"
-					(reference "#PWR036")
+					(reference "#PWR32")
 					(unit 1)
 				)
@@
 	(symbol
 		(lib_id "Power_symbols:GND")
-		(at 215.9 156.21 0)
+		(at 213.36 154.94 180)
 		(unit 1)
 		(exclude_from_sim no)
@@
 		(on_board no)
 		(dnp no)
-		(property "Reference" "#PWR033"
-			(at 215.646 147.574 0)
+		(property "Reference" "#PWR29"
+			(at 213.36 154.94 0)
 			(do_not_autoplace yes)
 			(effects
@@
 		)
 		(property "Value" "GND"
-			(at 213.36 160.274 0)
+			(at 213.36 161.29 0)
 			(effects
 				(font
@@
 		)
 		(property "Footprint" ""
-			(at 215.9 156.21 0)
+			(at 213.36 154.94 0)
 			(effects
 				(font
@@
 		)
 		(property "Datasheet" ""
-			(at 215.9 156.21 0)
+			(at 213.36 154.94 0)
 			(effects
 				(font
@@
 		)
 		(property "Description" "Power Symbol - Global Ground"
-			(at 215.9 163.068 0)
+			(at 213.36 154.94 0)
 			(effects
 				(font
@@
 			(project "Master_Hand_Kicad"
 				(path "/f9e05184-c88b-4a88-ae9c-ab2bdb32be7c/c5103ceb-5325-4a84-a025-9638a412984e/e744f3ce-03a6-44a6-8792-1447ef232b9a"
-					(reference "#PWR033")
+					(reference "#PWR29")
 					(unit 1)
 				)
