File: sch_backup_20260820_225926/MCU - Power.kicad_sch (KiCad schematic)
At the start: 22 parts, among them U6 STM32G474RET6, U7 STM32G474RET6

Commit message: Update Schematic
Parts:
- renumbered L2 to L3, L3 to L4
