File: sch_backup_20260820_225926/Motor Control - Index.kicad_sch (KiCad schematic)
At the start: 14 parts, among them J7 BM09B-SRSS-TB, U12 TB9051FTG,EL

Commit message: Update Schematic
Parts:
- removed C76, C77, C78, C79, C80, C81: CAP CER 0402, Duc_Library:C0402, symbol Duc-Capacitors:CAP CER 0402
- removed J7: BM09B-SRSS-TB, Duc:CONN-SMD_9P-P1.00_BM09B-SRSS-TB, symbol Duc-Connectors:BM09B-SRSS-TB
- removed R31, R32, R33, R34, R35, R36: RES 0402, Duc_Library:R0402, symbol Duc-Resistors:RES SMD 0402
- removed U12: TB9051FTG,EL, Duc_Library:UQFN-28_L6.0-W6.0-P0.65-BL-EP4.0, symbol Duc-ICs:TB9051FTG,EL
- added C52, C53, C54, C55, C56, C57: CAP CER 0402, Duc_Library:C0402, symbol Duc-Capacitors:CAP CER 0402
- added J3: BM09B-SRSS-TB, Duc:CONN-SMD_9P-P1.00_BM09B-SRSS-TB, symbol Duc-Connectors:BM09B-SRSS-TB
- added R10, R11, R12, R7, R8, R9: RES 0402, Duc_Library:R0402, symbol Duc-Resistors:RES SMD 0402
- added U8: TB9051FTG,EL, Duc_Library:UQFN-28_L6.0-W6.0-P0.65-BL-EP4.0, symbol Duc-ICs:TB9051FTG,EL
Connections:
- net +3V3: now also J3.8, R11.2
- net +5V: now also C52.2, R7.1
- net +A3V3: now also C56.2, J3.3
- net +VBAT: now also C54.2, U8.11 (VBAT), U8.12 (VBAT), U8.24 (VBAT), U8.25 (VBAT)
- net GND: now also C52.1, C53.1, C54.1, C55.1, C56.1, C57.1, J3.1, J3.10, J3.11, J3.5, R10.2, U8.1 (OCC), U8.15 (PGND), U8.16 (PGND), U8.17 (PGND), U8.19 (PGND), U8.20 (PGND), U8.21 (PGND), U8.27 (TEST1), U8.28 (TEST2), U8.29 (EP), U8.3 (ENB), U8.4 (AGND)
- new net DIAG_I: R9.2
- new net ECA_I: J3.6
- new net ECB_I: J3.7
- new net ECC_I: C57.2, R12.2
- new net EN_I: U8.5 (EN)
- new net OCM_I: R10.1, R8.1
- new net OUT1_I: J3.4, U8.13 (OUT1), U8.14 (OUT1)
- new net OUT2_I: J3.9, U8.22 (OUT2), U8.23 (OUT2)
- new net PWMA_I: U8.8 (PWM1)
- new net PWMB_I: U8.9 (PWM2)
- new net VCC_I: C53.2, R7.2, U8.2 (VCC)
- new net _DIAG_I: R11.1, R9.1, U8.18 (DIAG)
- new net _ECC_I: J3.2, R12.1
- new net _OCM_I: C55.2, R8.2, U8.7 (OCM)
