File: sch_backup_20260820_225926/Motor Control - Middle.kicad_sch (KiCad schematic)
At the start: 14 parts, among them J7 BM09B-SRSS-TB, U12 TB9051FTG,EL

Commit message: Update Schematic
Parts:
- removed C76, C77, C78, C79, C80, C81: CAP CER 0402, Duc_Library:C0402, symbol Duc-Capacitors:CAP CER 0402
- removed J7: BM09B-SRSS-TB, Duc:CONN-SMD_9P-P1.00_BM09B-SRSS-TB, symbol Duc-Connectors:BM09B-SRSS-TB
- removed R31, R32, R33, R34, R35, R36: RES 0402, Duc_Library:R0402, symbol Duc-Resistors:RES SMD 0402
- removed U12: TB9051FTG,EL, Duc_Library:UQFN-28_L6.0-W6.0-P0.65-BL-EP4.0, symbol Duc-ICs:TB9051FTG,EL
- added C58, C59, C60, C61, C62, C63: CAP CER 0402, Duc_Library:C0402, symbol Duc-Capacitors:CAP CER 0402
- added J4: BM09B-SRSS-TB, Duc:CONN-SMD_9P-P1.00_BM09B-SRSS-TB, symbol Duc-Connectors:BM09B-SRSS-TB
- added R13, R14, R15, R16, R17, R18: RES 0402, Duc_Library:R0402, symbol Duc-Resistors:RES SMD 0402
- added U9: TB9051FTG,EL, Duc_Library:UQFN-28_L6.0-W6.0-P0.65-BL-EP4.0, symbol Duc-ICs:TB9051FTG,EL
Connections:
- net +3V3: now also J4.8, R17.2
- net +5V: now also C58.2, R13.1
- net +A3V3: now also C62.2, J4.3
- net +VBAT: now also C60.2, U9.11 (VBAT), U9.12 (VBAT), U9.24 (VBAT), U9.25 (VBAT)
- net GND: now also C58.1, C59.1, C60.1, C61.1, C62.1, C63.1, J4.1, J4.10, J4.11, J4.5, R16.2, U9.1 (OCC), U9.15 (PGND), U9.16 (PGND), U9.17 (PGND), U9.19 (PGND), U9.20 (PGND), U9.21 (PGND), U9.27 (TEST1), U9.28 (TEST2), U9.29 (EP), U9.3 (ENB), U9.4 (AGND)
- new net DIAG_M: R15.2
- new net ECA_M: J4.6
- new net ECB_M: J4.7
- new net ECC_M: C63.2, R18.2
- new net EN_M: U9.5 (EN)
- new net OCM_M: R14.1, R16.1
- new net OUT1_M: J4.4, U9.13 (OUT1), U9.14 (OUT1)
- new net OUT2_M: J4.9, U9.22 (OUT2), U9.23 (OUT2)
- new net PWMA_M: U9.8 (PWM1)
- new net PWMB_M: U9.9 (PWM2)
- new net VCC_M: C59.2, R13.2, U9.2 (VCC)
- new net _DIAG_M: R15.1, R17.1, U9.18 (DIAG)
- new net _ECC_M: J4.2, R18.1
- new net _OCM_M: C61.2, R14.2, U9.7 (OCM)
