File: sch_backup_20260820_225926/Motor Control - Pinky.kicad_sch (KiCad schematic)
At the start: 14 parts, among them J7 BM09B-SRSS-TB, U12 TB9051FTG,EL

Commit message: Update Schematic
Parts:
- removed C76, C77, C78, C79, C80, C81: CAP CER 0402, Duc_Library:C0402, symbol Duc-Capacitors:CAP CER 0402
- removed J7: BM09B-SRSS-TB, Duc:CONN-SMD_9P-P1.00_BM09B-SRSS-TB, symbol Duc-Connectors:BM09B-SRSS-TB
- removed R31, R32, R33, R34, R35, R36: RES 0402, Duc_Library:R0402, symbol Duc-Resistors:RES SMD 0402
- removed U12: TB9051FTG,EL, Duc_Library:UQFN-28_L6.0-W6.0-P0.65-BL-EP4.0, symbol Duc-ICs:TB9051FTG,EL
- added C70, C71, C72, C73, C74, C75: CAP CER 0402, Duc_Library:C0402, symbol Duc-Capacitors:CAP CER 0402
- added J6: BM09B-SRSS-TB, Duc:CONN-SMD_9P-P1.00_BM09B-SRSS-TB, symbol Duc-Connectors:BM09B-SRSS-TB
- added R25, R26, R27, R28, R29, R30: RES 0402, Duc_Library:R0402, symbol Duc-Resistors:RES SMD 0402
- added U11: TB9051FTG,EL, Duc_Library:UQFN-28_L6.0-W6.0-P0.65-BL-EP4.0, symbol Duc-ICs:TB9051FTG,EL
Connections:
- net +3V3: now also J6.8, R29.2
- net +5V: now also C70.2, R25.1
- net +A3V3: now also C74.2, J6.3
- net +VBAT: now also C72.2, U11.11 (VBAT), U11.12 (VBAT), U11.24 (VBAT), U11.25 (VBAT)
- net GND: now also C70.1, C71.1, C72.1, C73.1, C74.1, C75.1, J6.1, J6.10, J6.11, J6.5, R28.2, U11.1 (OCC), U11.15 (PGND), U11.16 (PGND), U11.17 (PGND), U11.19 (PGND), U11.20 (PGND), U11.21 (PGND), U11.27 (TEST1), U11.28 (TEST2), U11.29 (EP), U11.3 (ENB), U11.4 (AGND)
- new net DIAG_P: R27.2
- new net ECA_P: J6.6
- new net ECB_P: J6.7
- new net ECC_P: C75.2, R30.2
- new net EN_P: U11.5 (EN)
- new net OCM_P: R26.1, R28.1
- new net OUT1_P: J6.4, U11.13 (OUT1), U11.14 (OUT1)
- new net OUT2_P: J6.9, U11.22 (OUT2), U11.23 (OUT2)
- new net PWMA_P: U11.8 (PWM1)
- new net PWMB_P: U11.9 (PWM2)
- new net VCC_P: C71.2, R25.2, U11.2 (VCC)
- new net _DIAG_P: R27.1, R29.1, U11.18 (DIAG)
- new net _ECC_P: J6.2, R30.1
- new net _OCM_P: C73.2, R26.2, U11.7 (OCM)
