File: sch_backup_20260820_225926/Motor Control - Ring.kicad_sch (KiCad schematic)
At the start: 14 parts, among them J7 BM09B-SRSS-TB, U12 TB9051FTG,EL

Commit message: Update Schematic
Parts:
- removed C76, C77, C78, C79, C80, C81: CAP CER 0402, Duc_Library:C0402, symbol Duc-Capacitors:CAP CER 0402
- removed J7: BM09B-SRSS-TB, Duc:CONN-SMD_9P-P1.00_BM09B-SRSS-TB, symbol Duc-Connectors:BM09B-SRSS-TB
- removed R31, R32, R33, R34, R35, R36: RES 0402, Duc_Library:R0402, symbol Duc-Resistors:RES SMD 0402
- removed U12: TB9051FTG,EL, Duc_Library:UQFN-28_L6.0-W6.0-P0.65-BL-EP4.0, symbol Duc-ICs:TB9051FTG,EL
- added C64, C65, C66, C67, C68, C69: CAP CER 0402, Duc_Library:C0402, symbol Duc-Capacitors:CAP CER 0402
- added J5: BM09B-SRSS-TB, Duc:CONN-SMD_9P-P1.00_BM09B-SRSS-TB, symbol Duc-Connectors:BM09B-SRSS-TB
- added R19, R20, R21, R22, R23, R24: RES 0402, Duc_Library:R0402, symbol Duc-Resistors:RES SMD 0402
- added U10: TB9051FTG,EL, Duc_Library:UQFN-28_L6.0-W6.0-P0.65-BL-EP4.0, symbol Duc-ICs:TB9051FTG,EL
Connections:
- net +3V3: now also J5.8, R23.2
- net +5V: now also C64.2, R19.1
- net +A3V3: now also C68.2, J5.3
- net +VBAT: now also C66.2, U10.11 (VBAT), U10.12 (VBAT), U10.24 (VBAT), U10.25 (VBAT)
- net GND: now also C64.1, C65.1, C66.1, C67.1, C68.1, C69.1, J5.1, J5.10, J5.11, J5.5, R22.2, U10.1 (OCC), U10.15 (PGND), U10.16 (PGND), U10.17 (PGND), U10.19 (PGND), U10.20 (PGND), U10.21 (PGND), U10.27 (TEST1), U10.28 (TEST2), U10.29 (EP), U10.3 (ENB), U10.4 (AGND)
- new net DIAG_R: R21.2
- new net ECA_R: J5.6
- new net ECB_R: J5.7
- new net ECC_R: C69.2, R24.2
- new net EN_R: U10.5 (EN)
- new net OCM_R: R20.1, R22.1
- new net OUT1_R: J5.4, U10.13 (OUT1), U10.14 (OUT1)
- new net OUT2_R: J5.9, U10.22 (OUT2), U10.23 (OUT2)
- new net PWMA_R: U10.8 (PWM1)
- new net PWMB_R: U10.9 (PWM2)
- new net VCC_R: C65.2, R19.2, U10.2 (VCC)
- new net _DIAG_R: R21.1, R23.1, U10.18 (DIAG)
- new net _ECC_R: J5.2, R24.1
- new net _OCM_R: C67.2, R20.2, U10.7 (OCM)
