File: sch_backup_20260820_225926/Motor Control - Thumb 2.kicad_sch (KiCad schematic)
At the start: 14 parts, among them J7 BM09B-SRSS-TB, U12 TB9051FTG,EL

Commit message: Update Schematic
Parts:
- removed C76, C77, C78, C79, C80, C81: CAP CER 0402, Duc_Library:C0402, symbol Duc-Capacitors:CAP CER 0402
- removed J7: BM09B-SRSS-TB, Duc:CONN-SMD_9P-P1.00_BM09B-SRSS-TB, symbol Duc-Connectors:BM09B-SRSS-TB
- removed R31, R32, R33, R34, R35, R36: RES 0402, Duc_Library:R0402, symbol Duc-Resistors:RES SMD 0402
- removed U12: TB9051FTG,EL, Duc_Library:UQFN-28_L6.0-W6.0-P0.65-BL-EP4.0, symbol Duc-ICs:TB9051FTG,EL
- added C82, C83, C84, C85, C86, C87: CAP CER 0402, Duc_Library:C0402, symbol Duc-Capacitors:CAP CER 0402
- added J8: BM09B-SRSS-TB, Duc:CONN-SMD_9P-P1.00_BM09B-SRSS-TB, symbol Duc-Connectors:BM09B-SRSS-TB
- added R37, R38, R39, R40, R41, R42: RES 0402, Duc_Library:R0402, symbol Duc-Resistors:RES SMD 0402
- added U13: TB9051FTG,EL, Duc_Library:UQFN-28_L6.0-W6.0-P0.65-BL-EP4.0, symbol Duc-ICs:TB9051FTG,EL
Connections:
- net +3V3: now also J8.8, R41.2
- net +5V: now also C82.2, R37.1
- net +A3V3: now also C86.2, J8.3
- net +VBAT: now also C84.2, U13.11 (VBAT), U13.12 (VBAT), U13.24 (VBAT), U13.25 (VBAT)
- net GND: now also C82.1, C83.1, C84.1, C85.1, C86.1, C87.1, J8.1, J8.10, J8.11, J8.5, R40.2, U13.1 (OCC), U13.15 (PGND), U13.16 (PGND), U13.17 (PGND), U13.19 (PGND), U13.20 (PGND), U13.21 (PGND), U13.27 (TEST1), U13.28 (TEST2), U13.29 (EP), U13.3 (ENB), U13.4 (AGND)
- new net DIAG_T2: R39.2
- new net ECA_T2: J8.6
- new net ECB_T2: J8.7
- new net ECC_T2: C87.2, R42.2
- new net EN_T2: U13.5 (EN)
- new net OCM_T2: R38.1, R40.1
- new net OUT1_T2: J8.4, U13.13 (OUT1), U13.14 (OUT1)
- new net OUT2_T2: J8.9, U13.22 (OUT2), U13.23 (OUT2)
- new net PWMA_T2: U13.8 (PWM1)
- new net PWMB_T2: U13.9 (PWM2)
- new net VCC_T2: C83.2, R37.2, U13.2 (VCC)
- new net _DIAG_T2: R39.1, R41.1, U13.18 (DIAG)
- new net _ECC_T2: J8.2, R42.1
- new net _OCM_T2: C85.2, R38.2, U13.7 (OCM)
