File: sch_backup_20260820_225926/Power - Connectors.kicad_sch (KiCad schematic)
At the start: 10 parts, among them J1 XT60PW-M, J2 DC-044A-20A, Q1 HV10N03, Q2 HV10N03, U4 LM74700QDBVRQ1, U5 LM74700QDBVRQ1

Commit message: Update Schematic
Changed lines of the file:
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@@
 	(wire
 		(pts
-			(xy 195.58 111.76) (xy 189.23 111.76)
-		)
-		(stroke
-			(width 0)
-			(type default)
-		)
-	)
-	(wire
-		(pts
 			(xy 111.76 40.64) (xy 111.76 45.72)
 		)
@@
 	(wire
 		(pts
-			(xy 189.23 68.58) (xy 195.58 68.58)
+			(xy 189.23 68.58) (xy 194.31 68.58)
 		)
 		(stroke
@@
 	(wire
 		(pts
-			(xy 195.58 114.3) (xy 195.58 111.76)
-		)
-		(stroke
-			(width 0)
-			(type default)
-		)
-	)
-	(wire
-		(pts
 			(xy 189.23 96.52) (xy 196.85 96.52)
 		)
@@
 	(wire
 		(pts
-			(xy 195.58 68.58) (xy 195.58 71.12)
+			(xy 189.23 111.76) (xy 194.31 111.76)
 		)
 		(stroke
@@
 	(symbol
 		(lib_id "Power_symbols:GND")
-		(at 198.12 71.12 0)
+		(at 193.04 68.58 270)
 		(unit 1)
 		(exclude_from_sim no)
@@
 		(on_board no)
 		(dnp no)
-		(property "Reference" "#PWR021"
-			(at 197.866 62.484 0)
+		(fields_autoplaced yes)
+		(property "Reference" "#PWR17"
+			(at 193.04 68.58 0)
 			(do_not_autoplace yes)
 			(effects
@@
 		)
 		(property "Value" "GND"
-			(at 195.58 75.184 0)
+			(at 198.12 68.5799 90)
 			(effects
 				(font
 					(size 1.27 1.27)
 				)
+				(justify left)
 			)
 		)
 		(property "Footprint" ""
-			(at 198.12 71.12 0)
+			(at 193.04 68.58 0)
 			(effects
 				(font
@@
 		)
 		(property "Datasheet" ""
-			(at 198.12 71.12 0)
+			(at 193.04 68.58 0)
 			(effects
 				(font
@@
 		)
 		(property "Description" "Power Symbol - Global Ground"
-			(at 198.12 77.978 0)
+			(at 193.04 68.58 0)
 			(effects
 				(font
@@
 			(project "Master_Hand_Kicad"
 				(path "/f9e05184-c88b-4a88-ae9c-ab2bdb32be7c/c5103ceb-5325-4a84-a025-9638a412984e/961411a1-6ec4-454f-96e4-c72953a40611"
-					(reference "#PWR021")
+					(reference "#PWR17")
 					(unit 1)
 				)
@@
 	(symbol
 		(lib_id "Power_symbols:GND")
-		(at 127 62.23 0)
+		(at 124.46 60.96 180)
 		(unit 1)
 		(exclude_from_sim no)
@@
 		(on_board no)
 		(dnp no)
-		(property "Reference" "#PWR020"
-			(at 126.746 53.594 0)
+		(property "Reference" "#PWR16"
+			(at 124.46 60.96 0)
 			(do_not_autoplace yes)
 			(effects
@@
 		)
 		(property "Value" "GND"
-			(at 122.682 66.04 0)
+			(at 127 66.04 0)
 			(effects
 				(font
@@
 		)
 		(property "Footprint" ""
-			(at 127 62.23 0)
+			(at 124.46 60.96 0)
 			(effects
 				(font
@@
 		)
 		(property "Datasheet" ""
-			(at 127 62.23 0)
+			(at 124.46 60.96 0)
 			(effects
 				(font
@@
 		)
 		(property "Description" "Power Symbol - Global Ground"
-			(at 127 69.088 0)
+			(at 124.46 60.96 0)
 			(effects
 				(font
@@
 			(project "Master_Hand_Kicad"
 				(path "/f9e05184-c88b-4a88-ae9c-ab2bdb32be7c/c5103ceb-5325-4a84-a025-9638a412984e/961411a1-6ec4-454f-96e4-c72953a40611"
-					(reference "#PWR020")
+					(reference "#PWR16")
 					(unit 1)
 				)
@@
 	(symbol
 		(lib_id "Power_symbols:GND")
-		(at 113.03 88.9 0)
+		(at 110.49 87.63 180)
 		(unit 1)
 		(exclude_from_sim no)
@@
 		(on_board no)
 		(dnp no)
-		(property "Reference" "#PWR022"
-			(at 112.776 80.264 0)
+		(fields_autoplaced yes)
+		(property "Reference" "#PWR18"
+			(at 110.49 87.63 0)
 			(do_not_autoplace yes)
 			(effects
@@
 		)
 		(property "Value" "GND"
-			(at 110.49 92.71 0)
+			(at 110.49 93.98 0)
 			(effects
 				(font
@@
 		)
 		(property "Footprint" ""
-			(at 113.03 88.9 0)
+			(at 110.49 87.63 0)
 			(effects
 				(font
@@
 		)
 		(property "Datasheet" ""
-			(at 113.03 88.9 0)
+			(at 110.49 87.63 0)
 			(effects
 				(font
@@
 		)
 		(property "Description" "Power Symbol - Global Ground"
-			(at 113.03 95.758 0)
+			(at 110.49 87.63 0)
 			(effects
 				(font
@@
 			(project "Master_Hand_Kicad"
 				(path "/f9e05184-c88b-4a88-ae9c-ab2bdb32be7c/c5103ceb-5325-4a84-a025-9638a412984e/961411a1-6ec4-454f-96e4-c72953a40611"
-					(reference "#PWR022")
+					(reference "#PWR18")
 					(unit 1)
 				)
@@
 	(symbol
 		(lib_id "Power_symbols:GND")
-		(at 127 105.41 0)
+		(at 124.46 104.14 180)
 		(unit 1)
 		(exclude_from_sim no)
@@
 		(on_board no)
 		(dnp no)
-		(property "Reference" "#PWR023"
-			(at 126.746 96.774 0)
+		(property "Reference" "#PWR19"
+			(at 124.46 104.14 0)
 			(do_not_autoplace yes)
 			(effects
@@
 		)
 		(property "Value" "GND"
-			(at 122.428 109.474 0)
+			(at 127 109.22 0)
 			(effects
 				(font
@@
 		)
 		(property "Footprint" ""
-			(at 127 105.41 0)
+			(at 124.46 104.14 0)
 			(effects
 				(font
@@
 		)
 		(property "Datasheet" ""
-			(at 127 105.41 0)
+			(at 124.46 104.14 0)
 			(effects
 				(font
@@
 		)
 		(property "Description" "Power Symbol - Global Ground"
-			(at 127 112.268 0)
+			(at 124.46 104.14 0)
 			(effects
 				(font
@@
 			(project "Master_Hand_Kicad"
 				(path "/f9e05184-c88b-4a88-ae9c-ab2bdb32be7c/c5103ceb-5325-4a84-a025-9638a412984e/961411a1-6ec4-454f-96e4-c72953a40611"
-					(reference "#PWR023")
+					(reference "#PWR19")
 					(unit 1)
 				)
@@
 	(symbol
 		(lib_id "Power_symbols:GND")
-		(at 114.3 45.72 0)
+		(at 111.76 44.45 180)
 		(unit 1)
 		(exclude_from_sim no)
@@
 		(on_board no)
 		(dnp no)
-		(property "Reference" "#PWR019"
-			(at 114.046 37.084 0)
+		(fields_autoplaced yes)
+		(property "Reference" "#PWR15"
+			(at 111.76 44.45 0)
 			(do_not_autoplace yes)
 			(effects
@@
 		)
 		(property "Value" "GND"
-			(at 111.76 49.784 0)
+			(at 111.76 50.8 0)
 			(effects
 				(font
@@
 		)
 		(property "Footprint" ""
-			(at 114.3 45.72 0)
+			(at 111.76 44.45 0)
 			(effects
 				(font
@@
 		)
 		(property "Datasheet" ""
-			(at 114.3 45.72 0)
+			(at 111.76 44.45 0)
 			(effects
 				(font
@@
 		)
 		(property "Description" "Power Symbol - Global Ground"
-			(at 114.3 52.578 0)
+			(at 111.76 44.45 0)
 			(effects
 				(font
@@
 			(project "Master_Hand_Kicad"
 				(path "/f9e05184-c88b-4a88-ae9c-ab2bdb32be7c/c5103ceb-5325-4a84-a025-9638a412984e/961411a1-6ec4-454f-96e4-c72953a40611"
-					(reference "#PWR019")
+					(reference "#PWR15")
 					(unit 1)
 				)
@@
 	(symbol
 		(lib_id "Power_symbols:GND")
-		(at 198.12 114.3 0)
+		(at 193.04 111.76 270)
 		(unit 1)
 		(exclude_from_sim no)
@@
 		(on_board no)
 		(dnp no)
-		(property "Reference" "#PWR024"
-			(at 197.866 105.664 0)
+		(fields_autoplaced yes)
+		(property "Reference" "#PWR20"
+			(at 193.04 111.76 0)
 			(do_not_autoplace yes)
 			(effects
@@
 		)
 		(property "Value" "GND"
-			(at 197.612 118.364 0)
+			(at 198.12 111.7599 90)
 			(effects
 				(font
 					(size 1.27 1.27)
 				)
-				(justify right)
+				(justify left)
 			)
 		)
 		(property "Footprint" ""
-			(at 198.12 114.3 0)
+			(at 193.04 111.76 0)
 			(effects
 				(font
@@
 		)
 		(property "Datasheet" ""
-			(at 198.12 114.3 0)
+			(at 193.04 111.76 0)
 			(effects
 				(font
@@
 		)
 		(property "Description" "Power Symbol - Global Ground"
-			(at 198.12 121.158 0)
+			(at 193.04 111.76 0)
 			(effects
 				(font
@@
 			(project "Master_Hand_Kicad"
 				(path "/f9e05184-c88b-4a88-ae9c-ab2bdb32be7c/c5103ceb-5325-4a84-a025-9638a412984e/961411a1-6ec4-454f-96e4-c72953a40611"
-					(reference "#PWR024")
+					(reference "#PWR20")
 					(unit 1)
 				)
