File: sch_backup_20260820_225926/Power - Generation.kicad_sch (KiCad schematic)
At the start: 38 parts, among them U1 TPSM63603RDHR, U2 TPS62162DSG, U3 TLV75533PDBVR

Commit message: Update Schematic
Connections:
- net +5V: now also FB2.; no longer FB2.1
- net +VBAT: now also FB1.; no longer FB1.1
- net F_VIN_3V3: now reaches C11.2, C12.2, U2.2 (VIN)
- net F_VIN_3V3: now also FB2.; no longer FB2.2
- net F_VIN_5V: now reaches C1.2, C2.2, C4.2, C5.2, R1.2, U1.18 (VIN), U1.19 (VIN), U1.3 (VIN), U1.4 (VIN)
- net F_VIN_5V: now also FB1.; no longer FB1.2
Other:
- moved on the sheet: C15, C8, U2, U3
