File: sch_backup_20260820_225926/Project Architecture.kicad_sch (KiCad schematic)
At the start: 0 parts

Commit message: Update Schematic
Other:
- sheet Interface - FD-CAN ports: added {FDCAN1_CNT}, {FDCAN2_CNT}; removed {FDCAN_CNT}
- sheet Interface - Interconnects ports: added {FDCAN1_CNT}, {FDCAN2_CNT}; removed {FDCAN_CNT}
- sheet MCU - IOs ports: added {LED_Finger 1}, {LED_Finger 2}; removed {LED_Finger1}, {LED_Finger2}
- sheet User - LED Indicators & Buzzer ports: added {LED_Finger 1}, {LED_Finger 2}; removed {LED_Finger1}, {LED_Finger2}
