File: sch_backup_20260820_225926/User - LED Indicators & Buzzer.kicad_sch (KiCad schematic)
At the start: 20 parts, among them Q3 2SC1815

Commit message: Update Schematic
Changed lines of the file:
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@@
 		)
 	)
-	(hierarchical_label "{LED_Finger1}"
+	(hierarchical_label "{LED_Finger 1}"
 		(shape output)
 		(at 229.87 31.75 0)
@@
 		)
 	)
-	(hierarchical_label "{LED_Finger2}"
+	(hierarchical_label "{LED_Finger 2}"
 		(shape output)
 		(at 229.87 44.45 0)
@@
 	(symbol
 		(lib_id "Power_symbols:GND")
-		(at 107.95 35.56 90)
+		(at 106.68 38.1 270)
 		(unit 1)
 		(exclude_from_sim no)
@@
 		(dnp no)
 		(fields_autoplaced yes)
-		(property "Reference" "#PWR0131"
-			(at 99.314 35.814 0)
+		(property "Reference" "#PWR127"
+			(at 106.68 38.1 0)
 			(do_not_autoplace yes)
 			(effects
@@
 					(size 1.27 1.27)
 				)
-				(justify right)
+				(justify left)
 			)
 		)
 		(property "Footprint" ""
-			(at 107.95 35.56 0)
+			(at 106.68 38.1 0)
 			(effects
 				(font
@@
 		)
 		(property "Datasheet" ""
-			(at 107.95 35.56 0)
+			(at 106.68 38.1 0)
 			(effects
 				(font
@@
 		)
 		(property "Description" "Power Symbol - Global Ground"
-			(at 114.808 35.56 0)
-			(effects
-				(font
-					(size 1.27 1.27)
-				)
-				(hide yes)
-			)
-		)
-		(pin "1"
-		)
-		(instances
-			(project "Master_Hand_Kicad"
-				(path "/f9e05184-c88b-4a88-ae9c-ab2bdb32be7c/c5103ceb-5325-4a84-a025-9638a412984e/28daf353-f3ef-4ecd-aedd-b1b76d334dfe"
-					(reference "#PWR0131")
+			(at 106.68 38.1 0)
+			(effects
+				(font
+					(size 1.27 1.27)
+				)
+				(hide yes)
+			)
+		)
+		(pin "1"
+		)
+		(instances
+			(project "Master_Hand_Kicad"
+				(path "/f9e05184-c88b-4a88-ae9c-ab2bdb32be7c/c5103ceb-5325-4a84-a025-9638a412984e/28daf353-f3ef-4ecd-aedd-b1b76d334dfe"
+					(reference "#PWR127")
 					(unit 1)
 				)
@@
 	(symbol
 		(lib_id "Power_symbols:GND")
-		(at 218.44 137.16 0)
+		(at 215.9 135.89 180)
 		(unit 1)
 		(exclude_from_sim no)
@@
 		(dnp no)
 		(fields_autoplaced yes)
-		(property "Reference" "#PWR0132"
-			(at 218.186 128.524 0)
+		(property "Reference" "#PWR128"
+			(at 215.9 135.89 0)
 			(do_not_autoplace yes)
 			(effects
@@
 		)
 		(property "Footprint" ""
-			(at 218.44 137.16 0)
+			(at 215.9 135.89 0)
 			(effects
 				(font
@@
 		)
 		(property "Datasheet" ""
-			(at 218.44 137.16 0)
+			(at 215.9 135.89 0)
 			(effects
 				(font
@@
 		)
 		(property "Description" "Power Symbol - Global Ground"
-			(at 218.44 144.018 0)
-			(effects
-				(font
-					(size 1.27 1.27)
-				)
-				(hide yes)
-			)
-		)
-		(pin "1"
-		)
-		(instances
-			(project "Master_Hand_Kicad"
-				(path "/f9e05184-c88b-4a88-ae9c-ab2bdb32be7c/c5103ceb-5325-4a84-a025-9638a412984e/28daf353-f3ef-4ecd-aedd-b1b76d334dfe"
-					(reference "#PWR0132")
-					(unit 1)
-				)
+			(at 215.9 135.89 0)
+			(effects
+				(font
+					(size 1.27 1.27)
+				)
+				(hide yes)
+			)
+		)
+		(pin "1"
+		)
+		(instances
+			(project "Master_Hand_Kicad"
+				(path "/f9e05184-c88b-4a88-ae9c-ab2bdb32be7c/c5103ceb-5325-4a84-a025-9638a412984e/28daf353-f3ef-4ecd-aedd-b1b76d334dfe"
+					(reference "#PWR128")
+					(unit 1)
+				)
